Commit message: Update relax_materials.gazebo.xacro

File: relax_urdf/urdf/gazebo/relax_materials.gazebo.xacro (robot description, xacro)
@@ -1,21 +1,19 @@
 <?xml version="1.0"?>
 <robot xmlns:xacro="http://ros.org/wiki/xacro">
-<!-- <gazebo reference="relax_link0">
+<!-- **** gazebo materials **** -->
+<gazebo reference="relax_link1">
   <material>Gazebo/Blue</material>
 </gazebo>
-<gazebo reference="relax_link1">
+<gazebo reference="relax_link2">
   <material>Gazebo/DarkGrey</material>
 </gazebo>
-<gazebo reference="relax_link2">
+<gazebo reference="relax_link3">
   <material>Gazebo/Blue</material>
 </gazebo>
-<gazebo reference="relax_link3">
-  <material>Gazebo/DarkGrey</material>
-</gazebo>
 <gazebo reference="relax_link4">
-  <material>Gazebo/DarkGrey</material>
+  <material>Gazebo/Blue</material>
 </gazebo>
 <gazebo reference="relax_link5">
   <material>Gazebo/Blue</material>
-</gazebo> -->
+</gazebo>
 </robot>
