Commit message: porting repo from old to new version - fixed bugs which does not allow visualizing the robot

File: relax_urdf/urdf/gazebo/materials.gazebo.xacro (robot description, xacro)
@@ -2,17 +2,17 @@
 <robot xmlns:xacro="http://ros.org/wiki/xacro">
 <!-- **** gazebo materials **** -->
-<gazebo reference="relax_link1">
+<gazebo reference="relax_arm1_link1">
   <material>Gazebo/Blue</material>
 </gazebo>
-<gazebo reference="relax_link2">
+<gazebo reference="relax_arm1_link2">
   <material>Gazebo/DarkGrey</material>
 </gazebo>
-<gazebo reference="relax_link3">
+<gazebo reference="relax_arm1_link3">
   <material>Gazebo/Blue</material>
 </gazebo>
-<gazebo reference="relax_link4">
+<gazebo reference="relax_arm1_link4">
   <material>Gazebo/Blue</material>
 </gazebo>
-<gazebo reference="relax_link5">
+<gazebo reference="relax_arm1_link5">
   <material>Gazebo/Blue</material>
 </gazebo>

File: relax_urdf/urdf/gazebo/relax.gazebo.xacro (robot description, xacro)
@@ -72,21 +72,17 @@
 </xacro:if>
 <xacro:if value="${RELAX_ARM}">
-    <gazebo reference="joint1">
+    <gazebo reference="relax_arm1_joint1">
         <implicitSpringDamper>1</implicitSpringDamper>
         <provideFeedback>true</provideFeedback>
     </gazebo>
-    <gazebo reference="joint2">
+    <gazebo reference="relax_arm1_joint2">
         <implicitSpringDamper>1</implicitSpringDamper>
         <provideFeedback>true</provideFeedback>
     </gazebo>
-    <gazebo reference="joint3">
+    <gazebo reference="relax_arm1_joint3">
         <implicitSpringDamper>1</implicitSpringDamper>
         <provideFeedback>true</provideFeedback>
     </gazebo>
-    <gazebo reference="joint4">
-        <implicitSpringDamper>1</implicitSpringDamper>
-        <provideFeedback>true</provideFeedback>
-    </gazebo>
-    <gazebo reference="joint5">
+    <gazebo reference="relax_arm1_joint4">
         <implicitSpringDamper>1</implicitSpringDamper>
         <provideFeedback>true</provideFeedback>

File: relax_urdf/urdf/gazebo/xbot.gazebo.xacro (robot description, xacro)
@@ -21,9 +21,8 @@
             <pid name="j_left_wheel_roll"     profile="wheel_mot"/>
             <pid name="j_right_wheel_roll"     profile="wheel_mot"/>
-            <pid name="joint1" profile="medium_mot"/>
-            <pid name="joint2" profile="medium_mot"/>
-            <pid name="joint3" profile="medium_mot"/>
-            <pid name="joint4" profile="small_mot"/>
-            <pid name="joint5" profile="small_mot"/>
+            <pid name="relax_arm1_joint1" profile="medium_mot"/>
+            <pid name="relax_arm1_joint2" profile="medium_mot"/>
+            <pid name="relax_arm1_joint3" profile="medium_mot"/>
+            <pid name="relax_arm1_joint4" profile="small_mot"/>
         </pid>
     </plugin>

File: relax_urdf/urdf/parts/arm.urdf.xacro (robot description, xacro)
@@ -4,7 +4,6 @@
 <xacro:include filename="$(find relax_urdf)/urdf/parts/relax_arm.urdf.xacro" />
 <!-- arms -->
-<xacro:relax_arm arm_num="1"  rot="1"  parent="relax_arm${arm_num}_link1">
-      <origin xyz="${Joint_1_Ox} ${Joint_1_Oy} ${Joint_1_Oz}" rpy="0 0 0"/>
-   </xacro:centauro_arm>
+<xacro:relax_arm arm_num="1" >
+   </xacro:relax_arm>
 <!-- end_effector attached -->
 <!-- <xacro:if value="${ADD_END_EFFECTOR}">

File: relax_urdf/urdf/parts/inertial_properties.urdf.xacro (robot description, xacro)
@@ -10,65 +10,65 @@
 <xacro:property name="Link_1_mass" value=" 5.9029271e+00 "/>
 <!-- Inertia -->
-<xacro:property name="Link_1_xx" value=" 6.2182861e+04*mm2Tom2 "/>
-<xacro:property name="Link_1_xy" value=" 8.1614096e+01*mm2Tom2 "/>
-<xacro:property name="Link_1_xz" value=" 1.0385066e+02*mm2Tom2 "/>
-<xacro:property name="Link_1_yy" value=" 5.5346023e+04*mm2Tom2 "/>
-<xacro:property name="Link_1_yz" value=" 1.2999920e+04*mm2Tom2 "/>
-<xacro:property name="Link_1_zz" value=" 1.6821722e+04*mm2Tom2 "/>
+<xacro:property name="Link_1_xx" value=" ${6.2182861e+04*mm2Tom2} "/>
+<xacro:property name="Link_1_xy" value=" ${8.1614096e+01*mm2Tom2} "/>
+<xacro:property name="Link_1_xz" value=" ${1.0385066e+02*mm2Tom2} "/>
+<xacro:property name="Link_1_yy" value=" ${5.5346023e+04*mm2Tom2} "/>
+<xacro:property name="Link_1_yz" value=" ${1.2999920e+04*mm2Tom2} "/>
+<xacro:property name="Link_1_zz" value=" ${1.6821722e+04*mm2Tom2} "/>
 <!-- Link 2 -->
 <!-- Center of Mass -->
-<xacro:property name="Link_2_x" value="  0.0000000e+00*mmTom "/>
-<xacro:property name="Link_2_y" value=" -7.1720374e+00*mmTom "/>
-<xacro:property name="Link_2_z" value=" -2.0000694e+02*mmTom "/>
+<xacro:property name="Link_2_x" value=" ${ 0.0000000e+00*mmTom} "/>
+<xacro:property name="Link_2_y" value=" ${-7.1720374e+00*mmTom} "/>
+<xacro:property name="Link_2_z" value=" ${-2.0000694e+02*mmTom} "/>
 <!-- Mass -->
 <xacro:property name="Link_2_mass" value=" 1.9989653e+00 "/>
 <!-- Inertia -->
-<xacro:property name="Link_2_xx" value="  4.9589547e+04*mm2Tom2 "/>
-<xacro:property name="Link_2_xy" value=" -2.3822174e-02*mm2Tom2 "/>
-<xacro:property name="Link_2_xz" value="  2.3476881e+02*mm2Tom2 "/>
-<xacro:property name="Link_2_yy" value="  5.1111593e+04*mm2Tom2 "/>
-<xacro:property name="Link_2_yz" value="  7.7698490e-01*mm2Tom2 "/>
-<xacro:property name="Link_2_zz" value="  4.0702979e+03*mm2Tom2 "/>
+<xacro:property name="Link_2_xx" value=" ${ 4.9589547e+04*mm2Tom2} "/>
+<xacro:property name="Link_2_xy" value=" ${-2.3822174e-02*mm2Tom2} "/>
+<xacro:property name="Link_2_xz" value=" ${ 2.3476881e+02*mm2Tom2} "/>
+<xacro:property name="Link_2_yy" value=" ${ 5.1111593e+04*mm2Tom2} "/>
+<xacro:property name="Link_2_yz" value=" ${ 7.7698490e-01*mm2Tom2} "/>
+<xacro:property name="Link_2_zz" value=" ${ 4.0702979e+03*mm2Tom2} "/>
 <!-- Link 3 -->
 <!-- Center of Mass -->
-<xacro:property name="Link_3_x" value=" -2.1052916e+00*mmTom "/>
-<xacro:property name="Link_3_y" value=" -1.0638552e+02*mmTom "/>
-<xacro:property name="Link_3_z" value=" -7.4903486e+01*mmTom "/>
+<xacro:property name="Link_3_x" value=" ${-2.1052916e+00*mmTom} "/>
+<xacro:property name="Link_3_y" value=" ${-1.0638552e+02*mmTom} "/>
+<xacro:property name="Link_3_z" value=" ${-7.4903486e+01*mmTom} "/>
 <!-- Mass -->
 <xacro:property name="Link_3_mass" value=" 5.8838845e+00 "/>
 <!-- Inertia -->
-<xacro:property name="Link_3_xx" value="  6.1043599e+04*mm2Tom2 "/>
-<xacro:property name="Link_3_xy" value=" -1.5340891e+02*mm2Tom2 "/>
-<xacro:property name="Link_3_xz" value=" -1.7833160e+02*mm2Tom2 "/>
-<xacro:property name="Link_3_yy" value="  5.3601310e+04*mm2Tom2 "/>
-<xacro:property name="Link_3_yz" value=" -1.1090900e+04*mm2Tom2 "/>
-<xacro:property name="Link_3_zz" value="  1.7380798e+04*mm2Tom2 "/>
+<xacro:property name="Link_3_xx" value=" ${ 6.1043599e+04*mm2Tom2} "/>
+<xacro:property name="Link_3_xy" value=" ${-1.5340891e+02*mm2Tom2} "/>
+<xacro:property name="Link_3_xz" value=" ${-1.7833160e+02*mm2Tom2} "/>
+<xacro:property name="Link_3_yy" value=" ${ 5.3601310e+04*mm2Tom2} "/>
+<xacro:property name="Link_3_yz" value=" ${-1.1090900e+04*mm2Tom2} "/>
+<xacro:property name="Link_3_zz" value=" ${ 1.7380798e+04*mm2Tom2} "/>
 <!-- Link 4 -->
 <!-- Center of Mass -->
-<xacro:property name="Link_4_x" value="  2.4496086e-01*mmTom "/>
-<xacro:property name="Link_4_y" value=" -1.0728501e+00*mmTom "/>
-<xacro:property name="Link_4_z" value=" -4.9015064e+01*mmTom "/>
+<xacro:property name="Link_4_x" value=" ${ 2.4496086e-01*mmTom} "/>
+<xacro:property name="Link_4_y" value=" ${-1.0728501e+00*mmTom} "/>
+<xacro:property name="Link_4_z" value=" ${-4.9015064e+01*mmTom} "/>
 <!-- Mass -->
 <xacro:property name="Link_4_mass" value=" 1.3982240e+00 "/>
 <!-- Inertia -->
-<xacro:property name="Link_4_xx" value="  1.4667270e+04*mm2Tom2 "/>
-<xacro:property name="Link_4_xy" value=" -2.0411012e+01*mm2Tom2 "/>
-<xacro:property name="Link_4_xz" value=" -4.4769570e+01*mm2Tom2 "/>
-<xacro:property name="Link_4_yy" value="  8.6598581e+03*mm2Tom2 "/>
-<xacro:property name="Link_4_yz" value=" -8.3199044e+01*mm2Tom2 "/>
-<xacro:property name="Link_4_zz" value="  1.0450923e+04*mm2Tom2 "/>
+<xacro:property name="Link_4_xx" value=" ${ 1.4667270e+04*mm2Tom2} "/>
+<xacro:property name="Link_4_xy" value=" ${-2.0411012e+01*mm2Tom2} "/>
+<xacro:property name="Link_4_xz" value=" ${-4.4769570e+01*mm2Tom2} "/>
+<xacro:property name="Link_4_yy" value=" ${ 8.6598581e+03*mm2Tom2} "/>
+<xacro:property name="Link_4_yz" value=" ${-8.3199044e+01*mm2Tom2} "/>
+<xacro:property name="Link_4_zz" value=" ${ 1.0450923e+04*mm2Tom2} "/>
 <!-- Link 5 -->
 <!-- Center of Mass -->
-<xacro:property name="Link_5_x" value=" -1.3228834e+00*mmTom "/>
-<xacro:property name="Link_5_y" value=" -8.4683010e+01*mmTom "/>
-<xacro:property name="Link_5_z" value=" -5.3211105e+01*mmTom "/>
+<xacro:property name="Link_5_x" value=" ${-1.3228834e+00*mmTom} "/>
+<xacro:property name="Link_5_y" value=" ${-8.4683010e+01*mmTom} "/>
+<xacro:property name="Link_5_z" value=" ${-5.3211105e+01*mmTom} "/>
 <!-- Mass -->
 <xacro:property name="Link_5_mass" value=" 5.7923846e+00 "/>
 <!-- Inertia -->
-<xacro:property name="Link_5_xx" value="  5.5109543e+04*mm2Tom2 "/>
-<xacro:property name="Link_5_xy" value=" -1.4003837e+02*mm2Tom2 "/>
-<xacro:property name="Link_5_xz" value="  2.1470743e+02*mm2Tom2 "/>
-<xacro:property name="Link_5_yy" value="  5.1309424e+04*mm2Tom2 "/>
-<xacro:property name="Link_5_yz" value=" -1.0289246e+03*mm2Tom2 "/>
-<xacro:property name="Link_5_zz" value="  1.3804762e+04*mm2Tom2 "/>
+<xacro:property name="Link_5_xx" value=" ${ 5.5109543e+04*mm2Tom2} "/>
+<xacro:property name="Link_5_xy" value=" ${-1.4003837e+02*mm2Tom2} "/>
+<xacro:property name="Link_5_xz" value=" ${ 2.1470743e+02*mm2Tom2} "/>
+<xacro:property name="Link_5_yy" value=" ${ 5.1309424e+04*mm2Tom2} "/>
+<xacro:property name="Link_5_yz" value=" ${-1.0289246e+03*mm2Tom2} "/>
+<xacro:property name="Link_5_zz" value=" ${ 1.3804762e+04*mm2Tom2} "/>
 </robot>

File: relax_urdf/urdf/parts/kinematics_properties.urdf.xacro (robot description, xacro)
@@ -4,18 +4,18 @@
 <!-- Joint 1 Origin -->
 <xacro:property name="Joint_1_Ox" value="  0.0 "/>
-<xacro:property name="Joint_1_Oy" value="  131.660*mmTom "/>
-<xacro:property name="Joint_1_Oz" value=" -249.660*mmTom "/>
+<xacro:property name="Joint_1_Oy" value=" ${ 131.660*mmTom} "/>
+<xacro:property name="Joint_1_Oz" value=" ${-249.660*mmTom} "/>
 <!-- Joint 2 Origin -->
 <xacro:property name="Joint_2_Ox" value="  0.0 "/>
 <xacro:property name="Joint_2_Oy" value="  0.0 "/>
-<xacro:property name="Joint_2_Oz" value=" -400*mmTom "/>
+<xacro:property name="Joint_2_Oz" value=" ${-400*mmTom} "/>
 <!-- Joint 3 Origin -->
 <xacro:property name="Joint_3_Ox" value="  0.0 "/>
-<xacro:property name="Joint_3_Oy" value=" -131.660*mmTom "/>
-<xacro:property name="Joint_3_Oz" value=" -249.660*mmTom "/>
+<xacro:property name="Joint_3_Oy" value=" ${-131.660*mmTom} "/>
+<xacro:property name="Joint_3_Oz" value=" ${-249.660*mmTom} "/>
 <!-- Joint 4 Origin -->
 <xacro:property name="Joint_4_Ox" value="  0.0 "/>
-<xacro:property name="Joint_4_Oy" value=" -88.1600*mmTom "/>
-<xacro:property name="Joint_4_Oz" value=" -153.500*mmTom "/>
+<xacro:property name="Joint_4_Oy" value=" ${-88.1600*mmTom} "/>
+<xacro:property name="Joint_4_Oz" value=" ${-153.500*mmTom} "/>
 <xacro:property name="Joint_4_Oroll" value="  0.0 "/>
 <xacro:property name="Joint_4_Opitch" value=" 0.0 "/>

File: relax_urdf/urdf/parts/relax_arm.urdf.xacro (robot description, xacro)
@@ -2,5 +2,5 @@
 <robot xmlns:xacro="http://ros.org/wiki/xacro">
 <!-- macro arm -->
-<xacro:macro name="relax_arm" params="arm_num rot parent *origin">
+<xacro:macro name="relax_arm" params="arm_num" >
 <!-- links -->
 <link name ="relax_arm${arm_num}_link1">  <!-- link 1 -->
@@ -32,5 +32,5 @@
     <visual>
       <origin xyz="0 0 0" rpy="0 0 0"/>
-      <geometry name="relax_link1_visual">
+      <geometry name="relax_link2_visual">
         <mesh filename="package://relax_urdf/meshes/mesh_link2.stl" scale="0.001 0.001 0.001" />
       </geometry>
@@ -106,7 +106,7 @@
 <!-- joints -->
 <joint name="relax_arm${arm_num}_joint1" type="revolute"> <!-- joint 1 -->
-    <parent link="${parent}"/>
+    <parent link="relax_arm${arm_num}_link1"/>
     <child link="relax_arm${arm_num}_link2"/>
-    <xacro:insert_block name="origin"/>
+    <origin xyz="${Joint_1_Ox} ${Joint_1_Oy} ${Joint_1_Oz}" rpy="0 0 0"/>
     <axis xyz="0 1 0"/>
     <limit velocity="${Joint_1_velocity}" effort="${Joint_1_effort}" lower="${Joint_1_lower}" upper="${Joint_1_upper}" />
@@ -119,5 +119,5 @@
     <axis xyz="0 1 0"/>
     <limit velocity="${Joint_2_velocity}" effort="${Joint_2_effort}" lower="${Joint_2_lower}" upper="${Joint_2_upper}" />
-    <dynamics damping="${Joint_2_damp}" friction="${Joint_1_fric}"/>
+    <dynamics damping="${Joint_2_damp}" friction="${Joint_2_fric}"/>
 </joint>
 <joint name="relax_arm${arm_num}_joint3" type="revolute"> <!-- joint 3 -->
@@ -127,5 +127,5 @@
     <axis xyz="0 0 1"/>
     <limit velocity="${Joint_3_velocity}" effort="${Joint_3_effort}" lower="${Joint_3_lower}" upper="${Joint_3_upper}" />
-    <dynamics damping="${Joint_3_damp}" friction="${Joint_1_fric}"/>
+    <dynamics damping="${Joint_3_damp}" friction="${Joint_3_fric}"/>
 </joint>
 <joint name="relax_arm${arm_num}_joint4" type="revolute"> <!-- joint 4 -->
@@ -135,5 +135,6 @@
     <axis xyz="0 1 0"/>
     <limit velocity="${Joint_4_velocity}" effort="${Joint_4_effort}" lower="${Joint_4_lower}" upper="${Joint_4_upper}" />
-    <dynamics damping="${Joint_4_damp}" friction="${Joint_1_fric}"/>
+    <dynamics damping="${Joint_4_damp}" friction="${Joint_4_fric}"/>
 </joint>
+  </xacro:macro>
 </robot>

File: relax_urdf/urdf/relax.urdf.xacro (robot description, xacro)
@@ -2,7 +2,7 @@
 <robot xmlns:xacro="http://ros.org/wiki/xacro" name="relax">
 <!-- ************ MODEL CONFIGURATION ************ -->
-<xacro:include filename="$(find relax_urdf)/urdf/config/relax.urdf.xacro" />
-<!-- ************ UTILS ************ -->
-<xacro:include filename="$(find relax_urdf)/urdf/relax_utils.urdf.xacro"/>
+<xacro:arg name="config" default="$(find relax_urdf)/urdf/config/relax.urdf.xacro" />
+<!-- ************ MODEL CONFIGURATION ************ -->
+<xacro:include filename="$(arg config)"/>
 <!-- ************ RELAX BASE ************ -->
 <xacro:include filename="$(find relax_urdf)/urdf/relax_base.urdf.xacro"/>

File: relax_urdf/urdf/relax_base.urdf.xacro (robot description, xacro)
@@ -21,5 +21,5 @@
             <joint name="base_joint" type="fixed">
                 <parent link="base_link"/>
-                <child link="relax_link1"/>
+                <child link="relax_arm1_link1"/>
                 <origin xyz="0 0 0" rpy="${PI} 0 0" />
             </joint>
@@ -41,5 +41,5 @@
             <joint name="base_joint" type="fixed">
                 <parent link="base_link"/>
-                <child link="relax_link1"/>
+                <child link="relax_arm1_link1"/>
                 <origin xyz="0 0 0" rpy="${PI} 0 0" />
             </joint>
@@ -56,5 +56,5 @@
         <joint name="mobile_base_joint" type="fixed"> <!-- mobile base joint -->
             <parent link="control_box"/>
-            <child link="relax_link1"/>
+            <child link="relax_arm1_link1"/>
             <origin xyz="0 0 0" rpy="3.1415927 0 0"/>
         </joint>

File: relax_urdf/urdf/relax_robot.urdf.xacro (robot description, xacro)
@@ -13,5 +13,5 @@
    	<joint name="world_joint" type="fixed">
         <parent link="world"/>
-        <child link="relax_link1"/>
+        <child link="relax_arm${arm_num}_link1"/>
         <origin xyz="0 0 0" rpy="0 0 0" />
   	</joint>
