Commit message: Integration with ros-navigation stack

File: relax_urdf/urdf/gazebo/materials.gazebo.xacro (robot description, xacro)
@@ -17,3 +17,6 @@
   <material>Gazebo/Blue</material>
 </gazebo>
+<gazebo reference="relax_arm1_link6">
+  <material>Gazebo/Blue</material>
+</gazebo>
 </robot>

File: relax_urdf/urdf/gazebo/relax.gazebo.xacro (robot description, xacro)
@@ -1,74 +1,15 @@
 <?xml version="1.0"?>
 <robot xmlns:xacro="http://ros.org/wiki/xacro">
-<xacro:if value="${RELAX_MOBILE_BASE}">
-    <gazebo reference="wheel_left">
-        <material>Gazebo/DarkGrey </material>
-        <collision>
-            <surface>
-                <friction>
-                    <ode>
-                        <mu>1.0</mu>
-                        <mu2>1.0</mu2>
-                    </ode>
-                    <bullet>
-                        <friction>1.0</friction>
-                        <friction2>1.0</friction2>
-                    </bullet>
-                </friction>
-                <contact>
-                    <ode>
-                        <kp>2100000</kp>
-                        <kd>1</kd>
-                        <max_vel>100</max_vel>
-                    </ode>
-                    <bullet>
-                        <soft_cfm>0.007</soft_cfm>
-                        <soft_erp>0.25</soft_erp>
-                        <kp>1000000</kp>
-                        <kd>5</kd>
-                    </bullet>
-                </contact>
-            </surface>
-        </collision>
-    </gazebo>
-    <gazebo reference="wheel_right">
-        <material>Gazebo/DarkGrey </material>
-        <collision>
-            <surface>
-                <friction>
-                    <ode>
-                        <mu>1.0</mu>
-                        <mu2>1.0</mu2>
-                    </ode>
-                    <bullet>
-                        <friction>1.0</friction>
-                        <friction2>1.0</friction2>
-                    </bullet>
-                </friction>
-                <contact>
-                    <ode>
-                        <kp>2100000</kp>
-                        <kd>1</kd>
-                        <max_vel>100</max_vel>
-                    </ode>
-                    <bullet>
-                        <soft_cfm>0.007</soft_cfm>
-                        <soft_erp>0.25</soft_erp>
-                        <kp>1000000</kp>
-                        <kd>5</kd>
-                    </bullet>
-                </contact>
-            </surface>
-        </collision>
-    </gazebo>
-    <gazebo reference="j_left_wheel">
-        <implicitSpringDamper>1</implicitSpringDamper>
-        <provideFeedback>true</provideFeedback>
-    </gazebo>
-    <gazebo reference="j_right_wheel">
-        <implicitSpringDamper>1</implicitSpringDamper>
-        <provideFeedback>true</provideFeedback>
-    </gazebo>
-</xacro:if>
+<xacro:macro name="controller_plugin_gazebo" params="robot_namespace">
+<gazebo>
+    <plugin name="gazebo_ros_control" filename="libgazebo_ros_control.so">
+    <xacro:unless value="${robot_namespace == ''}">
+        <robotNamespace>${robot_namespace}</robotNamespace>
+    </xacro:unless>
+    <controlPeriod>0.001</controlPeriod>
+    <legacyModeNS>false</legacyModeNS>
+    </plugin>
+</gazebo>
+</xacro:macro>
 <xacro:if value="${RELAX_ARM}">
     <gazebo reference="relax_arm1_joint1">
@@ -88,4 +29,8 @@
         <provideFeedback>true</provideFeedback>
     </gazebo>
+    <gazebo reference="relax_arm1_joint5">
+        <implicitSpringDamper>1</implicitSpringDamper>
+        <provideFeedback>true</provideFeedback>
+    </gazebo>
 </xacro:if>
 </robot>

File: relax_urdf/urdf/gazebo/xbot.gazebo.xacro (robot description, xacro)
@@ -5,5 +5,5 @@
         <links>
             <link name="base_link"/>
-            <link name="left_wheel"/>
+            <link name="left_wheel_link"/>
         </links>
     </plugin>
@@ -18,11 +18,20 @@
             <gain name="medium_mot" p="1000" d="10"/>
             <gain name="big_mot"    p="3000" d="10"/>
-            <gain name="wheel_mot"  p="0" d="10"/>
-            <pid name="j_left_wheel_roll"     profile="wheel_mot"/>
-            <pid name="j_right_wheel_roll"     profile="wheel_mot"/>
+            <gain name="wheel_mot"  p="1" d="1"/>
+            <pid name="left_wheel_joint"     profile="wheel_mot"/>
+            <pid name="right_wheel_joint"     profile="wheel_mot"/>
+            <pid name="front_left_caster_rotation_joint"     profile="wheel_mot"/>
+            <pid name="front_left_caster_wheel_joint"     profile="wheel_mot"/>
+            <pid name="front_right_caster_rotation_joint"     profile="wheel_mot"/>
+            <pid name="front_right_caster_wheel_joint"     profile="wheel_mot"/>
+            <pid name="rear_left_caster_rotation_joint"     profile="wheel_mot"/>
+            <pid name="rear_left_caster_wheel_joint"     profile="wheel_mot"/>
+            <pid name="rear_right_caster_rotation_joint"     profile="wheel_mot"/>
+            <pid name="rear_right_caster_wheel_joint"     profile="wheel_mot"/>
             <pid name="relax_arm1_joint1" profile="medium_mot"/>
             <pid name="relax_arm1_joint2" profile="medium_mot"/>
             <pid name="relax_arm1_joint3" profile="medium_mot"/>
             <pid name="relax_arm1_joint4" profile="small_mot"/>
+            <pid name="relax_arm1_joint5" profile="small_mot"/>
         </pid>
     </plugin>

File: relax_urdf/urdf/parts/mobile_base.urdf.xacro (robot description, xacro)
@@ -1,159 +1,99 @@
 <?xml version="1.0"?>
 <robot xmlns:xacro="http://ros.org/wiki/xacro">
-<!-- links -->
-<link name ="mobile_base_link">  <!-- mobile base link -->
-    <inertial>
-      <origin xyz="0.0 0.0 0.0" rpy="0 0 0"/>
-      <mass value="100.0"/>
-      <inertia ixx="17" ixy="0.0" ixz="0.0" iyy="17" iyz="0.0" izz="17" />
-    </inertial>
-    <visual>
-      <origin xyz="0 0 0" rpy="0 0 0"/>
-      <geometry name="mobile_base_link_visual">
-        <mesh filename="package://relax_urdf/meshes/mir_base.stl" scale="0.001 0.001 0.001" />
-      </geometry>
-      <material name="dark"/>
-    </visual>
-    <collision>
-      <origin xyz="0 0 0" rpy="0 0 0"/>
-      <geometry name="mobile_base_link_collision">
-        <mesh filename="package://relax_urdf/meshes/mir_base.stl" scale="0.001 0.001 0.001" />
-      </geometry>
-    </collision>
-</link>
-<link name ="control_box">
-    <inertial>
-      <origin xyz="0.0 0.0 0.0" rpy="0 0 0"/>
-      <mass value="1.0"/>
-      <inertia ixx="0.17" ixy="0.0" ixz="0.0" iyy="0.17" iyz="0.0" izz="0.17" />
-    </inertial>
-    <visual>
-      <origin xyz="0 0 0" rpy="0 0 0"/>
-      <geometry name="control_box_visual">
-          <box size="0.3 0.3 0.15" />
-      </geometry>
-      <material name="dark"/>
-    </visual>
-    <collision>
-      <origin xyz="0 0 0" rpy="0 0 0"/>
-      <geometry name="control_box_collision">
-          <box size="0.3 0.3 0.15" />
-      </geometry>
-    </collision>
-</link>
-<link name ="left_wheel">
-    <inertial>
-      <origin xyz="0.0 0.0 0.0" rpy="0 0 0"/>
-      <mass value="1.0"/>
-      <inertia ixx="0.17" ixy="0.0" ixz="0.0" iyy="0.17" iyz="0.0" izz="0.17" />
-    </inertial>
-    <visual>
-      <origin xyz="0 0 0" rpy="0 0 0"/>
-      <geometry name="left_wheel_link_visual">
-        <mesh filename="package://relax_urdf/meshes/mesh_left_wheel.stl" scale="0.001 0.001 0.001" />
-      </geometry>
-      <material name="dark"/>
-    </visual>
-    <collision>
-      <origin xyz="0 0 0" rpy="0 0 0"/>
-      <geometry name="left_wheel_link_collision">
-        <mesh filename="package://relax_urdf/meshes/mesh_left_wheel.stl" scale="0.001 0.001 0.001" />
-      </geometry>
-    </collision>
-</link>
-<link name ="right_wheel">
-    <inertial>
-      <origin xyz="0.0 0.0 0.0" rpy="0 0 0"/>
-      <mass value="1.0"/>
-      <inertia ixx="0.17" ixy="0.0" ixz="0.0" iyy="0.17" iyz="0.0" izz="0.17" />
-    </inertial>
-    <visual>
-      <origin xyz="0 0 0" rpy="0 0 0"/>
-      <geometry name="right_wheel_link_visual">
-        <mesh filename="package://relax_urdf/meshes/mesh_left_wheel.stl" scale="0.001 0.001 0.001" />
-      </geometry>
-      <material name="dark"/>
-    </visual>
-    <collision>
-      <origin xyz="0 0 0" rpy="0 0 0"/>
-      <geometry name="right_wheel_link_collision">
-        <mesh filename="package://relax_urdf/meshes/mesh_left_wheel.stl" scale="0.001 0.001 0.001" />
-      </geometry>
-    </collision>
-</link>
-<link name ="left_wheel_yaw">
-    <inertial>
-      <origin xyz="0.0 0.0 0.0" rpy="0 0 0"/>
-      <mass value="1.0"/>
-      <inertia ixx="0.17" ixy="0.0" ixz="0.0" iyy="0.17" iyz="0.0" izz="0.17" />
-    </inertial>
-    <visual>
-      <origin xyz="0 0 0" rpy="0 0 0"/>
-      <geometry name="left_wheel_yaw_link_visual">
-        <box size="0.001 0.001 0.001"/>
-      </geometry>
-      <material name="dark"/>
-    </visual>
-    <collision>
-      <origin xyz="0 0 0" rpy="0 0 0"/>
-      <geometry name="left_wheel_yaw_link_collision">
-        <box size="0.001 0.001 0.001"/>
-      </geometry>
-    </collision>
-</link>
-<link name ="right_wheel_yaw">
-    <inertial>
-      <origin xyz="0.0 0.0 0.0" rpy="0 0 0"/>
-      <mass value="1.0"/>
-      <inertia ixx="0.17" ixy="0.0" ixz="0.0" iyy="0.17" iyz="0.0" izz="0.17" />
-    </inertial>
-    <visual>
-      <origin xyz="0 0 0" rpy="0 0 0"/>
-      <geometry name="right_wheel_yaw_link_visual">
-        <box size="0.001 0.001 0.001"/>
-      </geometry>
-      <material name="dark"/>
-    </visual>
-    <collision>
-      <origin xyz="0 0 0" rpy="0 0 0"/>
-      <geometry name="right_wheel_yaw_link_collision">
-        <box size="0.001 0.001 0.001"/>
-      </geometry>
-    </collision>
-</link>
-<joint name="j_control" type="fixed">
-	<parent link="mobile_base_link"/>
-	<child link="control_box"/>
-    <origin xyz="0 0 ${225.000*mmTom+0.15}" rpy="0 0 0"/>
-	<axis xyz="0 0 1"/>
-</joint>
-<joint name="j_left_wheel_yaw" type="revolute">
-	<parent link="mobile_base_link"/>
-	<child link="left_wheel_yaw"/>
-    <origin xyz="-0.00448719 0.25 0.09" rpy="0 0 0"/>
-	<axis xyz="0 0 1"/>
-   <limit  effort="35" velocity="20" lower="-1" upper="1" />
-</joint>
-<joint name="j_right_wheel_yaw" type="revolute">
-	<parent link="mobile_base_link"/>
-	<child link="right_wheel_yaw"/>
-	<origin xyz="-0.00448719 -0.25 0.09" rpy="0 0 0"/>
-	<axis xyz="0 0 1"/>
-   <limit  effort="35" velocity="20" lower="-1" upper="1" />
-</joint>
-<joint name="j_left_wheel_roll" type="continuous">
-	<parent link="left_wheel_yaw"/>
-	<child link="left_wheel"/>
-    <origin xyz="0 0 0" rpy="0 0 0"/>
-	<axis xyz="0 1 0"/>
-   <limit  effort="35" velocity="20"/>
-</joint>
-<joint name="j_right_wheel_roll" type="continuous">
-	<parent link="right_wheel_yaw"/>
-	<child link="right_wheel"/>
-	<origin xyz="0 0 0" rpy="0 0 0"/>
-	<axis xyz="0 1 0"/>
-   <limit  effort="35" velocity="20"/>
-</joint>
+  <xacro:include filename="$(find relax_urdf)/urdf/parts/common_base_properties.urdf.xacro" />
+  <xacro:include filename="$(find relax_urdf)/urdf/gazebo/imu.gazebo.urdf.xacro" />
+  <xacro:include filename="$(find relax_urdf)/urdf/gazebo/mir.gazebo.xacro" />
+  <xacro:include filename="$(find relax_urdf)/urdf/parts/mir.transmission.xacro" />
+  <xacro:include filename="$(find relax_urdf)/urdf/parts/sick_s300.urdf.xacro" />
+  <xacro:include filename="$(find relax_urdf)/urdf/parts/wheels.urdf.xacro" />
+    <link name="${prefix}base_footprint" />
+    <joint name="${prefix}base_joint" type="fixed">
+      <parent link="${prefix}base_footprint" />
+      <child link="${prefix}base_link" />
+      <origin xyz="0 0 0" rpy="0 0 0" />
+    </joint>
+    <link name="${prefix}base_link">
+      <xacro:box_inertial mass="${mir_base_mass}" x="${mir_base_inertial_x_length}" y="${mir_base_inertial_y_length}" z="${mir_base_inertial_z_length}">
+        <origin xyz="${mir_base_inertial_x + mir_act_wheel_dx} ${mir_base_inertial_y} ${mir_base_inertial_z}" rpy="0 0 0" />
+      </xacro:box_inertial>
+      <visual>
+        <origin xyz="${mir_act_wheel_dx} 0 0" rpy="0 0 0" />
+        <geometry>
+          <mesh filename="package://relax_urdf/meshes/mesh_base_revised.stl" />
+        </geometry>
+        <xacro:insert_block name="material_dark_grey" />
+      </visual>
+      <collision>
+        <origin xyz="${mir_act_wheel_dx} 0 0" rpy="0 0 0" />
+        <geometry>
+          <mesh filename="package://relax_urdf/meshes/mesh_base_revised.stl" />
+        </geometry>
+      </collision>
+    </link>
+    <gazebo reference="${prefix}base_link">
+      <material>Gazebo/DarkGrey</material>
+    </gazebo>
+    <!-- IMU -->
+    <joint name="${prefix}base_link_to_imu_joint" type="fixed">
+      <parent link="${prefix}base_link" />
+      <child link="${prefix}imu_link" />
+      <origin xyz="0.0 0.0 0.25" rpy="0 0 0" />  <!-- same as real MiR -->
+    </joint>
+    <link name="${prefix}imu_link" />
+    <xacro:imu_gazebo link="${prefix}imu_link" imu_topic="imu_data" update_rate="50.0" />
+    <!-- Create an alias for imu_link. This is necessary because the real MiR's
+         TF has imu_link, but the imu_data topic is published in the imu_frame
+         frame. -->
+    <joint name="${prefix}imu_link_to_imu_frame_joint" type="fixed">
+      <parent link="${prefix}imu_link" />
+      <child link="${prefix}imu_frame" />
+      <origin xyz="0 0 0" rpy="0 0 0" />
+    </joint>
+    <link name="${prefix}imu_frame" />
+    <!-- Laser scanners -->
+    <joint name="${prefix}base_link_to_front_laser_joint" type="fixed">
+      <parent link="${prefix}base_link" />
+      <child link="${prefix}front_laser_link" />
+      <origin xyz="${laser_dx + mir_act_wheel_dx} ${laser_dy} ${laser_dz}" rpy="0.0 0.0 ${0.25 * pi}" />
+    </joint>
+    <xacro:sick_s300 prefix="${prefix}" link="front_laser_link" topic="f_scan" />
+    <joint name="${prefix}base_link_to_back_laser_joint" type="fixed">
+      <parent link="${prefix}base_link" />
+      <child link="${prefix}back_laser_link" />
+      <origin xyz="${-laser_dx + mir_act_wheel_dx} ${-laser_dy} ${laser_dz}" rpy="0.0 0.0 ${-0.75 * pi}" />
+    </joint>
+    <xacro:sick_s300 prefix="${prefix}" link="back_laser_link" topic="b_scan" />
+    <!-- Ultrasound sensors -->
+    <joint name="${prefix}us_1_joint" type="fixed">   <!-- right ultrasound -->
+      <parent link="${prefix}base_link" />
+      <child link="${prefix}us_1_frame" />
+      <origin xyz="0.45 -0.12 0.16 " rpy="0 0 0" />  <!-- from visually matching to the mesh of the MiR -->
+    </joint>
+    <link name="${prefix}us_1_frame" />
+    <joint name="${prefix}us_2_joint" type="fixed">   <!-- left ultrasound -->
+      <parent link="${prefix}base_link" />
+      <child link="${prefix}us_2_frame" />
+      <origin xyz="0.45 0.12 0.16 " rpy="0 0 0" />  <!-- from visually matching to the mesh of the MiR -->
+    </joint>
+    <link name="${prefix}us_2_frame" />
+    <!-- wheels -->
+    <xacro:actuated_wheel prefix="${prefix}" locationprefix="left" locationright="-1"/>
+    <xacro:actuated_wheel prefix="${prefix}" locationprefix="right" locationright="1"/>
+    <xacro:caster_wheel prefix="${prefix}" locationprefix="fl" locationright="-1" wheel_base_dx="${mir_front_caster_wheel_base_dx + mir_act_wheel_dx}"/>
+    <xacro:caster_wheel prefix="${prefix}" locationprefix="fr" locationright="1" wheel_base_dx="${mir_front_caster_wheel_base_dx + mir_act_wheel_dx}"/>
+    <xacro:caster_wheel prefix="${prefix}" locationprefix="bl" locationright="-1" wheel_base_dx="${-mir_back_caster_wheel_base_dx + mir_act_wheel_dx}"/>
+    <xacro:caster_wheel prefix="${prefix}" locationprefix="br" locationright="1" wheel_base_dx="${-mir_back_caster_wheel_base_dx + mir_act_wheel_dx}"/>
+    <joint name="${prefix}base_link_surface_joint" type="fixed">
+      <origin xyz="${mir_act_wheel_dx} 0 0.352" rpy="0 0 0" />
+      <parent link="${prefix}base_link" />
+      <child link="${prefix}surface" />
+      <axis xyz="0 0 1" />
+    </joint>
+    <link name="${prefix}surface"/>
+    <xacro:mir_wheel_transmissions prefix="${prefix}"/>
+    <!-- set the gazebo friction parameters for the wheels -->
+    <xacro:set_all_wheel_frictions prefix="${prefix}"/>
+    <xacro:p3d_base_controller prefix="${prefix}" />
+<!--
 <xacro:if value="${ADD_D435I_CONTROL_BOX}">
     <xacro:include filename="$(find realsense_gazebo_description)/urdf/_d435i.urdf.xacro" />
@@ -175,4 +115,4 @@
             <origin xyz="0.18 0 0" rpy="0 -0.5 0"/>
         </xacro:sensor_d435i>
-</xacro:if>
+</xacro:if>-->
 </robot>

File: relax_urdf/urdf/relax.urdf.xacro (robot description, xacro)
@@ -13,5 +13,5 @@
         <joint name="world_joint" type="floating">
             <parent link="world"/>
-            <child link="base_link"/>
+            <child link="base_footprint"/>
         </joint>
     </xacro:if>

File: relax_urdf/urdf/relax_base.urdf.xacro (robot description, xacro)
@@ -6,56 +6,17 @@
 <xacro:include filename="$(find relax_urdf)/urdf/parts/dynamic_properties.urdf.xacro" />
 <xacro:include filename="$(find relax_urdf)/urdf/parts/limits.urdf.xacro" />
-<!-- **** base attached to robot **** -->
-<xacro:if value="${RELAX_FLOATING_BASE}">
-    <xacro:if value="${RELAX_MOBILE_BASE}">
-        <link name="base_link"/>
-        <joint name="base_joint" type="fixed">
-            <parent link="base_link"/>
-            <child link="mobile_base_link"/>
-            <origin xyz="0 0 0" rpy="0 0 0" />
-        </joint>
-    </xacro:if>
-    <xacro:unless value="${RELAX_MOBILE_BASE}">
-        <xacro:if value="${RELAX_ARM}">
-            <link name="base_link"/>
-            <joint name="base_joint" type="fixed">
-                <parent link="base_link"/>
-                <child link="relax_arm1_link1"/>
-                <origin xyz="0 0 0" rpy="${PI} 0 0" />
-            </joint>
-        </xacro:if>
-    </xacro:unless>
-</xacro:if>
-<xacro:unless value="${RELAX_FLOATING_BASE}">
-    <xacro:if value="${RELAX_MOBILE_BASE}">
-        <link name="base_link"/>
-        <joint name="base_joint" type="fixed">
-            <parent link="base_link"/>
-            <child link="mobile_base_link"/>
-            <origin xyz="0 0 0" rpy="0 0 0" />
-        </joint>
-    </xacro:if>
-    <xacro:unless value="${RELAX_MOBILE_BASE}">
-        <xacro:if value="${RELAX_ARM}">
-            <link name="base_link"/>
-            <joint name="base_joint" type="fixed">
-                <parent link="base_link"/>
-                <child link="relax_arm1_link1"/>
-                <origin xyz="0 0 0" rpy="${PI} 0 0" />
-            </joint>
-        </xacro:if>
-    </xacro:unless>
-</xacro:unless>
 <!-- ********  attach robot  ******** -->
 <xacro:if value="${RELAX_ARM}">
     <xacro:include filename="$(find relax_urdf)/urdf/parts/arm.urdf.xacro" />
 </xacro:if>
+<!-- Add Base -->
 <xacro:if value="${RELAX_MOBILE_BASE}">
-<xacro:include filename="$(find relax_urdf)/urdf/parts/mobile_base.urdf.xacro" />
+    <xacro:include filename="$(find relax_urdf)/urdf/parts/mir_base.urdf.xacro" />
+    <xacro:mir prefix=""/>
     <xacro:if value="${RELAX_ARM}">
         <joint name="mobile_base_joint" type="fixed"> <!-- mobile base joint -->
-            <parent link="control_box"/>
+            <parent link="base_link"/>
             <child link="relax_arm1_link1"/>
-            <origin xyz="0 0 0" rpy="0 0 0"/>
+            <origin xyz="-0.130 0 0.3613" rpy="0 0 0"/>
         </joint>
     </xacro:if>

File: relax_urdf/urdf/relax_robot.urdf.xacro (robot description, xacro)
@@ -17,3 +17,6 @@
   	</joint>
 </xacro:unless>
+<xacro:if value="${RELAX_MOBILE_BASE}">
+  <xacro:controller_plugin_gazebo robot_namespace=""/>
+</xacro:if>
 </robot>
