Commit message: Add steering/rolling wheels

File: relax_urdf/urdf/gazebo/xbot.gazebo.xacro (robot description, xacro)
@@ -2,27 +2,28 @@
 <robot xmlns:xacro="http://ros.org/wiki/xacro">
 <gazebo>
-<!--
     <plugin name="xbot2_link_state_sensor" filename="libxbot2_gz_link_state_sensor.so">
         <links>
-            <link name="pelvis"/>
-            <link name="wheel_1"/>
+            <link name="base_link"/>
+            <link name="left_wheel"/>
         </links>
-    </plugin>-->
+    </plugin>
+    <!--
+    <plugin name="xbot2_ft_driver" filename="libxbot2_gz_ft_server.so"/>
+    <plugin name="xbot2_imu_driver" filename="libxbot2_gz_imu_server.so"/>-->
     <plugin name="xbot2_joint_driver" filename="libxbot2_gz_joint_server.so">
         <pid>
-            <!-- TODO -> CHANGE PARAMS              --><!--
+            <!-- TODO -> CHANGE PARAMS              -->
             <gain name="lowpwr_mot" p="50"  d="5"/>
             <gain name="small_mot"  p="250"  d="5"/>
             <gain name="medium_mot" p="1000" d="10"/>
-            <gain name="big_mot"    p="3000" d="10"/>-->
+            <gain name="big_mot"    p="3000" d="10"/>
             <gain name="wheel_mot"  p="0" d="10"/>
             <pid name="j_left_wheel"     profile="wheel_mot"/>
             <pid name="j_right_wheel"     profile="wheel_mot"/>
-            <!--
             <pid name="joint1" profile="medium_mot"/>
             <pid name="joint2" profile="medium_mot"/>
             <pid name="joint3" profile="medium_mot"/>
             <pid name="joint4" profile="small_mot"/>
-            <pid name="joint5" profile="small_mot"/>-->
+            <pid name="joint5" profile="small_mot"/>
         </pid>
     </plugin>

File: relax_urdf/urdf/parts/mobile_base.urdf.xacro (robot description, xacro)
@@ -30,5 +30,5 @@
     <visual>
       <origin xyz="0 0 0" rpy="0 0 0"/>
-      <geometry name="mobile_base_link_visual">
+      <geometry name="left_wheel_link_visual">
         <mesh filename="package://relax_urdf/meshes/mesh_left_wheel.stl" scale="0.001 0.001 0.001" />
       </geometry>
@@ -37,5 +37,5 @@
     <collision>
       <origin xyz="0 0 0" rpy="0 0 0"/>
-      <geometry name="mobile_base_link_collision">
+      <geometry name="left_wheel_link_collision">
         <mesh filename="package://relax_urdf/meshes/mir_base.stl" scale="0.001 0.001 0.001" />
       </geometry>
@@ -50,5 +50,5 @@
     <visual>
       <origin xyz="0 0 0" rpy="0 0 0"/>
-      <geometry name="mobile_base_link_visual">
+      <geometry name="right_wheel_link_visual">
         <mesh filename="package://relax_urdf/meshes/mesh_left_wheel.stl" scale="0.001 0.001 0.001" />
       </geometry>
@@ -57,20 +57,74 @@
     <collision>
       <origin xyz="0 0 0" rpy="0 0 0"/>
-      <geometry name="mobile_base_link_collision">
+      <geometry name="right_wheel_link_collision">
         <mesh filename="package://relax_urdf/meshes/mir_base.stl" scale="0.001 0.001 0.001" />
       </geometry>
     </collision>
 </link>
-<joint name="j_left_wheel" type="continuous">
+<link name ="left_wheel_yaw">
+    <inertial>
+      <origin xyz="0.0 0.0 0.0" rpy="0 0 0"/>
+      <mass value="1.0"/>
+      <inertia ixx="0.17" ixy="0.0" ixz="0.0" iyy="0.17" iyz="0.0" izz="0.17" />
+    </inertial>
+    <visual>
+      <origin xyz="0 0 0" rpy="0 0 0"/>
+      <geometry name="left_wheel_yaw_link_visual">
+        <box size="0.001 0.001 0.001"/>
+      </geometry>
+      <material name="dark"/>
+    </visual>
+    <collision>
+      <origin xyz="0 0 0" rpy="0 0 0"/>
+      <geometry name="left_wheel_yaw_link_collision">
+        <box size="0.001 0.001 0.001"/>
+      </geometry>
+    </collision>
+</link>
+<link name ="right_wheel_yaw">
+    <inertial>
+      <origin xyz="0.0 0.0 0.0" rpy="0 0 0"/>
+      <mass value="1.0"/>
+      <inertia ixx="0.17" ixy="0.0" ixz="0.0" iyy="0.17" iyz="0.0" izz="0.17" />
+    </inertial>
+    <visual>
+      <origin xyz="0 0 0" rpy="0 0 0"/>
+      <geometry name="right_wheel_yaw_link_visual">
+        <box size="0.001 0.001 0.001"/>
+      </geometry>
+      <material name="dark"/>
+    </visual>
+    <collision>
+      <origin xyz="0 0 0" rpy="0 0 0"/>
+      <geometry name="right_wheel_yaw_link_collision">
+        <box size="0.001 0.001 0.001"/>
+      </geometry>
+    </collision>
+</link>
+<joint name="j_left_wheel_yaw" type="revolute">
 	<parent link="mobile_base_link"/>
+	<child link="left_wheel_yaw"/>
+    <origin xyz="-0.00448719 0.25 0.09" rpy="0 0 0"/>
+	<axis xyz="0 0 1"/>
+   <limit  effort="35" velocity="20" lower="-1" upper="1" />
+</joint>
+<joint name="j_right_wheel_yaw" type="revolute">
+	<parent link="mobile_base_link"/>
+	<child link="right_wheel_yaw"/>
+	<origin xyz="-0.00448719 -0.25 0.09" rpy="0 0 0"/>
+	<axis xyz="0 0 1"/>
+   <limit  effort="35" velocity="20" lower="-1" upper="1" />
+</joint>
+<joint name="j_left_wheel_roll" type="continuous">
+	<parent link="left_wheel_yaw"/>
 	<child link="left_wheel"/>
-    <origin xyz="-0.00448719 0.25 0.09" rpy="0 0 0"/>
+    <origin xyz="0 0 0" rpy="0 0 0"/>
 	<axis xyz="0 1 0"/>
    <limit  effort="35" velocity="20"/>
 </joint>
-<joint name="j_right_wheel" type="continuous">
-	<parent link="mobile_base_link"/>
+<joint name="j_right_wheel_roll" type="continuous">
+	<parent link="right_wheel_yaw"/>
 	<child link="right_wheel"/>
-	<origin xyz="-0.00448719 -0.25 0.09" rpy="0 0 0"/>
+	<origin xyz="0 0 0" rpy="0 0 0"/>
 	<axis xyz="0 1 0"/>
    <limit  effort="35" velocity="20"/>

Commit message: using original mesh and changed pid gaind robot

File: relax_urdf/urdf/gazebo/xbot.gazebo.xacro (robot description, xacro)
@@ -18,13 +18,14 @@
             <!-- TODO -> CHANGE PARAMS              -->
             <gain name="lowpwr_mot" p="50"  d="5"/>
-            <gain name="small_mot"  p="250"  d="5"/>
-            <gain name="medium_mot" p="1000" d="10"/>
+            <gain name="small_mot"  p="250"  d="18"/>
+            <gain name="medium_mot" p="1000" d="37"/>
+            <gain name="high_mot"   p="2000" d="50"/>
             <gain name="big_mot"    p="3000" d="10"/>
             <gain name="wheel_mot"  p="10" d="2"/>
-            <pid name="relax_arm1_joint1" profile="medium_mot"/>
-            <pid name="relax_arm1_joint2" profile="medium_mot"/>
-            <pid name="relax_arm1_joint3" profile="medium_mot"/>
-            <pid name="relax_arm1_joint4" profile="small_mot"/>
-            <pid name="relax_arm1_joint5" profile="small_mot"/>
+            <pid name="relax_arm1_joint1" profile="high_mot"/>
+            <pid name="relax_arm1_joint2" profile="high_mot"/>
+            <pid name="relax_arm1_joint3" profile="high_mot"/>
+            <pid name="relax_arm1_joint4" profile="high_mot"/>
+            <pid name="relax_arm1_joint5" profile="high_mot"/>
         </pid>
     </plugin>

File: relax_urdf/urdf/parts/kinematics_properties.urdf.xacro (robot description, xacro)
@@ -3,5 +3,5 @@
 <!-- ARM -->
 <!-- Joint 0 Origin : Base - Link 1 -->
-<xacro:property name="Joint_0_Ox" value=" ${-130.000*mmTom} "/>
+<xacro:property name="Joint_0_Ox" value=" ${-134.485*mmTom} "/>
 <xacro:property name="Joint_0_Oy" value=" 0.0 "/>
 <xacro:property name="Joint_0_Oz" value=" ${ 361.300*mmTom} "/>

File: relax_urdf/urdf/relax_arm_teraflex.urdf (robot description, URDF)
Before this commit: robot relax, 17 links, 16 joints
Joints:
- joint relax_arm1_joint0: origin xyz=-0.13 0.0 0.3613 rpy=0.0 0.0 0.0 -> xyz=-0.134485 0.0 0.3613 rpy=0.0 0.0 0.0
