Commit message: push planner

File: relax_urdf/urdf/gazebo/mir.gazebo.xacro (robot description, xacro)
@@ -29,5 +29,5 @@
       <mu1 value="${friction}"/>
       <mu2 value="${friction}"/>
-      <kp value="10000000.0"/>
+      <kp value="100000000000.0"/>
       <kd value="1.0"/>
       <minDepth>0.01</minDepth>

File: relax_urdf/urdf/parts/wheels.urdf.xacro (robot description, xacro)
@@ -5,10 +5,10 @@
        the bounding box and also shifted a bit to the back, because most of the mass
        is in the lower center back (because of the batteries). -->
-  <xacro:property name="mir_base_inertial_x" value="-0.05" />
+  <xacro:property name="mir_base_inertial_x" value="0" />
   <xacro:property name="mir_base_inertial_y" value="0.0" />
   <xacro:property name="mir_base_inertial_z" value="0.15" />
-  <xacro:property name="mir_base_inertial_x_length" value="0.50" />
-  <xacro:property name="mir_base_inertial_y_length" value="0.30" />
-  <xacro:property name="mir_base_inertial_z_length" value="0.20" />
+  <xacro:property name="mir_base_inertial_x_length" value="0.80" />
+  <xacro:property name="mir_base_inertial_y_length" value="0.58" />
+  <xacro:property name="mir_base_inertial_z_length" value="0.30" />
   <xacro:property name="mir_base_mass" value="97.0" />
   <xacro:property name="mir_act_wheel_radius" value="0.100" />
