Commit message: Update relax_fixed_base.urdf.xacro

File: relax_urdf/urdf/config/relax_fixed_base.urdf.xacro (robot description, xacro)
@@ -7,3 +7,5 @@
 <!-- ************FIXED BASE*************-->
 <xacro:property name="RELAX_FIXED_BASE" value="true" />
+<!-- ************MOBILE BASE*************-->
+<xacro:property name="RELAX_MOBILE_BASE" value="false" />
 </robot>
