Commit message: Update relax_fake_base.urdf.xacro

File: relax_urdf/urdf/config/relax_fake_base.urdf.xacro (robot description, xacro)
@@ -9,3 +9,5 @@
 <!-- ************MOBILE BASE*************-->
 <xacro:property name="RELAX_MOBILE_BASE" value="false" />
+<!-- ************FAKE BASE*************-->
+<xacro:property name="RELAX_FAKE_BASE" value="true" />
 </robot>
