Commit message: Update relax_mobile_base.urdf.xacro

File: relax_urdf/urdf/config/relax_mobile_base.urdf.xacro (robot description, xacro)
@@ -9,3 +9,5 @@
 <!-- ************MOBILE BASE*************-->
 <xacro:property name="RELAX_MOBILE_BASE" value="true" />
+<!-- ************FAKE BASE*************-->
+<xacro:property name="RELAX_FAKE_BASE" value="false" />
 </robot>
