Commit message: porting repo from old to new version - relax_urdf changes made - ref issue #13

File: relax_urdf/urdf/config/relax_virtual_frame.urdf.xacro (robot description, xacro)
@@ -6,19 +6,9 @@
 <xacro:arg name="arm" default="true"/>
 <xacro:arg name="base" default="true"/>
-<!-- For sensors, you can use realsense=true argument to add all cameras (for now only d435i_control_box)
-or realsense=false togheter with d435_xxx=true to add single ones. This is like the centauro_urdf conf-->
-<xacro:arg name="realsense" default="true"/>
-<xacro:if value="$(arg realsense)">
-	<xacro:arg name="d435i_control_box" default="true"/>
-</xacro:if>
-<xacro:unless value="$(arg realsense)">
-	<xacro:arg name="d435i_control_box" default="false"/>
-</xacro:unless>
-<xacro:arg name="floating_joint" default="true"/>
 <!-- ************SELECT PARTS*************-->
 <!-- *************************************-->
 <!-- ************FLOATING BASE*************-->
 <xacro:property name="RELAX_FLOATING_BASE" value="$(arg floating_joint)" />
-<xacro:property name="ADD_VIRTUAL_FRAME" value="false" />
+<xacro:property name="ADD_VIRTUAL_FRAME" value="true" />
 <!-- ************ARM*************-->
 <xacro:property name="RELAX_ARM" value="$(arg arm)" />
@@ -26,4 +16,4 @@
 <xacro:property name="RELAX_MOBILE_BASE" value="$(arg base)" />
 <!--***************** CAMS **********-->
-<xacro:property name="ADD_D435I_CONTROL_BOX" value="$(arg d435i_control_box)" />
+<xacro:property name="ADD_D435I_CONTROL_BOX" value="false" />
 </robot>
