Commit message: Update relax.urdf.xacro

File: relax_urdf/urdf/config/relax.urdf.xacro (robot description, xacro)
@@ -0,0 +1,4 @@
+<?xml version="1.0"?>
+<robot xmlns:xacro="http://ros.org/wiki/xacro" name="RELAX">
+<xacro:property name="model_name" value="IIT RELAX" />
+<xacro:property name="model_version" value="0.1" />

Commit message: Update relax.urdf.xacro

File: relax_urdf/urdf/config/relax.urdf.xacro (robot description, xacro)
@@ -1,5 +1,9 @@
 <?xml version="1.0"?>
-<robot xmlns:xacro="http://ros.org/wiki/xacro" name="RELAX">
+<robot xmlns:xacro="http://ros.org/wiki/xacro" name="relax">
 <xacro:property name="model_name" value="IIT RELAX" />
 <xacro:property name="model_version" value="0.1" />
+<!-- ************FLOATING BASE*************-->
+<xacro:property name="RELAX_FLOATING_BASE" value="false" />
+<!-- ************FIXED BASE*************-->
+<xacro:property name="RELAX_FIXED_BASE" value="false" />
 </robot>

Commit message: Update relax.urdf.xacro

File: relax_urdf/urdf/config/relax.urdf.xacro (robot description, xacro)
@@ -9,3 +9,5 @@
 <!-- ************MOBILE BASE*************-->
 <xacro:property name="RELAX_MOBILE_BASE" value="false" />
+<!-- ************FAKE BASE*************-->
+<xacro:property name="RELAX_FAKE_BASE" value="false" />
 </robot>

Commit message: Update files

File: relax_urdf/urdf/config/relax.urdf.xacro (robot description, xacro)
@@ -4,9 +4,11 @@
 <xacro:property name="model_version" value="0.1" />
 <!-- ************FLOATING BASE*************-->
-<xacro:property name="RELAX_FLOATING_BASE" value="false" />
+<xacro:property name="RELAX_FLOATING_BASE" value="true" />
+<!-- ************ARM*************-->
+<xacro:property name="RELAX_ARM" value="true" />
 <!-- ************FIXED BASE*************-->
 <xacro:property name="RELAX_FIXED_BASE" value="false" />
 <!-- ************MOBILE BASE*************-->
-<xacro:property name="RELAX_MOBILE_BASE" value="false" />
+<xacro:property name="RELAX_MOBILE_BASE" value="true" />
 <!-- ************FAKE BASE*************-->
 <xacro:property name="RELAX_FAKE_BASE" value="false" />

File: relax_urdf/urdf/parts/mobile_base.urdf.xacro (robot description, xacro)
@@ -22,8 +22,10 @@
     </collision>
 </link>
-<joint name="mobile_base_joint" type="fixed"> <!-- mobile base joint -->
-    <parent link="mobile_base_link"/>
-    <child link="relax_link1"/>
-    <origin xyz="0 0 ${320.000*mmTom}" rpy="3.1415927 0 0"/>
-</joint>
+<xacro:if value="${RELAX_ARM}">
+    <joint name="mobile_base_joint" type="fixed"> <!-- mobile base joint -->
+        <parent link="mobile_base_link"/>
+        <child link="relax_link1"/>
+        <origin xyz="0 0 ${320.000*mmTom}" rpy="3.1415927 0 0"/>
+    </joint>
+</xacro:if>
 </robot>

File: relax_urdf/urdf/relax.urdf.xacro (robot description, xacro)
@@ -2,5 +2,5 @@
 <robot xmlns:xacro="http://ros.org/wiki/xacro" name="relax">
 <!-- ************ MODEL CONFIGURATION ************ -->
-<xacro:include filename="$(find relax_urdf)/urdf/relax_config.urdf.xacro" />
+<xacro:include filename="$(find relax_urdf)/urdf/config/relax.urdf.xacro" />
 <!-- ************ UTILS ************ -->
 <xacro:include filename="$(find relax_urdf)/urdf/relax_utils.urdf.xacro"/>

File: relax_urdf/urdf/relax_base.urdf.xacro (robot description, xacro)
@@ -3,18 +3,42 @@
 <!-- **** base attached to robot **** -->
 <xacro:if value="${RELAX_FLOATING_BASE}">
-	<link name="base_link"/>
-	<joint name="base_joint" type="fixed">
-    		<parent link="base_link"/>
-    		<child link="relax_link1"/>
-    		<origin xyz="0 0 0" rpy="0 0 0" />
-	</joint>
+    <xacro:if value="${RELAX_MOBILE_BASE}">
+        <link name="base_link"/>
+        <joint name="base_joint" type="fixed">
+                <parent link="base_link"/>
+                <child link="mobile_base_link"/>
+                <origin xyz="0 0 0" rpy="0 0 0" />
+        </joint>
+    </xacro:if>
+    <xacro:unless value="${RELAX_MOBILE_BASE}">
+        <xacro:if value="${RELAX_ARM}">
+            <link name="base_link"/>
+            <joint name="base_joint" type="fixed">
+                    <parent link="base_link"/>
+                    <child link="relax_link1"/>
+                    <origin xyz="0 0 0" rpy="0 0 0" />
+            </joint>
+        </xacro:if>
+    </xacro:unless>
 </xacro:if>
 <xacro:if value="${RELAX_FIXED_BASE}">
-	<link name="base_link"/>
-	<joint name="base_joint" type="fixed">
-    		<parent link="base_link"/>
-    		<child link="relax_link1"/>
-    		<origin xyz="0 0 0" rpy="0 0 0" />
-	</joint>
+    <xacro:if value="${RELAX_MOBILE_BASE}">
+        <link name="base_link"/>
+        <joint name="base_joint" type="fixed">
+                <parent link="base_link"/>
+                <child link="mobile_base_link"/>
+                <origin xyz="0 0 0" rpy="0 0 0" />
+        </joint>
+    </xacro:if>
+    <xacro:unless value="${RELAX_MOBILE_BASE}">
+        <xacro:if value="${RELAX_ARM}">
+            <link name="base_link"/>
+            <joint name="base_joint" type="fixed">
+                    <parent link="base_link"/>
+                    <child link="relax_link1"/>
+                    <origin xyz="0 0 0" rpy="0 0 0" />
+            </joint>
+        <xacro:if/>
+    </xacro:unless>
 </xacro:if>
 <!-- ********  attach robot  ******** -->

Commit message: Fix errors

File: relax_urdf/urdf/config/relax.urdf.xacro (robot description, xacro)
@@ -11,5 +11,3 @@
 <!-- ************MOBILE BASE*************-->
 <xacro:property name="RELAX_MOBILE_BASE" value="true" />
-<!-- ************FAKE BASE*************-->
-<xacro:property name="RELAX_FAKE_BASE" value="false" />
 </robot>

File: relax_urdf/urdf/relax_base.urdf.xacro (robot description, xacro)
@@ -39,5 +39,5 @@
                     <origin xyz="0 0 0" rpy="0 0 0" />
             </joint>
-        <xacro:if/>
+        </xacro:if>
     </xacro:unless>
 </xacro:if>
@@ -47,8 +47,6 @@
 </xacro:if>
 <!-- ********  attach robot  ******** -->
-<xacro:if value="${RELAX_FAKE_BASE}">
-<xacro:include filename="$(find relax_urdf)/urdf/parts/fake_base.urdf.xacro" />
+<xacro:if value="${RELAX_ARM}">
+    <xacro:include filename="$(find relax_urdf)/urdf/parts/arm.urdf.xacro" />
 </xacro:if>
-<!-- ********  attach robot  ******** -->
-<xacro:include filename="$(find relax_urdf)/urdf/parts/arm.urdf.xacro" />
 </robot>

Commit message: Adding srdf, based and adjust booleans

File: relax_urdf/urdf/config/relax.urdf.xacro (robot description, xacro)
@@ -7,6 +7,4 @@
 <!-- ************ARM*************-->
 <xacro:property name="RELAX_ARM" value="true" />
-<!-- ************FIXED BASE*************-->
-<xacro:property name="RELAX_FIXED_BASE" value="false" />
 <!-- ************MOBILE BASE*************-->
 <xacro:property name="RELAX_MOBILE_BASE" value="true" />

File: relax_urdf/urdf/gazebo/relax.gazebo.xacro (robot description, xacro)
@@ -1,4 +1,74 @@
 <?xml version="1.0"?>
 <robot xmlns:xacro="http://ros.org/wiki/xacro">
+<xacro:if value="${RELAX_MOBILE_BASE}">
+    <gazebo reference="wheel_left">
+        <material>Gazebo/DarkGrey </material>
+        <collision>
+            <surface>
+                <friction>
+                    <ode>
+                        <mu>0.5</mu>
+                        <mu2>0.5</mu2>
+                    </ode>
+                    <bullet>
+                        <friction>0.5</friction>
+                        <friction2>0.5</friction2>
+                    </bullet>
+                </friction>
+                <contact>
+                    <ode>
+                        <kp>2100000</kp>
+                        <kd>1</kd>
+                        <max_vel>100</max_vel>
+                    </ode>
+                    <bullet>
+                        <soft_cfm>0.007</soft_cfm>
+                        <soft_erp>0.25</soft_erp>
+                        <kp>1000000</kp>
+                        <kd>5</kd>
+                    </bullet>
+                </contact>
+            </surface>
+        </collision>
+    </gazebo>
+    <gazebo reference="wheel_right">
+        <material>Gazebo/DarkGrey </material>
+        <collision>
+            <surface>
+                <friction>
+                    <ode>
+                        <mu>0.5</mu>
+                        <mu2>0.5</mu2>
+                    </ode>
+                    <bullet>
+                        <friction>0.5</friction>
+                        <friction2>0.5</friction2>
+                    </bullet>
+                </friction>
+                <contact>
+                    <ode>
+                        <kp>2100000</kp>
+                        <kd>1</kd>
+                        <max_vel>100</max_vel>
+                    </ode>
+                    <bullet>
+                        <soft_cfm>0.007</soft_cfm>
+                        <soft_erp>0.25</soft_erp>
+                        <kp>1000000</kp>
+                        <kd>5</kd>
+                    </bullet>
+                </contact>
+            </surface>
+        </collision>
+    </gazebo>
+    <gazebo reference="j_wheel_left">
+        <implicitSpringDamper>1</implicitSpringDamper>
+        <provideFeedback>true</provideFeedback>
+    </gazebo>
+    <gazebo reference="j_wheel_right">
+        <implicitSpringDamper>1</implicitSpringDamper>
+        <provideFeedback>true</provideFeedback>
+    </gazebo>
+</xacro:if>
 <!-- <gazebo reference="joint1">
 	<implicitSpringDamper>1</implicitSpringDamper>

File: relax_urdf/urdf/parts/mobile_base.urdf.xacro (robot description, xacro)
@@ -5,6 +5,6 @@
     <inertial>
       <origin xyz="0.0 0.0 0.0" rpy="0 0 0"/>
-      <mass value="0.0"/>
-      <inertia ixx="0.0" ixy="0.0" ixz="0.0" iyy="0.0" iyz="0.0" izz="0.0" />
+      <mass value="10.0"/>
+      <inertia ixx="1.7" ixy="0.0" ixz="0.0" iyy="1.7" iyz="0.0" izz="1.7" />
     </inertial>
     <visual>
@@ -22,4 +22,94 @@
     </collision>
 </link>
+<link name ="left_wheel_motor">
+    <inertial>
+      <origin xyz="0.0 0.0 0.0" rpy="0 0 0"/>
+      <mass value="0.1"/>
+      <inertia ixx="0.017" ixy="0.0" ixz="0.0" iyy="0.017" iyz="0.0" izz="0.017" />
+    </inertial>
+    <visual>
+      <origin xyz="0 0 0" rpy="0 0 0"/>
+    </visual>
+    <collision>
+      <origin xyz="0 0 0" rpy="0 0 0"/>
+    </collision>
+</link>
+<link name ="left_wheel">
+    <inertial>
+      <origin xyz="0.0 0.0 0.0" rpy="0 0 0"/>
+      <mass value="1.0"/>
+      <inertia ixx="0.17" ixy="0.0" ixz="0.0" iyy="0.17" iyz="0.0" izz="0.17" />
+    </inertial>
+    <visual>
+      <origin xyz="0 0 0" rpy="0 0 0"/>
+      <geometry name="mobile_base_link_visual">
+        <mesh filename="package://relax_urdf/meshes/mesh_left_wheel.stl" scale="0.001 0.001 0.001" />
+      </geometry>
+      <material name="dark"/>
+    </visual>
+    <collision>
+      <origin xyz="0 0 0" rpy="0 0 0"/>
+      <geometry name="mobile_base_link_collision">
+        <mesh filename="package://relax_urdf/meshes/mir_base.stl" scale="0.001 0.001 0.001" />
+      </geometry>
+    </collision>
+</link>
+<link name ="right_wheel_motor">
+    <inertial>
+      <origin xyz="0.0 0.0 0.0" rpy="0 0 0"/>
+      <mass value="0.1"/>
+      <inertia ixx="0.017" ixy="0.0" ixz="0.0" iyy="0.017" iyz="0.0" izz="0.017" />
+    </inertial>
+    <visual>
+      <origin xyz="0 0 0" rpy="0 0 0"/>
+    </visual>
+    <collision>
+      <origin xyz="0 0 0" rpy="0 0 0"/>
+    </collision>
+</link>
+<link name ="right_wheel">
+    <inertial>
+      <origin xyz="0.0 0.0 0.0" rpy="0 0 0"/>
+      <mass value="1.0"/>
+      <inertia ixx="0.17" ixy="0.0" ixz="0.0" iyy="0.17" iyz="0.0" izz="0.17" />
+    </inertial>
+    <visual>
+      <origin xyz="0 0 0" rpy="0 0 0"/>
+      <geometry name="mobile_base_link_visual">
+        <mesh filename="package://relax_urdf/meshes/mesh_left_wheel.stl" scale="0.001 0.001 0.001" />
+      </geometry>
+      <material name="dark"/>
+    </visual>
+    <collision>
+      <origin xyz="0 0 0" rpy="0 0 0"/>
+      <geometry name="mobile_base_link_collision">
+        <mesh filename="package://relax_urdf/meshes/mir_base.stl" scale="0.001 0.001 0.001" />
+      </geometry>
+    </collision>
+</link>
+<joint name="j_l_motor" type="fixed">
+	<parent link="mobile_base_link"/>
+	<child link="left_wheel_motor"/>
+    <origin xyz="-0.00448719 0.25 0.09" rpy="0 0 0"/>
+</joint>
+<joint name="j_r_motor" type="fixed">
+	<parent link="mobile_base_link"/>
+	<child link="right_wheel_motor"/>
+	<origin xyz="-0.00448719 -0.25 0.09" rpy="0 0 0"/>
+</joint>
+<joint name="j_left_wheel" type="continuous">
+	<parent link="left_wheel_motor"/>
+	<child link="left_wheel"/>
+    <origin xyz="0 0 0" rpy="0 0 0"/>
+	<axis xyz="0 0 -1"/>
+   <limit  effort="35" velocity="20"/>
+</joint>
+<joint name="j_right_wheel" type="continuous">
+	<parent link="right_wheel_motor"/>
+	<child link="right_wheel"/>
+    <origin xyz="0 0 0" rpy="0 0 0"/>
+	<axis xyz="0 0 1"/>
+   <limit  effort="35" velocity="20"/>
+</joint>
 <xacro:if value="${RELAX_ARM}">
     <joint name="mobile_base_joint" type="fixed"> <!-- mobile base joint -->

File: relax_urdf/urdf/relax.urdf.xacro (robot description, xacro)
@@ -16,5 +16,5 @@
 	</joint>
 </xacro:if>
-<xacro:if value="${RELAX_FIXED_BASE}" > <!-- fixed base -->
+<xacro:unless value="${RELAX_FLOATING_BASE}" > <!-- fixed base -->
   	<link name="world"/>
    	<joint name="world_joint" type="fixed">
@@ -23,4 +23,4 @@
   	</joint>
     <origin xyz="0 0 0" rpy="0 0 0" />
-</xacro:if>
+</xacro:unless>
 </robot>

File: relax_urdf/urdf/relax_base.urdf.xacro (robot description, xacro)
@@ -6,7 +6,7 @@
         <link name="base_link"/>
         <joint name="base_joint" type="fixed">
-                <parent link="base_link"/>
-                <child link="mobile_base_link"/>
-                <origin xyz="0 0 0" rpy="0 0 0" />
+            <parent link="base_link"/>
+            <child link="mobile_base_link"/>
+            <origin xyz="0 0 0" rpy="0 0 0" />
         </joint>
     </xacro:if>
@@ -15,18 +15,18 @@
             <link name="base_link"/>
             <joint name="base_joint" type="fixed">
-                    <parent link="base_link"/>
-                    <child link="relax_link1"/>
-                    <origin xyz="0 0 0" rpy="0 0 0" />
+                <parent link="base_link"/>
+                <child link="relax_link1"/>
+                <origin xyz="0 0 0" rpy="${PI} 0 0" />
             </joint>
         </xacro:if>
     </xacro:unless>
 </xacro:if>
-<xacro:if value="${RELAX_FIXED_BASE}">
+<xacro:unless value="${RELAX_FLOATING_BASE}">
     <xacro:if value="${RELAX_MOBILE_BASE}">
         <link name="base_link"/>
         <joint name="base_joint" type="fixed">
-                <parent link="base_link"/>
-                <child link="mobile_base_link"/>
-                <origin xyz="0 0 0" rpy="0 0 0" />
+            <parent link="base_link"/>
+            <child link="mobile_base_link"/>
+            <origin xyz="0 0 0" rpy="0 0 0" />
         </joint>
     </xacro:if>
@@ -35,11 +35,11 @@
             <link name="base_link"/>
             <joint name="base_joint" type="fixed">
-                    <parent link="base_link"/>
-                    <child link="relax_link1"/>
-                    <origin xyz="0 0 0" rpy="0 0 0" />
+                <parent link="base_link"/>
+                <child link="relax_link1"/>
+                <origin xyz="0 0 0" rpy="${PI} 0 0" />
             </joint>
         </xacro:if>
     </xacro:unless>
-</xacro:if>
+</xacro:unless>
 <!-- ********  attach robot  ******** -->
 <xacro:if value="${RELAX_MOBILE_BASE}">

Commit message: add arguments in config similar to centauro urdf

File: relax_urdf/urdf/config/relax.urdf.xacro (robot description, xacro)
@@ -3,10 +3,24 @@
 <xacro:property name="model_name" value="IIT RELAX" />
 <xacro:property name="model_version" value="1.0" />
+<!-- command line arguments -->
+<xacro:arg name="arm" default="true"/>
+<xacro:arg name="base" default="true"/>
+<!-- For sensors, you can use realsense=true argument to add all cameras (for now only d435i_control_box)
+or realsense=false togheter with d435_xxx=true to add single ones. This is like the centauro_urdf conf-->
+<xacro:arg name="realsense" default="true"/>
+<xacro:if value="$(arg realsense)">
+	<xacro:arg name="d435i_control_box" default="true"/>
+</xacro:if>
+<xacro:unless value="$(arg realsense)">
+	<xacro:arg name="d435i_control_box" default="false"/>
+</xacro:unless>
+<xacro:arg name="floating_joint" default="true"/>
 <!-- ************FLOATING BASE*************-->
-<xacro:property name="RELAX_FLOATING_BASE" value="true" />
+<xacro:property name="RELAX_FLOATING_BASE" value="$(arg floating_joint)" />
 <!-- ************ARM*************-->
-<xacro:property name="RELAX_ARM" value="true" />
+<xacro:property name="RELAX_ARM" value="$(arg arm)" />
 <!-- ************MOBILE BASE*************-->
-<xacro:property name="RELAX_MOBILE_BASE" value="true" />
-<xacro:property name="USE_REALSENSE" value="true" />
+<xacro:property name="RELAX_MOBILE_BASE" value="$(arg base)" />
+<!--***************** CAMS **********-->
+<xacro:property name="ADD_D435I_CONTROL_BOX" value="$(arg d435i_control_box)" />
 </robot>

File: relax_urdf/urdf/parts/mobile_base.urdf.xacro (robot description, xacro)
@@ -156,5 +156,5 @@
    <limit  effort="35" velocity="20"/>
 </joint>
-<xacro:if value="${USE_REALSENSE}">
+<xacro:if value="${ADD_D435I_CONTROL_BOX}">
     <xacro:include filename="$(find realsense_gazebo_description)/urdf/_d435i.urdf.xacro" />
         <xacro:sensor_d435i parent="control_box" name="D435i_camera" topics_ns="D435i/D435i_camera"

Commit message: Add param for enabling controllers

File: relax_urdf/urdf/config/relax.urdf.xacro (robot description, xacro)
@@ -16,4 +16,5 @@
 </xacro:unless>
 <xacro:arg name="floating_joint" default="true"/>
+<xacro:arg name="use_nav_controllers" default="true"/>
 <!-- ************SELECT PARTS*************-->
 <!-- *************************************-->
@@ -27,3 +28,4 @@
 <!--***************** CAMS **********-->
 <xacro:property name="ADD_D435I_CONTROL_BOX" value="$(arg d435i_control_box)" />
+<xacro:property name="USE_NAV_CONTROLLERS" value="$(arg use_nav_controllers)" />
 </robot>

File: relax_urdf/urdf/parts/mobile_base.urdf.xacro (robot description, xacro)
@@ -91,8 +91,10 @@
     </joint>
     <link name="${prefix}surface"/>
-    <xacro:mir_wheel_transmissions prefix="${prefix}"/>
-    <!-- set the gazebo friction parameters for the wheels -->
-    <xacro:set_all_wheel_frictions prefix="${prefix}"/>
-    <xacro:p3d_base_controller prefix="${prefix}" />
+    <xacro:if value="${USE_NAV_CONTROLLERS}">
+        <xacro:mir_wheel_transmissions prefix="${prefix}"/>
+        <!-- set the gazebo friction parameters for the wheels -->
+        <xacro:set_all_wheel_frictions prefix="${prefix}"/>
+        <xacro:p3d_base_controller prefix="${prefix}" />
+    </xacro:if>
 <!--
 <xacro:if value="${ADD_D435I_CONTROL_BOX}">

File: relax_urdf/urdf/relax_robot.urdf.xacro (robot description, xacro)
@@ -18,5 +18,7 @@
 </xacro:unless>
 <xacro:if value="${RELAX_MOBILE_BASE}">
-  <xacro:controller_plugin_gazebo robot_namespace=""/>
+    <xacro:if value="${USE_NAV_CONTROLLERS}">
+        <xacro:controller_plugin_gazebo robot_namespace=""/>
+    </xacro:if>
 </xacro:if>
 </robot>
