Commit message: D435 camera mounted

File: relax_urdf/urdf/config/relax.urdf.xacro (robot description, xacro)
@@ -8,5 +8,5 @@
 <!-- For sensors, you can use realsense=true argument to add all cameras (for now only d435i_control_box)
 or realsense=false togheter with d435_xxx=true to add single ones. This is like the centauro_urdf conf-->
-<xacro:arg name="realsense" default="false"/>
+<xacro:arg name="realsense" default="true"/>
 <xacro:if value="$(arg realsense)">
 	<xacro:arg name="d435i_control_box" default="true"/>

File: relax_urdf/urdf/config/relax_xbot2.urdf.xacro (robot description, xacro)
@@ -8,5 +8,5 @@
 <!-- For sensors, you can use realsense=true argument to add all cameras (for now only d435i_control_box)
 or realsense=false togheter with d435_xxx=true to add single ones. This is like the centauro_urdf conf-->
-<xacro:arg name="realsense" default="false"/>
+<xacro:arg name="realsense" default="true"/>
 <xacro:if value="$(arg realsense)">
 	<xacro:arg name="d435i_control_box" default="true"/>

File: relax_urdf/urdf/parts/mir_base.urdf.xacro (robot description, xacro)
@@ -38,4 +38,283 @@
       <material>Gazebo/DarkGrey</material>
     </gazebo>
+  <!-- Depth Camera -->
+ <material name="D435i_camera_aluminum">
+    <color rgba="0.5 0.5 0.5 1"/>
+  </material>
+  <!-- camera body, with origin at bottom screw mount -->
+  <joint name="D435i_camera_joint" type="fixed">
+    <origin rpy="0 0.0 0" xyz="0.1 0 0.3815997"/>
+    <parent link="${prefix}base_link"/>
+    <child link="D435i_camera_bottom_screw_frame"/>
+  </joint>
+  <link name="D435i_camera_bottom_screw_frame"/>
+  <joint name="D435i_camera_link_joint" type="fixed">
+    <origin rpy="0 0 0" xyz="0 0.0175 0.0125"/>
+    <parent link="D435i_camera_bottom_screw_frame"/>
+    <child link="D435i_camera_link"/>
+  </joint>
+  <link name="D435i_camera_link">
+    <visual>
+      <origin rpy="1.57079632679 0 1.57079632679" xyz="0.0149 -0.0175 0"/>
+      <geometry>
+        <!-- <box size="${d435i_cam_width} ${d435i_cam_height} ${d435i_cam_depth}"/> -->
+        <mesh filename="package://realsense2_description/meshes/d435.dae"/>
+        <!--<mesh filename="package://realsense2_description/meshes/d435/d435.dae"/>-->
+      </geometry>
+      <material name="D435i_camera_aluminum"/>
+    </visual>
+    <collision>
+      <origin rpy="0 0 0" xyz="0 -0.0175 0"/>
+      <geometry>
+        <box size="0.02505 0.09 0.025"/>
+      </geometry>
+    </collision>
+    <inertial>
+      <!-- The following are not reliable values, and should not be used for modeling -->
+      <mass value="1e-5"/>
+      <origin xyz="0 0 0"/>
+      <inertia ixx="0.003881243" ixy="0.0" ixz="0.0" iyy="0.000498940" iyz="0.0" izz="0.003879257"/>
+    </inertial>
+  </link>
+  <!-- camera depth joints and links -->
+  <joint name="D435i_camera_depth_joint" type="fixed">
+    <origin rpy="0 0 0" xyz="0 0 0"/>
+    <parent link="D435i_camera_link"/>
+    <child link="D435i_camera_depth_frame"/>
+  </joint>
+  <link name="D435i_camera_depth_frame"/>
+  <joint name="D435i_camera_depth_optical_joint" type="fixed">
+    <origin rpy="-1.57079632679 0 -1.57079632679" xyz="0 0 0"/>
+    <parent link="D435i_camera_depth_frame"/>
+    <child link="D435i_camera_depth_optical_frame"/>
+  </joint>
+  <link name="D435i_camera_depth_optical_frame"/>
+  <!-- camera left IR joints and links -->
+  <joint name="D435i_camera_left_ir_joint" type="fixed">
+    <origin rpy="0 0 0" xyz="0 0.0 0"/>
+    <parent link="D435i_camera_depth_frame"/>
+    <child link="D435i_camera_left_ir_frame"/>
+  </joint>
+  <link name="D435i_camera_left_ir_frame"/>
+  <joint name="D435i_camera_left_ir_optical_joint" type="fixed">
+    <origin rpy="-1.57079632679 0 -1.57079632679" xyz="0 0 0"/>
+    <parent link="D435i_camera_left_ir_frame"/>
+    <child link="D435i_camera_left_ir_optical_frame"/>
+  </joint>
+  <link name="D435i_camera_left_ir_optical_frame"/>
+  <!-- camera right IR joints and links -->
+  <joint name="D435i_camera_right_ir_joint" type="fixed">
+    <origin rpy="0 0 0" xyz="0 -0.05 0"/>
+    <parent link="D435i_camera_depth_frame"/>
+    <child link="D435i_camera_right_ir_frame"/>
+  </joint>
+  <link name="D435i_camera_right_ir_frame"/>
+  <joint name="D435i_camera_right_ir_optical_joint" type="fixed">
+    <origin rpy="-1.57079632679 0 -1.57079632679" xyz="0 0 0"/>
+    <parent link="D435i_camera_right_ir_frame"/>
+    <child link="D435i_camera_right_ir_optical_frame"/>
+  </joint>
+  <link name="D435i_camera_right_ir_optical_frame"/>
+  <!-- camera color joints and links -->
+  <joint name="D435i_camera_color_joint" type="fixed">
+    <origin rpy="0 0 0" xyz="0 0.015 0"/>
+    <parent link="D435i_camera_depth_frame"/>
+    <child link="D435i_camera_color_frame"/>
+  </joint>
+  <link name="D435i_camera_color_frame"/>
+  <joint name="D435i_camera_color_optical_joint" type="fixed">
+    <origin rpy="-1.57079632679 0 -1.57079632679" xyz="0 0 0"/>
+    <parent link="D435i_camera_color_frame"/>
+    <child link="D435i_camera_color_optical_frame"/>
+  </joint>
+  <link name="D435i_camera_color_optical_frame"/>
+  <!-- camera accel joints and links -->
+  <joint name="D435i_camera_accel_joint" type="fixed">
+    <origin rpy="0 0 0" xyz="-0.00174 0.00552 0.0176"/>
+    <parent link="D435i_camera_link"/>
+    <child link="D435i_camera_accel_frame"/>
+  </joint>
+  <link name="D435i_camera_accel_frame"/>
+  <joint name="D435i_camera_accel_optical_joint" type="fixed">
+    <origin rpy="-1.57079632679 0 -1.57079632679" xyz="0 0 0"/>
+    <parent link="D435i_camera_accel_frame"/>
+    <child link="D435i_camera_accel_optical_frame"/>
+  </joint>
+  <link name="D435i_camera_accel_optical_frame"/>
+  <!-- camera gyro joints and links -->
+  <joint name="D435i_camera_gyro_joint" type="fixed">
+    <origin rpy="0 0 0" xyz="-0.00174 0.00552 0.0176"/>
+    <parent link="D435i_camera_link"/>
+    <child link="D435i_camera_gyro_frame"/>
+  </joint>
+  <link name="D435i_camera_gyro_frame"/>
+  <joint name="D435i_camera_gyro_optical_joint" type="fixed">
+    <origin rpy="-1.57079632679 0 -1.57079632679" xyz="0 0 0"/>
+    <parent link="D435i_camera_gyro_frame"/>
+    <child link="D435i_camera_gyro_optical_frame"/>
+  </joint>
+  <link name="D435i_camera_gyro_optical_frame"/>
+  <gazebo reference="D435i_camera_link">
+    <self_collide>0</self_collide>
+    <enable_wind>0</enable_wind>
+    <kinematic>0</kinematic>
+    <!-- <gravity>1</gravity> -->
+    <!--<mu>1</mu>-->
+    <mu2>1</mu2>
+    <fdir1>0 0 0</fdir1>
+    <!--<slip1>0</slip1>
+      <slip2>0</slip2>-->
+    <kp>1e+13</kp>
+    <kd>1</kd>
+    <!--<max_vel>0.01</max_vel>
+      <min_depth>0</min_depth>-->
+    <sensor name="D435i_cameracolor" type="camera">
+      <camera name="D435i_camera">
+        <horizontal_fov>1.21125850088</horizontal_fov>
+        <image>
+          <width>1280</width>
+          <height>720</height>
+          <format>RGB_INT8</format>
+        </image>
+        <clip>
+          <near>0.1</near>
+          <far>100</far>
+        </clip>
+        <noise>
+          <type>gaussian</type>
+          <mean>0.0</mean>
+          <stddev>0.007</stddev>
+        </noise>
+      </camera>
+      <always_on>1</always_on>
+      <update_rate>30</update_rate>
+      <visualize>False</visualize>
+    </sensor>
+    <sensor name="D435i_cameraired1" type="camera">
+      <camera name="D435i_camera">
+        <horizontal_fov>1.4870205227</horizontal_fov>
+        <image>
+          <width>1280</width>
+          <height>720</height>
+          <format>L_INT8</format>
+        </image>
+        <clip>
+          <near>0.1</near>
+          <far>100</far>
+        </clip>
+        <noise>
+          <type>gaussian</type>
+          <mean>0.0</mean>
+          <stddev>0.05</stddev>
+        </noise>
+      </camera>
+      <always_on>1</always_on>
+      <update_rate>90</update_rate>
+      <visualize>false</visualize>
+    </sensor>
+    <sensor name="D435i_cameraired2" type="camera">
+      <camera name="D435i_camera">
+        <horizontal_fov>1.4870205227</horizontal_fov>
+        <image>
+          <width>1280</width>
+          <height>720</height>
+          <format>L_INT8</format>
+        </image>
+        <clip>
+          <near>0.1</near>
+          <far>100</far>
+        </clip>
+        <noise>
+          <type>gaussian</type>
+          <mean>0.0</mean>
+          <stddev>0.05</stddev>
+        </noise>
+      </camera>
+      <always_on>1</always_on>
+      <update_rate>90</update_rate>
+      <visualize>false</visualize>
+    </sensor>
+    <sensor name="D435i_cameradepth" type="depth">
+      <camera name="D435i_camera">
+        <horizontal_fov>1.21125850088</horizontal_fov>
+        <image>
+          <width>1280</width>
+          <height>720</height>
+        </image>
+        <clip>
+          <near>0.1</near>
+          <far>100</far>
+        </clip>
+        <noise>
+          <type>gaussian</type>
+          <mean>0.0</mean>
+          <stddev>0.100</stddev>
+        </noise>
+      </camera>
+      <always_on>1</always_on>
+      <update_rate>30</update_rate>
+      <visualize>false</visualize>
+    </sensor>
+    <sensor name="D435i_cameraaccel" type="imu">
+      <always_on>true</always_on>
+      <update_rate>300</update_rate>
+      <topic>D435i/D435i_camera/accel/sample</topic>
+      <plugin filename="librealsense_gazebo_accel_sensor.so" name="D435i/D435i_camera_accel_plugin">
+        <topicName>D435i/D435i_camera/accel/sample</topicName>
+        <bodyName>D435i_camera_link</bodyName>
+        <updateRateHZ>300</updateRateHZ>
+        <gaussianNoise>0.1</gaussianNoise>
+        <xyzOffset>0 0 0</xyzOffset>
+        <rpyOffset>0 0 0</rpyOffset>
+        <frameName>D435i_camera_accel_optical_frame</frameName>
+        <initialOrientationAsReference>false</initialOrientationAsReference>
+      </plugin>
+      <pose>0 0 0 0 0 0</pose>
+    </sensor>
+    <sensor name="D435i_cameragyro" type="imu">
+      <always_on>true</always_on>
+      <update_rate>300</update_rate>
+      <topic>D435i_camera/gyro/sample</topic>
+      <plugin filename="librealsense_gazebo_gyro_sensor.so" name="D435i/D435i_camera_gyro_plugin">
+        <topicName>D435i/D435i_camera/gyro/sample</topicName>
+        <bodyName>D435i_camera_link</bodyName>
+        <updateRateHZ>300</updateRateHZ>
+        <gaussianNoise>0.1</gaussianNoise>
+        <xyzOffset>0 0 0</xyzOffset>
+        <rpyOffset>0 0 0</rpyOffset>
+        <frameName>D435i_camera_gyro_optical_frame</frameName>
+        <initialOrientationAsReference>false</initialOrientationAsReference>
+      </plugin>
+    </sensor>
+  </gazebo>
+  <gazebo>
+    <plugin filename="librealsense_gazebo_plugin.so" name="D435i/D435i_camera">
+      <prefix>D435i_camera</prefix>
+      <!-- Color camera settings -->
+      <colorUpdateRate>30</colorUpdateRate>
+      <colorTopicName>color/image_raw</colorTopicName>
+      <colorOpticalframeName>D435i_camera_color_optical_frame</colorOpticalframeName>
+      <colorCameraInfoTopicName>color/camera_info</colorCameraInfoTopicName>
+      <!-- Infrared camera settings -->
+      <infraredUpdateRate>90</infraredUpdateRate>
+      <infrared1TopicName>infra1/image_rect_raw</infrared1TopicName>
+      <infrared2TopicName>infra2/image_rect_raw</infrared2TopicName>
+      <infrared1CameraInfoTopicName>infra1/camera_info</infrared1CameraInfoTopicName>
+      <infrared2CameraInfoTopicName>infra2/camera_info</infrared2CameraInfoTopicName>
+      <infrared1OpticalframeName>D435i_camera_left_ir_optical_frame</infrared1OpticalframeName>
+      <infrared2OpticalframeName>D435i_camera_right_ir_optical_frame</infrared2OpticalframeName>
+      <!-- Depth camera settings -->
+      <rangeMinDepth>0.2</rangeMinDepth>
+      <rangeMaxDepth>10.0</rangeMaxDepth>
+      <depthUpdateRate>30</depthUpdateRate>
+      <depthTopicName>depth/image_rect_raw</depthTopicName>
+      <depthCameraInfoTopicName>depth/camera_info</depthCameraInfoTopicName>
+      <depthOpticalframeName>D435i_camera_depth_optical_frame</depthOpticalframeName>
+      <!-- Pointlcloud settings -->
+      <pointCloud>True</pointCloud>
+      <pointCloudTopicName>depth/color/points</pointCloudTopicName>
+      <pointCloudCutoff>0.5</pointCloudCutoff>
+    </plugin>
+  </gazebo>
     <!-- IMU -->
     <joint name="${prefix}base_link_to_imu_joint" type="fixed">

Commit message: added teraflex ring sensors to the model (by default it appears)

File: relax_urdf/urdf/config/relax.urdf.xacro (robot description, xacro)
@@ -6,4 +6,5 @@
 <xacro:arg name="arm" default="true"/>
 <xacro:arg name="base" default="true"/>
+<xacro:arg name="teraflex" default="true"/>
 <!-- For sensors, you can use realsense=true argument to add all cameras (for now only d435i_control_box)
 or realsense=false togheter with d435_xxx=true to add single ones. This is like the centauro_urdf conf-->
@@ -24,4 +25,6 @@
 <!-- ************ARM*************-->
 <xacro:property name="RELAX_ARM" value="$(arg arm)" />
+<!-- ************TERAFLEX*************-->
+<xacro:property name="TERAFLEX_RING" value="$(arg teraflex)" />
 <!-- ************MOBILE BASE*************-->
 <xacro:property name="RELAX_MOBILE_BASE" value="$(arg base)" />

File: relax_urdf/urdf/config/relax_arm.urdf.xacro (robot description, xacro)
@@ -7,4 +7,5 @@
 <xacro:arg name="base" default="false"/>
 <xacro:arg name="floating_joint" default="false"/>
+<xacro:arg name="teraflex" default="true"/>
 <!-- ************SELECT PARTS*************-->
 <!-- *************************************-->
@@ -14,4 +15,6 @@
 <!-- ************ARM*************-->
 <xacro:property name="RELAX_ARM" value="$(arg arm)" />
+<!-- ************TERAFLEX*************-->
+<xacro:property name="TERAFLEX_RING" value="$(arg teraflex)" />
 <!-- ************MOBILE BASE*************-->
 <xacro:property name="RELAX_MOBILE_BASE" value="$(arg base)" />

File: relax_urdf/urdf/parts/arm.urdf.xacro (robot description, xacro)
@@ -9,4 +9,11 @@
 <xacro:relax_arm arm_num="1" >
    </xacro:relax_arm>
+<!-- sensor ring (optionally) -->
+<xacro:if value="${TERAFLEX_RING}" > <!-- teraflex - ring -->
+    <xacro:include filename="$(find relax_urdf)/urdf/parts/teraflex_ring.urdf.xacro"/>
+    <xacro:teraflex_ring id="1" parent_link="relax_arm1_link5">
+        <origin xyz=" 0.0 0.142500 -0.0881600 " rpy="-1.5707963 -0.6404992 0" />
+    </xacro:teraflex_ring>
+</xacro:if>
 <xacro:unless value="${RELAX_MOBILE_BASE}">
   <link name="base_link">

Commit message: now relax can have hands!

File: relax_urdf/urdf/config/relax.urdf.xacro (robot description, xacro)
@@ -16,4 +16,5 @@
 </xacro:unless>
 <xacro:arg name="floating_joint" default="false"/>
+<xacro:arg name="end_effector" default="none"/> <!-- none, ball, dagana_fixed, dagana -->
 <xacro:arg name="use_nav_controllers" default="true"/>
 <!-- ************SELECT PARTS*************-->
@@ -28,4 +29,6 @@
 <!--***************** CAMS **********-->
 <xacro:property name="ADD_D435I_CONTROL_BOX" value="$(arg d435i_control_box)" />
+<!--***************** END EFFECTOR **********-->
+<xacro:property name="END_EFFECTOR" value="$(arg end_effector)" />
 <xacro:property name="USE_NAV_CONTROLLERS" value="$(arg use_nav_controllers)" />
 </robot>

File: relax_urdf/urdf/config/relax_arm.urdf.xacro (robot description, xacro)
@@ -7,4 +7,5 @@
 <xacro:arg name="base" default="false"/>
 <xacro:arg name="floating_joint" default="false"/>
+<xacro:arg name="end_effector" default="none"/> <!-- none, ball, dagana_fixed, dagana -->
 <!-- ************SELECT PARTS*************-->
 <!-- *************************************-->
@@ -18,3 +19,5 @@
 <!--***************** CAMS **********-->
 <xacro:property name="ADD_D435I_CONTROL_BOX" value="false" />
+<!--***************** END EFFECTOR **********-->
+<xacro:property name="END_EFFECTOR" value="$(arg end_effector)" />
 </robot>

File: relax_urdf/urdf/gazebo/materials.gazebo.xacro (robot description, xacro)
@@ -20,3 +20,16 @@
   <material>Gazebo/Blue</material>
 </gazebo>
+<xacro:if value="${END_EFFECTOR == 'ball'}">
+	<gazebo reference="ball1">
+		<material>Gazebo/BlackTransparent</material>
+	</gazebo>
+</xacro:if>
+<xacro:if value="${END_EFFECTOR == 'dagana' or END_EFFECTOR == 'dagana_fixed'}">
+	<gazebo reference="dagana_1_top_link">
+		<material>Gazebo/BlackTransparent</material>
+	</gazebo>
+	<gazebo reference="dagana_1_bottom_link">
+		<material>Gazebo/BlackTransparent</material>
+	</gazebo>
+</xacro:if>
 </robot>

File: relax_urdf/urdf/parts/arm.urdf.xacro (robot description, xacro)
@@ -6,7 +6,8 @@
 <xacro:include filename="$(find relax_urdf)/urdf/parts/wheels.urdf.xacro" />
 <xacro:include filename="$(find relax_urdf)/urdf/parts/common_base_properties.urdf.xacro" />
-<!-- arms -->
-<xacro:relax_arm arm_num="1" >
-   </xacro:relax_arm>
+<xacro:property name="arm_num" value="1" />
+<!-- *********************************************************************** arm **************************************************************** -->
+<xacro:relax_arm arm_num="${arm_num}" />
+<!-- ******************************************************************* mobile base **************************************************************** -->
 <xacro:unless value="${RELAX_MOBILE_BASE}">
   <link name="base_link">
@@ -32,13 +33,25 @@
   </gazebo>
 </xacro:unless>
-<!-- end_effector attached -->
-<!-- <xacro:if value="${ADD_END_EFFECTOR}">
-      <xacro:include filename="$(find relax_urdf)/urdf/parts/end_effector.urdf.xacro" />
-      <xacro:end_effector arm_num="1"  parent_link="arm1_7">
-                  <origin xyz="0. 0. 0." rpy="0. 0. 0."/>
-      </xacro:end_effector>
-      <xacro:end_effector arm_num="2"  parent_link="arm2_7">
-                  <origin xyz="0. 0. 0." rpy="0. 0. 0."/>
-      </xacroend_effector>
-</xacro:if> -->
+<!-- ******************************************************************* end_effector  **************************************************************** -->
+<xacro:if value="${END_EFFECTOR == 'none'}">
+    <!-- nothing to do -->
+</xacro:if>
+<xacro:if value="${END_EFFECTOR == 'ball'}">
+	<xacro:include filename="$(find centauro_urdf)/urdf/parts/ball.urdf.xacro" />
+	<xacro:ball_end_effector arm_num="${arm_num}"  parent_link="relax_arm${arm_num}_linkEndEffector">
+		      <origin xyz="0 0 0" rpy="0. ${PI} 0."/>
+	</xacro:ball_end_effector>
+</xacro:if>
+<xacro:if value="${END_EFFECTOR == 'dagana_fixed'}">
+	<xacro:include filename="$(find dagana_urdf)/urdf/dagana_macro.urdf.xacro" />
+	<xacro:dagana_gripper name="dagana_${arm_num}" parent_link="relax_arm${arm_num}_linkEndEffector" joint_type="fixed">
+		<origin xyz="0. 0 0" rpy="0. 0 0"/>
+	</xacro:dagana_gripper>
+</xacro:if>
+<xacro:if value="${END_EFFECTOR == 'dagana'}">
+	<xacro:include filename="$(find dagana_urdf)/urdf/dagana_macro.urdf.xacro" />
+	<xacro:dagana_gripper name="dagana_${arm_num}" parent_link="relax_arm${arm_num}_linkEndEffector" joint_type="revolute">
+		<origin xyz="0. 0 0" rpy="0. 0 0"/>
+	</xacro:dagana_gripper>
+</xacro:if>
 </robot>

Commit message: ee ball

File: relax_urdf/urdf/config/relax.urdf.xacro (robot description, xacro)
@@ -16,5 +16,5 @@
 </xacro:unless>
 <xacro:arg name="floating_joint" default="false"/>
-<xacro:arg name="end_effector" default="ball"/> <!-- none, ball, dagana_fixed, dagana -->
+<xacro:arg name="end_effector" default="none"/> <!-- none, ball, dagana_fixed, dagana -->
 <xacro:arg name="use_nav_controllers" default="true"/>
 <!-- ************SELECT PARTS*************-->

File: relax_urdf/urdf/config/relax_arm.urdf.xacro (robot description, xacro)
@@ -7,5 +7,5 @@
 <xacro:arg name="base" default="false"/>
 <xacro:arg name="floating_joint" default="false"/>
-<xacro:arg name="end_effector" default="none"/> <!-- none, ball, dagana_fixed, dagana -->
+<xacro:arg name="end_effector" default="ball"/> <!-- none, ball, dagana_fixed, dagana -->
 <!-- ************SELECT PARTS*************-->
 <!-- *************************************-->

File: relax_urdf/urdf/relax_arm.urdf (robot description, URDF)
Before this commit: robot relax, 9 links, 8 joints
Links:
- added link ball1, mass 1.27; collision mesh filename=package://relax_urdf/meshes/simple/BallHand.stl scale=0.001 0.001 0.001; visual mesh filename=package://relax_urdf/meshes/BallHand.stl scale=0.001 0.001 0.001
- added link ball1_tip
Joints:
- added joint j_arm1_ball_mount_joint: type fixed, parent relax_arm1_linkEndEffector, child ball1, origin xyz=0 0 0.02 rpy=0. 3.14159265359 0.
- added joint j_ball1_tip: type fixed, parent ball1, child ball1_tip, origin xyz=0 0 -0.07 rpy=0 0 0
