Commit message: wip

File: relax_urdf/urdf/config/relax.urdf.xacro (robot description, xacro)
@@ -1,34 +1,21 @@
 <?xml version="1.0"?>
 <robot xmlns:xacro="http://ros.org/wiki/xacro" name="relax">
-<xacro:property name="model_name" value="RELAX" />
-<xacro:property name="model_version" value="1.0" />
-<!-- command line arguments -->
-<xacro:arg name="arm" default="true"/>
-<xacro:arg name="base" default="true"/>
-<!-- For sensors, you can use realsense=true argument to add all cameras (for now only d435i_control_box)
-or realsense=false togheter with d435_xxx=true to add single ones. This is like the centauro_urdf conf-->
-<xacro:arg name="realsense" default="false"/>
-<xacro:if value="$(arg realsense)">
-	<xacro:arg name="d435i_control_box" default="true"/>
-</xacro:if>
-<xacro:unless value="$(arg realsense)">
-	<xacro:arg name="d435i_control_box" default="false"/>
-</xacro:unless>
-<xacro:arg name="floating_joint" default="false"/>
-<xacro:arg name="end_effector" default="none"/> <!-- none, ball, dagana_fixed, dagana -->
-<xacro:arg name="use_nav_controllers" default="true"/>
-<!-- ************SELECT PARTS*************-->
-<!-- *************************************-->
-<!-- ************FLOATING BASE*************-->
-<xacro:property name="RELAX_FLOATING_BASE" value="$(arg floating_joint)" />
-<xacro:property name="ADD_VIRTUAL_FRAME" value="false" />
-<!-- ************ARM*************-->
-<xacro:property name="RELAX_ARM" value="$(arg arm)" />
-<!-- ************MOBILE BASE*************-->
-<xacro:property name="RELAX_MOBILE_BASE" value="$(arg base)" />
-<!--***************** CAMS **********-->
-<xacro:property name="ADD_D435I_CONTROL_BOX" value="$(arg d435i_control_box)" />
-<!--***************** END EFFECTOR **********-->
-<xacro:property name="END_EFFECTOR" value="$(arg end_effector)" />
-<xacro:property name="USE_NAV_CONTROLLERS" value="$(arg use_nav_controllers)" />
+    <xacro:property name="model_name" value="RELAX" />
+    <xacro:property name="model_version" value="1.0" />
+    <xacro:arg name="arm" default="relax_arm"/>  <!-- none, relax_arm -->
+    <xacro:arg name="base" default="fixed"/> <!-- none, fixed, floating, mir -->
+    <xacro:arg name="end_effector" default="none"/> <!-- none, ball, dagana_fixed, dagana -->
+    <!-- For sensors, you can use realsense=true argument to add all cameras (for now only d435i_control_box)
+    or realsense=false togheter with d435_xxx=true to add single ones. This is like the centauro_urdf conf-->
+    <xacro:arg name="realsense" default="false"/>
+    <xacro:if value="$(arg realsense)">
+        <xacro:arg name="d435i_control_box" default="true"/>
+    </xacro:if>
+    <xacro:unless value="$(arg realsense)">
+        <xacro:arg name="d435i_control_box" default="false"/>
+    </xacro:unless>
+    <xacro:property name="RELAX_ARM" value="$(arg arm)" />
+    <xacro:property name="RELAX_MOBILE_BASE" value="$(arg base)" />
+    <xacro:property name="END_EFFECTOR" value="$(arg end_effector)" />
+    <xacro:property name="ADD_D435I_CONTROL_BOX" value="$(arg d435i_control_box)" />
 </robot>

File: relax_urdf/urdf/gazebo/materials.gazebo.xacro (robot description, xacro)
@@ -20,4 +20,7 @@
   <material>Gazebo/Blue</material>
 </gazebo>
+<gazebo reference="base_link">
+    <material>Gazebo/DarkGrey</material>
+</gazebo>
 <xacro:if value="${END_EFFECTOR == 'ball'}">
 	<gazebo reference="ball1">

File: relax_urdf/urdf/parts/relax_arm.urdf.xacro (robot description, xacro)
@@ -1,182 +1,17 @@
 <?xml version="1.0"?>
 <robot xmlns:xacro="http://ros.org/wiki/xacro">
-<!-- macro arm -->
-<xacro:macro name="relax_arm" params="arm_num" >
-<!-- links -->
-<link name ="relax_arm${arm_num}_link1">  <!-- link 1 -->
-    <inertial>
-      <origin xyz="${Link_1_x} ${Link_1_y} ${Link_1_z}" />
-      <mass value="${Link_1_mass}"/>
-      <inertia ixx="${Link_1_xx}" ixy="${Link_1_xy}" ixz="${Link_1_xz}" iyy="${Link_1_yy}" iyz="${Link_1_yz}" izz="${Link_1_zz}" />
-    </inertial>
-    <visual>
-      <origin xyz="0 0 0" rpy="0 0 0"/>
-      <geometry name="relax_link1_visual">
-        <mesh filename="package://relax_urdf/meshes/mesh_link1.stl" scale="0.001 0.001 0.001" />
-      </geometry>
-      <material name="darkblue"/>
-    </visual>
-    <collision>
-      <origin xyz="0 0 0" rpy="0 0 0"/>
-      <geometry name="relax_link1_collision">
-        <mesh filename="package://relax_urdf/meshes/mesh_link1.stl" scale="0.001 0.001 0.001" />
-      </geometry>
-    </collision>
-</link>
-<link name ="relax_arm${arm_num}_link2">  <!-- link 2 -->
-    <inertial>
-      <origin xyz="${Link_2_x} ${Link_2_y} ${Link_2_z}" />
-      <mass value="${Link_2_mass}"/>
-      <inertia ixx="${Link_2_xx}" ixy="${Link_2_xy}" ixz="${Link_2_xz}" iyy="${Link_2_yy}" iyz="${Link_2_yz}" izz="${Link_2_zz}" />
-    </inertial>
-    <visual>
-      <origin xyz="0 0 0" rpy="0 0 0"/>
-      <geometry name="relax_link2_visual">
-        <mesh filename="package://relax_urdf/meshes/mesh_link2.stl" scale="0.001 0.001 0.001" />
-      </geometry>
-      <material name="dark"/>
-    </visual>
-    <collision>
-      <origin xyz="0 0 0" rpy="0 0 0"/>
-      <geometry name="relax_link2_collision">
-        <mesh filename="package://relax_urdf/meshes/mesh_link2.stl" scale="0.001 0.001 0.001" />
-      </geometry>
-    </collision>
-</link>
-<link name ="relax_arm${arm_num}_link3">  <!-- link 3 -->
-    <inertial>
-      <origin xyz="${Link_3_x} ${Link_3_y} ${Link_3_z}" />
-      <mass value="${Link_3_mass}"/>
-      <inertia ixx="${Link_3_xx}" ixy="${Link_3_xy}" ixz="${Link_3_xz}" iyy="${Link_3_yy}" iyz="${Link_3_yz}" izz="${Link_3_zz}" />
-    </inertial>
-    <visual>
-      <origin xyz="0 0 0" rpy="0 0 0"/>
-      <geometry name="relax_link3_visual">
-        <mesh filename="package://relax_urdf/meshes/mesh_link3.stl" scale="0.001 0.001 0.001" />
-      </geometry>
-      <material name="darkblue"/>
-    </visual>
-    <collision>
-      <origin xyz="0 0 0" rpy="0 0 0"/>
-      <geometry name="relax_link3_collision">
-        <mesh filename="package://relax_urdf/meshes/mesh_link3.stl" scale="0.001 0.001 0.001" />
-      </geometry>
-    </collision>
-</link>
-<link name ="relax_arm${arm_num}_link4">  <!-- link 4 -->
-    <inertial>
-      <origin xyz="${Link_4_x} ${Link_4_y} ${Link_4_z}"/>
-      <mass value="${Link_4_mass}"/>
-      <inertia ixx="${Link_4_xx}" ixy="${Link_4_xy}" ixz="${Link_4_xz}" iyy="${Link_4_yy}" iyz="${Link_4_yz}" izz="${Link_4_zz}" />
-    </inertial>
-    <visual>
-      <origin xyz="0 0 0" rpy="0 0 0"/>
-      <geometry name="relax_link4_visual">
-        <mesh filename="package://relax_urdf/meshes/mesh_link4.stl" scale="0.001 0.001 0.001" />
-      </geometry>
-      <material name="darkblue"/>
-    </visual>
-    <collision>
-      <origin xyz="0 0 0" rpy="0 0 0"/>
-      <geometry name="relax_link4_collision">
-        <mesh filename="package://relax_urdf/meshes/mesh_link4.stl" scale="0.001 0.001 0.001" />
-      </geometry>
-    </collision>
-</link>
-<link name ="relax_arm${arm_num}_link5">  <!-- link 5 -->
-    <inertial>
-      <origin xyz="${Link_5_x} ${Link_5_y} ${Link_5_z}" />
-      <mass value="${Link_5_mass}"/>
-      <inertia ixx="${Link_5_xx}" ixy="${Link_5_xy}" ixz="${Link_5_xz}" iyy="${Link_5_yy}" iyz="${Link_5_yz}" izz="${Link_5_zz}" />
-    </inertial>
-    <visual>
-      <origin xyz="0 0 0" rpy="0 0 0"/>
-      <geometry name="relax_link5_visual">
-        <mesh filename="package://relax_urdf/meshes/mesh_link5.stl" scale="0.001 0.001 0.001" />
-      </geometry>
-      <material name="darkblue"/>
-    </visual>
-    <collision>
-      <origin xyz="0 0 0" rpy="0 0 0"/>
-      <geometry name="relax_link5_collision">
-        <mesh filename="package://relax_urdf/meshes/mesh_link5.stl" scale="0.001 0.001 0.001" />
-      </geometry>
-    </collision>
-</link>
-<link name ="relax_arm${arm_num}_link6">  <!-- link 6 -->
-    <inertial>
-      <origin xyz="${Link_6_x} ${Link_6_y} ${Link_6_z}" />
-      <mass value="${Link_6_mass}"/>
-      <inertia ixx="${Link_6_xx}" ixy="${Link_6_xy}" ixz="${Link_6_xz}" iyy="${Link_6_yy}" iyz="${Link_6_yz}" izz="${Link_6_zz}" />
-    </inertial>
-    <visual>
-      <origin xyz="0 0 0" rpy="0 0 0"/>
-      <geometry name="relax_link6_visual">
-        <mesh filename="package://relax_urdf/meshes/mesh_link6.stl" scale="0.001 0.001 0.001" />
-      </geometry>
-      <material name="darkblue"/>
-    </visual>
-    <collision>
-      <origin xyz="0 0 0" rpy="0 0 0"/>
-      <geometry name="relax_link6_collision">
-        <mesh filename="package://relax_urdf/meshes/mesh_link6.stl" scale="0.001 0.001 0.001" />
-      </geometry>
-    </collision>
-</link>
-<link name ="relax_arm${arm_num}_linkEndEffector" />  <!-- link End-Effector -->
-<!-- joints -->
-<joint name="relax_arm${arm_num}_joint0" type="revolute"> <!-- joint 1 -->
-    <parent link="base_link"/>
-    <child link="relax_arm${arm_num}_link1"/>
-    <origin xyz="${Joint_0_Ox} ${Joint_0_Oy} ${Joint_0_Oz}" rpy="${Joint_0_Oroll} ${Joint_0_Opitch} ${Joint_0_Oyaw}"/>
-    <axis xyz="0 0 1"/>
-    <limit velocity="${Joint_0_velocity}" effort="${Joint_0_effort}" lower="${Joint_0_lower}" upper="${Joint_0_upper}" />
-    <dynamics damping="${Joint_0_damp}" friction="${Joint_0_fric}"/>
-</joint>
-<joint name="relax_arm${arm_num}_joint1" type="revolute"> <!-- joint 1 -->
-    <parent link="relax_arm${arm_num}_link1"/>
-    <child link="relax_arm${arm_num}_link2"/>
-    <origin xyz="${Joint_1_Ox} ${Joint_1_Oy} ${Joint_1_Oz}" rpy="${Joint_1_Oroll} ${Joint_1_Opitch} ${Joint_1_Oyaw}"/>
-    <axis xyz="0 0 1"/>
-    <limit velocity="${Joint_1_velocity}" effort="${Joint_1_effort}" lower="${Joint_1_lower}" upper="${Joint_1_upper}" />
-    <dynamics damping="${Joint_1_damp}" friction="${Joint_1_fric}"/>
-</joint>
-<joint name="relax_arm${arm_num}_joint2" type="revolute"> <!-- joint 2 -->
-    <parent link="relax_arm${arm_num}_link2"/>
-    <child link="relax_arm${arm_num}_link3"/>
-    <origin xyz="${Joint_2_Ox} ${Joint_2_Oy} ${Joint_2_Oz}" rpy="${Joint_2_Oroll} ${Joint_2_Opitch} ${Joint_2_Oyaw}"/>
-    <axis xyz="0 0 -1"/>
-    <limit velocity="${Joint_2_velocity}" effort="${Joint_2_effort}" lower="${Joint_2_lower}" upper="${Joint_2_upper}" />
-    <dynamics damping="${Joint_2_damp}" friction="${Joint_2_fric}"/>
-</joint>
-<joint name="relax_arm${arm_num}_joint3" type="revolute"> <!-- joint 3 -->
-    <parent link="relax_arm${arm_num}_link3"/>
-    <child link="relax_arm${arm_num}_link4"/>
-    <origin xyz="${Joint_3_Ox} ${Joint_3_Oy} ${Joint_3_Oz}" rpy="${Joint_3_Oroll} ${Joint_3_Opitch} ${Joint_3_Oyaw}"/>
-    <axis xyz="0 0 1"/>
-    <limit velocity="${Joint_3_velocity}" effort="${Joint_3_effort}" lower="${Joint_3_lower}" upper="${Joint_3_upper}" />
-    <dynamics damping="${Joint_3_damp}" friction="${Joint_3_fric}"/>
-</joint>
-<joint name="relax_arm${arm_num}_joint4" type="revolute"> <!-- joint 4 -->
-    <parent link="relax_arm${arm_num}_link4"/>
-    <child link="relax_arm${arm_num}_link5"/>
-    <origin xyz="${Joint_4_Ox} ${Joint_4_Oy} ${Joint_4_Oz}" rpy="${Joint_4_Oroll} ${Joint_4_Opitch} ${Joint_4_Oyaw}"/>
-    <axis xyz="0 0 -1"/>
-    <limit velocity="${Joint_4_velocity}" effort="${Joint_4_effort}" lower="${Joint_4_lower}" upper="${Joint_4_upper}" />
-    <dynamics damping="${Joint_4_damp}" friction="${Joint_4_fric}"/>
-</joint>
-<joint name="relax_arm${arm_num}_joint5" type="revolute"> <!-- joint 5 -->
-    <parent link="relax_arm${arm_num}_link5"/>
-    <child link="relax_arm${arm_num}_link6"/>
-    <origin xyz="${Joint_5_Ox} ${Joint_5_Oy} ${Joint_5_Oz}" rpy="${Joint_5_Oroll} ${Joint_5_Opitch} ${Joint_5_Oyaw}"/>
-    <axis xyz="0 0 1"/>
-    <limit velocity="${Joint_5_velocity}" effort="${Joint_5_effort}" lower="${Joint_5_lower}" upper="${Joint_5_upper}" />
-    <dynamics damping="${Joint_5_damp}" friction="${Joint_5_fric}"/>
-</joint>
-<joint name="relax_arm${arm_num}_joint6" type="fixed"> <!-- joint 6 fake -->
-    <parent link="relax_arm${arm_num}_link6"/>
-    <child link="relax_arm${arm_num}_linkEndEffector"/>
-    <origin xyz="${Joint_6_Ox} ${Joint_6_Oy} ${Joint_6_Oz}" rpy="${Joint_6_Oroll} ${Joint_6_Opitch} ${Joint_6_Oyaw}"/>
-</joint>
-  </xacro:macro>
+<xacro:include filename="$(find relax_urdf)/urdf/properties/inertial_properties.urdf.xacro" />
+<xacro:include filename="$(find relax_urdf)/urdf/properties/kinematics_properties.urdf.xacro" />
+<xacro:include filename="$(find relax_urdf)/urdf/properties/dynamic_properties.urdf.xacro" />
+<xacro:include filename="$(find relax_urdf)/urdf/properties/limits.urdf.xacro" />
+<xacro:include filename="$(find relax_urdf)/urdf/parts/relax_arm_macro.urdf.xacro" />
+<xacro:include filename="$(find relax_urdf)/urdf/parts/relax_ee_macro.urdf.xacro" />
+<xacro:arg name="x" default="0"/>
+<xacro:arg name="y" default="0"/>
+<xacro:arg name="z" default="0"/>
+<xacro:property name="arm_num" value="1" />
+<xacro:relax_arm arm_num="${arm_num}" parent_link="base_link" >
+    <origin xyz="$(arg x) $(arg y) $(arg z)" rpy="0 0 0"/>
+</xacro:relax_arm>
+<xacro:relax_ee arm_num="${arm_num}" />
 </robot>

File: relax_urdf/urdf/relax.urdf.xacro (robot description, xacro)
@@ -1,31 +1,5 @@
 <?xml version="1.0"?>
 <robot xmlns:xacro="http://ros.org/wiki/xacro" name="relax">
-<!-- ************ MODEL CONFIGURATION ************ -->
-<xacro:arg name="config" default="$(find relax_urdf)/urdf/config/relax.urdf.xacro" />
-<!-- ************ MODEL CONFIGURATION ************ -->
-<xacro:include filename="$(arg config)"/>
-<!-- ************ RELAX BASE ************ -->
-<xacro:include filename="$(find relax_urdf)/urdf/relax_base.urdf.xacro"/>
-<!-- ***** attach base to the world ***** -->
-<xacro:if value="${RELAX_FLOATING_BASE}" > <!-- floating base -->
-    <xacro:if value="${RELAX_MOBILE_BASE}" >
-        <link name="world"/>
-        <joint name="world_joint" type="floating">
-            <parent link="world"/>
-            <child link="base_footprint"/>
-        </joint>
-    </xacro:if>
-</xacro:if>
-<xacro:unless value="${RELAX_MOBILE_BASE}" >
-  	<link name="world"/>
-   	<joint name="world_joint" type="fixed">
-        <parent link="world"/>
-<!--        <child link="base_footprint"/>-->
-        <child link="base_link"/>
-        <origin xyz="0 0 0" rpy="0 0 0" />
-  	</joint>
-</xacro:unless>
-<xacro:if value="${ADD_VIRTUAL_FRAME}">
-  <xacro:include filename="$(find relax_urdf)/urdf/parts/virtual_frame.urdf.xacro"/>
-</xacro:if>
+    <xacro:include filename="$(find relax_urdf)/urdf/config/relax.urdf.xacro"/>
+    <xacro:include filename="$(find relax_urdf)/urdf/parts/relax_core.urdf.xacro" />
 </robot>

File: relax_urdf/urdf/relax_robot.urdf.xacro (robot description, xacro)
@@ -1,14 +1,11 @@
 <?xml version="1.0"?>
 <robot xmlns:xacro="http://ros.org/wiki/xacro" name="relax">
-<!-- **** attach urdf robot model **** -->
-<xacro:include filename="$(find relax_urdf)/urdf/relax.urdf.xacro" />
-<!-- **** attach robot gazebo **** -->
-<xacro:include filename="$(find relax_urdf)/urdf/gazebo/relax.gazebo.xacro" />
-<xacro:include filename="$(find relax_urdf)/urdf/gazebo/xbot.gazebo.xacro" />
-<xacro:include filename="$(find relax_urdf)/urdf/gazebo/materials.gazebo.xacro" />
-<xacro:if value="${RELAX_MOBILE_BASE}">
-    <xacro:if value="${USE_NAV_CONTROLLERS}">
+    <xacro:include filename="$(find relax_urdf)/urdf/config/relax_gazebo.urdf.xacro"/>
+    <xacro:include filename="$(find relax_urdf)/urdf/gazebo/relax.gazebo.xacro" />
+    <xacro:include filename="$(find relax_urdf)/urdf/gazebo/xbot.gazebo.xacro" />
+    <xacro:include filename="$(find relax_urdf)/urdf/gazebo/materials.gazebo.xacro" />
+    <xacro:if value="${RELAX_MOBILE_BASE == 'mir'}">
         <xacro:controller_plugin_gazebo robot_namespace=""/>
     </xacro:if>
-</xacro:if>
+    <xacro:include filename="$(find relax_urdf)/urdf/parts/relax_core.urdf.xacro" />
 </robot>
