Commit message: Update fake_base.urdf.xacro

File: relax_urdf/urdf/parts/fake_base.urdf.xacro (robot description, xacro)
@@ -2,13 +2,9 @@
 <robot xmlns:xacro="http://ros.org/wiki/xacro">
 <!-- links -->
-<link name ="fake_link">  <!-- fake link -->
-    <visual>
-      <origin xyz="0 0 0" rpy="0 0 0"/>
-    </visual>
-</link>
-<joint name="fake_joint" type="fixed"> <!-- mobile base joint -->
+<link name ="fake_link" />  <!-- fake link -->
+<joint name="fake_joint" type="fixed"> <!-- fake joint -->
     <parent link="fake_link"/>
     <child link="relax_link1"/>
-    <origin xyz="0 0 0" rpy="0 0 0"/>
+    <origin xyz="0 0 0" rpy="3.1415927 0 0"/>
 </joint>
 </robot>
