Commit message: Update mobile_base.urdf.xacro

File: relax_urdf/urdf/parts/mobile_base.urdf.xacro (robot description, xacro)
@@ -1,3 +1,29 @@
 <?xml version="1.0"?>
 <robot xmlns:xacro="http://ros.org/wiki/xacro">
+<!-- links -->
+<link name ="mobile_base_link">  <!-- mobile base link -->
+    <inertial>
+      <origin xyz="0.0 0.0 0.0" rpy="0 0 0"/>
+      <mass value="0.0"/>
+      <inertia ixx="0.0" ixy="0.0" ixz="0.0" iyy="0.0" iyz="0.0" izz="0.0" />
+    </inertial>
+    <visual>
+      <origin xyz="0 0 0" rpy="0 0 0"/>
+      <geometry name="mobile_base_link_visual">
+        <mesh filename="package://relax_urdf/meshes/mir_base.stl" scale="0.001 0.001 0.001" />
+      </geometry>
+      <material name="dark"/>
+    </visual>
+    <collision>
+      <origin xyz="0 0 0" rpy="0 0 0"/>
+      <geometry name="mobile_base_link_collision">
+        <mesh filename="package://relax_urdf/meshes/mir_base.stl" scale="0.001 0.001 0.001" />
+      </geometry>
+    </collision>
+</link>
+<joint name="mobile_base_joint" type="fixed"> <!-- mobile base joint -->
+    <parent link="mobile_base_link"/>
+    <child link="relax_link1"/>
+    <origin xyz="0 0 ${320.000*mmTom}" rpy="3.1415927 0 0"/>
+</joint>
 </robot>

Commit message: Remove unneeded links for wheels

File: relax_urdf/urdf/parts/mobile_base.urdf.xacro (robot description, xacro)
@@ -22,17 +22,4 @@
     </collision>
 </link>
-<link name ="left_wheel_motor">
-    <inertial>
-      <origin xyz="0.0 0.0 0.0" rpy="0 0 0"/>
-      <mass value="0.1"/>
-      <inertia ixx="0.017" ixy="0.0" ixz="0.0" iyy="0.017" iyz="0.0" izz="0.017" />
-    </inertial>
-    <visual>
-      <origin xyz="0 0 0" rpy="0 0 0"/>
-    </visual>
-    <collision>
-      <origin xyz="0 0 0" rpy="0 0 0"/>
-    </collision>
-</link>
 <link name ="left_wheel">
     <inertial>
@@ -53,17 +40,4 @@
         <mesh filename="package://relax_urdf/meshes/mir_base.stl" scale="0.001 0.001 0.001" />
       </geometry>
-    </collision>
-</link>
-<link name ="right_wheel_motor">
-    <inertial>
-      <origin xyz="0.0 0.0 0.0" rpy="0 0 0"/>
-      <mass value="0.1"/>
-      <inertia ixx="0.017" ixy="0.0" ixz="0.0" iyy="0.017" iyz="0.0" izz="0.017" />
-    </inertial>
-    <visual>
-      <origin xyz="0 0 0" rpy="0 0 0"/>
-    </visual>
-    <collision>
-      <origin xyz="0 0 0" rpy="0 0 0"/>
     </collision>
 </link>
@@ -88,25 +62,15 @@
     </collision>
 </link>
-<joint name="j_l_motor" type="fixed">
+<joint name="j_left_wheel" type="continuous">
 	<parent link="mobile_base_link"/>
-	<child link="left_wheel_motor"/>
+	<child link="left_wheel"/>
     <origin xyz="-0.00448719 0.25 0.09" rpy="0 0 0"/>
-</joint>
-<joint name="j_r_motor" type="fixed">
-	<parent link="mobile_base_link"/>
-	<child link="right_wheel_motor"/>
-	<origin xyz="-0.00448719 -0.25 0.09" rpy="0 0 0"/>
-</joint>
-<joint name="j_left_wheel" type="continuous">
-	<parent link="left_wheel_motor"/>
-	<child link="left_wheel"/>
-    <origin xyz="0 0 0" rpy="0 0 0"/>
 	<axis xyz="0 0 -1"/>
    <limit  effort="35" velocity="20"/>
 </joint>
 <joint name="j_right_wheel" type="continuous">
-	<parent link="right_wheel_motor"/>
+	<parent link="mobile_base_link"/>
 	<child link="right_wheel"/>
-    <origin xyz="0 0 0" rpy="0 0 0"/>
+	<origin xyz="-0.00448719 -0.25 0.09" rpy="0 0 0"/>
 	<axis xyz="0 0 1"/>
    <limit  effort="35" velocity="20"/>

Commit message: Attach arm to base

File: relax_urdf/urdf/parts/mobile_base.urdf.xacro (robot description, xacro)
@@ -76,10 +76,3 @@
    <limit  effort="35" velocity="20"/>
 </joint>
-<xacro:if value="${RELAX_ARM}">
-    <joint name="mobile_base_joint" type="fixed"> <!-- mobile base joint -->
-        <parent link="mobile_base_link"/>
-        <child link="relax_link1"/>
-        <origin xyz="0 0 ${320.000*mmTom}" rpy="3.1415927 0 0"/>
-    </joint>
-</xacro:if>
 </robot>

File: relax_urdf/urdf/relax_base.urdf.xacro (robot description, xacro)
@@ -45,4 +45,11 @@
 <xacro:if value="${RELAX_MOBILE_BASE}">
 <xacro:include filename="$(find relax_urdf)/urdf/parts/mobile_base.urdf.xacro" />
+    <xacro:if value="${RELAX_ARM}">
+        <joint name="mobile_base_joint" type="fixed"> <!-- mobile base joint -->
+            <parent link="mobile_base_link"/>
+            <child link="relax_link1"/>
+            <origin xyz="0 0 ${240.000*mmTom}" rpy="3.1415927 0 0"/>
+        </joint>
+    </xacro:if>
 </xacro:if>
 <!-- ********  attach robot  ******** -->

Commit message: Small changes

File: relax_urdf/urdf/parts/mobile_base.urdf.xacro (robot description, xacro)
@@ -5,6 +5,6 @@
     <inertial>
       <origin xyz="0.0 0.0 0.0" rpy="0 0 0"/>
-      <mass value="10.0"/>
-      <inertia ixx="1.7" ixy="0.0" ixz="0.0" iyy="1.7" iyz="0.0" izz="1.7" />
+      <mass value="100.0"/>
+      <inertia ixx="17" ixy="0.0" ixz="0.0" iyy="17" iyz="0.0" izz="17" />
     </inertial>
     <visual>
