Commit message: added new meshes and updated inertial and kinematics properties in relax_urdf/urdf/parts

File: relax_urdf/urdf/parts/inertial_properties.urdf.xacro (robot description, xacro)
@@ -4,71 +4,85 @@
 <!-- Link 1 -->
 <!-- Center of Mass -->
-<xacro:property name="Link_1_x" value=" ${1.3955428e+00*mmTom} "/>
-<xacro:property name="Link_1_y" value=" ${2.5982581e+01*mmTom} "/>
-<xacro:property name="Link_1_z" value="${-1.6511476e+02*mmTom} "/>
+<xacro:property name="Link_1_x" value=" ${-1.8991406e+00*mmTom} "/>
+<xacro:property name="Link_1_y" value=" ${2.2645162e+01*mmTom} "/>
+<xacro:property name="Link_1_z" value="${1.6741297e+02*mmTom} "/>
 <!-- Mass -->
-<xacro:property name="Link_1_mass" value=" 5.9029271e+00 "/>
+<xacro:property name="Link_1_mass" value="6.2381702e+00"/>
 <!-- Inertia -->
-<xacro:property name="Link_1_xx" value=" ${6.2182861e+04*mm2Tom2} "/>
-<xacro:property name="Link_1_xy" value=" ${8.1614096e+01*mm2Tom2} "/>
-<xacro:property name="Link_1_xz" value=" ${1.0385066e+02*mm2Tom2} "/>
-<xacro:property name="Link_1_yy" value=" ${5.5346023e+04*mm2Tom2} "/>
-<xacro:property name="Link_1_yz" value=" ${1.2999920e+04*mm2Tom2} "/>
-<xacro:property name="Link_1_zz" value=" ${1.6821722e+04*mm2Tom2} "/>
+<xacro:property name="Link_1_xx" value=" ${6.5816037e+04*mm2Tom2} "/>
+<xacro:property name="Link_1_xy" value=" ${-1.1791629e+02*mm2Tom2} "/>
+<xacro:property name="Link_1_xz" value=" ${-4.0067927e+01*mm2Tom2} "/>
+<xacro:property name="Link_1_yy" value=" ${5.7828314e+04*mm2Tom2} "/>
+<xacro:property name="Link_1_yz" value=" ${-1.1584403e+04*mm2Tom2} "/>
+<xacro:property name="Link_1_zz" value=" ${1.9401960e+04*mm2Tom2} "/>
 <!-- Link 2 -->
 <!-- Center of Mass -->
-<xacro:property name="Link_2_x" value=" ${ 0.0000000e+00*mmTom} "/>
-<xacro:property name="Link_2_y" value=" ${-7.1720374e+00*mmTom} "/>
-<xacro:property name="Link_2_z" value=" ${-2.0000694e+02*mmTom} "/>
+<xacro:property name="Link_2_x" value=" ${-3.1494342e-02*mmTom} "/>
+<xacro:property name="Link_2_y" value=" ${-2.0005579e+02*mmTom} "/>
+<xacro:property name="Link_2_z" value=" ${-5.7041875e+00*mmTom} "/>
 <!-- Mass -->
-<xacro:property name="Link_2_mass" value=" 1.9989653e+00 "/>
+<xacro:property name="Link_2_mass" value="1.9989653e+00"/>
 <!-- Inertia -->
-<xacro:property name="Link_2_xx" value=" ${ 4.9589547e+04*mm2Tom2} "/>
-<xacro:property name="Link_2_xy" value=" ${-2.3822174e-02*mm2Tom2} "/>
-<xacro:property name="Link_2_xz" value=" ${ 2.3476881e+02*mm2Tom2} "/>
-<xacro:property name="Link_2_yy" value=" ${ 5.1111593e+04*mm2Tom2} "/>
-<xacro:property name="Link_2_yz" value=" ${ 7.7698490e-01*mm2Tom2} "/>
-<xacro:property name="Link_2_zz" value=" ${ 4.0702979e+03*mm2Tom2} "/>
+<xacro:property name="Link_2_xx" value=" ${ 6.4570453e+04*mm2Tom2} "/>
+<xacro:property name="Link_2_xy" value=" ${-1.9926538e+02*mm2Tom2} "/>
+<xacro:property name="Link_2_xz" value=" ${-1.6866046e+00*mm2Tom2} "/>
+<xacro:property name="Link_2_yy" value=" ${ 5.1512542e+03*mm2Tom2} "/>
+<xacro:property name="Link_2_yz" value=" ${-2.9627309e+00*mm2Tom2} "/>
+<xacro:property name="Link_2_zz" value=" ${ 6.6724653e+04*mm2Tom2} "/>
 <!-- Link 3 -->
 <!-- Center of Mass -->
-<xacro:property name="Link_3_x" value=" ${-2.1052916e+00*mmTom} "/>
-<xacro:property name="Link_3_y" value=" ${-1.0638552e+02*mmTom} "/>
-<xacro:property name="Link_3_z" value=" ${-7.4903486e+01*mmTom} "/>
+<xacro:property name="Link_3_x" value=" ${ 2.0858498e+00*mmTom} "/>
+<xacro:property name="Link_3_y" value=" ${-7.8452653e+01*mmTom} "/>
+<xacro:property name="Link_3_z" value=" ${-1.0797347e+02*mmTom} "/>
 <!-- Mass -->
-<xacro:property name="Link_3_mass" value=" 5.8838845e+00 "/>
+<xacro:property name="Link_3_mass" value="5.9482803e+00"/>
 <!-- Inertia -->
-<xacro:property name="Link_3_xx" value=" ${ 6.1043599e+04*mm2Tom2} "/>
-<xacro:property name="Link_3_xy" value=" ${-1.5340891e+02*mm2Tom2} "/>
-<xacro:property name="Link_3_xz" value=" ${-1.7833160e+02*mm2Tom2} "/>
-<xacro:property name="Link_3_yy" value=" ${ 5.3601310e+04*mm2Tom2} "/>
-<xacro:property name="Link_3_yz" value=" ${-1.1090900e+04*mm2Tom2} "/>
-<xacro:property name="Link_3_zz" value=" ${ 1.7380798e+04*mm2Tom2} "/>
+<xacro:property name="Link_3_xx" value=" ${ 6.2877846e+04*mm2Tom2} "/>
+<xacro:property name="Link_3_xy" value=" ${ 1.1665783e+02*mm2Tom2} "/>
+<xacro:property name="Link_3_xz" value=" ${ 1.2931181e+02*mm2Tom2} "/>
+<xacro:property name="Link_3_yy" value=" ${ 1.8390664e+04*mm2Tom2} "/>
+<xacro:property name="Link_3_yz" value=" ${-1.1034081e+04*mm2Tom2} "/>
+<xacro:property name="Link_3_zz" value=" ${ 5.5056826e+04*mm2Tom2} "/>
 <!-- Link 4 -->
 <!-- Center of Mass -->
-<xacro:property name="Link_4_x" value=" ${ 2.4496086e-01*mmTom} "/>
-<xacro:property name="Link_4_y" value=" ${-1.0728501e+00*mmTom} "/>
-<xacro:property name="Link_4_z" value=" ${-4.9015064e+01*mmTom} "/>
+<xacro:property name="Link_4_x" value=" ${ 9.6471566e-01*mmTom} "/>
+<xacro:property name="Link_4_y" value=" ${-4.2586853e+00*mmTom} "/>
+<xacro:property name="Link_4_z" value=" ${ 4.6169896e+01*mmTom} "/>
 <!-- Mass -->
-<xacro:property name="Link_4_mass" value=" 1.3982240e+00 "/>
+<xacro:property name="Link_4_mass" value="1.6710337e+00"/>
 <!-- Inertia -->
-<xacro:property name="Link_4_xx" value=" ${ 1.4667270e+04*mm2Tom2} "/>
-<xacro:property name="Link_4_xy" value=" ${-2.0411012e+01*mm2Tom2} "/>
-<xacro:property name="Link_4_xz" value=" ${-4.4769570e+01*mm2Tom2} "/>
-<xacro:property name="Link_4_yy" value=" ${ 8.6598581e+03*mm2Tom2} "/>
-<xacro:property name="Link_4_yz" value=" ${-8.3199044e+01*mm2Tom2} "/>
-<xacro:property name="Link_4_zz" value=" ${ 1.0450923e+04*mm2Tom2} "/>
+<xacro:property name="Link_4_xx" value=" ${ 1.7329394e+04*mm2Tom2} "/>
+<xacro:property name="Link_4_xy" value=" ${ 2.1094011e+02*mm2Tom2} "/>
+<xacro:property name="Link_4_xz" value=" ${-2.4511391e+02*mm2Tom2} "/>
+<xacro:property name="Link_4_yy" value=" ${ 1.0036061e+04*mm2Tom2} "/>
+<xacro:property name="Link_4_yz" value=" ${ 4.2230531e+02*mm2Tom2} "/>
+<xacro:property name="Link_4_zz" value=" ${ 1.2350325e+04*mm2Tom2} "/>
 <!-- Link 5 -->
 <!-- Center of Mass -->
-<xacro:property name="Link_5_x" value=" ${-1.3228834e+00*mmTom} "/>
-<xacro:property name="Link_5_y" value=" ${-8.4683010e+01*mmTom} "/>
-<xacro:property name="Link_5_z" value=" ${-5.3211105e+01*mmTom} "/>
+<xacro:property name="Link_5_x" value=" ${-1.3991722e+00*mmTom} "/>
+<xacro:property name="Link_5_y" value=" ${ 5.2618238e+01*mmTom} "/>
+<xacro:property name="Link_5_z" value=" ${-8.4259542e+01*mmTom} "/>
 <!-- Mass -->
-<xacro:property name="Link_5_mass" value=" 5.7923846e+00 "/>
+<xacro:property name="Link_5_mass" value="6.1811020e+00"/>
 <!-- Inertia -->
-<xacro:property name="Link_5_xx" value=" ${ 5.5109543e+04*mm2Tom2} "/>
-<xacro:property name="Link_5_xy" value=" ${-1.4003837e+02*mm2Tom2} "/>
-<xacro:property name="Link_5_xz" value=" ${ 2.1470743e+02*mm2Tom2} "/>
-<xacro:property name="Link_5_yy" value=" ${ 5.1309424e+04*mm2Tom2} "/>
-<xacro:property name="Link_5_yz" value=" ${-1.0289246e+03*mm2Tom2} "/>
-<xacro:property name="Link_5_zz" value=" ${ 1.3804762e+04*mm2Tom2} "/>
+<xacro:property name="Link_5_xx" value=" ${ 5.9736008e+04*mm2Tom2} "/>
+<xacro:property name="Link_5_xy" value=" ${-1.4975682e+02*mm2Tom2} "/>
+<xacro:property name="Link_5_xz" value=" ${-5.2815066e+01*mm2Tom2} "/>
+<xacro:property name="Link_5_yy" value=" ${ 1.5244195e+04*mm2Tom2} "/>
+<xacro:property name="Link_5_yz" value=" ${ 1.1994938e+03*mm2Tom2} "/>
+<xacro:property name="Link_5_zz" value=" ${ 5.5701504e+04*mm2Tom2} "/>
+<!-- Link 6 -->
+<!-- Center of Mass -->
+<xacro:property name="Link_6_x" value=" ${ 5.6879032e-01*mmTom} "/>
+<xacro:property name="Link_6_y" value=" ${ 0.0000000e+00*mmTom} "/>
+<xacro:property name="Link_6_z" value=" ${ 2.2653642e+00*mmTom} "/>
+<!-- Mass -->
+<xacro:property name="Link_6_mass" value="4.8141935e-01"/>
+<!-- Inertia -->
+<xacro:property name="Link_6_xx" value=" ${ 8.2206420e+02*mm2Tom2} "/>
+<xacro:property name="Link_6_xy" value=" ${ 1.0675057e-01*mm2Tom2} "/>
+<xacro:property name="Link_6_xz" value=" ${ 3.5319177e-01*mm2Tom2} "/>
+<xacro:property name="Link_6_yy" value=" ${ 8.3596992e+02*mm2Tom2} "/>
+<xacro:property name="Link_6_yz" value=" ${ 0.0000000e+00*mm2Tom2} "/>
+<xacro:property name="Link_6_zz" value=" ${ 1.2890535e+03*mm2Tom2} "/>
 </robot>

File: relax_urdf/urdf/parts/kinematics_properties.urdf.xacro (robot description, xacro)
@@ -2,22 +2,45 @@
 <robot  xmlns:xacro="http://ros.org/wiki/xacro">
 <!-- ARM -->
-<!-- Joint 1 Origin -->
+<!-- Joint 1 Origin : Link 1 - Link 2 -->
 <xacro:property name="Joint_1_Ox" value="  0.0 "/>
 <xacro:property name="Joint_1_Oy" value=" ${ 131.660*mmTom} "/>
-<xacro:property name="Joint_1_Oz" value=" ${-249.660*mmTom} "/>
-<!-- Joint 2 Origin -->
+<xacro:property name="Joint_1_Oz" value=" ${ 249.660*mmTom} "/>
+<xacro:property name="Joint_1_Oroll" value="  0.0 "/>
+<xacro:property name="Joint_1_Opitch" value=" 0.0 "/>
+<xacro:property name="Joint_1_Oyaw" value=" 0.0 "/>
+<!-- Joint 2 Origin : Link 2 - Link 3 -->
 <xacro:property name="Joint_2_Ox" value="  0.0 "/>
-<xacro:property name="Joint_2_Oy" value="  0.0 "/>
-<xacro:property name="Joint_2_Oz" value=" ${-400*mmTom} "/>
-<!-- Joint 3 Origin -->
+<xacro:property name="Joint_2_Oy" value=" ${-400*mmTom} "/>
+<xacro:property name="Joint_2_Oz" value="  0.0 "/>
+<xacro:property name="Joint_2_Oroll" value="  0.0 "/>
+<xacro:property name="Joint_2_Opitch" value=" 0.0 "/>
+<xacro:property name="Joint_2_Oyaw" value=" 0.0 "/>
+<!-- Joint 3 Origin : Link 3 - Link 4 -->
 <xacro:property name="Joint_3_Ox" value="  0.0 "/>
-<xacro:property name="Joint_3_Oy" value=" ${-131.660*mmTom} "/>
-<xacro:property name="Joint_3_Oz" value=" ${-249.660*mmTom} "/>
-<!-- Joint 4 Origin -->
+<xacro:property name="Joint_3_Oy" value=" ${-249.660*mmTom} "/>
+<xacro:property name="Joint_3_Oz" value=" ${-131.660*mmTom} "/>
+<xacro:property name="Joint_3_Oroll" value="  0.0 "/>
+<xacro:property name="Joint_3_Opitch" value=" 0.0 "/>
+<xacro:property name="Joint_3_Oyaw" value=" 0.0 "/>
+<!-- Joint 4 Origin : Link 4 - Link 5 -->
 <xacro:property name="Joint_4_Ox" value="  0.0 "/>
 <xacro:property name="Joint_4_Oy" value=" ${-88.1600*mmTom} "/>
-<xacro:property name="Joint_4_Oz" value=" ${-153.500*mmTom} "/>
+<xacro:property name="Joint_4_Oz" value=" ${153.500*mmTom} "/>
 <xacro:property name="Joint_4_Oroll" value="  0.0 "/>
 <xacro:property name="Joint_4_Opitch" value=" 0.0 "/>
 <xacro:property name="Joint_4_Oyaw" value=" 3.1415927 "/>
+<!-- Joint 5 Origin : Link 5 - Link 6 -->
+<xacro:property name="Joint_5_Ox" value="  0.0 "/>
+<xacro:property name="Joint_5_Oy" value=" ${222.160*mmTom} "/>
+<xacro:property name="Joint_5_Oz" value=" ${-88.1600*mmTom} "/>
+<xacro:property name="Joint_5_Oroll" value="  0.0 "/>
+<xacro:property name="Joint_5_Opitch" value=" 0.0 "/>
+<xacro:property name="Joint_5_Oyaw" value=" 0.0 "/>
+<!-- Fake Joint 6 Origin : Link 6 - End-Effector -->
+<xacro:property name="Joint_6_Ox" value="  0.0 "/>
+<xacro:property name="Joint_6_Oy" value=" 0.0 "/>
+<xacro:property name="Joint_6_Oz" value=" ${28.0000*mmTom} "/>
+<xacro:property name="Joint_6_Oroll" value="  0.0 "/>
+<xacro:property name="Joint_6_Opitch" value=" 0.0 "/>
+<xacro:property name="Joint_6_Oyaw" value=" 0.0 "/>
 </robot>

File: relax_urdf/urdf/parts/limits.urdf.xacro (robot description, xacro)
@@ -22,3 +22,8 @@
 <xacro:property name="Joint_4_lower" value=" -3.14 "/>
 <xacro:property name="Joint_4_upper" value=" 3.14 "/>
+<!-- Joint 5 -->
+<xacro:property name="Joint_5_velocity" value=" 3.86 "/>
+<xacro:property name="Joint_5_effort" value=" 147.0 "/>
+<xacro:property name="Joint_5_lower" value=" -3.14 "/>
+<xacro:property name="Joint_5_upper" value=" 3.14 "/>
 </robot>
