Commit message: Correct mesh path

File: relax_urdf/urdf/parts/wheels.urdf.xacro (robot description, xacro)
@@ -82,5 +82,5 @@
         <origin xyz="0 0 0" rpy="0 0 0" />
         <geometry>
-          <mesh filename="package://mir_description/meshes/visual/caster_wheel_base.stl" />
+          <mesh filename="package://relax_urdf/meshes/caster_wheel_base.stl" />
         </geometry>
         <xacro:insert_block name="material_black" />
@@ -89,5 +89,5 @@
         <origin xyz="0 0 0" rpy="0 0 0" />
         <geometry>
-          <mesh filename="package://mir_description/meshes/collision/caster_wheel_base.stl" />
+          <mesh filename="package://relax_urdf/meshes/caster_wheel_base.stl" />
         </geometry>
       </collision>
