Commit message: Update arm meshes (only on xacro)

File: relax_urdf/urdf/parts/dynamic_properties.urdf.xacro (robot description, xacro)
@@ -14,3 +14,6 @@
 <xacro:property name="Joint_4_damp" value="  0.2 "/>
 <xacro:property name="Joint_4_fric" value=" 10.0 "/>
+<!-- Joint 5 -->
+<xacro:property name="Joint_5_damp" value="  0.2 "/>
+<xacro:property name="Joint_5_fric" value=" 10.0 "/>
 </robot>

File: relax_urdf/urdf/parts/inertial_properties.urdf.xacro (robot description, xacro)
@@ -22,5 +22,5 @@
 <xacro:property name="Link_2_z" value=" ${-5.7041875e+00*mmTom} "/>
 <!-- Mass -->
-<xacro:property name="Link_2_mass" value="1.9989653e+00"/>
+<xacro:property name="Link_2_mass" value="2.6013710e+00"/>
 <!-- Inertia -->
 <xacro:property name="Link_2_xx" value=" ${ 6.4570453e+04*mm2Tom2} "/>

File: relax_urdf/urdf/parts/kinematics_properties.urdf.xacro (robot description, xacro)
@@ -6,7 +6,7 @@
 <xacro:property name="Joint_1_Oy" value=" ${ 131.660*mmTom} "/>
 <xacro:property name="Joint_1_Oz" value=" ${ 249.660*mmTom} "/>
-<xacro:property name="Joint_1_Oroll" value="  0.0 "/>
+<xacro:property name="Joint_1_Oroll" value="  -1.5707963 "/>
 <xacro:property name="Joint_1_Opitch" value=" 0.0 "/>
-<xacro:property name="Joint_1_Oyaw" value=" 0.0 "/>
+<xacro:property name="Joint_1_Oyaw" value=" 0.0"/>
 <!-- Joint 2 Origin : Link 2 - Link 3 -->
 <xacro:property name="Joint_2_Ox" value="  0.0 "/>
@@ -20,5 +20,5 @@
 <xacro:property name="Joint_3_Oy" value=" ${-249.660*mmTom} "/>
 <xacro:property name="Joint_3_Oz" value=" ${-131.660*mmTom} "/>
-<xacro:property name="Joint_3_Oroll" value="  0.0 "/>
+<xacro:property name="Joint_3_Oroll" value="  1.5707963 "/>
 <xacro:property name="Joint_3_Opitch" value=" 0.0 "/>
 <xacro:property name="Joint_3_Oyaw" value=" 0.0 "/>
@@ -27,12 +27,12 @@
 <xacro:property name="Joint_4_Oy" value=" ${-88.1600*mmTom} "/>
 <xacro:property name="Joint_4_Oz" value=" ${153.500*mmTom} "/>
-<xacro:property name="Joint_4_Oroll" value="  0.0 "/>
+<xacro:property name="Joint_4_Oroll" value="  1.5707963 "/>
 <xacro:property name="Joint_4_Opitch" value=" 0.0 "/>
-<xacro:property name="Joint_4_Oyaw" value=" 3.1415927 "/>
+<xacro:property name="Joint_4_Oyaw" value=" 0.0 "/>
 <!-- Joint 5 Origin : Link 5 - Link 6 -->
 <xacro:property name="Joint_5_Ox" value="  0.0 "/>
 <xacro:property name="Joint_5_Oy" value=" ${222.160*mmTom} "/>
 <xacro:property name="Joint_5_Oz" value=" ${-88.1600*mmTom} "/>
-<xacro:property name="Joint_5_Oroll" value="  0.0 "/>
+<xacro:property name="Joint_5_Oroll" value="  -1.5707963 "/>
 <xacro:property name="Joint_5_Opitch" value=" 0.0 "/>
 <xacro:property name="Joint_5_Oyaw" value=" 0.0 "/>

File: relax_urdf/urdf/parts/relax_arm.urdf.xacro (robot description, xacro)
@@ -13,5 +13,5 @@
       <origin xyz="0 0 0" rpy="0 0 0"/>
       <geometry name="relax_link1_visual">
-        <mesh filename="package://relax_urdf/meshes/mesh_link1.stl" scale="0.001 0.001 0.001" />
+        <mesh filename="package://relax_urdf/meshes/mesh_shoulder-yaw.stl" scale="0.001 0.001 0.001" />
       </geometry>
       <material name="darkblue"/>
@@ -20,5 +20,5 @@
       <origin xyz="0 0 0" rpy="0 0 0"/>
       <geometry name="relax_link1_collision">
-        <mesh filename="package://relax_urdf/meshes/mesh_link1.stl" scale="0.001 0.001 0.001" />
+        <mesh filename="package://relax_urdf/meshes/mesh_shoulder-yaw.stl" scale="0.001 0.001 0.001" />
       </geometry>
     </collision>
@@ -33,5 +33,5 @@
       <origin xyz="0 0 0" rpy="0 0 0"/>
       <geometry name="relax_link2_visual">
-        <mesh filename="package://relax_urdf/meshes/mesh_link2.stl" scale="0.001 0.001 0.001" />
+        <mesh filename="package://relax_urdf/meshes/mesh_shoulder-pitch.stl" scale="0.001 0.001 0.001" />
       </geometry>
       <material name="dark"/>
@@ -40,5 +40,5 @@
       <origin xyz="0 0 0" rpy="0 0 0"/>
       <geometry name="relax_link2_collision">
-        <mesh filename="package://relax_urdf/meshes/mesh_link2.stl" scale="0.001 0.001 0.001" />
+        <mesh filename="package://relax_urdf/meshes/mesh_shoulder-pitch.stl" scale="0.001 0.001 0.001" />
       </geometry>
     </collision>
@@ -53,5 +53,5 @@
       <origin xyz="0 0 0" rpy="0 0 0"/>
       <geometry name="relax_link3_visual">
-        <mesh filename="package://relax_urdf/meshes/mesh_link3.stl" scale="0.001 0.001 0.001" />
+        <mesh filename="package://relax_urdf/meshes/mesh_elbow.stl" scale="0.001 0.001 0.001" />
       </geometry>
       <material name="darkblue"/>
@@ -60,5 +60,5 @@
       <origin xyz="0 0 0" rpy="0 0 0"/>
       <geometry name="relax_link3_collision">
-        <mesh filename="package://relax_urdf/meshes/mesh_link3.stl" scale="0.001 0.001 0.001" />
+        <mesh filename="package://relax_urdf/meshes/mesh_elbow.stl" scale="0.001 0.001 0.001" />
       </geometry>
     </collision>
@@ -66,5 +66,5 @@
 <link name ="relax_arm${arm_num}_link4">  <!-- link 4 -->
     <inertial>
-      <origin xyz="${Link_4_x} ${Link_4_y} ${Link_4_z}" />
+      <origin xyz="${Link_4_x} ${Link_4_y} ${Link_4_z}" rpy="-2.6324601 1.5172034 -2.2584214"/>
       <mass value="${Link_4_mass}"/>
       <inertia ixx="${Link_4_xx}" ixy="${Link_4_xy}" ixz="${Link_4_xz}" iyy="${Link_4_yy}" iyz="${Link_4_yz}" izz="${Link_4_zz}" />
@@ -73,5 +73,5 @@
       <origin xyz="0 0 0" rpy="0 0 0"/>
       <geometry name="relax_link4_visual">
-        <mesh filename="package://relax_urdf/meshes/mesh_link4.stl" scale="0.001 0.001 0.001" />
+        <mesh filename="package://relax_urdf/meshes/mesh_forearm-yaw.stl" scale="0.001 0.001 0.001" />
       </geometry>
       <material name="darkblue"/>
@@ -80,5 +80,5 @@
       <origin xyz="0 0 0" rpy="0 0 0"/>
       <geometry name="relax_link4_collision">
-        <mesh filename="package://relax_urdf/meshes/mesh_link4.stl" scale="0.001 0.001 0.001" />
+        <mesh filename="package://relax_urdf/meshes/mesh_forearm-yaw.stl" scale="0.001 0.001 0.001" />
       </geometry>
     </collision>
@@ -93,5 +93,5 @@
       <origin xyz="0 0 0" rpy="0 0 0"/>
       <geometry name="relax_link5_visual">
-        <mesh filename="package://relax_urdf/meshes/mesh_link5.stl" scale="0.001 0.001 0.001" />
+        <mesh filename="package://relax_urdf/meshes/mesh_wrist-pitch.stl" scale="0.001 0.001 0.001" />
       </geometry>
       <material name="darkblue"/>
@@ -100,5 +100,25 @@
       <origin xyz="0 0 0" rpy="0 0 0"/>
       <geometry name="relax_link5_collision">
-        <mesh filename="package://relax_urdf/meshes/mesh_link5.stl" scale="0.001 0.001 0.001" />
+        <mesh filename="package://relax_urdf/meshes/mesh_wrist-pitch.stl" scale="0.001 0.001 0.001" />
+      </geometry>
+    </collision>
+</link>
+<link name ="relax_arm${arm_num}_link6">  <!-- link 5 -->
+    <inertial>
+      <origin xyz="${Link_6_x} ${Link_6_y} ${Link_6_z}" />
+      <mass value="${Link_6_mass}"/>
+      <inertia ixx="${Link_6_xx}" ixy="${Link_6_xy}" ixz="${Link_6_xz}" iyy="${Link_6_yy}" iyz="${Link_6_yz}" izz="${Link_6_zz}" />
+    </inertial>
+    <visual>
+      <origin xyz="0 0 0" rpy="0 0 0"/>
+      <geometry name="relax_link6_visual">
+        <mesh filename="package://relax_urdf/meshes/mesh_wrist-yaw.stl" scale="0.001 0.001 0.001" />
+      </geometry>
+      <material name="darkblue"/>
+    </visual>
+    <collision>
+      <origin xyz="0 0 0" rpy="0 0 0"/>
+      <geometry name="relax_link6_collision">
+        <mesh filename="package://relax_urdf/meshes/mesh_wrist-yaw.stl" scale="0.001 0.001 0.001" />
       </geometry>
     </collision>
@@ -108,6 +128,6 @@
     <parent link="relax_arm${arm_num}_link1"/>
     <child link="relax_arm${arm_num}_link2"/>
-    <origin xyz="${Joint_1_Ox} ${Joint_1_Oy} ${Joint_1_Oz}" rpy="0 0 0"/>
-    <axis xyz="0 1 0"/>
+    <origin xyz="${Joint_1_Ox} ${Joint_1_Oy} ${Joint_1_Oz}" rpy="${Joint_1_Oroll} ${Joint_1_Opitch} ${Joint_1_Oyaw}"/>
+    <axis xyz="0 0 1"/>
     <limit velocity="${Joint_1_velocity}" effort="${Joint_1_effort}" lower="${Joint_1_lower}" upper="${Joint_1_upper}" />
     <dynamics damping="${Joint_1_damp}" friction="${Joint_1_fric}"/>
@@ -116,6 +136,6 @@
     <parent link="relax_arm${arm_num}_link2"/>
     <child link="relax_arm${arm_num}_link3"/>
-    <origin xyz="${Joint_2_Ox} ${Joint_2_Oy} ${Joint_2_Oz}" rpy="0 0 0"/>
-    <axis xyz="0 1 0"/>
+    <origin xyz="${Joint_2_Ox} ${Joint_2_Oy} ${Joint_2_Oz}" rpy="${Joint_2_Oroll} ${Joint_2_Opitch} ${Joint_2_Oyaw}"/>
+    <axis xyz="0 0 1"/>
     <limit velocity="${Joint_2_velocity}" effort="${Joint_2_effort}" lower="${Joint_2_lower}" upper="${Joint_2_upper}" />
     <dynamics damping="${Joint_2_damp}" friction="${Joint_2_fric}"/>
@@ -124,5 +144,5 @@
     <parent link="relax_arm${arm_num}_link3"/>
     <child link="relax_arm${arm_num}_link4"/>
-    <origin xyz="${Joint_3_Ox} ${Joint_3_Oy} ${Joint_3_Oz}" rpy="0 0 0"/>
+    <origin xyz="${Joint_3_Ox} ${Joint_3_Oy} ${Joint_3_Oz}" rpy="${Joint_3_Oroll} ${Joint_3_Opitch} ${Joint_3_Oyaw}"/>
     <axis xyz="0 0 1"/>
     <limit velocity="${Joint_3_velocity}" effort="${Joint_3_effort}" lower="${Joint_3_lower}" upper="${Joint_3_upper}" />
@@ -133,8 +153,16 @@
     <child link="relax_arm${arm_num}_link5"/>
     <origin xyz="${Joint_4_Ox} ${Joint_4_Oy} ${Joint_4_Oz}" rpy="${Joint_4_Oroll} ${Joint_4_Opitch} ${Joint_4_Oyaw}"/>
-    <axis xyz="0 1 0"/>
+    <axis xyz="0 0 1"/>
     <limit velocity="${Joint_4_velocity}" effort="${Joint_4_effort}" lower="${Joint_4_lower}" upper="${Joint_4_upper}" />
     <dynamics damping="${Joint_4_damp}" friction="${Joint_4_fric}"/>
 </joint>
+<joint name="relax_arm${arm_num}_joint5" type="revolute"> <!-- joint 5 -->
+    <parent link="relax_arm${arm_num}_link5"/>
+    <child link="relax_arm${arm_num}_link6"/>
+    <origin xyz="${Joint_5_Ox} ${Joint_5_Oy} ${Joint_5_Oz}" rpy="${Joint_5_Oroll} ${Joint_5_Opitch} ${Joint_5_Oyaw}"/>
+    <axis xyz="0 0 1"/>
+    <limit velocity="${Joint_5_velocity}" effort="${Joint_5_effort}" lower="${Joint_5_lower}" upper="${Joint_5_upper}" />
+    <dynamics damping="${Joint_5_damp}" friction="${Joint_5_fric}"/>
+</joint>
   </xacro:macro>
 </robot>

File: relax_urdf/urdf/relax_base.urdf.xacro (robot description, xacro)
@@ -57,5 +57,5 @@
             <parent link="control_box"/>
             <child link="relax_arm1_link1"/>
-            <origin xyz="0 0 0" rpy="3.1415927 0 0"/>
+            <origin xyz="0 0 0" rpy="0 0 0"/>
         </joint>
     </xacro:if>

Commit message: added joint 0 between the base and the link1 of the arm

File: relax_urdf/urdf/parts/dynamic_properties.urdf.xacro (robot description, xacro)
@@ -2,4 +2,7 @@
 <robot  xmlns:xacro="http://ros.org/wiki/xacro">
 <!-- ARM -->
+<!-- Joint 0 -->
+<xacro:property name="Joint_0_damp" value="  0.2 "/>
+<xacro:property name="Joint_0_fric" value=" 10.0 "/>
 <!-- Joint 1 -->
 <xacro:property name="Joint_1_damp" value="  0.2 "/>
@@ -17,5 +20,5 @@
 <xacro:property name="Joint_5_damp" value="  0.2 "/>
 <xacro:property name="Joint_5_fric" value=" 10.0 "/>
-<!-- Joint 6 -->
+<!-- Joint 6 fake -->
 <xacro:property name="Joint_6_damp" value="  0.2 "/>
 <xacro:property name="Joint_6_fric" value=" 10.0 "/>

File: relax_urdf/urdf/parts/kinematics_properties.urdf.xacro (robot description, xacro)
@@ -2,4 +2,11 @@
 <robot  xmlns:xacro="http://ros.org/wiki/xacro">
 <!-- ARM -->
+<!-- Joint 0 Origin : Base - Link 1 -->
+<xacro:property name="Joint_0_Ox" value="  0.0 "/>
+<xacro:property name="Joint_0_Oy" value=" ${-130.000*mmTom} "/>
+<xacro:property name="Joint_0_Oz" value=" ${ 361.300*mmTom} "/>
+<xacro:property name="Joint_0_Oroll" value=" 0.0 "/>
+<xacro:property name="Joint_0_Opitch" value=" 0.0 "/>
+<xacro:property name="Joint_0_Oyaw" value=" 0.0 "/>
 <!-- Joint 1 Origin : Link 1 - Link 2 -->
 <xacro:property name="Joint_1_Ox" value="  0.0 "/>
@@ -8,5 +15,5 @@
 <xacro:property name="Joint_1_Oroll" value=" -1.5707963 "/>
 <xacro:property name="Joint_1_Opitch" value=" 0.0 "/>
-<xacro:property name="Joint_1_Oyaw" value=" 0.0"/>
+<xacro:property name="Joint_1_Oyaw" value=" 0.0 "/>
 <!-- Joint 2 Origin : Link 2 - Link 3 -->
 <xacro:property name="Joint_2_Ox" value="  0.0 "/>
@@ -37,5 +44,5 @@
 <xacro:property name="Joint_5_Opitch" value=" 0.0 "/>
 <xacro:property name="Joint_5_Oyaw" value=" 0.0 "/>
-<!-- Joint 6 Origin : Link 6 - End-Effector -->
+<!-- Joint 6 fake Origin : Link 6 - End-Effector -->
 <xacro:property name="Joint_6_Ox" value="  0.0 "/>
 <xacro:property name="Joint_6_Oy" value=" 0.0 "/>

File: relax_urdf/urdf/parts/limits.urdf.xacro (robot description, xacro)
@@ -2,4 +2,9 @@
 <robot  xmlns:xacro="http://ros.org/wiki/xacro">
 <!-- ARM -->
+<!-- Joint 0 -->
+<xacro:property name="Joint_0_velocity" value=" 3.86 "/>
+<xacro:property name="Joint_0_effort" value=" 147.0 "/>
+<xacro:property name="Joint_0_lower" value=" -3.14 "/>
+<xacro:property name="Joint_0_upper" value=" 3.14 "/>
 <!-- Joint 1 -->
 <xacro:property name="Joint_1_velocity" value=" 3.86 "/>
@@ -27,5 +32,5 @@
 <xacro:property name="Joint_5_lower" value=" -3.14 "/>
 <xacro:property name="Joint_5_upper" value=" 3.14 "/>
-<!-- Joint 6 -->
+<!-- Joint 6 fake -->
 <xacro:property name="Joint_6_velocity" value=" 3.86 "/>
 <xacro:property name="Joint_6_effort" value=" 147.0 "/>

File: relax_urdf/urdf/parts/relax_arm.urdf.xacro (robot description, xacro)
@@ -126,4 +126,12 @@
 <link name ="relax_arm${arm_num}_linkEndEffector" />  <!-- link End-Effector -->
 <!-- joints -->
+<joint name="relax_arm${arm_num}_joint0" type="revolute"> <!-- joint 1 -->
+    <parent link="base_link"/>
+    <child link="relax_arm${arm_num}_link1"/>
+    <origin xyz="${Joint_0_Ox} ${Joint_0_Oy} ${Joint_0_Oz}" rpy="${Joint_0_Oroll} ${Joint_0_Opitch} ${Joint_0_Oyaw}"/>
+    <axis xyz="0 0 1"/>
+    <limit velocity="${Joint_0_velocity}" effort="${Joint_0_effort}" lower="${Joint_0_lower}" upper="${Joint_0_upper}" />
+    <dynamics damping="${Joint_0_damp}" friction="${Joint_0_fric}"/>
+</joint>
 <joint name="relax_arm${arm_num}_joint1" type="revolute"> <!-- joint 1 -->
     <parent link="relax_arm${arm_num}_link1"/>
@@ -166,5 +174,5 @@
     <dynamics damping="${Joint_5_damp}" friction="${Joint_5_fric}"/>
 </joint>
-<joint name="relax_arm${arm_num}_joint6" type="revolute"> <!-- joint 6 -->
+<joint name="relax_arm${arm_num}_joint6" type="fixed"> <!-- joint 6 fake -->
     <parent link="relax_arm${arm_num}_link6"/>
     <child link="relax_arm${arm_num}_linkEndEffector"/>
