Commit message: inertia macro of wheels rotated correctly

File: relax_urdf/urdf/parts/common_base_properties.urdf.xacro (robot description, xacro)
@@ -70,4 +70,13 @@
     </inertial>
   </xacro:macro>
+  <xacro:macro name="wheel_inertial_y" params="radius length mass *origin">
+    <inertial>
+      <mass value="${mass}" />
+      <xacro:insert_block name="origin" />
+      <inertia ixx="${0.0833333 * mass * (3 * radius * radius + length * length)}" ixy="0.0" ixz="0.0"
+        iyy="${0.5 * mass * radius * radius}" iyz="0.0"
+        izz="${0.0833333 * mass * (3 * radius * radius + length * length)}"  />
+    </inertial>
+  </xacro:macro>
   <xacro:macro name="box_inertial" params="x y z mass *origin">
     <inertial>

File: relax_urdf/urdf/parts/wheels.urdf.xacro (robot description, xacro)
@@ -36,7 +36,7 @@
     </joint>
     <link name="${prefix}${locationprefix}_wheel_link">
-      <xacro:cylinder_inertial mass="${mir_act_wheel_mass}" radius="${mir_act_wheel_radius}" length="${mir_act_wheel_width}">
+      <xacro:wheel_inertial_y mass="${mir_act_wheel_mass}" radius="${mir_act_wheel_radius}" length="${mir_act_wheel_width}">
         <origin xyz="0 0 0" rpy="0 0 0" /> <!-- ${0.5 * pi} 0 0 -->
-      </xacro:cylinder_inertial>
+      </xacro:wheel_inertial_y>
       <visual>
         <origin xyz="0 0 0" rpy="${pi/2} 0 0" />
@@ -104,7 +104,7 @@
     </joint>
     <link name="${prefix}${locationprefix}_caster_wheel_link">
-      <xacro:cylinder_inertial mass="${mir_caster_wheel_mass}" radius="${mir_caster_wheel_radius}" length="${mir_caster_wheel_width}">
+      <xacro:wheel_inertial_y mass="${mir_caster_wheel_mass}" radius="${mir_caster_wheel_radius}" length="${mir_caster_wheel_width}">
         <origin xyz="0 0 0" rpy="0 0 0" /> <!--${0.5 * pi} -->
-      </xacro:cylinder_inertial>
+      </xacro:wheel_inertial_y>
       <visual>
         <origin xyz="0 0 0" rpy="${pi/2} 0 0" /> <!--${pi/2} 0 0 -->
