Commit message: Latest URDF: manually defining X and TETA control of the base using a prismatica and a revolute joint, all the rest is fixed

File: relax_urdf/urdf/parts/mir_base.urdf.xacro (robot description, xacro)
@@ -81,8 +81,107 @@
     </joint>
     <link name="${prefix}us_2_frame" />
-    <!-- wheels -->
-    <xacro:actuated_wheel prefix="${prefix}" locationprefix="left" locationright="-1"/>
+    <!-- wheels MANUALLY DONE FOR HIGH LEVEL CONTROL -->
+    <joint name="left_wheel_joint" type="revolute">
+      <origin rpy="0 0 0" xyz="0.0 0.2015 0.1"/>
+      <parent link="base_link"/>
+      <child link="left_wheel_link"/>
+      <axis xyz="0 0 1"/>
+      <limit upper="1e9" lower="-1e9" effort="2" velocity="2.0"/>
+    </joint>
+    <link name="left_wheel_link">
+    <inertial>
+      <mass value="1.0"/>
+      <origin rpy="0 0 0" xyz="0 0 0"/>
+      <inertia ixx="0.0026203322852000007" ixy="0.0" ixz="0.0" iyy="0.0026203322852000007" iyz="0.0" izz="0.005000000000000001"/>
+    </inertial>
+    <visual>
+      <origin rpy="1.5707963267948966 0 0" xyz="0 0 0"/>
+      <geometry>
+        <cylinder length="0.038" radius="0.1"/>
+      </geometry>
+      <material name="black">
+        <color rgba="0.1 0.1 0.1 1"/>
+      </material>
+    </visual>
+    <collision>
+      <origin rpy="1.5707963267948966 0 0" xyz="0 0 0"/>
+      <geometry>
+        <cylinder length="0.038" radius="0.1"/>
+      </geometry>
+    </collision>
+  </link>
+  <gazebo reference="left_wheel_link">
+    <material>Gazebo/FlatBlack</material>
+  </gazebo>
+  <joint name="fl_caster_rotation_joint" type="prismatic">
+    <origin rpy="0 0 0" xyz="0.299215 0.188 0.1565"/>
+    <parent link="base_link"/>
+    <child link="fl_caster_rotation_link"/>
+    <axis xyz="1 0 0"/>
+    <limit upper="1e9" lower="-1e9" effort="2" velocity="2.0"/>
+    <dynamics damping="0.01" friction="0.0"/>
+  </joint>
+  <link name="fl_caster_rotation_link">
+    <inertial>
+      <!-- <origin xyz="0 0 -0.042500000044" rpy="${0.5 * pi} ${24 * deg_to_rad} ${1.5 * pi}" /> -->
+      <origin rpy="0 0 0" xyz="0 0 -0.042500000044"/>
+      <!-- ${24 * deg_to_rad} 0 ${0.5 * pi} -->
+      <mass value="0.3097539019"/>
+      <inertia ixx="0.0005844517978" ixy="0" ixz="0" iyy="0.00052872551237" iyz="0" izz="0.00017923555074"/>
+    </inertial>
+    <visual>
+      <origin rpy="0 0 0" xyz="0 0 0"/>
+      <geometry>
+        <mesh filename="package://relax_urdf/meshes/caster_wheel_base.stl"/>
+      </geometry>
+      <material name="black">
+        <color rgba="0.1 0.1 0.1 1"/>
+      </material>
+    </visual>
+    <collision>
+      <origin rpy="0 0 0" xyz="0 0 0"/>
+      <geometry>
+        <mesh filename="package://relax_urdf/meshes/caster_wheel_base.stl"/>
+      </geometry>
+    </collision>
+  </link>
+  <gazebo reference="fl_caster_rotation_link">
+    <material>Gazebo/FlatBlack</material>
+  </gazebo>
+  <joint name="fl_caster_wheel_joint" type="fixed">
+    <origin rpy="0 0 0" xyz="-0.0382 0 -0.094"/>
+    <parent link="fl_caster_rotation_link"/>
+    <child link="fl_caster_wheel_link"/>
+    <axis xyz="0 1 0"/>
+    <limit upper="1e9" lower="-1e9" effort="2" velocity="2.0"/>
+  </joint>
+  <link name="fl_caster_wheel_link">
+    <inertial>
+      <mass value="1.0"/>
+      <origin rpy="0 0 0" xyz="0 0 0"/>
+      <inertia ixx="0.001061895408575" ixy="0.0" ixz="0.0" iyy="0.001061895408575" iyz="0.0" izz="0.001953125"/>
+    </inertial>
+    <visual>
+      <origin rpy="0 0 0" xyz="0 0 0"/>
+      <!--${pi/2} 0 0 -->
+      <geometry>
+        <cylinder length="0.032" radius="0.0625"/>
+      </geometry>
+      <material name="black">
+        <color rgba="0.1 0.1 0.1 1"/>
+      </material>
+    </visual>
+    <collision>
+      <origin rpy="0 0 0" xyz="0 0 0"/>
+      <!--${pi/2} 0 0 -->
+      <geometry>
+        <cylinder length="0.032" radius="0.0625"/>
+      </geometry>
+    </collision>
+  </link>
+  <gazebo reference="fl_caster_wheel_link">
+    <material>Gazebo/FlatBlack</material>
+  </gazebo>
     <xacro:actuated_wheel prefix="${prefix}" locationprefix="right" locationright="1"/>
-    <xacro:caster_wheel prefix="${prefix}" locationprefix="fl" locationright="-1" wheel_base_dx="${mir_front_caster_wheel_base_dx + mir_act_wheel_dx}"/>
     <xacro:caster_wheel prefix="${prefix}" locationprefix="fr" locationright="1" wheel_base_dx="${mir_front_caster_wheel_base_dx + mir_act_wheel_dx}"/>
     <xacro:caster_wheel prefix="${prefix}" locationprefix="bl" locationright="-1" wheel_base_dx="${-mir_back_caster_wheel_base_dx + mir_act_wheel_dx}"/>

File: relax_urdf/urdf/parts/wheels.urdf.xacro (robot description, xacro)
@@ -28,5 +28,5 @@
   <xacro:property name="mir_caster_wheel_base_dz" value="${mir_caster_wheel_radius - mir_caster_wheel_dz}" />
   <xacro:macro name="actuated_wheel" params="prefix locationprefix locationright">
-    <joint name="${prefix}${locationprefix}_wheel_joint" type="continuous">
+    <joint name="${prefix}${locationprefix}_wheel_joint" type="fixed">
       <origin xyz="0.0 ${-mir_act_wheel_dy * locationright} ${mir_act_wheel_radius}" rpy="0 0 0" />
       <parent link="${prefix}base_link" />
@@ -37,5 +37,5 @@
     <link name="${prefix}${locationprefix}_wheel_link">
       <xacro:cylinder_inertial mass="${mir_act_wheel_mass}" radius="${mir_act_wheel_radius}" length="${mir_act_wheel_width}">
-        <origin xyz="0 0 0" rpy="${0.5 * pi} 0 0" />
+        <origin xyz="0 0 0" rpy="0 0 0" /> <!-- ${0.5 * pi} 0 0 -->
       </xacro:cylinder_inertial>
       <visual>
@@ -59,5 +59,5 @@
   <xacro:macro name="caster_wheel" params="prefix locationprefix locationright wheel_base_dx">
     <!-- caster hub -->
-    <joint name="${prefix}${locationprefix}_caster_rotation_joint" type="continuous">
+    <joint name="${prefix}${locationprefix}_caster_rotation_joint" type="fixed">
       <origin xyz="${wheel_base_dx} ${-mir_caster_wheel_base_dy * locationright} ${mir_caster_wheel_base_dz}" rpy="0 0 0" />
       <parent link="${prefix}base_link" />
@@ -69,5 +69,5 @@
       <inertial>
         <!-- <origin xyz="0 0 -0.042500000044" rpy="${0.5 * pi} ${24 * deg_to_rad} ${1.5 * pi}" /> -->
-        <origin xyz="0 0 -0.042500000044" rpy="${24 * deg_to_rad} 0 ${0.5 * pi} " />
+        <origin xyz="0 0 -0.042500000044" rpy="0 0 0" /> <!-- ${24 * deg_to_rad} 0 ${0.5 * pi} -->
         <mass value="0.3097539019" />
         <inertia
@@ -97,5 +97,5 @@
     </gazebo>
     <!-- caster wheel -->
-    <joint name="${prefix}${locationprefix}_caster_wheel_joint" type="continuous">
+    <joint name="${prefix}${locationprefix}_caster_wheel_joint" type="fixed">
       <origin xyz="${mir_caster_wheel_dx} ${-mir_caster_wheel_dy * locationright} ${mir_caster_wheel_dz}" rpy="0 0 0" />
       <parent link="${prefix}${locationprefix}_caster_rotation_link" />
@@ -105,8 +105,8 @@
     <link name="${prefix}${locationprefix}_caster_wheel_link">
       <xacro:cylinder_inertial mass="${mir_caster_wheel_mass}" radius="${mir_caster_wheel_radius}" length="${mir_caster_wheel_width}">
-        <origin xyz="0 0 0" rpy="${0.5 * pi} 0 0" />
+        <origin xyz="0 0 0" rpy="0 0 0" /> <!--${0.5 * pi} -->
       </xacro:cylinder_inertial>
       <visual>
-        <origin xyz="0 0 0" rpy="${pi/2} 0 0" />
+        <origin xyz="0 0 0" rpy="0 0 0" /> <!--${pi/2} 0 0 -->
         <geometry>
           <cylinder radius="${mir_caster_wheel_radius}" length="${mir_caster_wheel_width}" />
@@ -115,5 +115,5 @@
       </visual>
       <collision>
-        <origin xyz="0 0 0" rpy="${pi/2} 0 0" />
+        <origin xyz="0 0 0" rpy="0 0 0" /> <!--${pi/2} 0 0 -->
         <geometry>
           <cylinder radius="${mir_caster_wheel_radius}" length="${mir_caster_wheel_width}" />

File: relax_urdf/urdf/relax_capsule.urdf (robot description, URDF)
Before this commit: robot relax, 27 links, 26 joints
Links:
- link back_laser_link: geometry collision cylinder length=0.08046897400091513 radius=0.0694408; collision sphere radius=0.0694408
- link base_link: geometry collision cylinder length=0.4739740000000168 radius=0.319357; collision sphere radius=0.319357
- link bl_caster_rotation_link: geometry collision cylinder length=0.08979176363609312 radius=0.0393866; collision sphere radius=0.0393866
- link bl_caster_wheel_link: geometry collision cylinder length=0.032 radius=0.0625; collision sphere radius=0.0625
- link br_caster_rotation_link: geometry collision cylinder length=0.08979176363609312 radius=0.0393866; collision sphere radius=0.0393866
- link br_caster_wheel_link: geometry collision cylinder length=0.032 radius=0.0625; collision sphere radius=0.0625
- link fl_caster_rotation_link: geometry collision cylinder length=0.08979176363609312 radius=0.0393866; collision sphere radius=0.0393866
- link fl_caster_wheel_link: geometry collision cylinder length=0.032 radius=0.0625; collision sphere radius=0.0625
- link fr_caster_rotation_link: geometry collision cylinder length=0.08979176363609312 radius=0.0393866; collision sphere radius=0.0393866
- link fr_caster_wheel_link: geometry collision cylinder length=0.032 radius=0.0625; collision sphere radius=0.0625
- link front_laser_link: geometry collision cylinder length=0.08046897400091513 radius=0.0694408; collision sphere radius=0.0694408
- link left_wheel_link: geometry collision cylinder length=0.038 radius=0.1; collision sphere radius=0.1
- link relax_arm1_link1: geometry collision cylinder length=0.13791276538840705 radius=0.0915579; collision sphere radius=0.0915579
- link relax_arm1_link2: geometry collision cylinder length=0.4002004224012504 radius=0.0779127; collision sphere radius=0.0779127
- link relax_arm1_link3: geometry collision cylinder length=0.1380269667138794 radius=0.0921787; collision sphere radius=0.0921787
- link relax_arm1_link4: geometry collision cylinder length=0.1319941011646182 radius=0.115074; collision sphere radius=0.115074
- link relax_arm1_link5: geometry collision cylinder length=0.13080711726714422 radius=0.104678; collision sphere radius=0.104678
- link relax_arm1_link6: geometry collision cylinder length=5.659878616105297e-07 radius=0.0752452; collision sphere radius=0.0752452
- link right_wheel_link: geometry collision cylinder length=0.038 radius=0.1; collision sphere radius=0.1
Joints:
- joint base_joint: origin xyz=0 0 0 rpy=0 0 0 -> xyz=0.0 0.0 0.0 rpy=0.0 0.0 0.0
- joint base_link_surface_joint: axis 0 0 1 -> 0.0 0.0 1.0; origin xyz=-0.004485 0 0.352 rpy=0 0 0 -> xyz=-0.004485 0.0 0.352 rpy=0.0 0.0 0.0
- joint base_link_to_imu_joint: origin xyz=0.0 0.0 0.25 rpy=0 0 0 -> xyz=0.0 0.0 0.25 rpy=0.0 0.0 0.0
- joint bl_caster_rotation_joint: axis 0 0 1 -> 0.0 0.0 1.0; origin xyz=-0.300485 0.188 0.1565 rpy=0 0 0 -> xyz=-0.300485 0.188 0.1565 rpy=0.0 0.0 0.0
- joint bl_caster_wheel_joint: axis 0 1 0 -> 0.0 1.0 0.0; origin xyz=-0.0382 0 -0.094 rpy=0 0 0 -> xyz=-0.0382 0.0 -0.094 rpy=0.0 0.0 0.0
- joint br_caster_rotation_joint: axis 0 0 1 -> 0.0 0.0 1.0; origin xyz=-0.300485 -0.188 0.1565 rpy=0 0 0 -> xyz=-0.300485 -0.188 0.1565 rpy=0.0 0.0 0.0
- joint br_caster_wheel_joint: axis 0 1 0 -> 0.0 1.0 0.0; origin xyz=-0.0382 0 -0.094 rpy=0 0 0 -> xyz=-0.0382 0.0 -0.094 rpy=0.0 0.0 0.0
- joint fl_caster_rotation_joint: axis 1 0 0 -> 1.0 0.0 0.0; limit lower=-1e9 upper=1e9 effort=2 velocity=2.0 -> lower=-1000000000.0 upper=1000000000.0 effort=2.0 velocity=2.0; origin xyz=0.299215 0.188 0.1565 rpy=0 0 0 -> xyz=0.299215 0.188 0.1565 rpy=0.0 0.0 0.0
- joint fl_caster_wheel_joint: axis 0 1 0 -> 0.0 1.0 0.0; limit lower=-1e9 upper=1e9 effort=2 velocity=2.0 -> lower=-1000000000.0 upper=1000000000.0 effort=2.0 velocity=2.0; origin xyz=-0.0382 0 -0.094 rpy=0 0 0 -> xyz=-0.0382 0.0 -0.094 rpy=0.0 0.0 0.0
- joint fr_caster_rotation_joint: axis 0 0 1 -> 0.0 0.0 1.0; origin xyz=0.299215 -0.188 0.1565 rpy=0 0 0 -> xyz=0.299215 -0.188 0.1565 rpy=0.0 0.0 0.0
- joint fr_caster_wheel_joint: axis 0 1 0 -> 0.0 1.0 0.0; origin xyz=-0.0382 0 -0.094 rpy=0 0 0 -> xyz=-0.0382 0.0 -0.094 rpy=0.0 0.0 0.0
- joint imu_link_to_imu_frame_joint: origin xyz=0 0 0 rpy=0 0 0 -> xyz=0.0 0.0 0.0 rpy=0.0 0.0 0.0
- joint left_wheel_joint: axis 0 0 1 -> 0.0 0.0 1.0; limit lower=-1e9 upper=1e9 effort=2 velocity=2.0 -> lower=-1000000000.0 upper=1000000000.0 effort=2.0 velocity=2.0; origin xyz=0.0 0.2015 0.1 rpy=0 0 0 -> xyz=0.0 0.2015 0.1 rpy=0.0 0.0 0.0
- joint relax_arm1_joint0: axis 0 0 1 -> 0.0 0.0 1.0
- joint relax_arm1_joint1: axis 0 0 1 -> 0.0 0.0 1.0
- joint relax_arm1_joint2: axis 0 0 1 -> 0.0 0.0 1.0
- joint relax_arm1_joint3: axis 0 0 1 -> 0.0 0.0 1.0
- joint relax_arm1_joint4: axis 0 0 1 -> 0.0 0.0 1.0
- joint relax_arm1_joint5: axis 0 0 1 -> 0.0 0.0 1.0
- joint relax_arm1_joint6: axis 0 0 1 -> 0.0 0.0 1.0
- joint right_wheel_joint: axis 0 1 0 -> 0.0 1.0 0.0; limit effort=100 velocity=20.0 -> lower=0 upper=0 effort=100.0 velocity=20.0; origin xyz=0.0 -0.2015 0.1 rpy=0 0 0 -> xyz=0.0 -0.2015 0.1 rpy=0.0 0.0 0.0
- joint us_1_joint: origin xyz=0.45 -0.12 0.16  rpy=0 0 0 -> xyz=0.45 -0.12 0.16 rpy=0.0 0.0 0.0
- joint us_2_joint: origin xyz=0.45 0.12 0.16  rpy=0 0 0 -> xyz=0.45 0.12 0.16 rpy=0.0 0.0 0.0

File: relax_urdf/urdf/relax_virtual_frame.urdf (robot description, URDF)
Before this commit: robot relax, 33 links, 32 joints
Links:
- removed link D435i_camera_accel_frame
- removed link D435i_camera_accel_optical_frame
- removed link D435i_camera_bottom_screw_frame
- removed link D435i_camera_color_frame
- removed link D435i_camera_color_optical_frame
- removed link D435i_camera_depth_frame
- removed link D435i_camera_depth_optical_frame
- removed link D435i_camera_gyro_frame
- removed link D435i_camera_gyro_optical_frame
- removed link D435i_camera_left_ir_frame
- removed link D435i_camera_left_ir_optical_frame
- removed link D435i_camera_link
- removed link D435i_camera_right_ir_frame
- removed link D435i_camera_right_ir_optical_frame
- removed link control_box
- removed link left_wheel
- removed link left_wheel_yaw
- removed link mobile_base_link
- removed link relax_link1
- removed link relax_link2
- removed link relax_link3
- removed link relax_link4
- removed link relax_link5
- removed link right_wheel
- removed link right_wheel_yaw
- added link back_laser_link, mass 1.2; collision mesh filename=package://relax_urdf/meshes/sick_lms-100.stl; visual mesh filename=package://relax_urdf/meshes/sick_lms-100.stl
- added link base_footprint
- added link bl_caster_rotation_link, mass 0.3097539019; collision mesh filename=package://relax_urdf/meshes/caster_wheel_base.stl; visual mesh filename=package://relax_urdf/meshes/caster_wheel_base.stl
- added link bl_caster_wheel_link, mass 1.0; collision cylinder length=0.032 radius=0.0625; visual cylinder length=0.032 radius=0.0625
- added link br_caster_rotation_link, mass 0.3097539019; collision mesh filename=package://relax_urdf/meshes/caster_wheel_base.stl; visual mesh filename=package://relax_urdf/meshes/caster_wheel_base.stl
- added link br_caster_wheel_link, mass 1.0; collision cylinder length=0.032 radius=0.0625; visual cylinder length=0.032 radius=0.0625
- added link fl_caster_rotation_link, mass 0.3097539019; collision mesh filename=package://relax_urdf/meshes/caster_wheel_base.stl; visual mesh filename=package://relax_urdf/meshes/caster_wheel_base.stl
- added link fl_caster_wheel_link, mass 1.0; collision cylinder length=0.032 radius=0.0625; visual cylinder length=0.032 radius=0.0625
- added link fr_caster_rotation_link, mass 0.3097539019; collision mesh filename=package://relax_urdf/meshes/caster_wheel_base.stl; visual mesh filename=package://relax_urdf/meshes/caster_wheel_base.stl
- added link fr_caster_wheel_link, mass 1.0; collision cylinder length=0.032 radius=0.0625; visual cylinder length=0.032 radius=0.0625
- added link front_laser_link, mass 1.2; collision mesh filename=package://relax_urdf/meshes/sick_lms-100.stl; visual mesh filename=package://relax_urdf/meshes/sick_lms-100.stl
- added link imu_frame
- added link imu_link
- added link left_wheel_link, mass 1.0; collision cylinder length=0.038 radius=0.1; visual cylinder length=0.038 radius=0.1
- added link relax_arm1_link1, mass 6.2381702; collision mesh filename=package://relax_urdf/meshes/mesh_link1.stl scale=0.001 0.001 0.001; visual mesh filename=package://relax_urdf/meshes/mesh_link1.stl scale=0.001 0.001 0.001
- added link relax_arm1_link2, mass 2.601371; collision mesh filename=package://relax_urdf/meshes/mesh_link2.stl scale=0.001 0.001 0.001; visual mesh filename=package://relax_urdf/meshes/mesh_link2.stl scale=0.001 0.001 0.001
- added link relax_arm1_link3, mass 5.9482803; collision mesh filename=package://relax_urdf/meshes/mesh_link3.stl scale=0.001 0.001 0.001; visual mesh filename=package://relax_urdf/meshes/mesh_link3.stl scale=0.001 0.001 0.001
- added link relax_arm1_link4, mass 1.6710337; collision mesh filename=package://relax_urdf/meshes/mesh_link4.stl scale=0.001 0.001 0.001; visual mesh filename=package://relax_urdf/meshes/mesh_link4.stl scale=0.001 0.001 0.001
- added link relax_arm1_link5, mass 6.181102; collision mesh filename=package://relax_urdf/meshes/mesh_link5.stl scale=0.001 0.001 0.001; visual mesh filename=package://relax_urdf/meshes/mesh_link5.stl scale=0.001 0.001 0.001
- added link relax_arm1_link6, mass 0.48141935; collision mesh filename=package://relax_urdf/meshes/mesh_link6.stl scale=0.001 0.001 0.001; visual mesh filename=package://relax_urdf/meshes/mesh_link6.stl scale=0.001 0.001 0.001
- added link relax_arm1_linkEndEffector
- added link right_wheel_link, mass 1.0; collision cylinder length=0.038 radius=0.1; visual cylinder length=0.038 radius=0.1
- added link surface
- added link us_1_frame
- added link us_2_frame
- link base_link: mass None -> 97.0; geometry collision mesh filename=package://relax_urdf/meshes/mesh_base_revised.stl scale=0.001 0.001 0.001; visual mesh filename=package://relax_urdf/meshes/mesh_base_revised.stl scale=0.001 0.001 0.001
Joints:
- removed joint D435i_camera_accel_joint
- removed joint D435i_camera_accel_optical_joint
- removed joint D435i_camera_color_joint
- removed joint D435i_camera_color_optical_joint
- removed joint D435i_camera_depth_joint
- removed joint D435i_camera_depth_optical_joint
- removed joint D435i_camera_gyro_joint
- removed joint D435i_camera_gyro_optical_joint
- removed joint D435i_camera_joint
- removed joint D435i_camera_left_ir_joint
- removed joint D435i_camera_left_ir_optical_joint
- removed joint D435i_camera_link_joint
- removed joint D435i_camera_right_ir_joint
- removed joint D435i_camera_right_ir_optical_joint
- removed joint j_control
- removed joint j_left_wheel_roll
- removed joint j_left_wheel_yaw
- removed joint j_right_wheel_roll
- removed joint j_right_wheel_yaw
- removed joint joint1
- removed joint joint2
- removed joint joint3
- removed joint joint4
- removed joint mobile_base_joint
- added joint base_link_surface_joint: type fixed, parent base_link, child surface, origin xyz=-0.004485 0 0.352 rpy=0 0 0, axis 0 0 1
- added joint base_link_to_back_laser_joint: type fixed, parent base_link, child back_laser_link, origin xyz=-0.319485 -0.205 0.1914 rpy=0.0 0.0 -2.356194490192345
- added joint base_link_to_front_laser_joint: type fixed, parent base_link, child front_laser_link, origin xyz=0.310515 0.205 0.1914 rpy=0.0 0.0 0.7853981633974483
- added joint base_link_to_imu_joint: type fixed, parent base_link, child imu_link, origin xyz=0.0 0.0 0.25 rpy=0 0 0
- added joint bl_caster_rotation_joint: type fixed, parent base_link, child bl_caster_rotation_link, origin xyz=-0.300485 0.188 0.1565 rpy=0 0 0, axis 0 0 1
- added joint bl_caster_wheel_joint: type fixed, parent bl_caster_rotation_link, child bl_caster_wheel_link, origin xyz=-0.0382 0 -0.094 rpy=0 0 0, axis 0 1 0
- added joint br_caster_rotation_joint: type fixed, parent base_link, child br_caster_rotation_link, origin xyz=-0.300485 -0.188 0.1565 rpy=0 0 0, axis 0 0 1
- added joint br_caster_wheel_joint: type fixed, parent br_caster_rotation_link, child br_caster_wheel_link, origin xyz=-0.0382 0 -0.094 rpy=0 0 0, axis 0 1 0
- added joint fl_caster_rotation_joint: type prismatic, parent base_link, child fl_caster_rotation_link, origin xyz=0.299215 0.188 0.1565 rpy=0 0 0, axis 1 0 0, limit lower=-1e9 upper=1e9 effort=2 velocity=2.0
- added joint fl_caster_wheel_joint: type fixed, parent fl_caster_rotation_link, child fl_caster_wheel_link, origin xyz=-0.0382 0 -0.094 rpy=0 0 0, axis 0 1 0, limit lower=-1e9 upper=1e9 effort=2 velocity=2.0
- added joint fr_caster_rotation_joint: type fixed, parent base_link, child fr_caster_rotation_link, origin xyz=0.299215 -0.188 0.1565 rpy=0 0 0, axis 0 0 1
- added joint fr_caster_wheel_joint: type fixed, parent fr_caster_rotation_link, child fr_caster_wheel_link, origin xyz=-0.0382 0 -0.094 rpy=0 0 0, axis 0 1 0
- added joint imu_link_to_imu_frame_joint: type fixed, parent imu_link, child imu_frame, origin xyz=0 0 0 rpy=0 0 0
- added joint left_wheel_joint: type revolute, parent base_link, child left_wheel_link, origin xyz=0.0 0.2015 0.1 rpy=0 0 0, axis 0 0 1, limit lower=-1e9 upper=1e9 effort=2 velocity=2.0
- added joint relax_arm1_joint0: type revolute, parent base_link, child relax_arm1_link1, origin xyz=-0.13 0.0 0.3613 rpy=0.0 0.0 0.0, axis 0 0 1, limit lower=-3.14 upper=3.14 effort=147.0 velocity=3.86
- added joint relax_arm1_joint1: type revolute, parent relax_arm1_link1, child relax_arm1_link2, origin xyz=0.0 0.13166 0.24966 rpy=-1.5707963 0.0 0.0, axis 0 0 1, limit lower=-3.14 upper=3.14 effort=147.0 velocity=3.86
- added joint relax_arm1_joint2: type revolute, parent relax_arm1_link2, child relax_arm1_link3, origin xyz=0.0 -0.4 0.0 rpy=0.0 0.0 0.0, axis 0 0 1, limit lower=-3.14 upper=3.14 effort=147.0 velocity=3.86
- added joint relax_arm1_joint3: type revolute, parent relax_arm1_link3, child relax_arm1_link4, origin xyz=0.0 -0.24966 -0.13166 rpy=1.5707963 0.0 0.0, axis 0 0 1, limit lower=-3.14 upper=3.14 effort=147.0 velocity=3.86
- added joint relax_arm1_joint4: type revolute, parent relax_arm1_link4, child relax_arm1_link5, origin xyz=0.0 -0.08816 0.1535 rpy=1.5707963 0.0 0.0, axis 0 0 1, limit lower=-3.14 upper=3.14 effort=147.0 velocity=3.86
- added joint relax_arm1_joint5: type revolute, parent relax_arm1_link5, child relax_arm1_link6, origin xyz=0.0 0.22216 -0.08816 rpy=-1.5707963 0.0 0.0, axis 0 0 1, limit lower=-3.14 upper=3.14 effort=147.0 velocity=3.86
- added joint relax_arm1_joint6: type fixed, parent relax_arm1_link6, child relax_arm1_linkEndEffector, origin xyz=0.0 0.0 0.028 rpy=0.0 0.0 0.0, axis 0 0 1, limit lower=-3.14 upper=3.14 effort=147.0 velocity=3.86
- added joint right_wheel_joint: type fixed, parent base_link, child right_wheel_link, origin xyz=0.0 -0.2015 0.1 rpy=0 0 0, axis 0 1 0, limit effort=100 velocity=20.0
- added joint us_1_joint: type fixed, parent base_link, child us_1_frame, origin xyz=0.45 -0.12 0.16  rpy=0 0 0
- added joint us_2_joint: type fixed, parent base_link, child us_2_frame, origin xyz=0.45 0.12 0.16  rpy=0 0 0
- joint base_joint: child mobile_base_link -> base_link; parent base_link -> base_footprint
- joint car_frame_tx: parent base_link -> base_footprint
- joint world_joint: child base_link -> base_footprint; origin xyz=0 0 0 rpy=0 0 0 -> (none)
