Commit message: clean models and fixed the caster issue

File: relax_urdf/urdf/parts/mir_base.urdf.xacro (robot description, xacro)
@@ -163,5 +163,5 @@
     </inertial>
     <visual>
-      <origin rpy="0 0 0" xyz="0 0 0"/>
+      <origin rpy="1.57 0 0" xyz="0 0 0"/>
       <!--${pi/2} 0 0 -->
       <geometry>
@@ -173,5 +173,5 @@
     </visual>
     <collision>
-      <origin rpy="0 0 0" xyz="0 0 0"/>
+      <origin rpy="1.57 0 0" xyz="0 0 0"/>
       <!--${pi/2} 0 0 -->
       <geometry>

File: relax_urdf/urdf/parts/wheels.urdf.xacro (robot description, xacro)
@@ -108,5 +108,5 @@
       </xacro:cylinder_inertial>
       <visual>
-        <origin xyz="0 0 0" rpy="0 0 0" /> <!--${pi/2} 0 0 -->
+        <origin xyz="0 0 0" rpy="${pi/2} 0 0" /> <!--${pi/2} 0 0 -->
         <geometry>
           <cylinder radius="${mir_caster_wheel_radius}" length="${mir_caster_wheel_width}" />
@@ -115,5 +115,5 @@
       </visual>
       <collision>
-        <origin xyz="0 0 0" rpy="0 0 0" /> <!--${pi/2} 0 0 -->
+        <origin xyz="0 0 0" rpy="${pi/2} 0 0" /> <!--${pi/2} 0 0 -->
         <geometry>
           <cylinder radius="${mir_caster_wheel_radius}" length="${mir_caster_wheel_width}" />

Commit message: added new meshes

File: relax_urdf/urdf/parts/mir_base.urdf.xacro (robot description, xacro)
@@ -24,5 +24,5 @@
         <origin xyz="${mir_act_wheel_dx} 0 0" rpy="0 0 0" />
         <geometry>
-          <mesh filename="package://relax_urdf/meshes/mesh_base_revised.stl" scale="0.001 0.001 0.001"/>
+          <mesh filename="package://relax_urdf/meshes/mesh_base_2.stl" scale="0.001 0.001 0.001"/>
         </geometry>
         <xacro:insert_block name="material_dark_grey" />
@@ -31,5 +31,5 @@
         <origin xyz="${mir_act_wheel_dx} 0 0" rpy="0 0 0" />
         <geometry>
-          <mesh filename="package://relax_urdf/meshes/mesh_base_revised.stl"  scale="0.001 0.001 0.001"/>
+          <mesh filename="package://relax_urdf/meshes/mesh_base_2.stl"  scale="0.001 0.001 0.001"/>
         </geometry>
       </collision>

File: relax_urdf/urdf/parts/relax_arm.urdf.xacro (robot description, xacro)
@@ -13,5 +13,5 @@
       <origin xyz="0 0 0" rpy="0 0 0"/>
       <geometry name="relax_link1_visual">
-        <mesh filename="package://relax_urdf/meshes/mesh_link1.stl" scale="0.001 0.001 0.001" />
+        <mesh filename="package://relax_urdf/meshes/mesh_link1_2.stl" scale="0.001 0.001 0.001" />
       </geometry>
       <material name="darkblue"/>
@@ -20,5 +20,5 @@
       <origin xyz="0 0 0" rpy="0 0 0"/>
       <geometry name="relax_link1_collision">
-        <mesh filename="package://relax_urdf/meshes/mesh_link1.stl" scale="0.001 0.001 0.001" />
+        <mesh filename="package://relax_urdf/meshes/mesh_link1_2.stl" scale="0.001 0.001 0.001" />
       </geometry>
     </collision>
