Commit message: Update relax_arm.urdf.xacro

File: relax_urdf/urdf/parts/relax_arm.urdf.xacro (robot description, xacro)
@@ -129,5 +129,5 @@
     <child link="relax_arm${arm_num}_link2"/>
     <origin xyz="${Joint_1_Ox} ${Joint_1_Oy} ${Joint_1_Oz}" rpy="${Joint_1_Oroll} ${Joint_1_Opitch} ${Joint_1_Oyaw}"/>
-    <axis xyz="0 0 1"/>
+    <axis xyz="0 1 0"/>
     <limit velocity="${Joint_1_velocity}" effort="${Joint_1_effort}" lower="${Joint_1_lower}" upper="${Joint_1_upper}" />
     <dynamics damping="${Joint_1_damp}" friction="${Joint_1_fric}"/>
@@ -137,5 +137,5 @@
     <child link="relax_arm${arm_num}_link3"/>
     <origin xyz="${Joint_2_Ox} ${Joint_2_Oy} ${Joint_2_Oz}" rpy="${Joint_2_Oroll} ${Joint_2_Opitch} ${Joint_2_Oyaw}"/>
-    <axis xyz="0 0 1"/>
+    <axis xyz="0 1 0"/>
     <limit velocity="${Joint_2_velocity}" effort="${Joint_2_effort}" lower="${Joint_2_lower}" upper="${Joint_2_upper}" />
     <dynamics damping="${Joint_2_damp}" friction="${Joint_2_fric}"/>

Commit message: modifying for new version of arm and mobile base - urdf and srdf consistency

File: relax_urdf/urdf/parts/relax_arm.urdf.xacro (robot description, xacro)
@@ -104,5 +104,5 @@
     </collision>
 </link>
-<link name ="relax_arm${arm_num}_link6">  <!-- link 5 -->
+<link name ="relax_arm${arm_num}_link6">  <!-- link 6 -->
     <inertial>
       <origin xyz="${Link_6_x} ${Link_6_y} ${Link_6_z}" />
@@ -129,5 +129,5 @@
     <child link="relax_arm${arm_num}_link2"/>
     <origin xyz="${Joint_1_Ox} ${Joint_1_Oy} ${Joint_1_Oz}" rpy="${Joint_1_Oroll} ${Joint_1_Opitch} ${Joint_1_Oyaw}"/>
-    <axis xyz="0 1 0"/>
+    <axis xyz="0 0 1"/>
     <limit velocity="${Joint_1_velocity}" effort="${Joint_1_effort}" lower="${Joint_1_lower}" upper="${Joint_1_upper}" />
     <dynamics damping="${Joint_1_damp}" friction="${Joint_1_fric}"/>
@@ -145,5 +145,5 @@
     <child link="relax_arm${arm_num}_link4"/>
     <origin xyz="${Joint_3_Ox} ${Joint_3_Oy} ${Joint_3_Oz}" rpy="${Joint_3_Oroll} ${Joint_3_Opitch} ${Joint_3_Oyaw}"/>
-    <axis xyz="0 0 1"/>
+    <axis xyz="0 1 0"/>
     <limit velocity="${Joint_3_velocity}" effort="${Joint_3_effort}" lower="${Joint_3_lower}" upper="${Joint_3_upper}" />
     <dynamics damping="${Joint_3_damp}" friction="${Joint_3_fric}"/>
@@ -161,5 +161,5 @@
     <child link="relax_arm${arm_num}_link6"/>
     <origin xyz="${Joint_5_Ox} ${Joint_5_Oy} ${Joint_5_Oz}" rpy="${Joint_5_Oroll} ${Joint_5_Opitch} ${Joint_5_Oyaw}"/>
-    <axis xyz="0 0 1"/>
+    <axis xyz="0 1 0"/>
     <limit velocity="${Joint_5_velocity}" effort="${Joint_5_effort}" lower="${Joint_5_lower}" upper="${Joint_5_upper}" />
     <dynamics damping="${Joint_5_damp}" friction="${Joint_5_fric}"/>

File: relax_urdf/urdf/relax.urdf (robot description, URDF)
Before this commit: robot relax, 27 links, 26 joints
Links:
- added link relax_arm1_link6, mass 5.7923846; collision mesh filename=package://relax_urdf/meshes/mesh_link5.stl scale=0.001 0.001 0.001; visual mesh filename=package://relax_urdf/meshes/mesh_link5.stl scale=0.001 0.001 0.001

Commit message: fixed joints axis - some mistakes were there

File: relax_urdf/urdf/parts/relax_arm.urdf.xacro (robot description, xacro)
@@ -138,5 +138,5 @@
     <child link="relax_arm${arm_num}_link3"/>
     <origin xyz="${Joint_2_Ox} ${Joint_2_Oy} ${Joint_2_Oz}" rpy="${Joint_2_Oroll} ${Joint_2_Opitch} ${Joint_2_Oyaw}"/>
-    <axis xyz="0 1 0"/>
+    <axis xyz="0 0 1"/>
     <limit velocity="${Joint_2_velocity}" effort="${Joint_2_effort}" lower="${Joint_2_lower}" upper="${Joint_2_upper}" />
     <dynamics damping="${Joint_2_damp}" friction="${Joint_2_fric}"/>
@@ -146,5 +146,5 @@
     <child link="relax_arm${arm_num}_link4"/>
     <origin xyz="${Joint_3_Ox} ${Joint_3_Oy} ${Joint_3_Oz}" rpy="${Joint_3_Oroll} ${Joint_3_Opitch} ${Joint_3_Oyaw}"/>
-    <axis xyz="0 1 0"/>
+    <axis xyz="0 0 1"/>
     <limit velocity="${Joint_3_velocity}" effort="${Joint_3_effort}" lower="${Joint_3_lower}" upper="${Joint_3_upper}" />
     <dynamics damping="${Joint_3_damp}" friction="${Joint_3_fric}"/>
@@ -162,5 +162,5 @@
     <child link="relax_arm${arm_num}_link6"/>
     <origin xyz="${Joint_5_Ox} ${Joint_5_Oy} ${Joint_5_Oz}" rpy="${Joint_5_Oroll} ${Joint_5_Opitch} ${Joint_5_Oyaw}"/>
-    <axis xyz="0 1 0"/>
+    <axis xyz="0 0 1"/>
     <limit velocity="${Joint_5_velocity}" effort="${Joint_5_effort}" lower="${Joint_5_lower}" upper="${Joint_5_upper}" />
     <dynamics damping="${Joint_5_damp}" friction="${Joint_5_fric}"/>

Commit message: Removing rpy to inertial data of link4 to solve https://github.com/ADVRHumanoids/iit-relax-ros-pkg/issues/28

File: relax_urdf/urdf/parts/relax_arm.urdf.xacro (robot description, xacro)
@@ -66,5 +66,5 @@
 <link name ="relax_arm${arm_num}_link4">  <!-- link 4 -->
     <inertial>
-      <origin xyz="${Link_4_x} ${Link_4_y} ${Link_4_z}" rpy="-2.6324601 1.5172034 -2.2584214"/>
+      <origin xyz="${Link_4_x} ${Link_4_y} ${Link_4_z}"/>
       <mass value="${Link_4_mass}"/>
       <inertia ixx="${Link_4_xx}" ixy="${Link_4_xy}" ixz="${Link_4_xz}" iyy="${Link_4_yy}" iyz="${Link_4_yz}" izz="${Link_4_zz}" />

Commit message: tests on real robot with cartesi/o

File: relax_urdf/urdf/parts/relax_arm.urdf.xacro (robot description, xacro)
@@ -154,5 +154,5 @@
     <child link="relax_arm${arm_num}_link4"/>
     <origin xyz="${Joint_3_Ox} ${Joint_3_Oy} ${Joint_3_Oz}" rpy="${Joint_3_Oroll} ${Joint_3_Opitch} ${Joint_3_Oyaw}"/>
-    <axis xyz="0 0 -1"/>
+    <axis xyz="0 0 1"/>
     <limit velocity="${Joint_3_velocity}" effort="${Joint_3_effort}" lower="${Joint_3_lower}" upper="${Joint_3_upper}" />
     <dynamics damping="${Joint_3_damp}" friction="${Joint_3_fric}"/>

File: relax_urdf/urdf/relax_arm.urdf (robot description, URDF)
Before this commit: robot relax, 8 links, 7 joints
Links:
- link base_link: mass 1 -> 97.0; geometry collision mesh filename=package://relax_urdf/meshes/mesh_base_revised.stl scale=0.001 0.001 0.001; visual mesh filename=package://relax_urdf/meshes/mesh_base_revised.stl scale=0.001 0.001 0.001
Joints:
- joint relax_arm1_joint3: axis 0 0 -1 -> 0 0 1

Commit message: attaching teraflex device

File: relax_urdf/urdf/parts/relax_arm.urdf.xacro (robot description, xacro)
@@ -166,5 +166,6 @@
     <dynamics damping="${Joint_4_damp}" friction="${Joint_4_fric}"/>
 </joint>
-<joint name="relax_arm${arm_num}_joint5" type="revolute"> <!-- joint 5 -->
+<!-- joint 5 -->
+<!-- <joint name="relax_arm${arm_num}_joint5" type="revolute">
     <parent link="relax_arm${arm_num}_link5"/>
     <child link="relax_arm${arm_num}_link6"/>
@@ -173,5 +174,5 @@
     <limit velocity="${Joint_5_velocity}" effort="${Joint_5_effort}" lower="${Joint_5_lower}" upper="${Joint_5_upper}" />
     <dynamics damping="${Joint_5_damp}" friction="${Joint_5_fric}"/>
-</joint>
+</joint> -->
 <joint name="relax_arm${arm_num}_joint6" type="fixed"> <!-- joint 6 fake -->
     <parent link="relax_arm${arm_num}_link6"/>

File: relax_urdf/urdf/parts/teraflex_ring.urdf.xacro (robot description, xacro)
@@ -80,4 +80,13 @@
     <origin xyz="${Joint_S6_S7_Ox} ${Joint_S6_S7_Oy} ${Joint_S6_S7_Oz}" rpy="${Joint_S6_S7_Oroll} ${Joint_S6_S7_Opitch} ${Joint_S6_S7_Oyaw}"/>
 </joint>
+<joint name="relax_arm1_joint5" type="revolute">
+    <!-- joint fake -->
+    <parent link="teraflex_1_sensor7_link"/>
+    <child link="relax_arm1_link6"/>
+    <origin rpy="0.0 0.0 2.9966942" xyz="-0.0776 0.0 0.0796600"/>
+    <axis xyz="0 0 1"/>
+    <limit effort="147.0" lower="-2.7" upper="2.7" velocity="3.86"/>
+    <dynamics damping="0.2" friction="10.0"/>
+  </joint>
 </xacro:macro>
 </robot>

File: relax_urdf/urdf/relax_arm_teraflex.urdf (robot description, URDF)
Before this commit: robot relax, 8 links, 7 joints
Links:
- added link teraflex_1_link, mass 0.03; collision mesh filename=package://relax_urdf/meshes/mesh_teraflex-ring.stl scale=0.001 0.001 0.001; visual mesh filename=package://relax_urdf/meshes/mesh_teraflex-ring.stl scale=0.001 0.001 0.001
- added link teraflex_1_sensor0_link
- added link teraflex_1_sensor1_link
- added link teraflex_1_sensor2_link
- added link teraflex_1_sensor3_link
- added link teraflex_1_sensor4_link
- added link teraflex_1_sensor5_link
- added link teraflex_1_sensor6_link
- added link teraflex_1_sensor7_link
Joints:
- added joint teraflex_1_mount_joint: type fixed, parent relax_arm1_link5, child teraflex_1_link, origin xyz= 0.0 0.142500 -0.0881600  rpy=-1.5707963 -0.6404992 0
- added joint teraflex_1_sensor0_joint: type fixed, parent relax_arm1_link5, child teraflex_1_sensor0_link, origin xyz=-0.0622195 0.142500 -0.1345334 rpy=1.5708 0.6405 3.1416
- added joint teraflex_1_sensor1_joint: type fixed, parent relax_arm1_link5, child teraflex_1_sensor1_link, origin xyz=-0.0112049 0.142500 -0.1649568 rpy=1.5708 1.4259 3.1416
- added joint teraflex_1_sensor2_joint: type fixed, parent relax_arm1_link5, child teraflex_1_sensor2_link, origin xyz=0.0463735 0.142500 -0.1503796 rpy=-1.5708 0.9303 0.0
- added joint teraflex_1_sensor3_joint: type fixed, parent relax_arm1_link5, child teraflex_1_sensor3_link, origin xyz=0.0767869 0.142500 -0.0993649 rpy=-1.5708 0.1449 0.0
- added joint teraflex_1_sensor4_joint: type fixed, parent relax_arm1_link5, child teraflex_1_sensor4_link, origin xyz=0.0622196 0.142500 -0.0417865 rpy=-1.5708 -0.6405 0.0
- added joint teraflex_1_sensor5_joint: type fixed, parent relax_arm1_link5, child teraflex_1_sensor5_link, origin xyz=0.0112049 0.142500 -0.0113731 rpy=-1.5708 -1.4259 0.0
- added joint teraflex_1_sensor6_joint: type fixed, parent relax_arm1_link5, child teraflex_1_sensor6_link, origin xyz=-0.0463735 0.142500 -0.0259404 rpy=1.5708 -0.9303 3.1416
- added joint teraflex_1_sensor7_joint: type fixed, parent relax_arm1_link5, child teraflex_1_sensor7_link, origin xyz=-0.0767870 0.142500 -0.0769551 rpy=1.5708 -0.1449 3.1416

Commit message: fix bugs in the xacros files - they were mismatching

File: relax_urdf/urdf/parts/relax_arm.urdf.xacro (robot description, xacro)
@@ -167,5 +167,5 @@
 </joint>
 <!-- joint 5 -->
-<!-- <joint name="relax_arm${arm_num}_joint5" type="revolute">
+<joint name="relax_arm${arm_num}_joint5" type="revolute">
     <parent link="relax_arm${arm_num}_link5"/>
     <child link="relax_arm${arm_num}_link6"/>
@@ -174,5 +174,5 @@
     <limit velocity="${Joint_5_velocity}" effort="${Joint_5_effort}" lower="${Joint_5_lower}" upper="${Joint_5_upper}" />
     <dynamics damping="${Joint_5_damp}" friction="${Joint_5_fric}"/>
-</joint> -->
+</joint>
 <joint name="relax_arm${arm_num}_joint6" type="fixed"> <!-- joint 6 fake -->
     <parent link="relax_arm${arm_num}_link6"/>

File: relax_urdf/urdf/parts/teraflex_ring.urdf.xacro (robot description, xacro)
@@ -41,52 +41,43 @@
 <link name ="teraflex_${id}_sensor7_link" />
 <joint name="teraflex_${id}_sensor0_joint" type="fixed"> <!-- joint fake -->
-    <parent link="teraflex_${id}_link"/>
+    <parent link="${parent_link}"/>
     <child link="teraflex_${id}_sensor0_link"/>
     <origin xyz="${Joint_TF_S0_Ox} ${Joint_TF_S0_Oy} ${Joint_TF_S0_Oz}" rpy="${Joint_TF_S0_Oroll} ${Joint_TF_S0_Opitch} ${Joint_TF_S0_Oyaw}"/>
 </joint>
-<joint name="teraflex_${id}_sensor01_joint" type="fixed"> <!-- joint fake -->
-    <parent link="teraflex_${id}_sensor0_link"/>
+<joint name="teraflex_${id}_sensor1_joint" type="fixed"> <!-- joint fake -->
+    <parent link="${parent_link}"/>
     <child link="teraflex_${id}_sensor1_link"/>
     <origin xyz="${Joint_S0_S1_Ox} ${Joint_S0_S1_Oy} ${Joint_S0_S1_Oz}" rpy="${Joint_S0_S1_Oroll} ${Joint_S0_S1_Opitch} ${Joint_S0_S1_Oyaw}"/>
 </joint>
-<joint name="teraflex_${id}_sensor12_joint" type="fixed"> <!-- joint fake -->
-    <parent link="teraflex_${id}_sensor1_link"/>
+<joint name="teraflex_${id}_sensor2_joint" type="fixed"> <!-- joint fake -->
+    <parent link="${parent_link}"/>
     <child link="teraflex_${id}_sensor2_link"/>
     <origin xyz="${Joint_S1_S2_Ox} ${Joint_S1_S2_Oy} ${Joint_S1_S2_Oz}" rpy="${Joint_S1_S2_Oroll} ${Joint_S1_S2_Opitch} ${Joint_S1_S2_Oyaw}"/>
 </joint>
-<joint name="teraflex_${id}_sensor23_joint" type="fixed"> <!-- joint fake -->
-    <parent link="teraflex_${id}_sensor2_link"/>
+<joint name="teraflex_${id}_sensor3_joint" type="fixed"> <!-- joint fake -->
+    <parent link="${parent_link}"/>
     <child link="teraflex_${id}_sensor3_link"/>
     <origin xyz="${Joint_S2_S3_Ox} ${Joint_S2_S3_Oy} ${Joint_S2_S3_Oz}" rpy="${Joint_S2_S3_Oroll} ${Joint_S2_S3_Opitch} ${Joint_S2_S3_Oyaw}"/>
 </joint>
-<joint name="teraflex_${id}_sensor34_joint" type="fixed"> <!-- joint fake -->
-    <parent link="teraflex_${id}_sensor3_link"/>
+<joint name="teraflex_${id}_sensor4_joint" type="fixed"> <!-- joint fake -->
+    <parent link="${parent_link}"/>
     <child link="teraflex_${id}_sensor4_link"/>
     <origin xyz="${Joint_S3_S4_Ox} ${Joint_S3_S4_Oy} ${Joint_S3_S4_Oz}" rpy="${Joint_S3_S4_Oroll} ${Joint_S3_S4_Opitch} ${Joint_S3_S4_Oyaw}"/>
 </joint>
-<joint name="teraflex_${id}_sensor45_joint" type="fixed"> <!-- joint fake -->
-    <parent link="teraflex_${id}_sensor4_link"/>
+<joint name="teraflex_${id}_sensor5_joint" type="fixed"> <!-- joint fake -->
+    <parent link="${parent_link}"/>
     <child link="teraflex_${id}_sensor5_link"/>
     <origin xyz="${Joint_S4_S5_Ox} ${Joint_S4_S5_Oy} ${Joint_S4_S5_Oz}" rpy="${Joint_S4_S5_Oroll} ${Joint_S4_S5_Opitch} ${Joint_S4_S5_Oyaw}"/>
 </joint>
-<joint name="teraflex_${id}_sensor56_joint" type="fixed"> <!-- joint fake -->
-    <parent link="teraflex_${id}_sensor5_link"/>
+<joint name="teraflex_${id}_sensor6_joint" type="fixed"> <!-- joint fake -->
+    <parent link="${parent_link}"/>
     <child link="teraflex_${id}_sensor6_link"/>
     <origin xyz="${Joint_S5_S6_Ox} ${Joint_S5_S6_Oy} ${Joint_S5_S6_Oz}" rpy="${Joint_S5_S6_Oroll} ${Joint_S5_S6_Opitch} ${Joint_S5_S6_Oyaw}"/>
 </joint>
-<joint name="teraflex_${id}_sensor67_joint" type="fixed"> <!-- joint fake -->
-    <parent link="teraflex_${id}_sensor6_link"/>
+<joint name="teraflex_${id}_sensor7_joint" type="fixed"> <!-- joint fake -->
+    <parent link="${parent_link}"/>
     <child link="teraflex_${id}_sensor7_link"/>
     <origin xyz="${Joint_S6_S7_Ox} ${Joint_S6_S7_Oy} ${Joint_S6_S7_Oz}" rpy="${Joint_S6_S7_Oroll} ${Joint_S6_S7_Opitch} ${Joint_S6_S7_Oyaw}"/>
 </joint>
-<joint name="relax_arm1_joint5" type="revolute">
-    <!-- joint fake -->
-    <parent link="teraflex_1_sensor7_link"/>
-    <child link="relax_arm1_link6"/>
-    <origin rpy="0.0 0.0 2.9966942" xyz="-0.0776 0.0 0.0796600"/>
-    <axis xyz="0 0 1"/>
-    <limit effort="147.0" lower="-2.7" upper="2.7" velocity="3.86"/>
-    <dynamics damping="0.2" friction="10.0"/>
-  </joint>
 </xacro:macro>
 </robot>

File: relax_urdf/urdf/parts/teraflex_ring_kinematics_properties.urdf.xacro (robot description, xacro)
@@ -2,51 +2,59 @@
 <robot  xmlns:xacro="http://ros.org/wiki/xacro">
 <!-- TERAFLEX RING -->
-<xacro:property name="Joint_TF_S0_Ox" value=" ${-77.6000*mmTom} "/>  <!-- Joint Origin TF To Sensor 0 -->
-<xacro:property name="Joint_TF_S0_Oy" value=" 0.0 "/>
-<xacro:property name="Joint_TF_S0_Oz" value=" 0.0 "/>
-<xacro:property name="Joint_TF_S0_Oroll" value=" 0.0 "/>
-<xacro:property name="Joint_TF_S0_Opitch" value=" 0.0"/>
-<xacro:property name="Joint_TF_S0_Oyaw" value=" -3.1415927 "/>
-<xacro:property name="Joint_S0_S1_Ox" value=" ${-22.7285*mmTom} "/>  <!-- Joint Sensor 0 To Sensor 1 -->
-<xacro:property name="Joint_S0_S1_Oy" value=" ${-54.8715*mmTom} "/>
-<xacro:property name="Joint_S0_S1_Oz" value=" 0.0 "/>
-<xacro:property name="Joint_S0_S1_Oroll" value=" 0.0 "/>
-<xacro:property name="Joint_S0_S1_Opitch" value=" 0.0"/>
-<xacro:property name="Joint_S0_S1_Oyaw" value=" -0.7853983 "/>
-<xacro:property name="Joint_S1_S2_Ox" value=" ${-22.7285*mmTom} "/>  <!-- Joint Sensor 1 To Sensor 2 -->
-<xacro:property name="Joint_S1_S2_Oy" value=" ${-54.8715*mmTom} "/>
-<xacro:property name="Joint_S1_S2_Oz" value=" 0.0 "/>
-<xacro:property name="Joint_S1_S2_Oroll" value=" 0.0 "/>
-<xacro:property name="Joint_S1_S2_Opitch" value=" 0.0"/>
-<xacro:property name="Joint_S1_S2_Oyaw" value=" -0.7853983 "/>
-<xacro:property name="Joint_S2_S3_Ox" value=" ${-22.7285*mmTom} "/>  <!-- Joint Sensor 2 To Sensor 3 -->
-<xacro:property name="Joint_S2_S3_Oy" value=" ${-54.8715*mmTom} "/>
-<xacro:property name="Joint_S2_S3_Oz" value=" 0.0 "/>
-<xacro:property name="Joint_S2_S3_Oroll" value=" 0.0 "/>
-<xacro:property name="Joint_S2_S3_Opitch" value=" 0.0"/>
-<xacro:property name="Joint_S2_S3_Oyaw" value=" -0.7853983 "/>
-<xacro:property name="Joint_S3_S4_Ox" value=" ${-22.7285*mmTom} "/>  <!-- Joint Sensor 3 To Sensor 4 -->
-<xacro:property name="Joint_S3_S4_Oy" value=" ${-54.8715*mmTom} "/>
-<xacro:property name="Joint_S3_S4_Oz" value=" 0.0 "/>
-<xacro:property name="Joint_S3_S4_Oroll" value=" 0.0 "/>
-<xacro:property name="Joint_S3_S4_Opitch" value=" 0.0"/>
-<xacro:property name="Joint_S3_S4_Oyaw" value=" -0.7853983 "/>
-<xacro:property name="Joint_S4_S5_Ox" value=" ${-22.7285*mmTom} "/>  <!-- Joint Sensor 4 To Sensor 5 -->
-<xacro:property name="Joint_S4_S5_Oy" value=" ${-54.8715*mmTom} "/>
-<xacro:property name="Joint_S4_S5_Oz" value=" 0.0 "/>
-<xacro:property name="Joint_S4_S5_Oroll" value=" 0.0 "/>
-<xacro:property name="Joint_S4_S5_Opitch" value=" 0.0"/>
-<xacro:property name="Joint_S4_S5_Oyaw" value=" -0.7853983 "/>
-<xacro:property name="Joint_S5_S6_Ox" value=" ${-22.7285*mmTom} "/>  <!-- Joint Sensor 5 To Sensor 6 -->
-<xacro:property name="Joint_S5_S6_Oy" value=" ${-54.8715*mmTom} "/>
-<xacro:property name="Joint_S5_S6_Oz" value=" 0.0 "/>
-<xacro:property name="Joint_S5_S6_Oroll" value=" 0.0 "/>
-<xacro:property name="Joint_S5_S6_Opitch" value=" 0.0"/>
-<xacro:property name="Joint_S5_S6_Oyaw" value=" -0.7853983 "/>
-<xacro:property name="Joint_S6_S7_Ox" value=" ${-22.7285*mmTom} "/>  <!-- Joint Sensor 6 To Sensor 7 -->
-<xacro:property name="Joint_S6_S7_Oy" value=" ${-54.8715*mmTom} "/>
-<xacro:property name="Joint_S6_S7_Oz" value=" 0.0 "/>
-<xacro:property name="Joint_S6_S7_Oroll" value=" 0.0 "/>
-<xacro:property name="Joint_S6_S7_Opitch" value=" 0.0"/>
-<xacro:property name="Joint_S6_S7_Oyaw" value=" -0.7853983 "/>
+<!-- Sensor 0 -->
+<xacro:property name="Joint_TF_S0_Ox" value=" -0.0622195 "/>
+<xacro:property name="Joint_TF_S0_Oy" value=" 0.142500 "/>
+<xacro:property name="Joint_TF_S0_Oz" value=" -0.1345334 "/>
+<xacro:property name="Joint_TF_S0_Oroll" value=" 1.5708 "/>
+<xacro:property name="Joint_TF_S0_Opitch" value=" 0.6405 "/>
+<xacro:property name="Joint_TF_S0_Oyaw" value=" 3.1416 "/>
+ <!-- Sensor 1 -->
+<xacro:property name="Joint_S0_S1_Ox" value=" -0.0112049 "/>
+<xacro:property name="Joint_S0_S1_Oy" value=" 0.142500 "/>
+<xacro:property name="Joint_S0_S1_Oz" value=" -0.1649568 "/>
+<xacro:property name="Joint_S0_S1_Oroll" value=" 1.5708 "/>
+<xacro:property name="Joint_S0_S1_Opitch" value=" 1.4259 "/>
+<xacro:property name="Joint_S0_S1_Oyaw" value=" 3.1416 "/>
+<!-- Sensor 2 -->
+<xacro:property name="Joint_S1_S2_Ox" value=" 0.0463735 "/>
+<xacro:property name="Joint_S1_S2_Oy" value=" 0.142500 "/>
+<xacro:property name="Joint_S1_S2_Oz" value=" -0.1503796 "/>
+<xacro:property name="Joint_S1_S2_Oroll" value=" -1.5708 "/>
+<xacro:property name="Joint_S1_S2_Opitch" value=" 0.9303 "/>
+<xacro:property name="Joint_S1_S2_Oyaw" value=" 0.0 "/>
+<!-- Sensor 3 -->
+<xacro:property name="Joint_S2_S3_Ox" value=" 0.0767869 "/>
+<xacro:property name="Joint_S2_S3_Oy" value=" 0.142500 "/>
+<xacro:property name="Joint_S2_S3_Oz" value=" -0.0993649 "/>
+<xacro:property name="Joint_S2_S3_Oroll" value=" -1.5708 "/>
+<xacro:property name="Joint_S2_S3_Opitch" value=" 0.1449 "/>
+<xacro:property name="Joint_S2_S3_Oyaw" value=" 0.0 "/>
+<!-- Sensor 4 -->
+<xacro:property name="Joint_S3_S4_Ox" value=" 0.0622196 "/>
+<xacro:property name="Joint_S3_S4_Oy" value=" 0.142500 "/>
+<xacro:property name="Joint_S3_S4_Oz" value=" -0.0417865 "/>
+<xacro:property name="Joint_S3_S4_Oroll" value=" -1.5708 "/>
+<xacro:property name="Joint_S3_S4_Opitch" value=" -0.6405 "/>
+<xacro:property name="Joint_S3_S4_Oyaw" value=" 0.0 "/>
+<!-- Sensor 5 -->
+<xacro:property name="Joint_S4_S5_Ox" value=" 0.0112049 "/>
+<xacro:property name="Joint_S4_S5_Oy" value=" 0.142500 "/>
+<xacro:property name="Joint_S4_S5_Oz" value=" -0.0113731 "/>
+<xacro:property name="Joint_S4_S5_Oroll" value=" -1.5708 "/>
+<xacro:property name="Joint_S4_S5_Opitch" value=" -1.4259 "/>
+<xacro:property name="Joint_S4_S5_Oyaw" value=" 0.0 "/>
+<!-- Sensor 6 -->
+<xacro:property name="Joint_S5_S6_Ox" value=" -0.0463735 "/>
+<xacro:property name="Joint_S5_S6_Oy" value=" 0.142500 "/>
+<xacro:property name="Joint_S5_S6_Oz" value=" -0.0259404 "/>
+<xacro:property name="Joint_S5_S6_Oroll" value=" 1.5708 "/>
+<xacro:property name="Joint_S5_S6_Opitch" value=" -0.9303 "/>
+<xacro:property name="Joint_S5_S6_Oyaw" value=" 3.1416 "/>
+<!-- Sensor 7 -->
+<xacro:property name="Joint_S6_S7_Ox" value=" -0.0767870 "/>
+<xacro:property name="Joint_S6_S7_Oy" value=" 0.142500 "/>
+<xacro:property name="Joint_S6_S7_Oz" value=" -0.0769551 "/>
+<xacro:property name="Joint_S6_S7_Oroll" value=" 1.5708 "/>
+<xacro:property name="Joint_S6_S7_Opitch" value=" -0.1449 "/>
+<xacro:property name="Joint_S6_S7_Oyaw" value=" 3.1416 "/>
 </robot>
