Commit message: fixed mistake

File: relax_urdf/urdf/parts/kinematics_properties.urdf.xacro (robot description, xacro)
@@ -3,6 +3,6 @@
 <!-- ARM -->
 <!-- Joint 0 Origin : Base - Link 1 -->
-<xacro:property name="Joint_0_Ox" value="  0.0 "/>
-<xacro:property name="Joint_0_Oy" value=" ${-130.000*mmTom} "/>
+<xacro:property name="Joint_0_Ox" value=" ${-130.000*mmTom} "/>
+<xacro:property name="Joint_0_Oy" value=" 0.0 "/>
 <xacro:property name="Joint_0_Oz" value=" ${ 361.300*mmTom} "/>
 <xacro:property name="Joint_0_Oroll" value=" 0.0 "/>

Commit message: issue #33

File: relax_urdf/urdf/parts/kinematics_properties.urdf.xacro (robot description, xacro)
@@ -3,5 +3,7 @@
 <!-- ARM -->
 <!-- Joint 0 Origin : Base - Link 1 -->
-<xacro:property name="Joint_0_Ox" value=" ${-130.000*mmTom} "/>
+<!-- See issue #33-->
+<!-- <xacro:property name="Joint_0_Ox" value=" ${-130.000*mmTom} "/> -->
+<xacro:property name="Joint_0_Ox" value=" ${-134.485*mmTom} "/>
 <xacro:property name="Joint_0_Oy" value=" 0.0 "/>
 <xacro:property name="Joint_0_Oz" value=" ${ 361.300*mmTom} "/>

Commit message: another gap was present

File: relax_urdf/urdf/parts/kinematics_properties.urdf.xacro (robot description, xacro)
@@ -7,5 +7,7 @@
 <xacro:property name="Joint_0_Ox" value=" ${-134.485*mmTom} "/>
 <xacro:property name="Joint_0_Oy" value=" 0.0 "/>
-<xacro:property name="Joint_0_Oz" value=" ${ 361.300*mmTom} "/>
+<!-- Manually-brute-forcely reduce this since a vertical gap was present -->
+<!--<xacro:property name="Joint_0_Oz" value=" ${ 361.300*mmTom} "/>-->
+<xacro:property name="Joint_0_Oz" value=" ${ 355.7*mmTom} "/>
 <xacro:property name="Joint_0_Oroll" value=" 0.0 "/>
 <xacro:property name="Joint_0_Opitch" value=" 0.0 "/>
