Commit message: Update arm.urdf.xacro

File: relax_urdf/urdf/parts/arm.urdf.xacro (robot description, xacro)
@@ -1,3 +1,124 @@
 <?xml version="1.0"?>
 <robot xmlns:xacro="http://ros.org/wiki/xacro">
+<!-- links -->
+<link name ="relax_link1">  <!-- link 1 -->
+    <inertial>
+      <origin xyz="0.0 0.0 0.0" rpy="0 0 0"/>
+      <mass value="0.0"/>
+      <inertia ixx="0.0" ixy="0.0" ixz="0.0" iyy="0.0" iyz="0.0" izz="0.0" />
+    </inertial>
+    <visual>
+      <origin xyz="0 0 0" rpy="0 0 0"/>
+      <geometry name="relax_link1_visual">
+        <mesh filename="package://teleop_urdf/meshes/mesh_link1.stl" scale="0.0 0.0 0.0" />
+      </geometry>
+      <material name=""/>
+    </visual>
+    <collision>
+      <origin xyz="0 0 0" rpy="0 0 0"/>
+      <geometry name="relax_link1_collision">
+        <mesh filename="package://relax_urdf/meshes/mesh_link1.stl" scale="0.0 0.0 0.0" />
+      </geometry>
+    </collision>
+</link>
+<link name ="relax_link2">  <!-- link 2 -->
+    <inertial>
+      <origin xyz="0.0 0.0 0.0" rpy="0 0 0"/>
+      <mass value="0.0"/>
+      <inertia ixx="0.0" ixy="0.0" ixz="0.0" iyy="0.0" iyz="0.0" izz="0.0" />
+    </inertial>
+    <visual>
+      <origin xyz="0 0 0" rpy="0 0 0"/>
+      <geometry name="relax_link1_visual">
+        <mesh filename="package://teleop_urdf/meshes/mesh_link2.stl" scale="0.0 0.0 0.0" />
+      </geometry>
+      <material name=""/>
+    </visual>
+    <collision>
+      <origin xyz="0 0 0" rpy="0 0 0"/>
+      <geometry name="relax_link2_collision">
+        <mesh filename="package://relax_urdf/meshes/mesh_link2.stl" scale="0.0 0.0 0.0" />
+      </geometry>
+    </collision>
+</link>
+<link name ="relax_link3">  <!-- link 3 -->
+    <inertial>
+      <origin xyz="0.0 0.0 0.0" rpy="0 0 0"/>
+      <mass value="0.0"/>
+      <inertia ixx="0.0" ixy="0.0" ixz="0.0" iyy="0.0" iyz="0.0" izz="0.0" />
+    </inertial>
+    <visual>
+      <origin xyz="0 0 0" rpy="0 0 0"/>
+      <geometry name="relax_link3_visual">
+        <mesh filename="package://teleop_urdf/meshes/mesh_link3.stl" scale="0.0 0.0 0.0" />
+      </geometry>
+      <material name=""/>
+    </visual>
+    <collision>
+      <origin xyz="0 0 0" rpy="0 0 0"/>
+      <geometry name="relax_link3_collision">
+        <mesh filename="package://relax_urdf/meshes/mesh_link3.stl" scale="0.0 0.0 0.0" />
+      </geometry>
+    </collision>
+</link>
+<link name ="relax_link4">  <!-- link 4 -->
+    <inertial>
+      <origin xyz="0.0 0.0 0.0" rpy="0 0 0"/>
+      <mass value="0.0"/>
+      <inertia ixx="0.0" ixy="0.0" ixz="0.0" iyy="0.0" iyz="0.0" izz="0.0" />
+    </inertial>
+    <visual>
+      <origin xyz="0 0 0" rpy="0 0 0"/>
+      <geometry name="relax_link4_visual">
+        <mesh filename="package://teleop_urdf/meshes/mesh_link4.stl" scale="0.0 0.0 0.0" />
+      </geometry>
+      <material name=""/>
+    </visual>
+    <collision>
+      <origin xyz="0 0 0" rpy="0 0 0"/>
+      <geometry name="relax_link4_collision">
+        <mesh filename="package://relax_urdf/meshes/mesh_link4.stl" scale="0.0 0.0 0.0" />
+      </geometry>
+    </collision>
+</link>
+<link name ="relax_link4">  <!-- link 4 -->
+    <inertial>
+      <origin xyz="0.0 0.0 0.0" rpy="0 0 0"/>
+      <mass value="0.0"/>
+      <inertia ixx="0.0" ixy="0.0" ixz="0.0" iyy="0.0" iyz="0.0" izz="0.0" />
+    </inertial>
+    <visual>
+      <origin xyz="0 0 0" rpy="0 0 0"/>
+      <geometry name="relax_link4_visual">
+        <mesh filename="package://teleop_urdf/meshes/mesh_link4.stl" scale="0.0 0.0 0.0" />
+      </geometry>
+      <material name=""/>
+    </visual>
+    <collision>
+      <origin xyz="0 0 0" rpy="0 0 0"/>
+      <geometry name="relax_link4_collision">
+        <mesh filename="package://relax_urdf/meshes/mesh_link4.stl" scale="0.0 0.0 0.0" />
+      </geometry>
+    </collision>
+</link>
+<link name ="relax_link5">  <!-- link 5 -->
+    <inertial>
+      <origin xyz="0.0 0.0 0.0" rpy="0 0 0"/>
+      <mass value="0.0"/>
+      <inertia ixx="0.0" ixy="0.0" ixz="0.0" iyy="0.0" iyz="0.0" izz="0.0" />
+    </inertial>
+    <visual>
+      <origin xyz="0 0 0" rpy="0 0 0"/>
+      <geometry name="relax_link5_visual">
+        <mesh filename="package://teleop_urdf/meshes/mesh_link5.stl" scale="0.0 0.0 0.0" />
+      </geometry>
+      <material name=""/>
+    </visual>
+    <collision>
+      <origin xyz="0 0 0" rpy="0 0 0"/>
+      <geometry name="relax_link5_collision">
+        <mesh filename="package://relax_urdf/meshes/mesh_link5.stl" scale="0.0 0.0 0.0" />
+      </geometry>
+    </collision>
+</link>
 </robot>

Commit message: Update arm.urdf.xacro

File: relax_urdf/urdf/parts/arm.urdf.xacro (robot description, xacro)
@@ -122,3 +122,36 @@
     </collision>
 </link>
+<!-- joints -->
+<joint name="joint1" type="revolute"> <!-- joint 1 -->
+    <parent link="relax_link1"/>
+    <child link="relax_link2"/>
+    <origin xyz="0 0 0" rpy="0 0 0"/>
+    <axis xyz="0 0 0"/>
+    <limit velocity="0" effort="0" lower="0" upper="0" />
+    <dynamics friction="0" damping="0"/>
+</joint>
+<joint name="joint2" type="revolute"> <!-- joint 2 -->
+    <parent link="relax_link2"/>
+    <child link="relax_link3"/>
+    <origin xyz="0 0 0" rpy="0 0 0"/>
+    <axis xyz="0 0 0"/>
+    <limit velocity="0" effort="0" lower="0" upper="0" />
+    <dynamics friction="0" damping="0"/>
+</joint>
+<joint name="joint3" type="revolute"> <!-- joint 3 -->
+    <parent link="relax_link3"/>
+    <child link="relax_link4"/>
+    <origin xyz="0 0 0" rpy="0 0 0"/>
+    <axis xyz="0 0 0"/>
+    <limit velocity="0" effort="0" lower="0" upper="0" />
+    <dynamics friction="0" damping="0"/>
+</joint>
+<joint name="joint4" type="revolute"> <!-- joint 4 -->
+    <parent link="relax_link4"/>
+    <child link="relax_link5"/>
+    <origin xyz="0 0 0" rpy="0 0 0"/>
+    <axis xyz="0 0 0"/>
+    <limit velocity="0" effort="0" lower="0" upper="0" />
+    <dynamics friction="0" damping="0"/>
+</joint>
 </robot>

Commit message: Update arm.urdf.xacro

File: relax_urdf/urdf/parts/arm.urdf.xacro (robot description, xacro)
@@ -1,4 +1,8 @@
 <?xml version="1.0"?>
 <robot xmlns:xacro="http://ros.org/wiki/xacro">
+<!-- color -->
+<material name="">
+  <color rgba="0.0 0.0 0.0 0.0"/>
+</material>
 <!-- links -->
 <link name ="relax_link1">  <!-- link 1 -->

Commit message: Update arm.urdf.xacro

File: relax_urdf/urdf/parts/arm.urdf.xacro (robot description, xacro)
@@ -86,24 +86,4 @@
     </collision>
 </link>
-<link name ="relax_link4">  <!-- link 4 -->
-    <inertial>
-      <origin xyz="0.0 0.0 0.0" rpy="0 0 0"/>
-      <mass value="0.0"/>
-      <inertia ixx="0.0" ixy="0.0" ixz="0.0" iyy="0.0" iyz="0.0" izz="0.0" />
-    </inertial>
-    <visual>
-      <origin xyz="0 0 0" rpy="0 0 0"/>
-      <geometry name="relax_link4_visual">
-        <mesh filename="package://teleop_urdf/meshes/mesh_link4.stl" scale="0.0 0.0 0.0" />
-      </geometry>
-      <material name=""/>
-    </visual>
-    <collision>
-      <origin xyz="0 0 0" rpy="0 0 0"/>
-      <geometry name="relax_link4_collision">
-        <mesh filename="package://relax_urdf/meshes/mesh_link4.stl" scale="0.0 0.0 0.0" />
-      </geometry>
-    </collision>
-</link>
 <link name ="relax_link5">  <!-- link 5 -->
     <inertial>

Commit message: Update arm.urdf.xacro

File: relax_urdf/urdf/parts/arm.urdf.xacro (robot description, xacro)
@@ -1,4 +1,6 @@
 <?xml version="1.0"?>
 <robot xmlns:xacro="http://ros.org/wiki/xacro">
+<!-- scale -->
+<xacro:property name="mmTom" value="0.001" />
 <!-- color -->
 <material name="">
@@ -110,6 +112,6 @@
     <parent link="relax_link1"/>
     <child link="relax_link2"/>
-    <origin xyz="0 0 0" rpy="0 0 0"/>
-    <axis xyz="0 0 0"/>
+    <origin xyz="0 ${131.660*mmTom} ${-249.660*mmTom}" rpy="0 0 0"/>
+    <axis xyz="0 1 0"/>
     <limit velocity="0" effort="0" lower="0" upper="0" />
     <dynamics friction="0" damping="0"/>
@@ -118,6 +120,6 @@
     <parent link="relax_link2"/>
     <child link="relax_link3"/>
-    <origin xyz="0 0 0" rpy="0 0 0"/>
-    <axis xyz="0 0 0"/>
+    <origin xyz="0 0 ${-400*mmTom}" rpy="0 0 0"/>
+    <axis xyz="0 1 0"/>
     <limit velocity="0" effort="0" lower="0" upper="0" />
     <dynamics friction="0" damping="0"/>
@@ -126,6 +128,6 @@
     <parent link="relax_link3"/>
     <child link="relax_link4"/>
-    <origin xyz="0 0 0" rpy="0 0 0"/>
-    <axis xyz="0 0 0"/>
+    <origin xyz="0 ${-131.660*mmTom} ${-249.660*mmTom}" rpy="0 0 0"/>
+    <axis xyz="0 0 1"/>
     <limit velocity="0" effort="0" lower="0" upper="0" />
     <dynamics friction="0" damping="0"/>
@@ -134,6 +136,6 @@
     <parent link="relax_link4"/>
     <child link="relax_link5"/>
-    <origin xyz="0 0 0" rpy="0 0 0"/>
-    <axis xyz="0 0 0"/>
+    <origin xyz="0 ${-88.1600*mmTom} ${-153.500*mmTom}" rpy="0 0 3.1415927"/>
+    <axis xyz="0 1 0"/>
     <limit velocity="0" effort="0" lower="0" upper="0" />
     <dynamics friction="0" damping="0"/>

Commit message: Update arm.urdf.xacro

File: relax_urdf/urdf/parts/arm.urdf.xacro (robot description, xacro)
@@ -17,5 +17,5 @@
       <origin xyz="0 0 0" rpy="0 0 0"/>
       <geometry name="relax_link1_visual">
-        <mesh filename="package://teleop_urdf/meshes/mesh_link1.stl" scale="0.0 0.0 0.0" />
+        <mesh filename="package://teleop_urdf/meshes/mesh_link1.stl" scale="0.001 0.001 0.001" />
       </geometry>
       <material name=""/>
@@ -24,5 +24,5 @@
       <origin xyz="0 0 0" rpy="0 0 0"/>
       <geometry name="relax_link1_collision">
-        <mesh filename="package://relax_urdf/meshes/mesh_link1.stl" scale="0.0 0.0 0.0" />
+        <mesh filename="package://relax_urdf/meshes/mesh_link1.stl" scale="0.001 0.001 0.001" />
       </geometry>
     </collision>
@@ -37,5 +37,5 @@
       <origin xyz="0 0 0" rpy="0 0 0"/>
       <geometry name="relax_link1_visual">
-        <mesh filename="package://teleop_urdf/meshes/mesh_link2.stl" scale="0.0 0.0 0.0" />
+        <mesh filename="package://teleop_urdf/meshes/mesh_link2.stl" scale="0.001 0.001 0.001" />
       </geometry>
       <material name=""/>
@@ -44,5 +44,5 @@
       <origin xyz="0 0 0" rpy="0 0 0"/>
       <geometry name="relax_link2_collision">
-        <mesh filename="package://relax_urdf/meshes/mesh_link2.stl" scale="0.0 0.0 0.0" />
+        <mesh filename="package://relax_urdf/meshes/mesh_link2.stl" scale="0.001 0.001 0.001" />
       </geometry>
     </collision>
@@ -57,5 +57,5 @@
       <origin xyz="0 0 0" rpy="0 0 0"/>
       <geometry name="relax_link3_visual">
-        <mesh filename="package://teleop_urdf/meshes/mesh_link3.stl" scale="0.0 0.0 0.0" />
+        <mesh filename="package://teleop_urdf/meshes/mesh_link3.stl" scale="0.001 0.001 0.001" />
       </geometry>
       <material name=""/>
@@ -64,5 +64,5 @@
       <origin xyz="0 0 0" rpy="0 0 0"/>
       <geometry name="relax_link3_collision">
-        <mesh filename="package://relax_urdf/meshes/mesh_link3.stl" scale="0.0 0.0 0.0" />
+        <mesh filename="package://relax_urdf/meshes/mesh_link3.stl" scale="0.001 0.001 0.001" />
       </geometry>
     </collision>
@@ -77,5 +77,5 @@
       <origin xyz="0 0 0" rpy="0 0 0"/>
       <geometry name="relax_link4_visual">
-        <mesh filename="package://teleop_urdf/meshes/mesh_link4.stl" scale="0.0 0.0 0.0" />
+        <mesh filename="package://teleop_urdf/meshes/mesh_link4.stl" scale="0.001 0.001 0.001" />
       </geometry>
       <material name=""/>
@@ -84,5 +84,5 @@
       <origin xyz="0 0 0" rpy="0 0 0"/>
       <geometry name="relax_link4_collision">
-        <mesh filename="package://relax_urdf/meshes/mesh_link4.stl" scale="0.0 0.0 0.0" />
+        <mesh filename="package://relax_urdf/meshes/mesh_link4.stl" scale="0.001 0.001 0.001" />
       </geometry>
     </collision>
@@ -97,5 +97,5 @@
       <origin xyz="0 0 0" rpy="0 0 0"/>
       <geometry name="relax_link5_visual">
-        <mesh filename="package://teleop_urdf/meshes/mesh_link5.stl" scale="0.0 0.0 0.0" />
+        <mesh filename="package://teleop_urdf/meshes/mesh_link5.stl" scale="0.001 0.001 0.001" />
       </geometry>
       <material name=""/>
@@ -104,5 +104,5 @@
       <origin xyz="0 0 0" rpy="0 0 0"/>
       <geometry name="relax_link5_collision">
-        <mesh filename="package://relax_urdf/meshes/mesh_link5.stl" scale="0.0 0.0 0.0" />
+        <mesh filename="package://relax_urdf/meshes/mesh_link5.stl" scale="0.001 0.001 0.001" />
       </geometry>
     </collision>

Commit message: Update arm.urdf.xacro

File: relax_urdf/urdf/parts/arm.urdf.xacro (robot description, xacro)
@@ -4,6 +4,9 @@
 <xacro:property name="mmTom" value="0.001" />
 <!-- color -->
-<material name="">
-  <color rgba="0.0 0.0 0.0 0.0"/>
+<material name="darkblue">
+    <color rgba="0.0 0.3 0.9 1"/>
+</material>
+<material name="dark">
+    <color rgba="0.1 0.1 0.1 1"/>
 </material>
 <!-- links -->
@@ -19,5 +22,5 @@
         <mesh filename="package://teleop_urdf/meshes/mesh_link1.stl" scale="0.001 0.001 0.001" />
       </geometry>
-      <material name=""/>
+      <material name="darkblue"/>
     </visual>
     <collision>
@@ -39,5 +42,5 @@
         <mesh filename="package://teleop_urdf/meshes/mesh_link2.stl" scale="0.001 0.001 0.001" />
       </geometry>
-      <material name=""/>
+      <material name="dark"/>
     </visual>
     <collision>
@@ -59,5 +62,5 @@
         <mesh filename="package://teleop_urdf/meshes/mesh_link3.stl" scale="0.001 0.001 0.001" />
       </geometry>
-      <material name=""/>
+      <material name="darkblue"/>
     </visual>
     <collision>
@@ -79,5 +82,5 @@
         <mesh filename="package://teleop_urdf/meshes/mesh_link4.stl" scale="0.001 0.001 0.001" />
       </geometry>
-      <material name=""/>
+      <material name="darkblue"/>
     </visual>
     <collision>
@@ -99,5 +102,5 @@
         <mesh filename="package://teleop_urdf/meshes/mesh_link5.stl" scale="0.001 0.001 0.001" />
       </geometry>
-      <material name=""/>
+      <material name="darkblue"/>
     </visual>
     <collision>

Commit message: Update arm.urdf.xacro

File: relax_urdf/urdf/parts/arm.urdf.xacro (robot description, xacro)
@@ -20,5 +20,5 @@
       <origin xyz="0 0 0" rpy="0 0 0"/>
       <geometry name="relax_link1_visual">
-        <mesh filename="package://teleop_urdf/meshes/mesh_link1.stl" scale="0.001 0.001 0.001" />
+        <mesh filename="package://relax_urdf/meshes/mesh_link1.stl" scale="0.001 0.001 0.001" />
       </geometry>
       <material name="darkblue"/>
@@ -40,5 +40,5 @@
       <origin xyz="0 0 0" rpy="0 0 0"/>
       <geometry name="relax_link1_visual">
-        <mesh filename="package://teleop_urdf/meshes/mesh_link2.stl" scale="0.001 0.001 0.001" />
+        <mesh filename="package://relax_urdf/meshes/mesh_link2.stl" scale="0.001 0.001 0.001" />
       </geometry>
       <material name="dark"/>
@@ -60,5 +60,5 @@
       <origin xyz="0 0 0" rpy="0 0 0"/>
       <geometry name="relax_link3_visual">
-        <mesh filename="package://teleop_urdf/meshes/mesh_link3.stl" scale="0.001 0.001 0.001" />
+        <mesh filename="package://relax_urdf/meshes/mesh_link3.stl" scale="0.001 0.001 0.001" />
       </geometry>
       <material name="darkblue"/>
@@ -80,5 +80,5 @@
       <origin xyz="0 0 0" rpy="0 0 0"/>
       <geometry name="relax_link4_visual">
-        <mesh filename="package://teleop_urdf/meshes/mesh_link4.stl" scale="0.001 0.001 0.001" />
+        <mesh filename="package://relax_urdf/meshes/mesh_link4.stl" scale="0.001 0.001 0.001" />
       </geometry>
       <material name="darkblue"/>
@@ -100,5 +100,5 @@
       <origin xyz="0 0 0" rpy="0 0 0"/>
       <geometry name="relax_link5_visual">
-        <mesh filename="package://teleop_urdf/meshes/mesh_link5.stl" scale="0.001 0.001 0.001" />
+        <mesh filename="package://relax_urdf/meshes/mesh_link5.stl" scale="0.001 0.001 0.001" />
       </geometry>
       <material name="darkblue"/>

Commit message: Update arm.urdf.xacro

File: relax_urdf/urdf/parts/arm.urdf.xacro (robot description, xacro)
@@ -1,13 +1,5 @@
 <?xml version="1.0"?>
 <robot xmlns:xacro="http://ros.org/wiki/xacro">
-<!-- scale -->
-<xacro:property name="mmTom" value="0.001" />
-<!-- color -->
-<material name="darkblue">
-    <color rgba="0.0 0.3 0.9 1"/>
-</material>
-<material name="dark">
-    <color rgba="0.1 0.1 0.1 1"/>
-</material>
+<!-- relax arm -->
 <!-- links -->
 <link name ="relax_link1">  <!-- link 1 -->

Commit message: Update arm.urdf.xacro

File: relax_urdf/urdf/parts/arm.urdf.xacro (robot description, xacro)
@@ -5,7 +5,7 @@
 <link name ="relax_link1">  <!-- link 1 -->
     <inertial>
-      <origin xyz="0.0 0.0 0.0" rpy="0 0 0"/>
-      <mass value="0.0"/>
-      <inertia ixx="0.0" ixy="0.0" ixz="0.0" iyy="0.0" iyz="0.0" izz="0.0" />
+      <origin xyz="${1.3955428e+00*mmTom} ${2.5982581e+01*mmTom} ${-1.6511476e+02*mmTom}" rpy="0 0 0"/>
+      <mass value="5.9029271e+00"/>
+      <inertia ixx="${6.2182861e+04*mm2Tom2}"  ixy="${8.1614096e+01*mm2Tom2}"  ixz="${1.0385066e+02*mm2Tom2}" iyy="${5.5346023e+04*mm2Tom2}" iyz="${1.2999920e+04*mm2Tom2}" izz="${1.6821722e+04*mm2Tom2}" />
     </inertial>
     <visual>
@@ -25,7 +25,9 @@
 <link name ="relax_link2">  <!-- link 2 -->
     <inertial>
-      <origin xyz="0.0 0.0 0.0" rpy="0 0 0"/>
-      <mass value="0.0"/>
-      <inertia ixx="0.0" ixy="0.0" ixz="0.0" iyy="0.0" iyz="0.0" izz="0.0" />
+       <inertial>
+      <origin xyz="${0.0000000e+00*mmTom} ${-7.1720374e+00*mmTom} ${-2.0000694e+02*mmTom}" rpy="0 0 0"/>
+      <mass value="1.9989653e+00"/>
+      <inertia ixx="${4.9589547e+04*mm2Tom2}"  ixy="${-2.3822174e-02*mm2Tom2}"  ixz="${2.3476881e+02*mm2Tom2}" iyy="${5.1111593e+04*mm2Tom2}" iyz="${7.7698490e-01*mm2Tom2}" izz="${4.0702979e+03*mm2Tom2}" />
+    </inertial>
     </inertial>
     <visual>
@@ -45,7 +47,7 @@
 <link name ="relax_link3">  <!-- link 3 -->
     <inertial>
-      <origin xyz="0.0 0.0 0.0" rpy="0 0 0"/>
-      <mass value="0.0"/>
-      <inertia ixx="0.0" ixy="0.0" ixz="0.0" iyy="0.0" iyz="0.0" izz="0.0" />
+      <origin xyz="${-2.1052916e+00*mmTom} ${-1.0638552e+02*mmTom} ${-7.4903486e+01*mmTom}" rpy="0 0 0"/>
+      <mass value="5.8838845e+00"/>
+      <inertia ixx="${6.1043599e+04*mm2Tom2}"  ixy="${-1.5340891e+02*mm2Tom2}"  ixz="${-1.7833160e+02*mm2Tom2}" iyy="${5.3601310e+04*mm2Tom2}" iyz="${-1.1090900e+04*mm2Tom2}" izz="${1.7380798e+04*mm2Tom2}" />
     </inertial>
     <visual>
@@ -65,7 +67,7 @@
 <link name ="relax_link4">  <!-- link 4 -->
     <inertial>
-      <origin xyz="0.0 0.0 0.0" rpy="0 0 0"/>
-      <mass value="0.0"/>
-      <inertia ixx="0.0" ixy="0.0" ixz="0.0" iyy="0.0" iyz="0.0" izz="0.0" />
+      <origin xyz="${2.4496086e-01*mmTom} ${-1.0728501e+00*mmTom} ${-4.9015064e+01*mmTom}" rpy="0 0 0"/>
+      <mass value="1.3982240e+00"/>
+      <inertia ixx="${1.4667270e+04*mm2Tom2}"  ixy="${-2.0411012e+01*mm2Tom2}"  ixz="${-4.4769570e+01*mm2Tom2}" iyy="${8.6598581e+03*mm2Tom2}" iyz="${-8.3199044e+01*mm2Tom2}" izz="${1.0450923e+04*mm2Tom2}" />
     </inertial>
     <visual>
@@ -84,8 +86,8 @@
 </link>
 <link name ="relax_link5">  <!-- link 5 -->
-    <inertial>
-      <origin xyz="0.0 0.0 0.0" rpy="0 0 0"/>
-      <mass value="0.0"/>
-      <inertia ixx="0.0" ixy="0.0" ixz="0.0" iyy="0.0" iyz="0.0" izz="0.0" />
+     <inertial>
+      <origin xyz="${-1.3228834e+00*mmTom} ${-8.4683010e+01*mmTom} ${-5.3211105e+01*mmTom}" rpy="0 0 0"/>
+      <mass value="5.7923846e+00"/>
+      <inertia ixx="${5.5109543e+04*mm2Tom2}"  ixy="${-1.4003837e+02*mm2Tom2}"  ixz="${ 2.1470743e+02*mm2Tom2}" iyy="${5.1309424e+04*mm2Tom2}" iyz="${-1.0289246e+03*mm2Tom2}" izz="${1.3804762e+04*mm2Tom2}" />
     </inertial>
     <visual>

Commit message: Update arm.urdf.xacro

File: relax_urdf/urdf/parts/arm.urdf.xacro (robot description, xacro)
@@ -29,5 +29,4 @@
       <mass value="1.9989653e+00"/>
       <inertia ixx="${4.9589547e+04*mm2Tom2}"  ixy="${-2.3822174e-02*mm2Tom2}"  ixz="${2.3476881e+02*mm2Tom2}" iyy="${5.1111593e+04*mm2Tom2}" iyz="${7.7698490e-01*mm2Tom2}" izz="${4.0702979e+03*mm2Tom2}" />
-    </inertial>
     </inertial>
     <visual>

Commit message: Update arm.urdf.xacro

File: relax_urdf/urdf/parts/arm.urdf.xacro (robot description, xacro)
@@ -25,5 +25,4 @@
 <link name ="relax_link2">  <!-- link 2 -->
     <inertial>
-       <inertial>
       <origin xyz="${0.0000000e+00*mmTom} ${-7.1720374e+00*mmTom} ${-2.0000694e+02*mmTom}" rpy="0 0 0"/>
       <mass value="1.9989653e+00"/>
