Commit message: porting repo from old to new version - parametric urdf model parts changed - ref issue 13 and 18

File: relax_urdf/urdf/parts/arm.urdf.xacro (robot description, xacro)
@@ -2,137 +2,18 @@
 <robot xmlns:xacro="http://ros.org/wiki/xacro">
 <!-- relax arm -->
-<!-- links -->
-<link name ="relax_link1">  <!-- link 1 -->
-    <inertial>
-      <origin xyz="${1.3955428e+00*mmTom} ${2.5982581e+01*mmTom} ${-1.6511476e+02*mmTom}" rpy="0 0 0"/>
-      <mass value="5.9029271e+00"/>
-      <inertia ixx="${6.2182861e+04*mm2Tom2}"  ixy="${8.1614096e+01*mm2Tom2}"  ixz="${1.0385066e+02*mm2Tom2}" iyy="${5.5346023e+04*mm2Tom2}" iyz="${1.2999920e+04*mm2Tom2}" izz="${1.6821722e+04*mm2Tom2}" />
-    </inertial>
-    <visual>
-      <origin xyz="0 0 0" rpy="0 0 0"/>
-      <geometry name="relax_link1_visual">
-        <mesh filename="package://relax_urdf/meshes/mesh_link1.stl" scale="0.001 0.001 0.001" />
-      </geometry>
-      <material name="darkblue"/>
-    </visual>
-    <collision>
-      <origin xyz="0 0 0" rpy="0 0 0"/>
-      <geometry name="relax_link1_collision">
-        <mesh filename="package://relax_urdf/meshes/mesh_link1.stl" scale="0.001 0.001 0.001" />
-      </geometry>
-    </collision>
-</link>
-<link name ="relax_link2">  <!-- link 2 -->
-    <inertial>
-      <origin xyz="${0.0000000e+00*mmTom} ${-7.1720374e+00*mmTom} ${-2.0000694e+02*mmTom}" rpy="0 0 0"/>
-      <mass value="1.9989653e+00"/>
-      <inertia ixx="${4.9589547e+04*mm2Tom2}"  ixy="${-2.3822174e-02*mm2Tom2}"  ixz="${2.3476881e+02*mm2Tom2}" iyy="${5.1111593e+04*mm2Tom2}" iyz="${7.7698490e-01*mm2Tom2}" izz="${4.0702979e+03*mm2Tom2}" />
-    </inertial>
-    <visual>
-      <origin xyz="0 0 0" rpy="0 0 0"/>
-      <geometry name="relax_link1_visual">
-        <mesh filename="package://relax_urdf/meshes/mesh_link2.stl" scale="0.001 0.001 0.001" />
-      </geometry>
-      <material name="dark"/>
-    </visual>
-    <collision>
-      <origin xyz="0 0 0" rpy="0 0 0"/>
-      <geometry name="relax_link2_collision">
-        <mesh filename="package://relax_urdf/meshes/mesh_link2.stl" scale="0.001 0.001 0.001" />
-      </geometry>
-    </collision>
-</link>
-<link name ="relax_link3">  <!-- link 3 -->
-    <inertial>
-      <origin xyz="${-2.1052916e+00*mmTom} ${-1.0638552e+02*mmTom} ${-7.4903486e+01*mmTom}" rpy="0 0 0"/>
-      <mass value="5.8838845e+00"/>
-      <inertia ixx="${6.1043599e+04*mm2Tom2}"  ixy="${-1.5340891e+02*mm2Tom2}"  ixz="${-1.7833160e+02*mm2Tom2}" iyy="${5.3601310e+04*mm2Tom2}" iyz="${-1.1090900e+04*mm2Tom2}" izz="${1.7380798e+04*mm2Tom2}" />
-    </inertial>
-    <visual>
-      <origin xyz="0 0 0" rpy="0 0 0"/>
-      <geometry name="relax_link3_visual">
-        <mesh filename="package://relax_urdf/meshes/mesh_link3.stl" scale="0.001 0.001 0.001" />
-      </geometry>
-      <material name="darkblue"/>
-    </visual>
-    <collision>
-      <origin xyz="0 0 0" rpy="0 0 0"/>
-      <geometry name="relax_link3_collision">
-        <mesh filename="package://relax_urdf/meshes/mesh_link3.stl" scale="0.001 0.001 0.001" />
-      </geometry>
-    </collision>
-</link>
-<link name ="relax_link4">  <!-- link 4 -->
-    <inertial>
-      <origin xyz="${2.4496086e-01*mmTom} ${-1.0728501e+00*mmTom} ${-4.9015064e+01*mmTom}" rpy="0 0 0"/>
-      <mass value="1.3982240e+00"/>
-      <inertia ixx="${1.4667270e+04*mm2Tom2}"  ixy="${-2.0411012e+01*mm2Tom2}"  ixz="${-4.4769570e+01*mm2Tom2}" iyy="${8.6598581e+03*mm2Tom2}" iyz="${-8.3199044e+01*mm2Tom2}" izz="${1.0450923e+04*mm2Tom2}" />
-    </inertial>
-    <visual>
-      <origin xyz="0 0 0" rpy="0 0 0"/>
-      <geometry name="relax_link4_visual">
-        <mesh filename="package://relax_urdf/meshes/mesh_link4.stl" scale="0.001 0.001 0.001" />
-      </geometry>
-      <material name="darkblue"/>
-    </visual>
-    <collision>
-      <origin xyz="0 0 0" rpy="0 0 0"/>
-      <geometry name="relax_link4_collision">
-        <mesh filename="package://relax_urdf/meshes/mesh_link4.stl" scale="0.001 0.001 0.001" />
-      </geometry>
-    </collision>
-</link>
-<link name ="relax_link5">  <!-- link 5 -->
-     <inertial>
-      <origin xyz="${-1.3228834e+00*mmTom} ${-8.4683010e+01*mmTom} ${-5.3211105e+01*mmTom}" rpy="0 0 0"/>
-      <mass value="5.7923846e+00"/>
-      <inertia ixx="${5.5109543e+04*mm2Tom2}"  ixy="${-1.4003837e+02*mm2Tom2}"  ixz="${ 2.1470743e+02*mm2Tom2}" iyy="${5.1309424e+04*mm2Tom2}" iyz="${-1.0289246e+03*mm2Tom2}" izz="${1.3804762e+04*mm2Tom2}" />
-    </inertial>
-    <visual>
-      <origin xyz="0 0 0" rpy="0 0 0"/>
-      <geometry name="relax_link5_visual">
-        <mesh filename="package://relax_urdf/meshes/mesh_link5.stl" scale="0.001 0.001 0.001" />
-      </geometry>
-      <material name="darkblue"/>
-    </visual>
-    <collision>
-      <origin xyz="0 0 0" rpy="0 0 0"/>
-      <geometry name="relax_link5_collision">
-        <mesh filename="package://relax_urdf/meshes/mesh_link5.stl" scale="0.001 0.001 0.001" />
-      </geometry>
-    </collision>
-</link>
-<!-- joints -->
-<joint name="joint1" type="revolute"> <!-- joint 1 -->
-    <parent link="relax_link1"/>
-    <child link="relax_link2"/>
-    <origin xyz="0 ${131.660*mmTom} ${-249.660*mmTom}" rpy="0 0 0"/>
-    <axis xyz="0 1 0"/>
-    <limit velocity="3.86" effort="147.0" lower="-3.14" upper="3.14" />
-    <dynamics damping="0.2" friction="10.0"/>
-</joint>
-<joint name="joint2" type="revolute"> <!-- joint 2 -->
-    <parent link="relax_link2"/>
-    <child link="relax_link3"/>
-    <origin xyz="0 0 ${-400*mmTom}" rpy="0 0 0"/>
-    <axis xyz="0 1 0"/>
-    <limit velocity="3.86" effort="147.0" lower="-3.14" upper="3.14" />
-    <dynamics damping="0.2" friction="10.0"/>
-</joint>
-<joint name="joint3" type="revolute"> <!-- joint 3 -->
-    <parent link="relax_link3"/>
-    <child link="relax_link4"/>
-    <origin xyz="0 ${-131.660*mmTom} ${-249.660*mmTom}" rpy="0 0 0"/>
-    <axis xyz="0 0 1"/>
-    <limit velocity="3.86" effort="147.0" lower="-3.14" upper="3.14" />
-    <dynamics damping="0.2" friction="10.0"/>
-</joint>
-<joint name="joint4" type="revolute"> <!-- joint 4 -->
-    <parent link="relax_link4"/>
-    <child link="relax_link5"/>
-    <origin xyz="0 ${-88.1600*mmTom} ${-153.500*mmTom}" rpy="0 0 3.1415927"/>
-    <axis xyz="0 1 0"/>
-    <limit velocity="3.86" effort="147.0" lower="-3.14" upper="3.14" />
-    <dynamics damping="0.2" friction="10.0"/>
-</joint>
+<xacro:include filename="$(find relax_urdf)/urdf/parts/relax_arm.urdf.xacro" />
+<!-- arms -->
+<xacro:relax_arm arm_num="1"  rot="1"  parent="relax_arm${arm_num}_link1">
+      <origin xyz="${Joint_1_Ox} ${Joint_1_Oy} ${Joint_1_Oz}" rpy="0 0 0"/>
+   </xacro:centauro_arm>
+<!-- end_effector attached -->
+<!-- <xacro:if value="${ADD_END_EFFECTOR}">
+      <xacro:include filename="$(find relax_urdf)/urdf/parts/end_effector.urdf.xacro" />
+      <xacro:end_effector arm_num="1"  parent_link="arm1_7">
+                  <origin xyz="0. 0. 0." rpy="0. 0. 0."/>
+      </xacro:end_effector>
+      <xacro:end_effector arm_num="2"  parent_link="arm2_7">
+                  <origin xyz="0. 0. 0." rpy="0. 0. 0."/>
+      </xacroend_effector>
+</xacro:if> -->
 </robot>

File: relax_urdf/urdf/relax_base.urdf.xacro (robot description, xacro)
@@ -1,4 +1,9 @@
 <?xml version="1.0"?>
 <robot xmlns:xacro="http://ros.org/wiki/xacro">
+<xacro:include filename="$(find relax_urdf)/urdf/relax_utils.urdf.xacro" />
+<xacro:include filename="$(find relax_urdf)/urdf/parts/inertial_properties.urdf.xacro" />
+<xacro:include filename="$(find relax_urdf)/urdf/parts/kinematics_properties.urdf.xacro" />
+<xacro:include filename="$(find relax_urdf)/urdf/parts/dynamic_properties.urdf.xacro" />
+<xacro:include filename="$(find relax_urdf)/urdf/parts/limits.urdf.xacro" />
 <!-- **** base attached to robot **** -->
 <xacro:if value="${RELAX_FLOATING_BASE}">

File: relax_urdf/urdf/relax_robot.urdf.xacro (robot description, xacro)
@@ -8,6 +8,5 @@
 <xacro:include filename="$(find relax_urdf)/urdf/gazebo/relax.gazebo.xacro" />
 <xacro:include filename="$(find relax_urdf)/urdf/gazebo/xbot.gazebo.xacro" />
-<!-- **** attach robot material gazebo **** -->
-<xacro:include filename="$(find relax_urdf)/urdf/gazebo/relax_materials.gazebo.xacro" />
+<xacro:include filename="$(find relax_urdf)/urdf/gazebo/materials.gazebo.xacro" />
 <xacro:unless value="${RELAX_MOBILE_BASE}" > <!-- fixed base -->
   	<link name="world"/>

Commit message: adding draft base_link inertial and visual

File: relax_urdf/urdf/parts/arm.urdf.xacro (robot description, xacro)
@@ -7,5 +7,17 @@
    </xacro:relax_arm>
 <xacro:unless value="${RELAX_MOBILE_BASE}">
-      <link name="base_link"/>
+  <link name="base_link">
+    <inertial>
+      <origin rpy="0 0 0" xyz="0 0 0"/>
+      <mass value="1"/>
+      <inertia ixx="1e-4" ixy="0" ixz="0" iyy="1e-4" iyz="0" izz="1e-4"/>
+    </inertial>
+    <visual>
+      <geometry>
+        <mesh filename="package://relax_urdf/meshes/mesh_base.stl" scale="0.001 0.001 0.001"/>
+      </geometry>
+      <material name="dark_grey"/>
+    </visual>
+  </link>
 </xacro:unless>
 <!-- end_effector attached -->

Commit message: relax_arm corrected inertia and mesh

File: relax_urdf/urdf/parts/arm.urdf.xacro (robot description, xacro)
@@ -3,4 +3,7 @@
 <!-- relax arm -->
 <xacro:include filename="$(find relax_urdf)/urdf/parts/relax_arm.urdf.xacro" />
+<!-- TODO: in wheels.urdf.xacro base link properties are defined, they should be shift into another file -->
+<xacro:include filename="$(find relax_urdf)/urdf/parts/wheels.urdf.xacro" />
+<xacro:include filename="$(find relax_urdf)/urdf/parts/common_base_properties.urdf.xacro" />
 <!-- arms -->
 <xacro:relax_arm arm_num="1" >
@@ -8,16 +11,24 @@
 <xacro:unless value="${RELAX_MOBILE_BASE}">
   <link name="base_link">
-    <inertial>
-      <origin rpy="0 0 0" xyz="0 0 0"/>
-      <mass value="1"/>
-      <inertia ixx="1e-4" ixy="0" ixz="0" iyy="1e-4" iyz="0" izz="1e-4"/>
-    </inertial>
+    <xacro:box_inertial mass="${mir_base_mass}" x="${mir_base_inertial_x_length}" y="${mir_base_inertial_y_length}" z="${mir_base_inertial_z_length}">
+        <origin xyz="${mir_base_inertial_x + mir_act_wheel_dx} ${mir_base_inertial_y} ${mir_base_inertial_z}" rpy="0 0 0" />
+    </xacro:box_inertial>
     <visual>
-      <geometry>
-        <mesh filename="package://relax_urdf/meshes/mesh_base.stl" scale="0.001 0.001 0.001"/>
-      </geometry>
-      <material name="dark_grey"/>
+        <origin xyz="${mir_act_wheel_dx} 0 0" rpy="0 0 0" />
+        <geometry>
+            <mesh filename="package://relax_urdf/meshes/mesh_base_revised.stl" scale="0.001 0.001 0.001"/>
+        </geometry>
+        <material name="dark_grey"/>
     </visual>
+    <collision>
+        <origin xyz="${mir_act_wheel_dx} 0 0" rpy="0 0 0" />
+        <geometry>
+            <mesh filename="package://relax_urdf/meshes/mesh_base_revised.stl"  scale="0.001 0.001 0.001"/>
+        </geometry>
+    </collision>
   </link>
+  <gazebo reference="base_link">
+        <material>Gazebo/DarkGrey</material>
+  </gazebo>
 </xacro:unless>
 <!-- end_effector attached -->

File: relax_urdf/urdf/relax_arm.urdf (robot description, URDF)
Before this commit: robot relax, 8 links, 7 joints
Links:
- link base_link: mass 1 -> 97.0; geometry collision mesh filename=package://relax_urdf/meshes/mesh_base_revised.stl scale=0.001 0.001 0.001; visual mesh filename=package://relax_urdf/meshes/mesh_base_revised.stl scale=0.001 0.001 0.001

Commit message: ball better positioned

File: relax_urdf/urdf/parts/arm.urdf.xacro (robot description, xacro)
@@ -40,5 +40,5 @@
 	<xacro:include filename="$(find centauro_urdf)/urdf/parts/ball.urdf.xacro" />
 	<xacro:ball_end_effector arm_num="${arm_num}"  parent_link="relax_arm${arm_num}_linkEndEffector">
-		      <origin xyz="0 0 0" rpy="0. ${PI} 0."/>
+		      <origin xyz="0 0 0.02" rpy="0. ${PI} 0."/>
 	</xacro:ball_end_effector>
 </xacro:if>

Commit message: ball better positioned

File: relax_urdf/urdf/parts/arm.urdf.xacro (robot description, xacro)
@@ -14,5 +14,5 @@
 	<xacro:include filename="$(find relax_urdf)/urdf/parts/ball.urdf.xacro" />
 	<xacro:ball_end_effector arm_num="${arm_num}"  parent_link="relax_arm${arm_num}_linkEndEffector">
-		      <origin xyz="0 0 0" rpy="0. ${PI} 0."/>
+		      <origin xyz="0 0 0.02" rpy="0. ${PI} 0."/>
 	</xacro:ball_end_effector>
 </xacro:if>

Commit message: move base definition in relax_base (from arm.urdf.xacro), regenerated urdf according also to some updated params

File: relax_urdf/urdf/parts/arm.urdf.xacro (robot description, xacro)
@@ -3,34 +3,8 @@
 <!-- relax arm -->
 <xacro:include filename="$(find relax_urdf)/urdf/parts/relax_arm.urdf.xacro" />
-<!-- TODO: in wheels.urdf.xacro base link properties are defined, they should be shift into another file -->
-<xacro:include filename="$(find relax_urdf)/urdf/parts/wheels.urdf.xacro" />
-<xacro:include filename="$(find relax_urdf)/urdf/parts/common_base_properties.urdf.xacro" />
 <xacro:property name="arm_num" value="1" />
+<xacro:property name="relax_arm_base_link" value="relax_arm_base_link" />
 <!-- *********************************************************************** arm **************************************************************** -->
 <xacro:relax_arm arm_num="${arm_num}" />
-<!-- ******************************************************************* mobile base **************************************************************** -->
-<xacro:unless value="${RELAX_MOBILE_BASE}">
-  <link name="base_link">
-    <xacro:box_inertial mass="${mir_base_mass}" x="${mir_base_inertial_x_length}" y="${mir_base_inertial_y_length}" z="${mir_base_inertial_z_length}">
-        <origin xyz="${mir_base_inertial_x + mir_act_wheel_dx} ${mir_base_inertial_y} ${mir_base_inertial_z}" rpy="0 0 0" />
-    </xacro:box_inertial>
-    <visual>
-        <origin xyz="${mir_act_wheel_dx} 0 0" rpy="0 0 0" />
-        <geometry>
-            <mesh filename="package://relax_urdf/meshes/mesh_base_revised.stl" scale="0.001 0.001 0.001"/>
-        </geometry>
-        <material name="dark_grey"/>
-    </visual>
-    <collision>
-        <origin xyz="${mir_act_wheel_dx} 0 0" rpy="0 0 0" />
-        <geometry>
-            <mesh filename="package://relax_urdf/meshes/mesh_base_revised.stl"  scale="0.001 0.001 0.001"/>
-        </geometry>
-    </collision>
-  </link>
-  <gazebo reference="base_link">
-        <material>Gazebo/DarkGrey</material>
-  </gazebo>
-</xacro:unless>
 <!-- ******************************************************************* end_effector  **************************************************************** -->
 <xacro:if value="${END_EFFECTOR == 'none'}">

File: relax_urdf/urdf/relax.urdf (robot description, URDF)
Before this commit: robot relax, 26 links, 25 joints
Joints:
- joint relax_arm1_joint0: limit lower=-3.14 upper=3.14 effort=147.0 velocity=3.86 -> lower=-2.7 upper=2.7 effort=147.0 velocity=3.86; origin xyz=-0.13 0.0 0.3613 rpy=0.0 0.0 0.0 -> xyz=-0.13448500000000002 0.0 0.3613 rpy=0.0 0.0 0.0
- joint relax_arm1_joint1: limit lower=-3.14 upper=3.14 effort=147.0 velocity=3.86 -> lower=-2.7 upper=2.7 effort=147.0 velocity=3.86
- joint relax_arm1_joint2: axis 0 0 1 -> 0 0 -1; limit lower=-3.14 upper=3.14 effort=147.0 velocity=3.86 -> lower=-2.7 upper=2.7 effort=147.0 velocity=3.86
- joint relax_arm1_joint3: limit lower=-3.14 upper=3.14 effort=147.0 velocity=3.86 -> lower=-2.7 upper=2.7 effort=147.0 velocity=3.86
- joint relax_arm1_joint4: axis 0 0 1 -> 0 0 -1; limit lower=-3.14 upper=3.14 effort=147.0 velocity=3.86 -> lower=-2.0 upper=2.0 effort=147.0 velocity=3.86
- joint relax_arm1_joint5: limit lower=-3.14 upper=3.14 effort=147.0 velocity=3.86 -> lower=-2.7 upper=2.7 effort=147.0 velocity=3.86
- joint relax_arm1_joint6: axis 0 0 1 -> (none); limit lower=-3.14 upper=3.14 effort=147.0 velocity=3.86 -> (none)

File: relax_urdf/urdf/relax_arm.urdf (robot description, URDF)
Before this commit: robot relax, 8 links, 7 joints
Joints:
- joint relax_arm1_joint0: origin xyz=-0.13 0.0 0.3613 rpy=0.0 0.0 0.0 -> xyz=-0.13448500000000002 0.0 0.3613 rpy=0.0 0.0 0.0

File: relax_urdf/urdf/relax_base.urdf.xacro (robot description, xacro)
@@ -6,12 +6,39 @@
 <xacro:include filename="$(find relax_urdf)/urdf/parts/dynamic_properties.urdf.xacro" />
 <xacro:include filename="$(find relax_urdf)/urdf/parts/limits.urdf.xacro" />
-<!-- ********  attach robot  ******** -->
+<!-- TODO: in wheels.urdf.xacro base link properties are defined, they should be shift into another file -->
+<xacro:include filename="$(find relax_urdf)/urdf/parts/wheels.urdf.xacro" />
+<xacro:include filename="$(find relax_urdf)/urdf/parts/common_base_properties.urdf.xacro" />
+<!-- ********************* MOBILE BASE ******************************************** -->
+<xacro:if value="${RELAX_MOBILE_BASE}">
+    <xacro:property name="prefix" value="" />
+    <xacro:include filename="$(find relax_urdf)/urdf/parts/mir_base.urdf.xacro" />
+    <xacro:mir prefix="${prefix}"/>
+</xacro:if>
+<xacro:unless value="${RELAX_MOBILE_BASE}">
+    <link name="base_link">
+        <xacro:box_inertial mass="${mir_base_mass}" x="${mir_base_inertial_x_length}" y="${mir_base_inertial_y_length}" z="${mir_base_inertial_z_length}">
+            <origin xyz="${mir_base_inertial_x + mir_act_wheel_dx} ${mir_base_inertial_y} ${mir_base_inertial_z}" rpy="0 0 0" />
+        </xacro:box_inertial>
+        <visual>
+            <origin xyz="${mir_act_wheel_dx} 0 0" rpy="0 0 0" />
+            <geometry>
+                <mesh filename="package://relax_urdf/meshes/mesh_base_revised.stl" scale="0.001 0.001 0.001"/>
+            </geometry>
+            <material name="dark_grey"/>
+        </visual>
+        <collision>
+            <origin xyz="${mir_act_wheel_dx} 0 0" rpy="0 0 0" />
+            <geometry>
+                <mesh filename="package://relax_urdf/meshes/mesh_base_revised.stl"  scale="0.001 0.001 0.001"/>
+            </geometry>
+        </collision>
+    </link>
+    <gazebo reference="base_link">
+        <material>Gazebo/DarkGrey</material>
+  </gazebo>
+</xacro:unless>
+<!-- ********************* ARM ******************************************** -->
 <xacro:if value="${RELAX_ARM}">
     <xacro:include filename="$(find relax_urdf)/urdf/parts/arm.urdf.xacro" />
 </xacro:if>
-<!-- Add Base -->
-<xacro:if value="${RELAX_MOBILE_BASE}">
-    <xacro:include filename="$(find relax_urdf)/urdf/parts/mir_base.urdf.xacro" />
-    <xacro:mir prefix=""/>
-</xacro:if>
 </robot>

Commit message: tcp for all EE and disc EE

File: relax_urdf/urdf/parts/arm.urdf.xacro (robot description, xacro)
@@ -9,11 +9,22 @@
 <!-- ******************************************************************* end_effector  **************************************************************** -->
 <xacro:if value="${END_EFFECTOR == 'none'}">
-    <!-- nothing to do -->
+    <link name="tcp_${arm_num}" />
+    <joint name="j_tcp_${arm_num}" type="fixed">
+        <parent link="relax_arm${arm_num}_linkEndEffector" />
+        <child link="tcp_${arm_num}" />
+        <origin xyz="0 0 0" rpy="0 0 0"/>
+    </joint>
 </xacro:if>
 <xacro:if value="${END_EFFECTOR == 'ball'}">
 	<xacro:include filename="$(find relax_urdf)/urdf/parts/ball.urdf.xacro" />
 	<xacro:ball_end_effector arm_num="${arm_num}"  parent_link="relax_arm${arm_num}_linkEndEffector">
-		      <origin xyz="0 0 0.02" rpy="0. ${PI} 0."/>
+        <origin xyz="0 0 0.02" rpy="0. ${PI} 0."/>
 	</xacro:ball_end_effector>
+    <link name="tcp_${arm_num}" />
+    <joint name="j_tcp_${arm_num}" type="fixed">
+        <parent link="ball${arm_num}_tip" />
+        <child link="tcp_${arm_num}" />
+        <origin xyz="0 0 0" rpy="0 0 0"/>
+    </joint>
 </xacro:if>
 <xacro:if value="${END_EFFECTOR == 'dagana_fixed'}">
@@ -22,10 +33,54 @@
 		<origin xyz="0. 0 0" rpy="0. 0 0"/>
 	</xacro:dagana_gripper>
+    <link name="tcp_${arm_num}" />
+    <joint name="j_tcp_${arm_num}" type="fixed">
+        <parent link="dagana_${arm_num}_tcp" />
+        <child link="tcp_${arm_num}" />
+        <origin xyz="0 0 0" rpy="0 0 0"/>
+    </joint>
 </xacro:if>
 <xacro:if value="${END_EFFECTOR == 'dagana'}">
 	<xacro:include filename="$(find dagana_urdf)/urdf/dagana_macro.urdf.xacro" />
-	<xacro:dagana_gripper name="dagana_${arm_num}" parent_link="relax_arm${arm_num}_linkEndEffector" joint_type="revolute">
-		<origin xyz="0. 0 0" rpy="0. 0 0"/>
-	</xacro:dagana_gripper>
+    <xacro:dagana_gripper name="dagana_${arm_num}" parent_link="relax_arm${arm_num}_linkEndEffector" joint_type="revolute">
+        <origin xyz="0. 0 0" rpy="0. 0 0"/>
+    </xacro:dagana_gripper>
+    <!--     to have the same final link as when "none" option is used     -->
+    <link name="tcp_${arm_num}" />
+    <joint name="j_tcp_${arm_num}" type="fixed">
+        <parent link="dagana_${arm_num}_tcp" />
+        <child link="tcp_${arm_num}" />
+        <origin xyz="0 0 0" rpy="0 0 0"/>
+    </joint>
+</xacro:if>
+<xacro:if value="${END_EFFECTOR == 'disc'}">
+    <link name="tool_disc">
+        <visual>
+            <geometry>
+                <cylinder length="0.01" radius="0.1"/>
+            </geometry>
+            <material name="dark_grey"/>
+        </visual>
+        <collision>
+            <geometry>
+                <cylinder length="0.01" radius="0.1"/>
+            </geometry>
+        </collision>
+        <inertial>
+            <mass value="1"/>
+            <origin xyz="0 0 0" rpy="0 0 0"/>
+            <inertia ixx="0.001" ixy="0" ixz="0" iyy="0.001" iyz="0" izz="0.002"/>
+        </inertial>
+    </link>
+    <joint name="tool_disc_joint" type="fixed">
+        <parent link="relax_arm${arm_num}_linkEndEffector"/>
+        <child link="tool_disc"/>
+        <origin xyz="0 0 0" rpy="0 0 0"/>
+    </joint>
+    <link name="tcp_${arm_num}" />
+    <joint name="j_tcp_${arm_num}" type="fixed">
+        <parent link="tool_disc" />
+        <child link="tcp_${arm_num}" />
+        <origin xyz="0 0 ${0.001/2}" rpy="0 0 0"/>
+    </joint>
 </xacro:if>
 </robot>
