Commit message: ball with z axis pointing out

File: relax_urdf/urdf/parts/ball.urdf.xacro (robot description, xacro)
@@ -31,5 +31,5 @@
 	<parent link="ball${arm_num}"/>
 	<child link="ball${arm_num}_tip"/>
-	<origin xyz="0 0 -0.07" rpy="0 0 0"/>
+	<origin xyz="0 0 -0.07" rpy="0 ${-PI} 0"/>
 </joint>
 </xacro:macro>

Commit message: ball better tcp

File: relax_urdf/urdf/parts/ball.urdf.xacro (robot description, xacro)
@@ -31,5 +31,5 @@
 	<parent link="ball${arm_num}"/>
 	<child link="ball${arm_num}_tip"/>
-	<origin xyz="0 0 -0.07" rpy="0 ${-PI} 0"/>
+	<origin xyz="0 0 -0.078" rpy="0 ${-PI} 0"/>
 </joint>
 </xacro:macro>
