Commit message: generated correct relax.urdf model

File: relax_urdf/urdf/relax.urdf (robot description, URDF)
Before this commit: robot relax, 27 links, 26 joints
Links:
- removed link relax_link1
- removed link relax_link2
- removed link relax_link3
- removed link relax_link4
- removed link relax_link5
- added link relax_arm1_link1, mass 5.9029271; collision mesh filename=package://relax_urdf/meshes/mesh_link1.stl scale=0.001 0.001 0.001; visual mesh filename=package://relax_urdf/meshes/mesh_link1.stl scale=0.001 0.001 0.001
- added link relax_arm1_link2, mass 1.9989653; collision mesh filename=package://relax_urdf/meshes/mesh_link2.stl scale=0.001 0.001 0.001; visual mesh filename=package://relax_urdf/meshes/mesh_link2.stl scale=0.001 0.001 0.001
- added link relax_arm1_link3, mass 5.8838845; collision mesh filename=package://relax_urdf/meshes/mesh_link3.stl scale=0.001 0.001 0.001; visual mesh filename=package://relax_urdf/meshes/mesh_link3.stl scale=0.001 0.001 0.001
- added link relax_arm1_link4, mass 1.398224; collision mesh filename=package://relax_urdf/meshes/mesh_link4.stl scale=0.001 0.001 0.001; visual mesh filename=package://relax_urdf/meshes/mesh_link4.stl scale=0.001 0.001 0.001
- added link relax_arm1_link5, mass 5.7923846; collision mesh filename=package://relax_urdf/meshes/mesh_link5.stl scale=0.001 0.001 0.001; visual mesh filename=package://relax_urdf/meshes/mesh_link5.stl scale=0.001 0.001 0.001
- link left_wheel: geometry collision mesh filename=package://relax_urdf/meshes/mesh_left_wheel.stl scale=0.001 0.001 0.001; visual mesh filename=package://relax_urdf/meshes/mesh_left_wheel.stl scale=0.001 0.001 0.001
- link right_wheel: geometry collision mesh filename=package://relax_urdf/meshes/mesh_left_wheel.stl scale=0.001 0.001 0.001; visual mesh filename=package://relax_urdf/meshes/mesh_left_wheel.stl scale=0.001 0.001 0.001
Joints:
- removed joint joint1
- removed joint joint2
- removed joint joint3
- removed joint joint4
- added joint relax_arm1_joint1: type revolute, parent relax_arm1_link1, child relax_arm1_link2, origin xyz=0.0 0.13166 -0.24966 rpy=0 0 0, axis 0 1 0, limit lower=-3.14 upper=3.14 effort=147.0 velocity=3.86
- added joint relax_arm1_joint2: type revolute, parent relax_arm1_link2, child relax_arm1_link3, origin xyz=0.0 0.0 -0.4 rpy=0 0 0, axis 0 1 0, limit lower=-3.14 upper=3.14 effort=147.0 velocity=3.86
- added joint relax_arm1_joint3: type revolute, parent relax_arm1_link3, child relax_arm1_link4, origin xyz=0.0 -0.13166 -0.24966 rpy=0 0 0, axis 0 0 1, limit lower=-3.14 upper=3.14 effort=147.0 velocity=3.86
- added joint relax_arm1_joint4: type revolute, parent relax_arm1_link4, child relax_arm1_link5, origin xyz=0.0 -0.08816 -0.1535 rpy=0.0 0.0 3.1415927, axis 0 1 0, limit lower=-3.14 upper=3.14 effort=147.0 velocity=3.86
- joint mobile_base_joint: child relax_link1 -> relax_arm1_link1

Commit message: updated relax.urdf-manually generated with rosrun xacro

File: relax_urdf/urdf/relax.urdf (robot description, URDF)
Before this commit: robot relax, 25 links, 24 joints
Links:
- added link relax_arm1_linkEndEffector
Joints:
- added joint relax_arm1_joint0: type revolute, parent base_link, child relax_arm1_link1, origin xyz=-0.13 0.0 0.3613 rpy=0.0 0.0 0.0, axis 0 0 1, limit lower=-3.14 upper=3.14 effort=147.0 velocity=3.86
- added joint relax_arm1_joint6: type fixed, parent relax_arm1_link6, child relax_arm1_linkEndEffector, origin xyz=0.0 0.0 0.028 rpy=0.0 0.0 0.0, axis 0 0 1, limit lower=-3.14 upper=3.14 effort=147.0 velocity=3.86
- joint relax_arm1_joint2: axis 0 1 0 -> 0 0 1
- joint relax_arm1_joint3: axis 0 1 0 -> 0 0 1
- joint relax_arm1_joint5: axis 0 1 0 -> 0 0 1
