Commit message: Update relax_base.urdf.xacro

File: relax_urdf/urdf/relax_base.urdf.xacro (robot description, xacro)
@@ -1,4 +1,22 @@
 <?xml version="1.0"?>
 <robot xmlns:xacro="http://ros.org/wiki/xacro" name="relax">
+<!-- **** base attached to robot **** -->
+<xacro:if value="${RELAX_FLOATING_BASE}">
+	<link name="base_link"/>
+	<joint name="base_joint" type="fixed">
+    		<parent link="base_link"/>
+    		<child link="relax_link1">
+    		<origin xyz="0 0 0" rpy="0 0 0" />
+	</joint>
+</xacro:if>
+<xacro:if value="${RELAX_FIXED_BASE}">
+	<link name="base_link"/>
+	<joint name="base_joint" type="fixed">
+    		<parent link="base_link"/>
+    		<child link="relax_link1"/>
+    		<origin xyz="0 0 0" rpy="0 0 0" />
+	</joint>
+</xacro:if>
+<!-- ********  attach robot  ******** -->
 <xacro:include filename="$(find relax_urdf)/urdf/parts/arm.urdf.xacro" />
 </robot>

Commit message: Update relax_base.urdf.xacro

File: relax_urdf/urdf/relax_base.urdf.xacro (robot description, xacro)
@@ -4,5 +4,5 @@
 <xacro:if value="${RELAX_FLOATING_BASE}">
 	<link name="base_link"/>
-	<joint name="base_joint" type="fixed">
+	<joint name="base_joint" type="floating">
     		<parent link="base_link"/>
     		<child link="relax_link1">

Commit message: Update relax_base.urdf.xacro

File: relax_urdf/urdf/relax_base.urdf.xacro (robot description, xacro)
@@ -4,5 +4,5 @@
 <xacro:if value="${RELAX_FLOATING_BASE}">
 	<link name="base_link"/>
-	<joint name="base_joint" type="floating">
+	<joint name="base_joint" type="fixed">
     		<parent link="base_link"/>
     		<child link="relax_link1">

Commit message: Update relax_base.urdf.xacro

File: relax_urdf/urdf/relax_base.urdf.xacro (robot description, xacro)
@@ -6,5 +6,5 @@
 	<joint name="base_joint" type="fixed">
     		<parent link="base_link"/>
-    		<child link="relax_link1">
+    		<child link="relax_link1"/>
     		<origin xyz="0 0 0" rpy="0 0 0" />
 	</joint>

Commit message: Removing mobile_base_joint causing https://github.com/ADVRHumanoids/iit-relax-ros-pkg/issues/27

File: relax_urdf/urdf/relax_base.urdf.xacro (robot description, xacro)
@@ -14,11 +14,4 @@
     <xacro:include filename="$(find relax_urdf)/urdf/parts/mir_base.urdf.xacro" />
     <xacro:mir prefix=""/>
-    <xacro:if value="${RELAX_ARM}">
-        <joint name="mobile_base_joint" type="fixed"> <!-- mobile base joint -->
-            <parent link="base_link"/>
-            <child link="relax_arm1_link1"/>
-            <origin xyz="-0.130 0 0.3613" rpy="0 0 0"/>
-        </joint>
-    </xacro:if>
 </xacro:if>
 </robot>
