Commit message: Update relax_utils.urdf.xacro

File: relax_urdf/urdf/relax_utils.urdf.xacro (robot description, xacro)
@@ -3,4 +3,8 @@
 <!-- scale -->
 <xacro:property name="mmTom" value="0.001" />
+<xacro:property name="mm2Tom2" value="${0.001*0.001}" />
+<xacro:property name="tonsToKg" value="1000.0" />
+<xacro:property name="PI" value="3.14159265359" />
+<xacro:property name="PI_2" value="1.57079632679" />
 <!-- color -->
 <material name="darkblue">

Commit message: materials and utils

File: relax_urdf/urdf/relax_utils.urdf.xacro (robot description, xacro)
@@ -7,5 +7,10 @@
 <xacro:property name="PI" value="3.14159265359" />
 <xacro:property name="PI_2" value="1.57079632679" />
+<xacro:property name="toRad" value="${PI/180.0}" />
+<xacro:property name="toDeg" value="${180.0/PI}" />
 <!-- color -->
+<material name="black">
+    <color rgba="0.4 0.4 0.4 1"/>
+</material>
 <material name="darkblue">
     <color rgba="0.0 0.3 0.9 1"/>
@@ -14,3 +19,6 @@
     <color rgba="0.1 0.1 0.1 1"/>
 </material>
+<material name="dark_grey">
+    <color rgba="0.2 0.2 0.2 1"/>
+</material>
 </robot>
