Commit message: rbdl wants a first world link with fixed joint, see also #48

File: relax_urdf/urdf/relax_arm.urdf (robot description, URDF)
Before this commit: robot relax, 8 links, 7 joints
Links:
- added link world
Joints:
- added joint world_joint: type fixed, parent world, child base_link

File: relax_urdf/urdf/relax_arm.urdf.xacro (robot description, xacro)
@@ -17,4 +17,11 @@
     </xacro:if>
 </xacro:if>
+<xacro:unless value="${RELAX_FLOATING_BASE}" > <!-- floating base -->
+    <link name="world"/>
+    <joint name="world_joint" type="fixed">
+        <parent link="world"/>
+        <child link="base_link"/>
+    </joint>
+</xacro:unless>
 <xacro:if value="${ADD_VIRTUAL_FRAME}">
   <xacro:include filename="$(find relax_urdf)/urdf/parts/virtual_frame.urdf.xacro"/>
