Commit message: Update relax.urdf.xacro

File: relax_urdf/urdf/relax.urdf.xacro (robot description, xacro)
@@ -5,3 +5,18 @@
 <!-- ************ RELAX BASE ************ -->
 <xacro:include filename="$(find relax_urdf)/urdf/relax_base.urdf.xacro"/>
+<!-- **** attach to the world **** -->
+<xacro:if value="${ADD_FLOATING_BASE}">
+<link name="world"/>
+  <joint name="world_joint" type="floating">
+    <parent link="world"/>
+    <child link=""/>
+</joint>
+</xacro:if>
+<xacro:unless value="${ADD_FLOATING_BASE}">
+<link name="world"/>
+  <joint name="world_joint" type="fixed">
+    <parent link="world"/>
+    <child link=""/>
+</joint>
+</xacro:unless>
 </robot>

Commit message: Update relax.urdf.xacro

File: relax_urdf/urdf/relax.urdf.xacro (robot description, xacro)
@@ -7,16 +7,16 @@
 <!-- **** attach to the world **** -->
 <xacro:if value="${ADD_FLOATING_BASE}">
-<link name="world"/>
-  <joint name="world_joint" type="floating">
-    <parent link="world"/>
-    <child link=""/>
-</joint>
+    <link name="world"/>
+    <joint name="world_joint" type="floating">
+      <parent link="world"/>
+      <child link=""/>
+    </joint>
 </xacro:if>
 <xacro:unless value="${ADD_FLOATING_BASE}">
-<link name="world"/>
-  <joint name="world_joint" type="fixed">
-    <parent link="world"/>
-    <child link=""/>
-</joint>
+    <link name="world"/>
+    <joint name="world_joint" type="fixed">
+      <parent link="world"/>
+      <child link=""/>
+    </joint>
 </xacro:unless>
 </robot>

Commit message: Update relax.urdf.xacro

File: relax_urdf/urdf/relax.urdf.xacro (robot description, xacro)
@@ -1,14 +1,12 @@
 <?xml version="1.0"?>
 <robot xmlns:xacro="http://ros.org/wiki/xacro" name="relax">
-<!-- ************ MODEL CONFIGURATION ************ -->
-<xacro:include filename="$(find relax_urdf)/urdf/relax_config.urdf.xacro" />
 <!-- ************ RELAX BASE ************ -->
 <xacro:include filename="$(find relax_urdf)/urdf/relax_base.urdf.xacro"/>
-<!-- **** attach to the world **** -->
+<!-- ***** attach base to the world **** -->
 <xacro:if value="${ADD_FLOATING_BASE}">
     <link name="world"/>
     <joint name="world_joint" type="floating">
       <parent link="world"/>
-      <child link=""/>
+      <child link="base_link"/>
     </joint>
 </xacro:if>
@@ -17,5 +15,5 @@
     <joint name="world_joint" type="fixed">
       <parent link="world"/>
-      <child link=""/>
+      <child link="base_link"/>
     </joint>
 </xacro:unless>

Commit message: Update relax.urdf.xacro

File: relax_urdf/urdf/relax.urdf.xacro (robot description, xacro)
@@ -4,17 +4,19 @@
 <xacro:include filename="$(find relax_urdf)/urdf/relax_base.urdf.xacro"/>
 <!-- ***** attach base to the world ***** -->
-<xacro:if value="${RELAX_FLOATING_BASE}">
-    <link name="world"/>
-    <joint name="world_joint" type="floating">
-      <parent link="world"/>
-      <child link="base_link"/>
-    </joint>
+<xacro:if value="${RELAX_FLOATING_BASE}" > <!-- floating base -->
+	<link name="world"/>
+  <joint name="world_joint" type="floating">
+    	<parent link="world"/>
+    	<child link="base_link"/>
+		<origin xyz="0 0 0" rpy="0 0 0" />
+	</joint>
 </xacro:if>
-<xacro:unless value="${RELAX_FLOATING_BASE}">
-    <link name="world"/>
-    <joint name="world_joint" type="fixed">
-      <parent link="world"/>
-      <child link="base_link"/>
-    </joint>
-</xacro:unless>
+<xacro:if value="${RELAX_FIXED_BASE}" > <!-- fixed base -->
+  	<link name="world"/>
+   	<joint name="world_joint" type="fixed">
+    		<parent link="world"/>
+    		<child link="base_link"/>
+  	</joint>
+    <origin xyz="0 0 0" rpy="0 0 0" />
+</xacro:if>
 </robot>

Commit message: Update relax.urdf.xacro

File: relax_urdf/urdf/relax.urdf.xacro (robot description, xacro)
@@ -8,5 +8,5 @@
 <xacro:if value="${RELAX_FLOATING_BASE}" > <!-- floating base -->
 	<link name="world"/>
-  <joint name="world_joint" type="floating">
+  	<joint name="world_joint" type="floating">
     	<parent link="world"/>
     	<child link="base_link"/>

Commit message: gazebo launch with rviz optional conf && world to base joint also in relax if mobile base not used

File: relax_urdf/urdf/relax.urdf.xacro (robot description, xacro)
@@ -17,4 +17,12 @@
     </xacro:if>
 </xacro:if>
+<xacro:unless value="${RELAX_MOBILE_BASE}" > <!-- fixed base -->
+  	<link name="world"/>
+   	<joint name="world_joint" type="fixed">
+        <parent link="world"/>
+        <child link="base_link"/>
+        <origin xyz="0 0 0" rpy="0 0 0" />
+  	</joint>
+</xacro:unless>
 <xacro:if value="${ADD_VIRTUAL_FRAME}">
   <xacro:include filename="$(find relax_urdf)/urdf/parts/virtual_frame.urdf.xacro"/>

Commit message: fixed. now if no floating joint the robot will not move in gazebo as intended (I suppose)

File: relax_urdf/urdf/relax.urdf.xacro (robot description, xacro)
@@ -17,9 +17,9 @@
     </xacro:if>
 </xacro:if>
-<xacro:unless value="${RELAX_MOBILE_BASE}" > <!-- fixed base -->
+<xacro:unless value="${RELAX_FLOATING_BASE}" > <!-- fixed base -->
   	<link name="world"/>
    	<joint name="world_joint" type="fixed">
         <parent link="world"/>
-        <child link="base_link"/>
+        <child link="base_footprint"/>
         <origin xyz="0 0 0" rpy="0 0 0" />
   	</joint>

Commit message: please refactor me :C

File: relax_urdf/urdf/relax.urdf.xacro (robot description, xacro)
@@ -21,5 +21,6 @@
    	<joint name="world_joint" type="fixed">
         <parent link="world"/>
-        <child link="base_footprint"/>
+<!--        <child link="base_footprint"/>-->
+        <child link="base_link"/>
         <origin xyz="0 0 0" rpy="0 0 0" />
   	</joint>
