Commit message: Latest working model in simulation

File: relax_srdf/srdf/relax_arm.srdf.xacro (robot description, xacro)
@@ -5,5 +5,5 @@
 -->
 <robot xmlns:xacro="http://ros.org/wiki/xacro" name="relax">
-    <xacro:include filename="$(find relax_urdf)/urdf/config/relax.urdf.xacro" />
+    <xacro:include filename="$(find relax_urdf)/urdf/config/relax_arm.urdf.xacro" />
 <xacro:if value="${RELAX_MOBILE_BASE}">
     <group name="base">
@@ -16,5 +16,5 @@
 <xacro:if value="${RELAX_ARM}">
     <group name="arm">
-            <chain base_link="base_link" tip_link="relax_arm1_linkEndEffector" />
+        <chain base_link="base_link" tip_link="relax_arm1_linkEndEffector" />
     </group>
     <xacro:unless  value="${RELAX_MOBILE_BASE}">

File: relax_urdf/urdf/config/relax_arm.urdf.xacro (robot description, xacro)
@@ -1,9 +1,9 @@
 <?xml version="1.0"?>
-<robot xmlns:xacro="http://ros.org/wiki/xacro" name="relax_mir">
-<xacro:property name="model_name" value="RELAX MIR250" />
+<robot xmlns:xacro="http://ros.org/wiki/xacro" name="relax_arm">
+<xacro:property name="model_name" value="RELAX ARM" />
 <xacro:property name="model_version" value="1.0" />
 <!-- command line arguments -->
-<xacro:arg name="arm" default="false"/>
-<xacro:arg name="base" default="true"/>
+<xacro:arg name="arm" default="true"/>
+<xacro:arg name="base" default="false"/>
 <xacro:arg name="floating_joint" default="false"/>
 <!-- ************SELECT PARTS*************-->

File: relax_urdf/urdf/gazebo/xbot.gazebo.xacro (robot description, xacro)
@@ -2,14 +2,17 @@
 <robot xmlns:xacro="http://ros.org/wiki/xacro">
 <gazebo>
-    <plugin name="xbot2_link_state_sensor" filename="libxbot2_gz_link_state_sensor.so">
-        <links>
-            <link name="base_link"/>
-            <link name="left_wheel_link"/>
-        </links>
-    </plugin>
-    <!--
-    <plugin name="xbot2_ft_driver" filename="libxbot2_gz_ft_server.so"/>
-    <plugin name="xbot2_imu_driver" filename="libxbot2_gz_imu_server.so"/>-->
     <plugin name="xbot2_joint_driver" filename="libxbot2_gz_joint_server.so">
+        <ignore_joints>
+            <joint_to_ignore name="left_wheel_joint"/>
+            <joint_to_ignore name="right_wheel_joint"/>
+            <joint_to_ignore name="bl_caster_rotation_joint"/>
+            <joint_to_ignore name="bl_caster_wheel_joint"/>
+            <joint_to_ignore name="br_caster_rotation_joint"/>
+            <joint_to_ignore name="br_caster_wheel_joint"/>
+            <joint_to_ignore name="fl_caster_rotation_joint"/>
+            <joint_to_ignore name="fl_caster_wheel_joint"/>
+            <joint_to_ignore name="fr_caster_rotation_joint"/>
+            <joint_to_ignore name="fr_caster_wheel_joint"/>
+        </ignore_joints>
         <pid>
             <!-- TODO -> CHANGE PARAMS              -->
@@ -18,15 +21,5 @@
             <gain name="medium_mot" p="1000" d="10"/>
             <gain name="big_mot"    p="3000" d="10"/>
-            <gain name="wheel_mot"  p="1" d="1"/>
-            <pid name="left_wheel_joint"     profile="wheel_mot"/>
-            <pid name="right_wheel_joint"     profile="wheel_mot"/>
-            <pid name="front_left_caster_rotation_joint"     profile="wheel_mot"/>
-            <pid name="front_left_caster_wheel_joint"     profile="wheel_mot"/>
-            <pid name="front_right_caster_rotation_joint"     profile="wheel_mot"/>
-            <pid name="front_right_caster_wheel_joint"     profile="wheel_mot"/>
-            <pid name="rear_left_caster_rotation_joint"     profile="wheel_mot"/>
-            <pid name="rear_left_caster_wheel_joint"     profile="wheel_mot"/>
-            <pid name="rear_right_caster_rotation_joint"     profile="wheel_mot"/>
-            <pid name="rear_right_caster_wheel_joint"     profile="wheel_mot"/>
+            <gain name="wheel_mot"  p="10" d="2"/>
             <pid name="relax_arm1_joint1" profile="medium_mot"/>
             <pid name="relax_arm1_joint2" profile="medium_mot"/>

File: relax_urdf/urdf/parts/arm.urdf.xacro (robot description, xacro)
@@ -6,4 +6,7 @@
 <xacro:relax_arm arm_num="1" >
    </xacro:relax_arm>
+<xacro:unless value="${RELAX_MOBILE_BASE}">
+      <link name="base_link"/>
+</xacro:unless>
 <!-- end_effector attached -->
 <!-- <xacro:if value="${ADD_END_EFFECTOR}">

File: relax_urdf/urdf/parts/mir_base_xbot2.urdf.xacro (robot description, xacro)
@@ -81,4 +81,38 @@
     </joint>
     <link name="${prefix}us_2_frame" />
+    <!-- HACK: manually defining fake joints for cartesian control -->
+    <link name="world"/>
+    <joint name="lin_x_joint" type="prismatic">
+      <parent link="world"/>
+      <child link="lin_x_link"/>
+      <limit upper="1e9" lower="-1e9" velocity="2" effort="100"/>
+      <axis xyz="1 0 0"/>
+    </joint>
+    <joint name="lin_y_joint" type="prismatic">
+      <parent link="lin_x_link"/>
+      <child link="lin_y_link"/>
+      <limit upper="1e9" lower="-1e9" velocity="2" effort="100"/>
+      <axis xyz="0 1 0"/>
+    </joint>
+    <joint name="rot_z_joint" type="revolute">
+      <parent link="lin_y_link"/>
+      <child link="base_footprint"/>
+      <limit upper="1e9" lower="-1e9" velocity="2" effort="100"/>
+      <axis xyz="0 0 1"/>
+    </joint>
+    <link name="lin_x_link">
+      <inertial>
+        <mass value="0.01"/>
+        <origin xyz="0 0 0"/>
+        <inertia ixx="0.0001" ixy="0.0" ixz="0.0" iyy="0.0001" iyz="0.0" izz="0.0001"/>
+      </inertial>
+    </link>
+    <link name="lin_y_link">
+      <inertial>
+        <mass value="0.01"/>
+        <origin xyz="0 0 0"/>
+        <inertia ixx="0.0001" ixy="0.0" ixz="0.0" iyy="0.0001" iyz="0.0" izz="0.0001"/>
+      </inertial>
+    </link>
     <xacro:actuated_wheel prefix="${prefix}" locationprefix="left" locationright="-1"/>
     <xacro:actuated_wheel prefix="${prefix}" locationprefix="right" locationright="1"/>

File: relax_urdf/urdf/relax.urdf (robot description, URDF)
Before this commit: robot relax, 29 links, 28 joints
Links:
- removed link lin_x_link
- removed link lin_y_link
- removed link world
Joints:
- removed joint lin_x_joint
- removed joint lin_y_joint
- removed joint rot_z_joint

File: relax_urdf/urdf/relax_capsule.urdf (robot description, URDF)
Before this commit: robot relax, 29 links, 28 joints
Links:
- removed link lin_x_link
- removed link lin_y_link
- removed link world
Joints:
- removed joint lin_x_joint
- removed joint lin_y_joint
- removed joint rot_z_joint

File: relax_urdf/urdf/relax_mir.urdf (robot description, URDF)
Before this commit: robot relax, 28 links, 27 joints
Links:
- removed link car_frame
- removed link car_frame_intermediate_1
- removed link car_frame_intermediate_2
- removed link car_frame_intermediate_3
- removed link car_frame_intermediate_4
- removed link car_frame_intermediate_5
- removed link lin_x_link
- removed link lin_y_link
- removed link world
Joints:
- removed joint car_frame_rx
- removed joint car_frame_ry
- removed joint car_frame_rz
- removed joint car_frame_tx
- removed joint car_frame_ty
- removed joint car_frame_tz
- removed joint lin_x_joint
- removed joint lin_y_joint
- removed joint rot_z_joint

File: relax_urdf/urdf/relax_robot.urdf.xacro (robot description, xacro)
@@ -13,5 +13,5 @@
    	<joint name="world_joint" type="fixed">
         <parent link="world"/>
-        <child link="relax_arm${arm_num}_link1"/>
+        <child link="base_link"/>
         <origin xyz="0 0 0" rpy="0 0 0" />
   	</joint>

File: relax_urdf/urdf/relax_xbot2.urdf (robot description, URDF)
Before this commit: robot relax, 29 links, 28 joints
Joints:
- joint bl_caster_rotation_joint: type fixed -> continuous
- joint bl_caster_wheel_joint: type fixed -> continuous
- joint br_caster_rotation_joint: type fixed -> continuous
- joint br_caster_wheel_joint: type fixed -> continuous
- joint fl_caster_rotation_joint: type fixed -> continuous
- joint fl_caster_wheel_joint: type fixed -> continuous
- joint fr_caster_rotation_joint: type fixed -> continuous
- joint fr_caster_wheel_joint: type fixed -> continuous
- joint left_wheel_joint: type fixed -> continuous
- joint lin_x_joint: limit lower=-1e9 upper=1e9 effort=1 velocity=1 -> lower=-1e9 upper=1e9 effort=100 velocity=2
- joint lin_y_joint: limit lower=-1e9 upper=1e9 effort=1 velocity=1 -> lower=-1e9 upper=1e9 effort=100 velocity=2
- joint right_wheel_joint: type fixed -> continuous
- joint rot_z_joint: limit lower=-1e9 upper=1e9 effort=1 velocity=1 -> lower=-1e9 upper=1e9 effort=100 velocity=2

Commit message: right limits and axes wrt real robot

File: relax_srdf/srdf/relax_arm.srdf.xacro (robot description, xacro)
@@ -42,10 +42,10 @@
 <!-- homing posture -->
   <group_state name="home" group="chains">
-    <joint name="relax_arm1_joint0" value="0.0"/>
-    <joint name="relax_arm1_joint1" value="0.8"/>
-    <joint name="relax_arm1_joint2" value="0.6"/>
-    <joint name="relax_arm1_joint3" value="0.0"/>
-    <joint name="relax_arm1_joint4" value="-0.5"/>
-    <joint name="relax_arm1_joint5" value="0.0"/>
+    <joint name="relax_arm1_joint0" value="0"/>
+        <joint name="relax_arm1_joint1" value="-0.4"/>
+        <joint name="relax_arm1_joint2" value="-1.8"/>
+        <joint name="relax_arm1_joint3" value="0"/>
+        <joint name="relax_arm1_joint4" value="0.8"/>
+        <joint name="relax_arm1_joint5" value="0"/>
   </group_state>
 </robot>

File: relax_urdf/urdf/parts/limits.urdf.xacro (robot description, xacro)
@@ -5,35 +5,30 @@
 <xacro:property name="Joint_0_velocity" value=" 3.86 "/>
 <xacro:property name="Joint_0_effort" value=" 147.0 "/>
-<xacro:property name="Joint_0_lower" value=" -3.14 "/>
-<xacro:property name="Joint_0_upper" value=" 3.14 "/>
+<xacro:property name="Joint_0_lower" value=" -2.70 "/>
+<xacro:property name="Joint_0_upper" value=" 2.70 "/>
 <!-- Joint 1 -->
 <xacro:property name="Joint_1_velocity" value=" 3.86 "/>
 <xacro:property name="Joint_1_effort" value=" 147.0 "/>
-<xacro:property name="Joint_1_lower" value=" -3.14 "/>
-<xacro:property name="Joint_1_upper" value=" 3.14 "/>
+<xacro:property name="Joint_1_lower" value=" -2.70 "/>
+<xacro:property name="Joint_1_upper" value=" 2.70 "/>
 <!-- Joint 2 -->
 <xacro:property name="Joint_2_velocity" value=" 3.86 "/>
 <xacro:property name="Joint_2_effort" value=" 147.0 "/>
-<xacro:property name="Joint_2_lower" value=" -3.14 "/>
-<xacro:property name="Joint_2_upper" value=" 3.14 "/>
+<xacro:property name="Joint_2_lower" value=" -2.70 "/>
+<xacro:property name="Joint_2_upper" value=" 2.70 "/>
 <!-- Joint 3 -->
 <xacro:property name="Joint_3_velocity" value=" 3.86 "/>
 <xacro:property name="Joint_3_effort" value=" 147.0 "/>
-<xacro:property name="Joint_3_lower" value=" -3.14 "/>
-<xacro:property name="Joint_3_upper" value=" 3.14 "/>
+<xacro:property name="Joint_3_lower" value=" -2.70 "/>
+<xacro:property name="Joint_3_upper" value=" 2.70 "/>
 <!-- Joint 4 -->
 <xacro:property name="Joint_4_velocity" value=" 3.86 "/>
 <xacro:property name="Joint_4_effort" value=" 147.0 "/>
-<xacro:property name="Joint_4_lower" value=" -3.14 "/>
-<xacro:property name="Joint_4_upper" value=" 3.14 "/>
+<xacro:property name="Joint_4_lower" value=" -2.0 "/>
+<xacro:property name="Joint_4_upper" value=" 2.0 "/>
 <!-- Joint 5 -->
 <xacro:property name="Joint_5_velocity" value=" 3.86 "/>
 <xacro:property name="Joint_5_effort" value=" 147.0 "/>
-<xacro:property name="Joint_5_lower" value=" -3.14 "/>
-<xacro:property name="Joint_5_upper" value=" 3.14 "/>
-<!-- Joint 6 fake -->
-<xacro:property name="Joint_6_velocity" value=" 3.86 "/>
-<xacro:property name="Joint_6_effort" value=" 147.0 "/>
-<xacro:property name="Joint_6_lower" value=" -3.14 "/>
-<xacro:property name="Joint_6_upper" value=" 3.14 "/>
+<xacro:property name="Joint_5_lower" value=" -2.70 "/>
+<xacro:property name="Joint_5_upper" value=" 2.70 "/>
 </robot>

File: relax_urdf/urdf/parts/relax_arm.urdf.xacro (robot description, xacro)
@@ -146,5 +146,5 @@
     <child link="relax_arm${arm_num}_link3"/>
     <origin xyz="${Joint_2_Ox} ${Joint_2_Oy} ${Joint_2_Oz}" rpy="${Joint_2_Oroll} ${Joint_2_Opitch} ${Joint_2_Oyaw}"/>
-    <axis xyz="0 0 1"/>
+    <axis xyz="0 0 -1"/>
     <limit velocity="${Joint_2_velocity}" effort="${Joint_2_effort}" lower="${Joint_2_lower}" upper="${Joint_2_upper}" />
     <dynamics damping="${Joint_2_damp}" friction="${Joint_2_fric}"/>
@@ -154,5 +154,5 @@
     <child link="relax_arm${arm_num}_link4"/>
     <origin xyz="${Joint_3_Ox} ${Joint_3_Oy} ${Joint_3_Oz}" rpy="${Joint_3_Oroll} ${Joint_3_Opitch} ${Joint_3_Oyaw}"/>
-    <axis xyz="0 0 1"/>
+    <axis xyz="0 0 -1"/>
     <limit velocity="${Joint_3_velocity}" effort="${Joint_3_effort}" lower="${Joint_3_lower}" upper="${Joint_3_upper}" />
     <dynamics damping="${Joint_3_damp}" friction="${Joint_3_fric}"/>
@@ -162,5 +162,5 @@
     <child link="relax_arm${arm_num}_link5"/>
     <origin xyz="${Joint_4_Ox} ${Joint_4_Oy} ${Joint_4_Oz}" rpy="${Joint_4_Oroll} ${Joint_4_Opitch} ${Joint_4_Oyaw}"/>
-    <axis xyz="0 0 1"/>
+    <axis xyz="0 0 -1"/>
     <limit velocity="${Joint_4_velocity}" effort="${Joint_4_effort}" lower="${Joint_4_lower}" upper="${Joint_4_upper}" />
     <dynamics damping="${Joint_4_damp}" friction="${Joint_4_fric}"/>
@@ -178,7 +178,4 @@
     <child link="relax_arm${arm_num}_linkEndEffector"/>
     <origin xyz="${Joint_6_Ox} ${Joint_6_Oy} ${Joint_6_Oz}" rpy="${Joint_6_Oroll} ${Joint_6_Opitch} ${Joint_6_Oyaw}"/>
-    <axis xyz="0 0 1"/>
-    <limit velocity="${Joint_6_velocity}" effort="${Joint_6_effort}" lower="${Joint_6_lower}" upper="${Joint_6_upper}" />
-    <dynamics damping="${Joint_6_damp}" friction="${Joint_6_fric}"/>
 </joint>
   </xacro:macro>

File: relax_urdf/urdf/relax_arm.urdf (robot description, URDF)
Before this commit: robot relax, 8 links, 7 joints
Links:
- link base_link: geometry visual mesh filename=package://relax_urdf/meshes/mesh_base.stl scale=0.001 0.001 0.001
Joints:
- joint relax_arm1_joint0: limit lower=-3.14 upper=3.14 effort=147.0 velocity=3.86 -> lower=-2.7 upper=2.7 effort=147.0 velocity=3.86
- joint relax_arm1_joint1: limit lower=-3.14 upper=3.14 effort=147.0 velocity=3.86 -> lower=-2.7 upper=2.7 effort=147.0 velocity=3.86
- joint relax_arm1_joint2: axis 0 0 1 -> 0 0 -1; limit lower=-3.14 upper=3.14 effort=147.0 velocity=3.86 -> lower=-2.7 upper=2.7 effort=147.0 velocity=3.86
- joint relax_arm1_joint3: axis 0 0 1 -> 0 0 -1; limit lower=-3.14 upper=3.14 effort=147.0 velocity=3.86 -> lower=-2.7 upper=2.7 effort=147.0 velocity=3.86
- joint relax_arm1_joint4: axis 0 0 1 -> 0 0 -1; limit lower=-3.14 upper=3.14 effort=147.0 velocity=3.86 -> lower=-2.0 upper=2.0 effort=147.0 velocity=3.86
- joint relax_arm1_joint5: limit lower=-3.14 upper=3.14 effort=147.0 velocity=3.86 -> lower=-2.7 upper=2.7 effort=147.0 velocity=3.86
- joint relax_arm1_joint6: axis 0 0 1 -> (none); limit lower=-3.14 upper=3.14 effort=147.0 velocity=3.86 -> (none)

Commit message: dagana fixed joint

File: relax_srdf/srdf/relax_arm.srdf.xacro (robot description, xacro)
@@ -14,5 +14,5 @@
     </group>
 </xacro:if>
-<xacro:if value="${END_EFFECTOR == 'dagana' or END_EFFECTOR == 'dagana_fixed'}">
+<xacro:if value="${END_EFFECTOR == 'dagana'}">
     <group name="dagana">
         <chain base_link="relax_arm1_linkEndEffector" tip_link="dagana_1_bottom_link"/>
@@ -44,5 +44,5 @@
         <group name="car_frame_chain"/>
     </xacro:if>
-    <xacro:if value="${END_EFFECTOR == 'dagana' or END_EFFECTOR == 'dagana_fixed'}">
+    <xacro:if value="${END_EFFECTOR == 'dagana'}">
         <group name="dagana"></group>
     </xacro:if>
@@ -52,7 +52,7 @@
     <joint name="relax_arm1_joint0" value="0"/>
     <joint name="relax_arm1_joint1" value="-0.4"/>
-    <joint name="relax_arm1_joint2" value="-1.8"/>
+    <joint name="relax_arm1_joint2" value="-1.67"/>
     <joint name="relax_arm1_joint3" value="0"/>
-    <joint name="relax_arm1_joint4" value="0.8"/>
+    <joint name="relax_arm1_joint4" value="-1.46"/>
     <joint name="relax_arm1_joint5" value="0"/>
   </group_state>
