Commit message: Start adding xbot and cartesio files

File: relax_srdf/srdf/relax.srdf.xacro (robot description, xacro)
@@ -10,8 +10,8 @@
     </group>
 <xacro:if value="${RELAX_MOBILE_BASE}">
-    <group name="left_wheel">
+    <group name="left_locomotion">
         <chain base_link="mobile_base_link" tip_link="left_wheel" />
     </group>
-    <group name="right_wheel">
+    <group name="right_locomotion">
         <chain base_link="mobile_base_link" tip_link="right_wheel" />
     </group>
@@ -31,6 +31,6 @@
 <group name="chains"> <!--THIS HAS TO BE THE LAST GROUP IN THE FILE -->
     <xacro:if value="${RELAX_MOBILE_BASE}">
-        <group name="right_wheel" />
-        <group name="left_wheel" />
+        <group name="right_locomotion" />
+        <group name="left_locomotion" />
     </xacro:if>
     <xacro:if value="${RELAX_ARM}">

File: relax_urdf/urdf/gazebo/relax.gazebo.xacro (robot description, xacro)
@@ -62,9 +62,9 @@
         </collision>
     </gazebo>
-    <gazebo reference="j_wheel_left">
+    <gazebo reference="j_left_wheel">
         <implicitSpringDamper>1</implicitSpringDamper>
         <provideFeedback>true</provideFeedback>
     </gazebo>
-    <gazebo reference="j_wheel_right">
+    <gazebo reference="j_right_wheel">
         <implicitSpringDamper>1</implicitSpringDamper>
         <provideFeedback>true</provideFeedback>

File: relax_urdf/urdf/parts/arm.urdf.xacro (robot description, xacro)
@@ -109,6 +109,6 @@
     <origin xyz="0 ${131.660*mmTom} ${-249.660*mmTom}" rpy="0 0 0"/>
     <axis xyz="0 1 0"/>
-    <limit velocity="0" effort="0" lower="0" upper="0" />
-    <dynamics friction="0" damping="0"/>
+    <limit velocity="3.86" effort="147.0" lower="-3.14" upper="3.14" />
+    <dynamics damping="0.2" friction="10.0"/>
 </joint>
 <joint name="joint2" type="revolute"> <!-- joint 2 -->
@@ -117,6 +117,6 @@
     <origin xyz="0 0 ${-400*mmTom}" rpy="0 0 0"/>
     <axis xyz="0 1 0"/>
-    <limit velocity="0" effort="0" lower="0" upper="0" />
-    <dynamics friction="0" damping="0"/>
+    <limit velocity="3.86" effort="147.0" lower="-3.14" upper="3.14" />
+    <dynamics damping="0.2" friction="10.0"/>
 </joint>
 <joint name="joint3" type="revolute"> <!-- joint 3 -->
@@ -125,6 +125,6 @@
     <origin xyz="0 ${-131.660*mmTom} ${-249.660*mmTom}" rpy="0 0 0"/>
     <axis xyz="0 0 1"/>
-    <limit velocity="0" effort="0" lower="0" upper="0" />
-    <dynamics friction="0" damping="0"/>
+    <limit velocity="3.86" effort="147.0" lower="-3.14" upper="3.14" />
+    <dynamics damping="0.2" friction="10.0"/>
 </joint>
 <joint name="joint4" type="revolute"> <!-- joint 4 -->
@@ -133,6 +133,6 @@
     <origin xyz="0 ${-88.1600*mmTom} ${-153.500*mmTom}" rpy="0 0 3.1415927"/>
     <axis xyz="0 1 0"/>
-    <limit velocity="0" effort="0" lower="0" upper="0" />
-    <dynamics friction="0" damping="0"/>
+    <limit velocity="3.86" effort="147.0" lower="-3.14" upper="3.14" />
+    <dynamics damping="0.2" friction="10.0"/>
 </joint>
 </robot>

File: relax_urdf/urdf/parts/mobile_base.urdf.xacro (robot description, xacro)
@@ -66,5 +66,5 @@
 	<child link="left_wheel"/>
     <origin xyz="-0.00448719 0.25 0.09" rpy="0 0 0"/>
-	<axis xyz="0 0 -1"/>
+	<axis xyz="0 1 0"/>
    <limit  effort="35" velocity="20"/>
 </joint>
@@ -73,5 +73,5 @@
 	<child link="right_wheel"/>
 	<origin xyz="-0.00448719 -0.25 0.09" rpy="0 0 0"/>
-	<axis xyz="0 0 1"/>
+	<axis xyz="0 1 0"/>
    <limit  effort="35" velocity="20"/>
 </joint>

File: relax_urdf/urdf/relax.urdf.xacro (robot description, xacro)
@@ -7,4 +7,6 @@
 <!-- ************ RELAX BASE ************ -->
 <xacro:include filename="$(find relax_urdf)/urdf/relax_base.urdf.xacro"/>
+<!-- ************ XBOT-CORE ************ -->
+<!-- <xacro:include filename="$(find relax_urdf)/urdf/gazebo/xbot.gazebo.xacro" /> -->
 <!-- ***** attach base to the world ***** -->
 <xacro:if value="${RELAX_FLOATING_BASE}" > <!-- floating base -->

Commit message: Control Box + D435i

File: relax_srdf/srdf/relax.srdf.xacro (robot description, xacro)
@@ -7,5 +7,5 @@
     <xacro:include filename="$(find relax_urdf)/urdf/config/relax.urdf.xacro" />
     <group name="base">
-        <link name="base_link"/>
+        <link name="mobile_base_link"/>
     </group>
 <xacro:if value="${RELAX_MOBILE_BASE}">
@@ -20,5 +20,5 @@
     <xacro:if value="${RELAX_MOBILE_BASE}">
         <group name="arm">
-            <chain base_link="mobile_base_link" tip_link="relax_link5" />
+            <chain base_link="control_box" tip_link="relax_link5" />
         </group>
     </xacro:if>

File: relax_urdf/urdf/config/relax.urdf.xacro (robot description, xacro)
@@ -2,5 +2,5 @@
 <robot xmlns:xacro="http://ros.org/wiki/xacro" name="relax">
 <xacro:property name="model_name" value="IIT RELAX" />
-<xacro:property name="model_version" value="0.1" />
+<xacro:property name="model_version" value="1.0" />
 <!-- ************FLOATING BASE*************-->
 <xacro:property name="RELAX_FLOATING_BASE" value="true" />
@@ -9,3 +9,4 @@
 <!-- ************MOBILE BASE*************-->
 <xacro:property name="RELAX_MOBILE_BASE" value="true" />
+<xacro:property name="USE_REALSENSE" value="true" />
 </robot>

File: relax_urdf/urdf/gazebo/relax.gazebo.xacro (robot description, xacro)
@@ -8,10 +8,10 @@
                 <friction>
                     <ode>
-                        <mu>0.5</mu>
-                        <mu2>0.5</mu2>
+                        <mu>1.0</mu>
+                        <mu2>1.0</mu2>
                     </ode>
                     <bullet>
-                        <friction>0.5</friction>
-                        <friction2>0.5</friction2>
+                        <friction>1.0</friction>
+                        <friction2>1.0</friction2>
                     </bullet>
                 </friction>
@@ -38,10 +38,10 @@
                 <friction>
                     <ode>
-                        <mu>0.5</mu>
-                        <mu2>0.5</mu2>
+                        <mu>1.0</mu>
+                        <mu2>1.0</mu2>
                     </ode>
                     <bullet>
-                        <friction>0.5</friction>
-                        <friction2>0.5</friction2>
+                        <friction>1.0</friction>
+                        <friction2>1.0</friction2>
                     </bullet>
                 </friction>
@@ -71,23 +71,25 @@
     </gazebo>
 </xacro:if>
-<!-- <gazebo reference="joint1">
-	<implicitSpringDamper>1</implicitSpringDamper>
-	<provideFeedback>true</provideFeedback>
-</gazebo>
-<gazebo reference="joint2">
-	<implicitSpringDamper>1</implicitSpringDamper>
-	<provideFeedback>true</provideFeedback>
-</gazebo>
-<gazebo reference="joint3">
-	<implicitSpringDamper>1</implicitSpringDamper>
-	<provideFeedback>true</provideFeedback>
-</gazebo>
-<gazebo reference="joint4">
-	<implicitSpringDamper>1</implicitSpringDamper>
-	<provideFeedback>true</provideFeedback>
-</gazebo>
-<gazebo reference="joint5">
-	<implicitSpringDamper>1</implicitSpringDamper>
-	<provideFeedback>true</provideFeedback>
-</gazebo> -->
+<xacro:if value="${RELAX_ARM}">
+    <gazebo reference="joint1">
+        <implicitSpringDamper>1</implicitSpringDamper>
+        <provideFeedback>true</provideFeedback>
+    </gazebo>
+    <gazebo reference="joint2">
+        <implicitSpringDamper>1</implicitSpringDamper>
+        <provideFeedback>true</provideFeedback>
+    </gazebo>
+    <gazebo reference="joint3">
+        <implicitSpringDamper>1</implicitSpringDamper>
+        <provideFeedback>true</provideFeedback>
+    </gazebo>
+    <gazebo reference="joint4">
+        <implicitSpringDamper>1</implicitSpringDamper>
+        <provideFeedback>true</provideFeedback>
+    </gazebo>
+    <gazebo reference="joint5">
+        <implicitSpringDamper>1</implicitSpringDamper>
+        <provideFeedback>true</provideFeedback>
+    </gazebo>
+</xacro:if>
 </robot>

File: relax_urdf/urdf/parts/mobile_base.urdf.xacro (robot description, xacro)
@@ -19,4 +19,24 @@
       <geometry name="mobile_base_link_collision">
         <mesh filename="package://relax_urdf/meshes/mir_base.stl" scale="0.001 0.001 0.001" />
+      </geometry>
+    </collision>
+</link>
+<link name ="control_box">
+    <inertial>
+      <origin xyz="0.0 0.0 0.0" rpy="0 0 0"/>
+      <mass value="1.0"/>
+      <inertia ixx="0.17" ixy="0.0" ixz="0.0" iyy="0.17" iyz="0.0" izz="0.17" />
+    </inertial>
+    <visual>
+      <origin xyz="0 0 0" rpy="0 0 0"/>
+      <geometry name="control_box_visual">
+          <box size="0.3 0.3 0.15" />
+      </geometry>
+      <material name="dark"/>
+    </visual>
+    <collision>
+      <origin xyz="0 0 0" rpy="0 0 0"/>
+      <geometry name="control_box_collision">
+          <box size="0.3 0.3 0.15" />
       </geometry>
     </collision>
@@ -102,4 +122,10 @@
     </collision>
 </link>
+<joint name="j_control" type="fixed">
+	<parent link="mobile_base_link"/>
+	<child link="control_box"/>
+    <origin xyz="0 0 ${225.000*mmTom+0.15}" rpy="0 0 0"/>
+	<axis xyz="0 0 1"/>
+</joint>
 <joint name="j_left_wheel_yaw" type="revolute">
 	<parent link="mobile_base_link"/>
@@ -130,3 +156,23 @@
    <limit  effort="35" velocity="20"/>
 </joint>
+<xacro:if value="${USE_REALSENSE}">
+    <xacro:include filename="$(find realsense_gazebo_description)/urdf/_d435i.urdf.xacro" />
+        <xacro:sensor_d435i parent="control_box" name="D435i_camera" topics_ns="D435i/D435i_camera"
+                      enable_pointCloud="true" align_depth="true"
+                      unite_imu_method="false"
+                      visualize="false"
+                      accel_fps="300"
+                      gyro_fps="300"
+                      depth_width="1280"
+                      depth_height="720"
+                      depth_fps="90"
+                      infra_width="1280"
+                      infra_height="720"
+                      infra_fps="90"
+                      color_width="1280"
+                      color_height="720"
+                      color_fps="30">
+            <origin xyz="0.18 0 0" rpy="0 -0.5 0"/>
+        </xacro:sensor_d435i>
+</xacro:if>
 </robot>

File: relax_urdf/urdf/relax.urdf.xacro (robot description, xacro)
@@ -7,6 +7,8 @@
 <!-- ************ RELAX BASE ************ -->
 <xacro:include filename="$(find relax_urdf)/urdf/relax_base.urdf.xacro"/>
-<!-- ************ XBOT-CORE ************ -->
-<!-- <xacro:include filename="$(find relax_urdf)/urdf/gazebo/xbot.gazebo.xacro" /> -->
+<!-- **** attach robot gazebo **** -->
+<xacro:include filename="$(find relax_urdf)/urdf/gazebo/relax.gazebo.xacro" />
+<!-- **** XBotCore **** -->
+<xacro:include filename="$(find relax_urdf)/urdf/gazebo/xbot.gazebo.xacro" />
 <!-- ***** attach base to the world ***** -->
 <xacro:if value="${RELAX_FLOATING_BASE}" > <!-- floating base -->
@@ -15,5 +17,5 @@
     	<parent link="world"/>
     	<child link="base_link"/>
-		<origin xyz="0 0 0" rpy="0 0 0" />
+        <origin xyz="0 0 0" rpy="0 0 0" />
 	</joint>
 </xacro:if>
@@ -21,8 +23,8 @@
   	<link name="world"/>
    	<joint name="world_joint" type="fixed">
-    		<parent link="world"/>
-    		<child link="base_link"/>
+        <parent link="world"/>
+        <child link="base_link"/>
+        <origin xyz="0 0 0" rpy="0 0 0" />
   	</joint>
-    <origin xyz="0 0 0" rpy="0 0 0" />
 </xacro:unless>
 </robot>

File: relax_urdf/urdf/relax_base.urdf.xacro (robot description, xacro)
@@ -43,17 +43,16 @@
 </xacro:unless>
 <!-- ********  attach robot  ******** -->
+<xacro:if value="${RELAX_ARM}">
+    <xacro:include filename="$(find relax_urdf)/urdf/parts/arm.urdf.xacro" />
+</xacro:if>
 <xacro:if value="${RELAX_MOBILE_BASE}">
 <xacro:include filename="$(find relax_urdf)/urdf/parts/mobile_base.urdf.xacro" />
     <xacro:if value="${RELAX_ARM}">
         <joint name="mobile_base_joint" type="fixed"> <!-- mobile base joint -->
-            <parent link="mobile_base_link"/>
+            <parent link="control_box"/>
             <child link="relax_link1"/>
-            <origin xyz="0 0 ${240.000*mmTom}" rpy="3.1415927 0 0"/>
+            <origin xyz="0 0 0" rpy="3.1415927 0 0"/>
         </joint>
     </xacro:if>
 </xacro:if>
-<!-- ********  attach robot  ******** -->
-<xacro:if value="${RELAX_ARM}">
-    <xacro:include filename="$(find relax_urdf)/urdf/parts/arm.urdf.xacro" />
-</xacro:if>
 </robot>

Commit message: porting repo from old to new version - homing posture changes made - ref issue 13 and 15

File: relax_srdf/srdf/relax.srdf.xacro (robot description, xacro)
@@ -38,3 +38,14 @@
     </xacro:if>
 </group>
+<!-- homing posture -->
+  <group_state name="home" group="chains">
+    <joint name="joint1" value="0.6"/>
+    <joint name="joint2" value="-1.7"/>
+    <joint name="joint3" value="0.0"/>
+    <joint name="joint4" value="0.6"/>
+    <joint name="j_left_wheel_roll" value="0.0"/>
+    <joint name="j_left_wheel_yaw" value="0.0"/>
+    <joint name="j_right_wheel_roll" value="0.0"/>
+    <joint name="j_right_wheel_yaw" value="0.0"/>
+  </group_state>
 </robot>

Commit message: Correction collision wheel, floating base and add virtual chain files

File: relax_srdf/srdf/relax.srdf.xacro (robot description, xacro)
@@ -25,7 +25,12 @@
     <xacro:unless value="${RELAX_MOBILE_BASE}">
         <group name="arm">
-            <chain base_link="base_link" tip_link="relax_link5" />
+            <chain base_link="mobile_base_link" tip_link="relax_link5" />
         </group>
     </xacro:unless>
+</xacro:if>
+<xacro:if value="${ADD_VIRTUAL_FRAME}">
+    <group name="car_frame_chain">
+        <chain base_link="base_link" tip_link="car_frame"/>
+    </group>
 </xacro:if>
 <group name="chains"> <!--THIS HAS TO BE THE LAST GROUP IN THE FILE -->
@@ -36,4 +41,7 @@
     <xacro:if value="${RELAX_ARM}">
         <group name="arm" />
+    </xacro:if>
+    <xacro:if value="${ADD_VIRTUAL_FRAME}">
+        <group name="car_frame_chain"/>
     </xacro:if>
 </group>

File: relax_urdf/urdf/config/relax.urdf.xacro (robot description, xacro)
@@ -1,5 +1,5 @@
 <?xml version="1.0"?>
 <robot xmlns:xacro="http://ros.org/wiki/xacro" name="relax">
-<xacro:property name="model_name" value="IIT RELAX" />
+<xacro:property name="model_name" value="relax" />
 <xacro:property name="model_version" value="1.0" />
 <!-- command line arguments -->

File: relax_urdf/urdf/parts/mobile_base.urdf.xacro (robot description, xacro)
@@ -58,5 +58,5 @@
       <origin xyz="0 0 0" rpy="0 0 0"/>
       <geometry name="left_wheel_link_collision">
-        <mesh filename="package://relax_urdf/meshes/mir_base.stl" scale="0.001 0.001 0.001" />
+        <mesh filename="package://relax_urdf/meshes/mesh_left_wheel.stl" scale="0.001 0.001 0.001" />
       </geometry>
     </collision>
@@ -78,5 +78,5 @@
       <origin xyz="0 0 0" rpy="0 0 0"/>
       <geometry name="right_wheel_link_collision">
-        <mesh filename="package://relax_urdf/meshes/mir_base.stl" scale="0.001 0.001 0.001" />
+        <mesh filename="package://relax_urdf/meshes/mesh_left_wheel.stl" scale="0.001 0.001 0.001" />
       </geometry>
     </collision>

File: relax_urdf/urdf/relax.urdf.xacro (robot description, xacro)
@@ -9,18 +9,14 @@
 <!-- ***** attach base to the world ***** -->
 <xacro:if value="${RELAX_FLOATING_BASE}" > <!-- floating base -->
-	<link name="world"/>
-  	<joint name="world_joint" type="floating">
-    	<parent link="world"/>
-    	<child link="base_link"/>
-        <origin xyz="0 0 0" rpy="0 0 0" />
-	</joint>
+    <xacro:if value="${RELAX_MOBILE_BASE}" >
+        <link name="world"/>
+        <joint name="world_joint" type="floating">
+            <parent link="world"/>
+            <child link="base_link"/>
+        </joint>
+    </xacro:if>
 </xacro:if>
-<xacro:unless value="${RELAX_FLOATING_BASE}" > <!-- fixed base -->
-  	<link name="world"/>
-   	<joint name="world_joint" type="fixed">
-        <parent link="world"/>
-        <child link="base_link"/>
-        <origin xyz="0 0 0" rpy="0 0 0" />
-  	</joint>
-</xacro:unless>
+<xacro:if value="${ADD_VIRTUAL_FRAME}">
+  <xacro:include filename="$(find relax_urdf)/urdf/parts/virtual_frame.urdf.xacro"/>
+</xacro:if>
 </robot>

File: relax_urdf/urdf/relax_robot.urdf.xacro (robot description, xacro)
@@ -10,3 +10,11 @@
 <!-- **** attach robot material gazebo **** -->
 <xacro:include filename="$(find relax_urdf)/urdf/gazebo/relax_materials.gazebo.xacro" />
+<xacro:unless value="${RELAX_MOBILE_BASE}" > <!-- fixed base -->
+  	<link name="world"/>
+   	<joint name="world_joint" type="fixed">
+        <parent link="world"/>
+        <child link="relax_link1"/>
+        <origin xyz="0 0 0" rpy="0 0 0" />
+  	</joint>
+</xacro:unless>
 </robot>

File: relax_urdf/urdf/relax_virutal_frame.urdf (robot description, URDF)
Before this commit: robot relax, 27 links, 26 joints
Links:
- added link car_frame, mass 0.0
- added link car_frame_intermediate_1, mass 0.0
- added link car_frame_intermediate_2, mass 0.0
- added link car_frame_intermediate_3, mass 0.0
- added link car_frame_intermediate_4, mass 0.0
- added link car_frame_intermediate_5, mass 0.0
Joints:
- added joint car_frame_rx: type revolute, parent car_frame_intermediate_3, child car_frame_intermediate_4, origin xyz=0.0 0.0 0.0, axis 1 0 0, limit lower=-1e9 upper=1e9 effort=1000 velocity=10.0
- added joint car_frame_ry: type revolute, parent car_frame_intermediate_4, child car_frame_intermediate_5, origin xyz=0.0 0.0 0.0, axis 0 1 0, limit lower=-1e9 upper=1e9 effort=1000 velocity=10.0
- added joint car_frame_rz: type revolute, parent car_frame_intermediate_5, child car_frame, origin xyz=0.0 0.0 0.0, axis 0 0 1, limit lower=-1e9 upper=1e9 effort=1000 velocity=10.0
- added joint car_frame_tx: type prismatic, parent base_link, child car_frame_intermediate_1, origin xyz=0.0 0.0 0.0, axis 1 0 0, limit lower=-1e9 upper=1e9 effort=1000 velocity=10.0
- added joint car_frame_ty: type prismatic, parent car_frame_intermediate_1, child car_frame_intermediate_2, origin xyz=0.0 0.0 0.0, axis 0 1 0, limit lower=-1e9 upper=1e9 effort=1000 velocity=10.0
- added joint car_frame_tz: type prismatic, parent car_frame_intermediate_2, child car_frame_intermediate_3, origin xyz=0.0 0.0 0.0, axis 0 0 1, limit lower=-1e9 upper=1e9 effort=1000 velocity=10.0
- joint world_joint: origin (none) -> xyz=0 0 0 rpy=0 0 0

Commit message: fixed srdf arm names and added rviz config

File: relax_srdf/srdf/relax.srdf.xacro (robot description, xacro)
@@ -20,10 +20,10 @@
     <xacro:if value="${RELAX_MOBILE_BASE}">
         <group name="arm">
-            <chain base_link="control_box" tip_link="relax_link5" />
+            <chain base_link="control_box" tip_link="relax_arm1_link5" />
         </group>
     </xacro:if>
     <xacro:unless value="${RELAX_MOBILE_BASE}">
         <group name="arm">
-            <chain base_link="mobile_base_link" tip_link="relax_link5" />
+            <chain base_link="mobile_base_link" tip_link="relax_arm1_link5" />
         </group>
     </xacro:unless>
@@ -48,8 +48,8 @@
 <!-- homing posture -->
   <group_state name="home" group="chains">
-    <joint name="joint1" value="0.6"/>
-    <joint name="joint2" value="-1.7"/>
-    <joint name="joint3" value="0.0"/>
-    <joint name="joint4" value="0.6"/>
+    <joint name="relax_arm1_joint1" value="0.6"/>
+    <joint name="relax_arm1_joint2" value="-1.7"/>
+    <joint name="relax_arm1_joint3" value="0.0"/>
+    <joint name="relax_arm1_joint4" value="0.6"/>
     <joint name="j_left_wheel_roll" value="0.0"/>
     <joint name="j_left_wheel_yaw" value="0.0"/>

Commit message: Update srdf

File: relax_srdf/srdf/relax.srdf.xacro (robot description, xacro)
@@ -7,12 +7,12 @@
     <xacro:include filename="$(find relax_urdf)/urdf/config/relax.urdf.xacro" />
     <group name="base">
-        <link name="mobile_base_link"/>
+        <link name="base_footprint"/>
     </group>
 <xacro:if value="${RELAX_MOBILE_BASE}">
     <group name="left_locomotion">
-        <chain base_link="mobile_base_link" tip_link="left_wheel" />
+        <chain base_link="base_footprint" tip_link="left_wheel_link" />
     </group>
     <group name="right_locomotion">
-        <chain base_link="mobile_base_link" tip_link="right_wheel" />
+        <chain base_link="base_footprint" tip_link="right_wheel_link" />
     </group>
 </xacro:if>
@@ -20,10 +20,10 @@
     <xacro:if value="${RELAX_MOBILE_BASE}">
         <group name="arm">
-            <chain base_link="control_box" tip_link="relax_arm1_link5" />
+            <chain base_link="world" tip_link="relax_arm1_link6" />
         </group>
     </xacro:if>
     <xacro:unless value="${RELAX_MOBILE_BASE}">
         <group name="arm">
-            <chain base_link="mobile_base_link" tip_link="relax_arm1_link5" />
+            <chain base_link="relax_arm1_link1" tip_link="relax_arm1_link6" />
         </group>
     </xacro:unless>
@@ -31,5 +31,5 @@
 <xacro:if value="${ADD_VIRTUAL_FRAME}">
     <group name="car_frame_chain">
-        <chain base_link="base_link" tip_link="car_frame"/>
+        <chain base_link="base_footprint" tip_link="car_frame"/>
     </group>
 </xacro:if>
@@ -48,12 +48,11 @@
 <!-- homing posture -->
   <group_state name="home" group="chains">
-    <joint name="relax_arm1_joint1" value="0.6"/>
-    <joint name="relax_arm1_joint2" value="-1.7"/>
-    <joint name="relax_arm1_joint3" value="0.0"/>
-    <joint name="relax_arm1_joint4" value="0.6"/>
-    <joint name="j_left_wheel_roll" value="0.0"/>
-    <joint name="j_left_wheel_yaw" value="0.0"/>
-    <joint name="j_right_wheel_roll" value="0.0"/>
-    <joint name="j_right_wheel_yaw" value="0.0"/>
+    <joint name="relax_arm1_joint1" value="0.0"/>
+    <joint name="relax_arm1_joint2" value="0.6"/>
+    <joint name="relax_arm1_joint3" value="-1.7"/>
+    <joint name="relax_arm1_joint4" value="0.0"/>
+    <joint name="relax_arm1_joint5" value="0.6"/>
+    <joint name="left_wheel_joint" value="0.0"/>
+    <joint name="right_wheel_joint" value="0.0"/>
   </group_state>
 </robot>

File: relax_urdf/urdf/parts/virtual_frame.urdf.xacro (robot description, xacro)
@@ -3,5 +3,5 @@
 <!-- car frame virtual joints -->
 <joint name="car_frame_tx" type="prismatic">
-    <parent link="base_link"/>
+    <parent link="base_footprint"/>
     <origin xyz="0.0 0.0 0.0"/>
     <child link="car_frame_intermediate_1"/>
