Commit message: adding last joint (#6) and last fictitious link (end effector link)

File: relax_srdf/srdf/relax.srdf.xacro (robot description, xacro)
@@ -20,10 +20,10 @@
     <xacro:if value="${RELAX_MOBILE_BASE}">
         <group name="arm">
-            <chain base_link="world" tip_link="relax_arm1_link6" />
+            <chain base_link="world" tip_link="relax_arm1_linkEndEffector" />
         </group>
     </xacro:if>
     <xacro:unless value="${RELAX_MOBILE_BASE}">
         <group name="arm">
-            <chain base_link="relax_arm1_link1" tip_link="relax_arm1_link6" />
+            <chain base_link="relax_arm1_link1" tip_link="relax_arm1_linkEndEffector" />
         </group>
     </xacro:unless>
@@ -53,4 +53,5 @@
     <joint name="relax_arm1_joint4" value="0.0"/>
     <joint name="relax_arm1_joint5" value="0.6"/>
+    <joint name="relax_arm1_joint6" value="0.0"/>
     <joint name="left_wheel_joint" value="0.0"/>
     <joint name="right_wheel_joint" value="0.0"/>

File: relax_urdf/urdf/parts/dynamic_properties.urdf.xacro (robot description, xacro)
@@ -17,3 +17,6 @@
 <xacro:property name="Joint_5_damp" value="  0.2 "/>
 <xacro:property name="Joint_5_fric" value=" 10.0 "/>
+<!-- Joint 6 -->
+<xacro:property name="Joint_6_damp" value="  0.2 "/>
+<xacro:property name="Joint_6_fric" value=" 10.0 "/>
 </robot>

File: relax_urdf/urdf/parts/inertial_properties.urdf.xacro (robot description, xacro)
@@ -5,15 +5,15 @@
 <!-- Center of Mass -->
 <xacro:property name="Link_1_x" value=" ${-1.8991406e+00*mmTom} "/>
-<xacro:property name="Link_1_y" value=" ${2.2645162e+01*mmTom} "/>
-<xacro:property name="Link_1_z" value="${1.6741297e+02*mmTom} "/>
+<xacro:property name="Link_1_y" value=" ${ 2.2645162e+01*mmTom} "/>
+<xacro:property name="Link_1_z" value=" ${ 1.6741297e+02*mmTom} "/>
 <!-- Mass -->
 <xacro:property name="Link_1_mass" value="6.2381702e+00"/>
 <!-- Inertia -->
-<xacro:property name="Link_1_xx" value=" ${6.5816037e+04*mm2Tom2} "/>
+<xacro:property name="Link_1_xx" value=" ${ 6.5816037e+04*mm2Tom2} "/>
 <xacro:property name="Link_1_xy" value=" ${-1.1791629e+02*mm2Tom2} "/>
 <xacro:property name="Link_1_xz" value=" ${-4.0067927e+01*mm2Tom2} "/>
-<xacro:property name="Link_1_yy" value=" ${5.7828314e+04*mm2Tom2} "/>
+<xacro:property name="Link_1_yy" value=" ${ 5.7828314e+04*mm2Tom2} "/>
 <xacro:property name="Link_1_yz" value=" ${-1.1584403e+04*mm2Tom2} "/>
-<xacro:property name="Link_1_zz" value=" ${1.9401960e+04*mm2Tom2} "/>
+<xacro:property name="Link_1_zz" value=" ${ 1.9401960e+04*mm2Tom2} "/>
 <!-- Link 2 -->
 <!-- Center of Mass -->

File: relax_urdf/urdf/parts/kinematics_properties.urdf.xacro (robot description, xacro)
@@ -6,5 +6,5 @@
 <xacro:property name="Joint_1_Oy" value=" ${ 131.660*mmTom} "/>
 <xacro:property name="Joint_1_Oz" value=" ${ 249.660*mmTom} "/>
-<xacro:property name="Joint_1_Oroll" value="  -1.5707963 "/>
+<xacro:property name="Joint_1_Oroll" value=" -1.5707963 "/>
 <xacro:property name="Joint_1_Opitch" value=" 0.0 "/>
 <xacro:property name="Joint_1_Oyaw" value=" 0.0"/>
@@ -26,6 +26,6 @@
 <xacro:property name="Joint_4_Ox" value="  0.0 "/>
 <xacro:property name="Joint_4_Oy" value=" ${-88.1600*mmTom} "/>
-<xacro:property name="Joint_4_Oz" value=" ${153.500*mmTom} "/>
-<xacro:property name="Joint_4_Oroll" value="  1.5707963 "/>
+<xacro:property name="Joint_4_Oz" value=" ${ 153.500*mmTom} "/>
+<xacro:property name="Joint_4_Oroll" value=" 1.5707963 "/>
 <xacro:property name="Joint_4_Opitch" value=" 0.0 "/>
 <xacro:property name="Joint_4_Oyaw" value=" 0.0 "/>
@@ -37,5 +37,5 @@
 <xacro:property name="Joint_5_Opitch" value=" 0.0 "/>
 <xacro:property name="Joint_5_Oyaw" value=" 0.0 "/>
-<!-- Fake Joint 6 Origin : Link 6 - End-Effector -->
+<!-- Joint 6 Origin : Link 6 - End-Effector -->
 <xacro:property name="Joint_6_Ox" value="  0.0 "/>
 <xacro:property name="Joint_6_Oy" value=" 0.0 "/>

File: relax_urdf/urdf/parts/limits.urdf.xacro (robot description, xacro)
@@ -27,3 +27,8 @@
 <xacro:property name="Joint_5_lower" value=" -3.14 "/>
 <xacro:property name="Joint_5_upper" value=" 3.14 "/>
+<!-- Joint 6 -->
+<xacro:property name="Joint_6_velocity" value=" 3.86 "/>
+<xacro:property name="Joint_6_effort" value=" 147.0 "/>
+<xacro:property name="Joint_6_lower" value=" -3.14 "/>
+<xacro:property name="Joint_6_upper" value=" 3.14 "/>
 </robot>

File: relax_urdf/urdf/parts/relax_arm.urdf.xacro (robot description, xacro)
@@ -13,5 +13,5 @@
       <origin xyz="0 0 0" rpy="0 0 0"/>
       <geometry name="relax_link1_visual">
-        <mesh filename="package://relax_urdf/meshes/mesh_shoulder-yaw.stl" scale="0.001 0.001 0.001" />
+        <mesh filename="package://relax_urdf/meshes/mesh_link1.stl" scale="0.001 0.001 0.001" />
       </geometry>
       <material name="darkblue"/>
@@ -20,5 +20,5 @@
       <origin xyz="0 0 0" rpy="0 0 0"/>
       <geometry name="relax_link1_collision">
-        <mesh filename="package://relax_urdf/meshes/mesh_shoulder-yaw.stl" scale="0.001 0.001 0.001" />
+        <mesh filename="package://relax_urdf/meshes/mesh_link1.stl" scale="0.001 0.001 0.001" />
       </geometry>
     </collision>
@@ -33,5 +33,5 @@
       <origin xyz="0 0 0" rpy="0 0 0"/>
       <geometry name="relax_link2_visual">
-        <mesh filename="package://relax_urdf/meshes/mesh_shoulder-pitch.stl" scale="0.001 0.001 0.001" />
+        <mesh filename="package://relax_urdf/meshes/mesh_link2.stl" scale="0.001 0.001 0.001" />
       </geometry>
       <material name="dark"/>
@@ -40,5 +40,5 @@
       <origin xyz="0 0 0" rpy="0 0 0"/>
       <geometry name="relax_link2_collision">
-        <mesh filename="package://relax_urdf/meshes/mesh_shoulder-pitch.stl" scale="0.001 0.001 0.001" />
+        <mesh filename="package://relax_urdf/meshes/mesh_link2.stl" scale="0.001 0.001 0.001" />
       </geometry>
     </collision>
@@ -53,5 +53,5 @@
       <origin xyz="0 0 0" rpy="0 0 0"/>
       <geometry name="relax_link3_visual">
-        <mesh filename="package://relax_urdf/meshes/mesh_elbow.stl" scale="0.001 0.001 0.001" />
+        <mesh filename="package://relax_urdf/meshes/mesh_link3.stl" scale="0.001 0.001 0.001" />
       </geometry>
       <material name="darkblue"/>
@@ -60,5 +60,5 @@
       <origin xyz="0 0 0" rpy="0 0 0"/>
       <geometry name="relax_link3_collision">
-        <mesh filename="package://relax_urdf/meshes/mesh_elbow.stl" scale="0.001 0.001 0.001" />
+        <mesh filename="package://relax_urdf/meshes/mesh_link3.stl" scale="0.001 0.001 0.001" />
       </geometry>
     </collision>
@@ -73,5 +73,5 @@
       <origin xyz="0 0 0" rpy="0 0 0"/>
       <geometry name="relax_link4_visual">
-        <mesh filename="package://relax_urdf/meshes/mesh_forearm-yaw.stl" scale="0.001 0.001 0.001" />
+        <mesh filename="package://relax_urdf/meshes/mesh_link4.stl" scale="0.001 0.001 0.001" />
       </geometry>
       <material name="darkblue"/>
@@ -80,5 +80,5 @@
       <origin xyz="0 0 0" rpy="0 0 0"/>
       <geometry name="relax_link4_collision">
-        <mesh filename="package://relax_urdf/meshes/mesh_forearm-yaw.stl" scale="0.001 0.001 0.001" />
+        <mesh filename="package://relax_urdf/meshes/mesh_link4.stl" scale="0.001 0.001 0.001" />
       </geometry>
     </collision>
@@ -93,5 +93,5 @@
       <origin xyz="0 0 0" rpy="0 0 0"/>
       <geometry name="relax_link5_visual">
-        <mesh filename="package://relax_urdf/meshes/mesh_wrist-pitch.stl" scale="0.001 0.001 0.001" />
+        <mesh filename="package://relax_urdf/meshes/mesh_link5.stl" scale="0.001 0.001 0.001" />
       </geometry>
       <material name="darkblue"/>
@@ -100,5 +100,5 @@
       <origin xyz="0 0 0" rpy="0 0 0"/>
       <geometry name="relax_link5_collision">
-        <mesh filename="package://relax_urdf/meshes/mesh_wrist-pitch.stl" scale="0.001 0.001 0.001" />
+        <mesh filename="package://relax_urdf/meshes/mesh_link5.stl" scale="0.001 0.001 0.001" />
       </geometry>
     </collision>
@@ -113,5 +113,5 @@
       <origin xyz="0 0 0" rpy="0 0 0"/>
       <geometry name="relax_link6_visual">
-        <mesh filename="package://relax_urdf/meshes/mesh_wrist-yaw.stl" scale="0.001 0.001 0.001" />
+        <mesh filename="package://relax_urdf/meshes/mesh_link6.stl" scale="0.001 0.001 0.001" />
       </geometry>
       <material name="darkblue"/>
@@ -120,8 +120,9 @@
       <origin xyz="0 0 0" rpy="0 0 0"/>
       <geometry name="relax_link6_collision">
-        <mesh filename="package://relax_urdf/meshes/mesh_wrist-yaw.stl" scale="0.001 0.001 0.001" />
+        <mesh filename="package://relax_urdf/meshes/mesh_link6.stl" scale="0.001 0.001 0.001" />
       </geometry>
     </collision>
 </link>
+<link name ="relax_arm${arm_num}_linkEndEffector" />  <!-- link End-Effector -->
 <!-- joints -->
 <joint name="relax_arm${arm_num}_joint1" type="revolute"> <!-- joint 1 -->
@@ -165,4 +166,12 @@
     <dynamics damping="${Joint_5_damp}" friction="${Joint_5_fric}"/>
 </joint>
+<joint name="relax_arm${arm_num}_joint6" type="revolute"> <!-- joint 6 -->
+    <parent link="relax_arm${arm_num}_link6"/>
+    <child link="relax_arm${arm_num}_linkEndEffector"/>
+    <origin xyz="${Joint_6_Ox} ${Joint_6_Oy} ${Joint_6_Oz}" rpy="${Joint_6_Oroll} ${Joint_6_Opitch} ${Joint_6_Oyaw}"/>
+    <axis xyz="0 0 1"/>
+    <limit velocity="${Joint_6_velocity}" effort="${Joint_6_effort}" lower="${Joint_6_lower}" upper="${Joint_6_upper}" />
+    <dynamics damping="${Joint_6_damp}" friction="${Joint_6_fric}"/>
+</joint>
   </xacro:macro>
 </robot>

File: relax_urdf/urdf/relax.urdf (robot description, URDF)
Before this commit: robot relax, 28 links, 26 joints
Links:
- removed link D435i_camera_accel_frame
- removed link D435i_camera_accel_optical_frame
- removed link D435i_camera_bottom_screw_frame
- removed link D435i_camera_color_frame
- removed link D435i_camera_color_optical_frame
- removed link D435i_camera_depth_frame
- removed link D435i_camera_depth_optical_frame
- removed link D435i_camera_gyro_frame
- removed link D435i_camera_gyro_optical_frame
- removed link D435i_camera_left_ir_frame
- removed link D435i_camera_left_ir_optical_frame
- removed link D435i_camera_link
- removed link D435i_camera_right_ir_frame
- removed link D435i_camera_right_ir_optical_frame
- removed link control_box
- removed link left_wheel
- removed link left_wheel_yaw
- removed link mobile_base_link
- removed link right_wheel
- removed link right_wheel_yaw
- removed link world
- added link back_laser_link, mass 1.2; collision mesh filename=package://relax_urdf/meshes/sick_lms-100.stl; visual mesh filename=package://relax_urdf/meshes/sick_lms-100.stl
- added link base_footprint
- added link bl_caster_rotation_link, mass 0.3097539019; collision mesh filename=package://relax_urdf/meshes/caster_wheel_base.stl; visual mesh filename=package://relax_urdf/meshes/caster_wheel_base.stl
- added link bl_caster_wheel_link, mass 1.0; collision cylinder length=0.032 radius=0.0625; visual cylinder length=0.032 radius=0.0625
- added link br_caster_rotation_link, mass 0.3097539019; collision mesh filename=package://relax_urdf/meshes/caster_wheel_base.stl; visual mesh filename=package://relax_urdf/meshes/caster_wheel_base.stl
- added link br_caster_wheel_link, mass 1.0; collision cylinder length=0.032 radius=0.0625; visual cylinder length=0.032 radius=0.0625
- added link fl_caster_rotation_link, mass 0.3097539019; collision mesh filename=package://relax_urdf/meshes/caster_wheel_base.stl; visual mesh filename=package://relax_urdf/meshes/caster_wheel_base.stl
- added link fl_caster_wheel_link, mass 1.0; collision cylinder length=0.032 radius=0.0625; visual cylinder length=0.032 radius=0.0625
- added link fr_caster_rotation_link, mass 0.3097539019; collision mesh filename=package://relax_urdf/meshes/caster_wheel_base.stl; visual mesh filename=package://relax_urdf/meshes/caster_wheel_base.stl
- added link fr_caster_wheel_link, mass 1.0; collision cylinder length=0.032 radius=0.0625; visual cylinder length=0.032 radius=0.0625
- added link front_laser_link, mass 1.2; collision mesh filename=package://relax_urdf/meshes/sick_lms-100.stl; visual mesh filename=package://relax_urdf/meshes/sick_lms-100.stl
- added link imu_frame
- added link imu_link
- added link left_wheel_link, mass 1.0; collision cylinder length=0.038 radius=0.1; visual cylinder length=0.038 radius=0.1
- added link right_wheel_link, mass 1.0; collision cylinder length=0.038 radius=0.1; visual cylinder length=0.038 radius=0.1
- added link surface
- added link us_1_frame
- added link us_2_frame
- link base_link: mass None -> 97.0; geometry collision mesh filename=package://relax_urdf/meshes/mesh_base_revised.stl scale=0.001 0.001 0.001; visual mesh filename=package://relax_urdf/meshes/mesh_base_revised.stl scale=0.001 0.001 0.001
- link relax_arm1_link1: mass 5.9029271 -> 6.2381702
- link relax_arm1_link2: mass 1.9989653 -> 2.601371
- link relax_arm1_link3: mass 5.8838845 -> 5.9482803
- link relax_arm1_link4: mass 1.398224 -> 1.6710337
- link relax_arm1_link5: mass 5.7923846 -> 6.181102
- link relax_arm1_link6: mass 5.7923846 -> 0.48141935; geometry collision mesh filename=package://relax_urdf/meshes/mesh_link6.stl scale=0.001 0.001 0.001; visual mesh filename=package://relax_urdf/meshes/mesh_link6.stl scale=0.001 0.001 0.001
Joints:
- removed joint D435i_camera_accel_joint
- removed joint D435i_camera_accel_optical_joint
- removed joint D435i_camera_color_joint
- removed joint D435i_camera_color_optical_joint
- removed joint D435i_camera_depth_joint
- removed joint D435i_camera_depth_optical_joint
- removed joint D435i_camera_gyro_joint
- removed joint D435i_camera_gyro_optical_joint
- removed joint D435i_camera_joint
- removed joint D435i_camera_left_ir_joint
- removed joint D435i_camera_left_ir_optical_joint
- removed joint D435i_camera_link_joint
- removed joint D435i_camera_right_ir_joint
- removed joint D435i_camera_right_ir_optical_joint
- removed joint j_control
- removed joint j_left_wheel_roll
- removed joint j_left_wheel_yaw
- removed joint j_right_wheel_roll
- removed joint j_right_wheel_yaw
- removed joint world_joint
- added joint base_link_surface_joint: type fixed, parent base_link, child surface, origin xyz=-0.004485 0 0.352 rpy=0 0 0, axis 0 0 1
- added joint base_link_to_back_laser_joint: type fixed, parent base_link, child back_laser_link, origin xyz=-0.319485 -0.205 0.1914 rpy=0.0 0.0 -2.356194490192345
- added joint base_link_to_front_laser_joint: type fixed, parent base_link, child front_laser_link, origin xyz=0.310515 0.205 0.1914 rpy=0.0 0.0 0.7853981633974483
- added joint base_link_to_imu_joint: type fixed, parent base_link, child imu_link, origin xyz=0.0 0.0 0.25 rpy=0 0 0
- added joint bl_caster_rotation_joint: type continuous, parent base_link, child bl_caster_rotation_link, origin xyz=-0.300485 0.188 0.1565 rpy=0 0 0, axis 0 0 1
- added joint bl_caster_wheel_joint: type continuous, parent bl_caster_rotation_link, child bl_caster_wheel_link, origin xyz=-0.0382 0 -0.094 rpy=0 0 0, axis 0 1 0
- added joint br_caster_rotation_joint: type continuous, parent base_link, child br_caster_rotation_link, origin xyz=-0.300485 -0.188 0.1565 rpy=0 0 0, axis 0 0 1
- added joint br_caster_wheel_joint: type continuous, parent br_caster_rotation_link, child br_caster_wheel_link, origin xyz=-0.0382 0 -0.094 rpy=0 0 0, axis 0 1 0
- added joint fl_caster_rotation_joint: type continuous, parent base_link, child fl_caster_rotation_link, origin xyz=0.299215 0.188 0.1565 rpy=0 0 0, axis 0 0 1
- added joint fl_caster_wheel_joint: type continuous, parent fl_caster_rotation_link, child fl_caster_wheel_link, origin xyz=-0.0382 0 -0.094 rpy=0 0 0, axis 0 1 0
- added joint fr_caster_rotation_joint: type continuous, parent base_link, child fr_caster_rotation_link, origin xyz=0.299215 -0.188 0.1565 rpy=0 0 0, axis 0 0 1
- added joint fr_caster_wheel_joint: type continuous, parent fr_caster_rotation_link, child fr_caster_wheel_link, origin xyz=-0.0382 0 -0.094 rpy=0 0 0, axis 0 1 0
- added joint imu_link_to_imu_frame_joint: type fixed, parent imu_link, child imu_frame, origin xyz=0 0 0 rpy=0 0 0
- added joint left_wheel_joint: type continuous, parent base_link, child left_wheel_link, origin xyz=0.0 0.2015 0.1 rpy=0 0 0, axis 0 1 0, limit effort=100 velocity=20.0
- added joint relax_arm1_joint5: type revolute, parent relax_arm1_link5, child relax_arm1_link6, origin xyz=0.0 0.22216 -0.08816 rpy=-1.5707963 0.0 0.0, axis 0 1 0, limit lower=-3.14 upper=3.14 effort=147.0 velocity=3.86
- added joint right_wheel_joint: type continuous, parent base_link, child right_wheel_link, origin xyz=0.0 -0.2015 0.1 rpy=0 0 0, axis 0 1 0, limit effort=100 velocity=20.0
- added joint us_1_joint: type fixed, parent base_link, child us_1_frame, origin xyz=0.45 -0.12 0.16  rpy=0 0 0
- added joint us_2_joint: type fixed, parent base_link, child us_2_frame, origin xyz=0.45 0.12 0.16  rpy=0 0 0
- joint base_joint: child mobile_base_link -> base_link; parent base_link -> base_footprint
- joint mobile_base_joint: origin xyz=0 0 0 rpy=3.1415927 0 0 -> xyz=-0.130 0 0.3613 rpy=0 0 0; parent control_box -> base_link
- joint relax_arm1_joint1: axis 0 1 0 -> 0 0 1; origin xyz=0.0 0.13166 -0.24966 rpy=0 0 0 -> xyz=0.0 0.13166 0.24966 rpy=-1.5707963 0.0 0.0
- joint relax_arm1_joint2: origin xyz=0.0 0.0 -0.4 rpy=0 0 0 -> xyz=0.0 -0.4 0.0 rpy=0.0 0.0 0.0
- joint relax_arm1_joint3: axis 0 0 1 -> 0 1 0; origin xyz=0.0 -0.13166 -0.24966 rpy=0 0 0 -> xyz=0.0 -0.24966 -0.13166 rpy=1.5707963 0.0 0.0
- joint relax_arm1_joint4: axis 0 1 0 -> 0 0 1; origin xyz=0.0 -0.08816 -0.1535 rpy=0.0 0.0 3.1415927 -> xyz=0.0 -0.08816 0.1535 rpy=1.5707963 0.0 0.0

Commit message: fixed srdf files due to the last change for the joint 0 of the arm

File: relax_srdf/srdf/relax.srdf.xacro (robot description, xacro)
@@ -20,10 +20,10 @@
     <xacro:if value="${RELAX_MOBILE_BASE}">
         <group name="arm">
-            <chain base_link="world" tip_link="relax_arm1_linkEndEffector" />
+            <chain base_link="world" tip_link="relax_arm1_link6" />
         </group>
     </xacro:if>
     <xacro:unless value="${RELAX_MOBILE_BASE}">
         <group name="arm">
-            <chain base_link="relax_arm1_link1" tip_link="relax_arm1_linkEndEffector" />
+            <chain base_link="base_link" tip_link="relax_arm1_link6" />
         </group>
     </xacro:unless>
@@ -48,4 +48,5 @@
 <!-- homing posture -->
   <group_state name="home" group="chains">
+    <joint name="relax_arm1_joint0" value="0.0"/>
     <joint name="relax_arm1_joint1" value="0.0"/>
     <joint name="relax_arm1_joint2" value="0.6"/>
@@ -53,5 +54,4 @@
     <joint name="relax_arm1_joint4" value="0.0"/>
     <joint name="relax_arm1_joint5" value="0.6"/>
-    <joint name="relax_arm1_joint6" value="0.0"/>
     <joint name="left_wheel_joint" value="0.0"/>
     <joint name="right_wheel_joint" value="0.0"/>

Commit message: new SRDF with two groups for linear and rotation control of the base

File: relax_srdf/srdf/relax.srdf.xacro (robot description, xacro)
@@ -10,9 +10,9 @@
     </group>
 <xacro:if value="${RELAX_MOBILE_BASE}">
-    <group name="left_locomotion">
+    <group name="cartesian_base_linear">
+        <chain base_link="base_footprint" tip_link="fl_caster_wheel_link" />
+    </group>
+    <group name="cartesian_base_rot">
         <chain base_link="base_footprint" tip_link="left_wheel_link" />
-    </group>
-    <group name="right_locomotion">
-        <chain base_link="base_footprint" tip_link="right_wheel_link" />
     </group>
 </xacro:if>
@@ -20,10 +20,10 @@
     <xacro:if value="${RELAX_MOBILE_BASE}">
         <group name="arm">
-            <chain base_link="world" tip_link="relax_arm1_link6" />
+            <chain base_link="base_link" tip_link="relax_arm1_linkEndEffector" />
         </group>
     </xacro:if>
     <xacro:unless value="${RELAX_MOBILE_BASE}">
         <group name="arm">
-            <chain base_link="base_link" tip_link="relax_arm1_link6" />
+            <chain base_link="base_link" tip_link="relax_arm1_linkEndEffector" />
         </group>
     </xacro:unless>
@@ -34,8 +34,8 @@
     </group>
 </xacro:if>
-<group name="chains"> <!--THIS HAS TO BE THE LAST GROUP IN THE FILE -->
+<group name="chains">
     <xacro:if value="${RELAX_MOBILE_BASE}">
-        <group name="right_locomotion" />
-        <group name="left_locomotion" />
+        <group name="cartesian_base_linear" />
+        <group name="cartesian_base_rot" />
     </xacro:if>
     <xacro:if value="${RELAX_ARM}">
@@ -54,6 +54,4 @@
     <joint name="relax_arm1_joint4" value="0.0"/>
     <joint name="relax_arm1_joint5" value="0.6"/>
-    <joint name="left_wheel_joint" value="0.0"/>
-    <joint name="right_wheel_joint" value="0.0"/>
   </group_state>
 </robot>
