Commit message: Working version in simulation using a separate fake chain for the base cartesian control

File: relax_srdf/srdf/relax.srdf.xacro (robot description, xacro)
@@ -10,22 +10,12 @@
     </group>
 <xacro:if value="${RELAX_MOBILE_BASE}">
-    <group name="cartesian_base_linear">
-        <chain base_link="base_footprint" tip_link="fl_caster_wheel_link" />
-    </group>
-    <group name="cartesian_base_rot">
-        <chain base_link="base_footprint" tip_link="left_wheel_link" />
+    <group name="cartesian_base">
+        <chain base_link="world" tip_link="base_footprint"/>
     </group>
 </xacro:if>
 <xacro:if value="${RELAX_ARM}">
-    <xacro:if value="${RELAX_MOBILE_BASE}">
-        <group name="arm">
-            <chain base_link="base_link" tip_link="relax_arm1_linkEndEffector" />
-        </group>
-    </xacro:if>
-    <xacro:unless value="${RELAX_MOBILE_BASE}">
-        <group name="arm">
-            <chain base_link="base_link" tip_link="relax_arm1_linkEndEffector" />
-        </group>
-    </xacro:unless>
+    <group name="arm">
+        <chain base_link="base_link" tip_link="relax_arm1_linkEndEffector" />
+    </group>
 </xacro:if>
 <xacro:if value="${ADD_VIRTUAL_FRAME}">
@@ -36,6 +26,5 @@
 <group name="chains">
     <xacro:if value="${RELAX_MOBILE_BASE}">
-        <group name="cartesian_base_linear" />
-        <group name="cartesian_base_rot" />
+        <group name="cartesian_base"/>
     </xacro:if>
     <xacro:if value="${RELAX_ARM}">
@@ -49,9 +38,9 @@
   <group_state name="home" group="chains">
     <joint name="relax_arm1_joint0" value="0.0"/>
-    <joint name="relax_arm1_joint1" value="0.0"/>
+    <joint name="relax_arm1_joint1" value="0.8"/>
     <joint name="relax_arm1_joint2" value="0.6"/>
-    <joint name="relax_arm1_joint3" value="-1.7"/>
-    <joint name="relax_arm1_joint4" value="0.0"/>
-    <joint name="relax_arm1_joint5" value="0.6"/>
+    <joint name="relax_arm1_joint3" value="0.0"/>
+    <joint name="relax_arm1_joint4" value="-0.5"/>
+    <joint name="relax_arm1_joint5" value="0.0"/>
   </group_state>
 </robot>

File: relax_urdf/urdf/config/relax.urdf.xacro (robot description, xacro)
@@ -1,5 +1,5 @@
 <?xml version="1.0"?>
 <robot xmlns:xacro="http://ros.org/wiki/xacro" name="relax">
-<xacro:property name="model_name" value="relax" />
+<xacro:property name="model_name" value="RELAX" />
 <xacro:property name="model_version" value="1.0" />
 <!-- command line arguments -->
@@ -8,5 +8,5 @@
 <!-- For sensors, you can use realsense=true argument to add all cameras (for now only d435i_control_box)
 or realsense=false togheter with d435_xxx=true to add single ones. This is like the centauro_urdf conf-->
-<xacro:arg name="realsense" default="true"/>
+<xacro:arg name="realsense" default="false"/>
 <xacro:if value="$(arg realsense)">
 	<xacro:arg name="d435i_control_box" default="true"/>
@@ -15,5 +15,5 @@
 	<xacro:arg name="d435i_control_box" default="false"/>
 </xacro:unless>
-<xacro:arg name="floating_joint" default="true"/>
+<xacro:arg name="floating_joint" default="false"/>
 <xacro:arg name="use_nav_controllers" default="true"/>
 <!-- ************SELECT PARTS*************-->

File: relax_urdf/urdf/config/relax_mir.urdf.xacro (robot description, xacro)
@@ -1,10 +1,10 @@
 <?xml version="1.0"?>
 <robot xmlns:xacro="http://ros.org/wiki/xacro" name="relax">
-<xacro:property name="model_name" value="IIT RELAX" />
+<xacro:property name="model_name" value="RELAX MIR250" />
 <xacro:property name="model_version" value="1.0" />
 <!-- command line arguments -->
-<xacro:arg name="arm" default="true"/>
+<xacro:arg name="arm" default="false"/>
 <xacro:arg name="base" default="true"/>
-<xacro:arg name="floating_joint" default="true"/>
+<xacro:arg name="floating_joint" default="false"/>
 <!-- ************SELECT PARTS*************-->
 <!-- *************************************-->

File: relax_urdf/urdf/parts/mir_base.urdf.xacro (robot description, xacro)
@@ -81,107 +81,41 @@
     </joint>
     <link name="${prefix}us_2_frame" />
-    <!-- wheels MANUALLY DONE FOR HIGH LEVEL CONTROL -->
-    <joint name="left_wheel_joint" type="revolute">
-      <origin rpy="0 0 0" xyz="0.0 0.2015 0.1"/>
-      <parent link="base_link"/>
-      <child link="left_wheel_link"/>
+    <!-- HACK: manually defining fake joints for cartesian control -->
+    <link name="world"/>
+    <joint name="lin_x_joint" type="prismatic">
+      <parent link="world"/>
+      <child link="lin_x_link"/>
+      <limit upper="1e9" lower="-1e9" velocity="1" effort="1"/>
+      <axis xyz="1 0 0"/>
+    </joint>
+    <joint name="lin_y_joint" type="prismatic">
+      <parent link="lin_x_link"/>
+      <child link="lin_y_link"/>
+      <limit upper="1e9" lower="-1e9" velocity="1" effort="1"/>
+      <axis xyz="0 1 0"/>
+    </joint>
+    <joint name="rot_z_joint" type="revolute">
+      <parent link="lin_y_link"/>
+      <child link="base_footprint"/>
+      <limit upper="1e9" lower="-1e9" velocity="1" effort="1"/>
       <axis xyz="0 0 1"/>
-      <limit upper="1e9" lower="-1e9" effort="2" velocity="2.0"/>
     </joint>
-    <link name="left_wheel_link">
-    <inertial>
-      <mass value="1.0"/>
-      <origin rpy="0 0 0" xyz="0 0 0"/>
-      <inertia ixx="0.0026203322852000007" ixy="0.0" ixz="0.0" iyy="0.0026203322852000007" iyz="0.0" izz="0.005000000000000001"/>
-    </inertial>
-    <visual>
-      <origin rpy="1.5707963267948966 0 0" xyz="0 0 0"/>
-      <geometry>
-        <cylinder length="0.038" radius="0.1"/>
-      </geometry>
-      <material name="black">
-        <color rgba="0.1 0.1 0.1 1"/>
-      </material>
-    </visual>
-    <collision>
-      <origin rpy="1.5707963267948966 0 0" xyz="0 0 0"/>
-      <geometry>
-        <cylinder length="0.038" radius="0.1"/>
-      </geometry>
-    </collision>
-  </link>
-  <gazebo reference="left_wheel_link">
-    <material>Gazebo/FlatBlack</material>
-  </gazebo>
-  <joint name="fl_caster_rotation_joint" type="prismatic">
-    <origin rpy="0 0 0" xyz="0.299215 0.188 0.1565"/>
-    <parent link="base_link"/>
-    <child link="fl_caster_rotation_link"/>
-    <axis xyz="1 0 0"/>
-    <limit upper="1e9" lower="-1e9" effort="2" velocity="2.0"/>
-    <dynamics damping="0.01" friction="0.0"/>
-  </joint>
-  <link name="fl_caster_rotation_link">
-    <inertial>
-      <!-- <origin xyz="0 0 -0.042500000044" rpy="${0.5 * pi} ${24 * deg_to_rad} ${1.5 * pi}" /> -->
-      <origin rpy="0 0 0" xyz="0 0 -0.042500000044"/>
-      <!-- ${24 * deg_to_rad} 0 ${0.5 * pi} -->
-      <mass value="0.3097539019"/>
-      <inertia ixx="0.0005844517978" ixy="0" ixz="0" iyy="0.00052872551237" iyz="0" izz="0.00017923555074"/>
-    </inertial>
-    <visual>
-      <origin rpy="0 0 0" xyz="0 0 0"/>
-      <geometry>
-        <mesh filename="package://relax_urdf/meshes/caster_wheel_base.stl"/>
-      </geometry>
-      <material name="black">
-        <color rgba="0.1 0.1 0.1 1"/>
-      </material>
-    </visual>
-    <collision>
-      <origin rpy="0 0 0" xyz="0 0 0"/>
-      <geometry>
-        <mesh filename="package://relax_urdf/meshes/caster_wheel_base.stl"/>
-      </geometry>
-    </collision>
-  </link>
-  <gazebo reference="fl_caster_rotation_link">
-    <material>Gazebo/FlatBlack</material>
-  </gazebo>
-  <joint name="fl_caster_wheel_joint" type="fixed">
-    <origin rpy="0 0 0" xyz="-0.0382 0 -0.094"/>
-    <parent link="fl_caster_rotation_link"/>
-    <child link="fl_caster_wheel_link"/>
-    <axis xyz="0 1 0"/>
-    <limit upper="1e9" lower="-1e9" effort="2" velocity="2.0"/>
-  </joint>
-  <link name="fl_caster_wheel_link">
-    <inertial>
-      <mass value="1.0"/>
-      <origin rpy="0 0 0" xyz="0 0 0"/>
-      <inertia ixx="0.001061895408575" ixy="0.0" ixz="0.0" iyy="0.001061895408575" iyz="0.0" izz="0.001953125"/>
-    </inertial>
-    <visual>
-      <origin rpy="1.57 0 0" xyz="0 0 0"/>
-      <!--${pi/2} 0 0 -->
-      <geometry>
-        <cylinder length="0.032" radius="0.0625"/>
-      </geometry>
-      <material name="black">
-        <color rgba="0.1 0.1 0.1 1"/>
-      </material>
-    </visual>
-    <collision>
-      <origin rpy="1.57 0 0" xyz="0 0 0"/>
-      <!--${pi/2} 0 0 -->
-      <geometry>
-        <cylinder length="0.032" radius="0.0625"/>
-      </geometry>
-    </collision>
-  </link>
-  <gazebo reference="fl_caster_wheel_link">
-    <material>Gazebo/FlatBlack</material>
-  </gazebo>
+    <link name="lin_x_link">
+      <inertial>
+        <mass value="0.01"/>
+        <origin xyz="0 0 0"/>
+        <inertia ixx="0.0001" ixy="0.0" ixz="0.0" iyy="0.0001" iyz="0.0" izz="0.0001"/>
+      </inertial>
+    </link>
+    <link name="lin_y_link">
+      <inertial>
+        <mass value="0.01"/>
+        <origin xyz="0 0 0"/>
+        <inertia ixx="0.0001" ixy="0.0" ixz="0.0" iyy="0.0001" iyz="0.0" izz="0.0001"/>
+      </inertial>
+    </link>
+    <xacro:actuated_wheel prefix="${prefix}" locationprefix="left" locationright="-1"/>
     <xacro:actuated_wheel prefix="${prefix}" locationprefix="right" locationright="1"/>
+    <xacro:caster_wheel prefix="${prefix}" locationprefix="fl" locationright="-1" wheel_base_dx="${mir_front_caster_wheel_base_dx + mir_act_wheel_dx}"/>
     <xacro:caster_wheel prefix="${prefix}" locationprefix="fr" locationright="1" wheel_base_dx="${mir_front_caster_wheel_base_dx + mir_act_wheel_dx}"/>
     <xacro:caster_wheel prefix="${prefix}" locationprefix="bl" locationright="-1" wheel_base_dx="${-mir_back_caster_wheel_base_dx + mir_act_wheel_dx}"/>

File: relax_urdf/urdf/parts/wheels.urdf.xacro (robot description, xacro)
@@ -28,5 +28,5 @@
   <xacro:property name="mir_caster_wheel_base_dz" value="${mir_caster_wheel_radius - mir_caster_wheel_dz}" />
   <xacro:macro name="actuated_wheel" params="prefix locationprefix locationright">
-    <joint name="${prefix}${locationprefix}_wheel_joint" type="fixed">
+    <joint name="${prefix}${locationprefix}_wheel_joint" type="continuous">
       <origin xyz="0.0 ${-mir_act_wheel_dy * locationright} ${mir_act_wheel_radius}" rpy="0 0 0" />
       <parent link="${prefix}base_link" />
@@ -59,5 +59,5 @@
   <xacro:macro name="caster_wheel" params="prefix locationprefix locationright wheel_base_dx">
     <!-- caster hub -->
-    <joint name="${prefix}${locationprefix}_caster_rotation_joint" type="fixed">
+    <joint name="${prefix}${locationprefix}_caster_rotation_joint" type="continuous">
       <origin xyz="${wheel_base_dx} ${-mir_caster_wheel_base_dy * locationright} ${mir_caster_wheel_base_dz}" rpy="0 0 0" />
       <parent link="${prefix}base_link" />
@@ -97,5 +97,5 @@
     </gazebo>
     <!-- caster wheel -->
-    <joint name="${prefix}${locationprefix}_caster_wheel_joint" type="fixed">
+    <joint name="${prefix}${locationprefix}_caster_wheel_joint" type="continuous">
       <origin xyz="${mir_caster_wheel_dx} ${-mir_caster_wheel_dy * locationright} ${mir_caster_wheel_dz}" rpy="0 0 0" />
       <parent link="${prefix}${locationprefix}_caster_rotation_link" />

File: relax_urdf/urdf/relax_capsule.urdf (robot description, URDF)
Before this commit: robot relax, 27 links, 26 joints
Links:
- added link lin_x_link, mass 0.01
- added link lin_y_link, mass 0.01
Joints:
- removed joint world_joint
- added joint lin_x_joint: type prismatic, parent world, child lin_x_link, axis 1.0 0.0 0.0, limit lower=-1000000000.0 upper=1000000000.0 effort=1.0 velocity=1.0
- added joint lin_y_joint: type prismatic, parent lin_x_link, child lin_y_link, axis 0.0 1.0 0.0, limit lower=-1000000000.0 upper=1000000000.0 effort=1.0 velocity=1.0
- added joint rot_z_joint: type revolute, parent lin_y_link, child base_footprint, axis 0.0 0.0 1.0, limit lower=-1000000000.0 upper=1000000000.0 effort=1.0 velocity=1.0
- joint bl_caster_rotation_joint: type fixed -> continuous
- joint bl_caster_wheel_joint: type fixed -> continuous
- joint br_caster_rotation_joint: type fixed -> continuous
- joint br_caster_wheel_joint: type fixed -> continuous
- joint fl_caster_rotation_joint: axis 1.0 0.0 0.0 -> 0.0 0.0 1.0; limit lower=-1000000000.0 upper=1000000000.0 effort=2.0 velocity=2.0 -> (none); type prismatic -> continuous
- joint fl_caster_wheel_joint: limit lower=-1000000000.0 upper=1000000000.0 effort=2.0 velocity=2.0 -> (none); type fixed -> continuous
- joint fr_caster_rotation_joint: type fixed -> continuous
- joint fr_caster_wheel_joint: type fixed -> continuous
- joint left_wheel_joint: axis 0.0 0.0 1.0 -> 0.0 1.0 0.0; limit lower=-1000000000.0 upper=1000000000.0 effort=2.0 velocity=2.0 -> lower=0 upper=0 effort=100.0 velocity=20.0; type revolute -> continuous
- joint right_wheel_joint: type fixed -> continuous

File: relax_urdf/urdf/relax_mir.urdf (robot description, URDF)
Before this commit: robot mir, 20 links, 19 joints
Links:
- added link car_frame, mass 0.0
- added link car_frame_intermediate_1, mass 0.0
- added link car_frame_intermediate_2, mass 0.0
- added link car_frame_intermediate_3, mass 0.0
- added link car_frame_intermediate_4, mass 0.0
- added link car_frame_intermediate_5, mass 0.0
- added link lin_x_link, mass 0.01
- added link lin_y_link, mass 0.01
Joints:
- removed joint world_joint
- added joint car_frame_rx: type revolute, parent car_frame_intermediate_3, child car_frame_intermediate_4, origin xyz=0.0 0.0 0.0, axis 1 0 0, limit lower=-1e9 upper=1e9 effort=1000 velocity=10.0
- added joint car_frame_ry: type revolute, parent car_frame_intermediate_4, child car_frame_intermediate_5, origin xyz=0.0 0.0 0.0, axis 0 1 0, limit lower=-1e9 upper=1e9 effort=1000 velocity=10.0
- added joint car_frame_rz: type revolute, parent car_frame_intermediate_5, child car_frame, origin xyz=0.0 0.0 0.0, axis 0 0 1, limit lower=-1e9 upper=1e9 effort=1000 velocity=10.0
- added joint car_frame_tx: type prismatic, parent base_footprint, child car_frame_intermediate_1, origin xyz=0.0 0.0 0.0, axis 1 0 0, limit lower=-1e9 upper=1e9 effort=1000 velocity=10.0
- added joint car_frame_ty: type prismatic, parent car_frame_intermediate_1, child car_frame_intermediate_2, origin xyz=0.0 0.0 0.0, axis 0 1 0, limit lower=-1e9 upper=1e9 effort=1000 velocity=10.0
- added joint car_frame_tz: type prismatic, parent car_frame_intermediate_2, child car_frame_intermediate_3, origin xyz=0.0 0.0 0.0, axis 0 0 1, limit lower=-1e9 upper=1e9 effort=1000 velocity=10.0
- added joint lin_x_joint: type prismatic, parent world, child lin_x_link, axis 1 0 0, limit lower=-1e9 upper=1e9 effort=1 velocity=1
- added joint lin_y_joint: type prismatic, parent lin_x_link, child lin_y_link, axis 0 1 0, limit lower=-1e9 upper=1e9 effort=1 velocity=1
- added joint rot_z_joint: type revolute, parent lin_y_link, child base_footprint, axis 0 0 1, limit lower=-1e9 upper=1e9 effort=1 velocity=1
- joint bl_caster_rotation_joint: type fixed -> continuous
- joint bl_caster_wheel_joint: type fixed -> continuous
- joint br_caster_rotation_joint: type fixed -> continuous
- joint br_caster_wheel_joint: type fixed -> continuous
- joint fl_caster_rotation_joint: axis 1 0 0 -> 0 0 1; limit lower=-1e9 upper=1e9 effort=2 velocity=2.0 -> (none); type revolute -> continuous
- joint fl_caster_wheel_joint: limit lower=-1e9 upper=1e9 effort=2 velocity=2.0 -> (none); type fixed -> continuous
- joint fr_caster_rotation_joint: type fixed -> continuous
- joint fr_caster_wheel_joint: type fixed -> continuous
- joint left_wheel_joint: axis 0 0 1 -> 0 1 0; limit lower=-1e9 upper=1e9 effort=2 velocity=2.0 -> effort=100 velocity=20.0; type revolute -> continuous
- joint right_wheel_joint: type fixed -> continuous

File: relax_urdf/urdf/relax_xbot2.urdf (robot description, URDF)
Before this commit: robot relax, 29 links, 28 joints
Joints:
- joint bl_caster_rotation_joint: type continuous -> fixed
- joint bl_caster_wheel_joint: type continuous -> fixed
- joint br_caster_rotation_joint: type continuous -> fixed
- joint br_caster_wheel_joint: type continuous -> fixed
- joint fl_caster_rotation_joint: type continuous -> fixed
- joint fl_caster_wheel_joint: type continuous -> fixed
- joint fr_caster_rotation_joint: type continuous -> fixed
- joint fr_caster_wheel_joint: type continuous -> fixed
- joint left_wheel_joint: type continuous -> fixed
- joint right_wheel_joint: type continuous -> fixed
