Commit message: just srdf collisions

File: relax_srdf/srdf/relax.srdf.xacro (robot description, xacro)
@@ -49,3 +49,116 @@
     <joint name="relax_arm1_joint5" value="0.0"/>
   </group_state>
+  <xacro:if value="${RELAX_MOBILE_BASE}">
+    <disable_collisions link1="back_laser_link" link2="base_link" reason="Adjacent"/>
+    <disable_collisions link1="back_laser_link" link2="bl_caster_rotation_link" reason="Never"/>
+    <disable_collisions link1="back_laser_link" link2="bl_caster_wheel_link" reason="Never"/>
+    <disable_collisions link1="back_laser_link" link2="br_caster_rotation_link" reason="Default"/>
+    <disable_collisions link1="back_laser_link" link2="br_caster_wheel_link" reason="Never"/>
+    <disable_collisions link1="back_laser_link" link2="fl_caster_rotation_link" reason="Never"/>
+    <disable_collisions link1="back_laser_link" link2="fl_caster_wheel_link" reason="Never"/>
+    <disable_collisions link1="back_laser_link" link2="fr_caster_rotation_link" reason="Never"/>
+    <disable_collisions link1="back_laser_link" link2="fr_caster_wheel_link" reason="Never"/>
+    <disable_collisions link1="back_laser_link" link2="front_laser_link" reason="Never"/>
+    <disable_collisions link1="back_laser_link" link2="left_wheel_link" reason="Never"/>
+    <disable_collisions link1="back_laser_link" link2="relax_arm1_link1" reason="Never"/>
+    <disable_collisions link1="back_laser_link" link2="right_wheel_link" reason="Never"/>
+    <disable_collisions link1="base_link" link2="bl_caster_rotation_link" reason="Adjacent"/>
+    <disable_collisions link1="base_link" link2="bl_caster_wheel_link" reason="Never"/>
+    <disable_collisions link1="base_link" link2="br_caster_rotation_link" reason="Adjacent"/>
+    <disable_collisions link1="base_link" link2="br_caster_wheel_link" reason="Never"/>
+    <disable_collisions link1="base_link" link2="fl_caster_rotation_link" reason="Adjacent"/>
+    <disable_collisions link1="base_link" link2="fl_caster_wheel_link" reason="Never"/>
+    <disable_collisions link1="base_link" link2="fr_caster_rotation_link" reason="Adjacent"/>
+    <disable_collisions link1="base_link" link2="fr_caster_wheel_link" reason="Never"/>
+    <disable_collisions link1="base_link" link2="front_laser_link" reason="Adjacent"/>
+    <disable_collisions link1="base_link" link2="left_wheel_link" reason="Adjacent"/>
+    <disable_collisions link1="base_link" link2="relax_arm1_link1" reason="Adjacent"/>
+    <disable_collisions link1="base_link" link2="right_wheel_link" reason="Adjacent"/>
+    <disable_collisions link1="bl_caster_rotation_link" link2="bl_caster_wheel_link" reason="Adjacent"/>
+    <disable_collisions link1="bl_caster_rotation_link" link2="br_caster_rotation_link" reason="Never"/>
+    <disable_collisions link1="bl_caster_rotation_link" link2="br_caster_wheel_link" reason="Never"/>
+    <disable_collisions link1="bl_caster_rotation_link" link2="fl_caster_rotation_link" reason="Never"/>
+    <disable_collisions link1="bl_caster_rotation_link" link2="fl_caster_wheel_link" reason="Never"/>
+    <disable_collisions link1="bl_caster_rotation_link" link2="fr_caster_rotation_link" reason="Never"/>
+    <disable_collisions link1="bl_caster_rotation_link" link2="fr_caster_wheel_link" reason="Never"/>
+    <disable_collisions link1="bl_caster_rotation_link" link2="front_laser_link" reason="Never"/>
+    <disable_collisions link1="bl_caster_rotation_link" link2="left_wheel_link" reason="Never"/>
+    <disable_collisions link1="bl_caster_rotation_link" link2="relax_arm1_link1" reason="Never"/>
+    <disable_collisions link1="bl_caster_rotation_link" link2="relax_arm1_link2" reason="Never"/>
+    <disable_collisions link1="bl_caster_rotation_link" link2="right_wheel_link" reason="Never"/>
+    <disable_collisions link1="bl_caster_wheel_link" link2="br_caster_rotation_link" reason="Never"/>
+    <disable_collisions link1="bl_caster_wheel_link" link2="br_caster_wheel_link" reason="Never"/>
+    <disable_collisions link1="bl_caster_wheel_link" link2="fl_caster_rotation_link" reason="Never"/>
+    <disable_collisions link1="bl_caster_wheel_link" link2="fl_caster_wheel_link" reason="Never"/>
+    <disable_collisions link1="bl_caster_wheel_link" link2="fr_caster_rotation_link" reason="Never"/>
+    <disable_collisions link1="bl_caster_wheel_link" link2="fr_caster_wheel_link" reason="Never"/>
+    <disable_collisions link1="bl_caster_wheel_link" link2="front_laser_link" reason="Never"/>
+    <disable_collisions link1="bl_caster_wheel_link" link2="left_wheel_link" reason="Never"/>
+    <disable_collisions link1="bl_caster_wheel_link" link2="relax_arm1_link1" reason="Never"/>
+    <disable_collisions link1="bl_caster_wheel_link" link2="relax_arm1_link2" reason="Never"/>
+    <disable_collisions link1="bl_caster_wheel_link" link2="right_wheel_link" reason="Never"/>
+    <disable_collisions link1="br_caster_rotation_link" link2="br_caster_wheel_link" reason="Adjacent"/>
+    <disable_collisions link1="br_caster_rotation_link" link2="fl_caster_rotation_link" reason="Never"/>
+    <disable_collisions link1="br_caster_rotation_link" link2="fl_caster_wheel_link" reason="Never"/>
+    <disable_collisions link1="br_caster_rotation_link" link2="fr_caster_rotation_link" reason="Never"/>
+    <disable_collisions link1="br_caster_rotation_link" link2="fr_caster_wheel_link" reason="Never"/>
+    <disable_collisions link1="br_caster_rotation_link" link2="front_laser_link" reason="Never"/>
+    <disable_collisions link1="br_caster_rotation_link" link2="left_wheel_link" reason="Never"/>
+    <disable_collisions link1="br_caster_rotation_link" link2="relax_arm1_link1" reason="Never"/>
+    <disable_collisions link1="br_caster_rotation_link" link2="relax_arm1_link2" reason="Never"/>
+    <disable_collisions link1="br_caster_rotation_link" link2="right_wheel_link" reason="Never"/>
+    <disable_collisions link1="br_caster_wheel_link" link2="fl_caster_rotation_link" reason="Never"/>
+    <disable_collisions link1="br_caster_wheel_link" link2="fl_caster_wheel_link" reason="Never"/>
+    <disable_collisions link1="br_caster_wheel_link" link2="fr_caster_rotation_link" reason="Never"/>
+    <disable_collisions link1="br_caster_wheel_link" link2="fr_caster_wheel_link" reason="Never"/>
+    <disable_collisions link1="br_caster_wheel_link" link2="front_laser_link" reason="Never"/>
+    <disable_collisions link1="br_caster_wheel_link" link2="left_wheel_link" reason="Never"/>
+    <disable_collisions link1="br_caster_wheel_link" link2="relax_arm1_link1" reason="Never"/>
+    <disable_collisions link1="br_caster_wheel_link" link2="relax_arm1_link2" reason="Never"/>
+    <disable_collisions link1="br_caster_wheel_link" link2="right_wheel_link" reason="Never"/>
+    <disable_collisions link1="fl_caster_rotation_link" link2="fl_caster_wheel_link" reason="Adjacent"/>
+    <disable_collisions link1="fl_caster_rotation_link" link2="fr_caster_rotation_link" reason="Never"/>
+    <disable_collisions link1="fl_caster_rotation_link" link2="fr_caster_wheel_link" reason="Never"/>
+    <disable_collisions link1="fl_caster_rotation_link" link2="front_laser_link" reason="Default"/>
+    <disable_collisions link1="fl_caster_rotation_link" link2="left_wheel_link" reason="Never"/>
+    <disable_collisions link1="fl_caster_rotation_link" link2="relax_arm1_link1" reason="Never"/>
+    <disable_collisions link1="fl_caster_rotation_link" link2="relax_arm1_link2" reason="Never"/>
+    <disable_collisions link1="fl_caster_rotation_link" link2="relax_arm1_link3" reason="Never"/>
+    <disable_collisions link1="fl_caster_rotation_link" link2="right_wheel_link" reason="Never"/>
+    <disable_collisions link1="fl_caster_wheel_link" link2="fr_caster_rotation_link" reason="Never"/>
+    <disable_collisions link1="fl_caster_wheel_link" link2="fr_caster_wheel_link" reason="Never"/>
+    <disable_collisions link1="fl_caster_wheel_link" link2="front_laser_link" reason="Never"/>
+    <disable_collisions link1="fl_caster_wheel_link" link2="left_wheel_link" reason="Never"/>
+    <disable_collisions link1="fl_caster_wheel_link" link2="relax_arm1_link1" reason="Never"/>
+    <disable_collisions link1="fl_caster_wheel_link" link2="relax_arm1_link2" reason="Never"/>
+    <disable_collisions link1="fl_caster_wheel_link" link2="relax_arm1_link3" reason="Never"/>
+    <disable_collisions link1="fl_caster_wheel_link" link2="right_wheel_link" reason="Never"/>
+    <disable_collisions link1="fr_caster_rotation_link" link2="fr_caster_wheel_link" reason="Adjacent"/>
+    <disable_collisions link1="fr_caster_rotation_link" link2="front_laser_link" reason="Never"/>
+    <disable_collisions link1="fr_caster_rotation_link" link2="left_wheel_link" reason="Never"/>
+    <disable_collisions link1="fr_caster_rotation_link" link2="relax_arm1_link1" reason="Never"/>
+    <disable_collisions link1="fr_caster_rotation_link" link2="relax_arm1_link2" reason="Never"/>
+    <disable_collisions link1="fr_caster_rotation_link" link2="relax_arm1_link3" reason="Never"/>
+    <disable_collisions link1="fr_caster_rotation_link" link2="right_wheel_link" reason="Never"/>
+    <disable_collisions link1="fr_caster_wheel_link" link2="front_laser_link" reason="Never"/>
+    <disable_collisions link1="fr_caster_wheel_link" link2="left_wheel_link" reason="Never"/>
+    <disable_collisions link1="fr_caster_wheel_link" link2="relax_arm1_link1" reason="Never"/>
+    <disable_collisions link1="fr_caster_wheel_link" link2="relax_arm1_link2" reason="Never"/>
+    <disable_collisions link1="fr_caster_wheel_link" link2="relax_arm1_link3" reason="Never"/>
+    <disable_collisions link1="fr_caster_wheel_link" link2="right_wheel_link" reason="Never"/>
+    <disable_collisions link1="front_laser_link" link2="left_wheel_link" reason="Never"/>
+    <disable_collisions link1="front_laser_link" link2="relax_arm1_link1" reason="Never"/>
+    <disable_collisions link1="front_laser_link" link2="relax_arm1_link2" reason="Never"/>
+    <disable_collisions link1="front_laser_link" link2="right_wheel_link" reason="Never"/>
+    <disable_collisions link1="left_wheel_link" link2="relax_arm1_link1" reason="Never"/>
+    <disable_collisions link1="left_wheel_link" link2="right_wheel_link" reason="Never"/>
+  </xacro:if>
+  <xacro:if value="${RELAX_ARM}">
+    <disable_collisions link1="relax_arm1_link1" link2="relax_arm1_link2" reason="Adjacent"/>
+    <disable_collisions link1="relax_arm1_link2" link2="relax_arm1_link3" reason="Adjacent"/>
+    <disable_collisions link1="relax_arm1_link3" link2="relax_arm1_link4" reason="Adjacent"/>
+    <disable_collisions link1="relax_arm1_link3" link2="relax_arm1_link5" reason="Never"/>
+    <disable_collisions link1="relax_arm1_link4" link2="relax_arm1_link5" reason="Adjacent"/>
+    <disable_collisions link1="relax_arm1_link5" link2="relax_arm1_link6" reason="Adjacent"/>
+  </xacro:if>
 </robot>

File: relax_srdf/srdf/relax_arm.srdf.xacro (robot description, xacro)
@@ -43,9 +43,17 @@
   <group_state name="home" group="chains">
     <joint name="relax_arm1_joint0" value="0"/>
-        <joint name="relax_arm1_joint1" value="-0.4"/>
-        <joint name="relax_arm1_joint2" value="-1.8"/>
-        <joint name="relax_arm1_joint3" value="0"/>
-        <joint name="relax_arm1_joint4" value="0.8"/>
-        <joint name="relax_arm1_joint5" value="0"/>
+    <joint name="relax_arm1_joint1" value="-0.4"/>
+    <joint name="relax_arm1_joint2" value="-1.8"/>
+    <joint name="relax_arm1_joint3" value="0"/>
+    <joint name="relax_arm1_joint4" value="0.8"/>
+    <joint name="relax_arm1_joint5" value="0"/>
   </group_state>
+  <xacro:if value="${RELAX_ARM}">
+    <disable_collisions link1="relax_arm1_link1" link2="relax_arm1_link2" reason="Adjacent"/>
+    <disable_collisions link1="relax_arm1_link2" link2="relax_arm1_link3" reason="Adjacent"/>
+    <disable_collisions link1="relax_arm1_link3" link2="relax_arm1_link4" reason="Adjacent"/>
+    <disable_collisions link1="relax_arm1_link3" link2="relax_arm1_link5" reason="Never"/>
+    <disable_collisions link1="relax_arm1_link4" link2="relax_arm1_link5" reason="Adjacent"/>
+    <disable_collisions link1="relax_arm1_link5" link2="relax_arm1_link6" reason="Adjacent"/>
+  </xacro:if>
 </robot>
