Commit message: end big refactor

File: relax_srdf/srdf/relax.srdf.xacro (robot description, xacro)
@@ -5,49 +5,43 @@
 -->
 <robot xmlns:xacro="http://ros.org/wiki/xacro" name="relax">
-    <xacro:include filename="$(find relax_urdf)/urdf/config/relax.urdf.xacro" />
-<xacro:if value="${RELAX_MOBILE_BASE}">
-    <group name="base">
-        <link name="base_footprint"/>
-    </group>
-    <!--<group name="cartesian_base">
-        <chain base_link="world" tip_link="base_footprint"/>
-    </group>-->
-</xacro:if>
-<xacro:if value="${RELAX_ARM}">
-    <group name="arm">
-            <chain base_link="base_link" tip_link="relax_arm1_linkEndEffector" />
-    </group>
-    <xacro:unless  value="${RELAX_MOBILE_BASE}">
-        <group name="base">
-            <link name="base_link"/>
-        </group>
-    </xacro:unless>
-</xacro:if>
-<xacro:if value="${ADD_VIRTUAL_FRAME}">
+<xacro:include filename="$(find relax_urdf)/urdf/config/relax.urdf.xacro" />
+<xacro:if value="${RELAX_MOBILE_BASE == 'floating'}">
     <group name="car_frame_chain">
         <chain base_link="base_footprint" tip_link="car_frame"/>
     </group>
 </xacro:if>
+<xacro:if value="${RELAX_ARM == 'relax_arm'}">
+    <group name="arm">
+        <chain base_link="base_link" tip_link="relax_arm1_linkEndEffector" />
+    </group>
+</xacro:if>
+<xacro:if value="${END_EFFECTOR == 'dagana'}">
+    <group name="dagana">
+        <chain base_link="relax_arm1_linkEndEffector" tip_link="dagana_1_bottom_link"/>
+    </group>
+</xacro:if>
 <group name="chains">
-    <!--<xacro:if value="${RELAX_MOBILE_BASE}">
-        <group name="cartesian_base"/>
-    </xacro:if>-->
-    <xacro:if value="${RELAX_ARM}">
+    <xacro:if value="${RELAX_MOBILE_BASE == 'floating'}">
+        <group name="car_frame_chain"/>
+    </xacro:if>
+    <xacro:if value="${RELAX_ARM == 'relax_arm'}">
         <group name="arm" />
     </xacro:if>
-    <xacro:if value="${ADD_VIRTUAL_FRAME}">
-        <group name="car_frame_chain"/>
+    <xacro:if value="${END_EFFECTOR == 'dagana'}">
+        <group name="dagana"></group>
     </xacro:if>
 </group>
-<!-- homing posture -->
-  <group_state name="home" group="chains">
-    <joint name="relax_arm1_joint0" value="0.0"/>
-    <joint name="relax_arm1_joint1" value="0.8"/>
-    <joint name="relax_arm1_joint2" value="0.6"/>
-    <joint name="relax_arm1_joint3" value="0.0"/>
-    <joint name="relax_arm1_joint4" value="-0.5"/>
-    <joint name="relax_arm1_joint5" value="0.0"/>
-  </group_state>
-  <xacro:if value="${RELAX_MOBILE_BASE}">
+<xacro:if value="${RELAX_ARM == 'relax_arm'}">
+    <group_state name="home" group="chains">
+        <joint name="relax_arm1_joint0" value="0"/>
+        <joint name="relax_arm1_joint1" value="-0.4"/>
+        <joint name="relax_arm1_joint2" value="-1.67"/>
+        <joint name="relax_arm1_joint3" value="0"/>
+        <joint name="relax_arm1_joint4" value="-1.46"/>
+        <joint name="relax_arm1_joint5" value="0"/>
+    </group_state>
+</xacro:if>
+<disable_collisions link1="base_link" link2="relax_arm1_link1" reason="Adjacent"/>
+<xacro:if value="${RELAX_MOBILE_BASE == 'floating'}">
     <disable_collisions link1="back_laser_link" link2="base_link" reason="Adjacent"/>
     <disable_collisions link1="back_laser_link" link2="bl_caster_rotation_link" reason="Never"/>
@@ -73,5 +67,4 @@
     <disable_collisions link1="base_link" link2="front_laser_link" reason="Adjacent"/>
     <disable_collisions link1="base_link" link2="left_wheel_link" reason="Adjacent"/>
-    <disable_collisions link1="base_link" link2="relax_arm1_link1" reason="Adjacent"/>
     <disable_collisions link1="base_link" link2="right_wheel_link" reason="Adjacent"/>
     <disable_collisions link1="bl_caster_rotation_link" link2="bl_caster_wheel_link" reason="Adjacent"/>
@@ -153,6 +146,6 @@
     <disable_collisions link1="left_wheel_link" link2="relax_arm1_link1" reason="Never"/>
     <disable_collisions link1="left_wheel_link" link2="right_wheel_link" reason="Never"/>
-  </xacro:if>
-  <xacro:if value="${RELAX_ARM}">
+</xacro:if>
+<xacro:if value="${RELAX_ARM == 'relax_arm'}">
     <disable_collisions link1="relax_arm1_link1" link2="relax_arm1_link2" reason="Adjacent"/>
     <disable_collisions link1="relax_arm1_link2" link2="relax_arm1_link3" reason="Adjacent"/>
@@ -161,4 +154,9 @@
     <disable_collisions link1="relax_arm1_link4" link2="relax_arm1_link5" reason="Adjacent"/>
     <disable_collisions link1="relax_arm1_link5" link2="relax_arm1_link6" reason="Adjacent"/>
-  </xacro:if>
+</xacro:if>
+<xacro:if value="${END_EFFECTOR == 'dagana' or END_EFFECTOR == 'dagana_fixed'}">
+    <disable_collisions link1="relax_arm1_link6" link2="dagana_1_bottom_link" reason="Adjacent"/>
+    <disable_collisions link1="relax_arm1_link6" link2="dagana_1_top_link" reason="Adjacent"/>
+    <disable_collisions link1="dagana_1_bottom_link" link2="dagana_1_top_link" reason="Adjacent"/>
+</xacro:if>
 </robot>

File: relax_urdf/urdf/config/relax_gazebo.urdf.xacro (robot description, xacro)
@@ -1,6 +1,6 @@
 <?xml version="1.0"?>
 <robot xmlns:xacro="http://ros.org/wiki/xacro" name="relax">
-<xacro:property name="model_name" value="RELAX" />
-<xacro:property name="model_version" value="1.0" />
+    <xacro:property name="model_name" value="RELAX" />
+    <xacro:property name="model_version" value="1.0" />
     <xacro:arg name="arm" default="relax_arm"/>  <!-- none, relax_arm -->
     <xacro:arg name="base" default="mir"/> <!-- none, fixed, floating, mir -->

File: relax_urdf/urdf/gazebo/relax.gazebo.xacro (robot description, xacro)
@@ -12,5 +12,5 @@
 </gazebo>
 </xacro:macro>
-<xacro:if value="${RELAX_ARM}">
+<xacro:if value="${RELAX_ARM == 'relax_arm'}">
     <gazebo reference="relax_arm1_joint1">
         <implicitSpringDamper>1</implicitSpringDamper>

File: relax_urdf/urdf/gazebo/xbot.gazebo.xacro (robot description, xacro)
@@ -3,4 +3,5 @@
 <gazebo>
     <plugin name="xbot2_joint_driver" filename="libxbot2_gz_joint_server.so">
+        <xacro:if value="${RELAX_MOBILE_BASE == 'mir'}">
         <ignore_joints>
             <joint_to_ignore name="left_wheel_joint"/>
@@ -15,6 +16,6 @@
             <joint_to_ignore name="fr_caster_wheel_joint"/>
         </ignore_joints>
+        </xacro:if>
         <pid>
-            <!-- TODO -> CHANGE PARAMS              -->
             <gain name="lowpwr_mot" p="50"  d="5"/>
             <gain name="small_mot"  p="250"  d="5"/>
@@ -22,9 +23,11 @@
             <gain name="big_mot"    p="3000" d="10"/>
             <gain name="wheel_mot"  p="10" d="2"/>
-            <pid name="relax_arm1_joint1" profile="medium_mot"/>
-            <pid name="relax_arm1_joint2" profile="medium_mot"/>
-            <pid name="relax_arm1_joint3" profile="medium_mot"/>
-            <pid name="relax_arm1_joint4" profile="small_mot"/>
-            <pid name="relax_arm1_joint5" profile="small_mot"/>
+            <xacro:if value="${RELAX_ARM == 'relax_arm'}">
+                <pid name="relax_arm1_joint1" profile="medium_mot"/>
+                <pid name="relax_arm1_joint2" profile="medium_mot"/>
+                <pid name="relax_arm1_joint3" profile="medium_mot"/>
+                <pid name="relax_arm1_joint4" profile="small_mot"/>
+                <pid name="relax_arm1_joint5" profile="small_mot"/>
+            </xacro:if>
         </pid>
     </plugin>

File: relax_urdf/urdf/parts/mir/mir_base_macro.urdf.xacro (robot description, xacro)
@@ -87,11 +87,4 @@
     <xacro:caster_wheel prefix="${prefix}" locationprefix="bl" locationright="-1" wheel_base_dx="${-mir_back_caster_wheel_base_dx + mir_act_wheel_dx}"/>
     <xacro:caster_wheel prefix="${prefix}" locationprefix="br" locationright="1" wheel_base_dx="${-mir_back_caster_wheel_base_dx + mir_act_wheel_dx}"/>
-    <joint name="${prefix}base_link_surface_joint" type="fixed">
-      <origin xyz="${mir_act_wheel_dx} 0 0.352" rpy="0 0 0" />
-      <parent link="${prefix}base_link" />
-      <child link="${prefix}surface" />
-      <axis xyz="0 0 1" />
-    </joint>
-    <link name="${prefix}surface"/>
     <xacro:mir_wheel_transmissions prefix="${prefix}"/>
     <!-- set the gazebo friction parameters for the wheels -->

File: relax_urdf/urdf/parts/relax_arm_macro.urdf.xacro (robot description, xacro)
@@ -13,5 +13,5 @@
       <origin xyz="0 0 0" rpy="0 0 0"/>
       <geometry name="relax_link1_visual">
-        <mesh filename="package://relax_urdf/meshes/untitled.stl" scale="0.001 0.001 0.001" />
+        <mesh filename="package://relax_urdf/meshes/mesh_link1.stl" scale="0.001 0.001 0.001" />
       </geometry>
       <material name="darkblue"/>

File: relax_urdf/urdf/parts/relax_core.urdf.xacro (robot description, xacro)
@@ -11,11 +11,10 @@
         <origin xyz="0 0 0" rpy="0 0 0" />
     </joint>
-    <link name="base_link"/>
-    <link name="relax_arm_base_link"/>
-    <joint name="relax_arm_base_link_joint" type="fixed">
-        <parent link="base_link"/>
-        <child link="relax_arm_base_link"/>
-        <origin xyz="0 0 0" rpy="0 0 0"/>
-    </joint>
+    <link name="base_link">
+        <!--  a inertia is necessary for gazebo... solved in future version? https://github.com/gazebosim/sdformat/pull/1238  -->
+        <xacro:box_inertial mass="0.001" x="0.001" y="0.001" z="0.001">
+            <origin xyz="0 0 0" rpy="0 0 0" />
+        </xacro:box_inertial>
+    </link>
 </xacro:if>
 <xacro:if value="${RELAX_MOBILE_BASE == 'fixed'}">
@@ -47,11 +46,4 @@
         </collision>
     </link>
-    <xacro:include filename="$(find relax_urdf)/urdf/properties/kinematics_properties.urdf.xacro" />
-    <link name="relax_arm_base_link"/>
-    <joint name="relax_arm_base_link_joint" type="fixed">
-        <parent link="base_link"/>
-        <child link="relax_arm_base_link"/>
-        <origin xyz="${Joint_0_Ox} ${Joint_0_Oy} ${Joint_0_Oz}" rpy="${Joint_0_Oroll} ${Joint_0_Opitch} ${Joint_0_Oyaw}"/>
-    </joint>
 </xacro:if>
 <xacro:if value="${RELAX_MOBILE_BASE == 'floating'}">
@@ -59,7 +51,28 @@
     <joint name="world_joint" type="floating">
         <parent link="world"/>
-        <child link="base_footprint"/>
+        <child link="base_link"/>
     </joint>
     <xacro:include filename="$(find relax_urdf)/urdf/parts/virtual_frame.urdf.xacro"/>
+    <!--  mir_act_wheel_dx is used so also wheels xacro is necessary here    -->
+    <xacro:include filename="$(find relax_urdf)/urdf/parts/mir/base_properties.urdf.xacro" />
+    <xacro:include filename="$(find relax_urdf)/urdf/parts/mir/wheels.urdf.xacro" />
+    <link name="base_link">
+        <xacro:box_inertial mass="${mir_base_mass}" x="${mir_base_inertial_x_length}" y="${mir_base_inertial_y_length}" z="${mir_base_inertial_z_length}">
+            <origin xyz="${mir_base_inertial_x + mir_act_wheel_dx} ${mir_base_inertial_y} ${mir_base_inertial_z}" rpy="0 0 0" />
+        </xacro:box_inertial>
+        <visual>
+            <origin xyz="${mir_act_wheel_dx} 0 0" rpy="0 0 0" />
+            <geometry>
+                <mesh filename="package://relax_urdf/meshes/mesh_base_revised.stl" scale="0.001 0.001 0.001"/>
+            </geometry>
+            <material name="dark_grey"/>
+        </visual>
+        <collision>
+            <origin xyz="${mir_act_wheel_dx} 0 0" rpy="0 0 0" />
+            <geometry>
+                <mesh filename="package://relax_urdf/meshes/mesh_base_revised.stl"  scale="0.001 0.001 0.001"/>
+            </geometry>
+        </collision>
+    </link>
 </xacro:if>
 <xacro:if value="${RELAX_MOBILE_BASE == 'mir'}">
@@ -86,7 +99,14 @@
     <xacro:include filename="$(find relax_urdf)/urdf/parts/relax_ee_macro.urdf.xacro" />
     <xacro:property name="arm_num" value="1" />
-    <xacro:relax_arm arm_num="${arm_num}" parent_link="relax_arm_base_link" >
-        <origin xyz="0 0 0" rpy="0 0 0"/>
-    </xacro:relax_arm>
+    <xacro:if value="${RELAX_MOBILE_BASE == 'none'}">
+        <xacro:relax_arm arm_num="${arm_num}" parent_link="base_link" >
+            <origin xyz="0 0 0" rpy="0 0 0"/>
+        </xacro:relax_arm>
+    </xacro:if>
+    <xacro:unless value="${RELAX_MOBILE_BASE == 'none'}">
+        <xacro:relax_arm arm_num="${arm_num}" parent_link="base_link" >
+            <origin xyz="${Joint_0_Ox} ${Joint_0_Oy} ${Joint_0_Oz}" rpy="${Joint_0_Oroll} ${Joint_0_Opitch} ${Joint_0_Oyaw}"/>
+        </xacro:relax_arm>
+    </xacro:unless>
     <xacro:relax_ee arm_num="${arm_num}" />
 </xacro:if>

File: relax_urdf/urdf/parts/virtual_frame.urdf.xacro (robot description, xacro)
@@ -3,5 +3,5 @@
 <!-- car frame virtual joints -->
 <joint name="car_frame_tx" type="prismatic">
-    <parent link="base_footprint"/>
+    <parent link="base_link"/>
     <origin xyz="0.0 0.0 0.0"/>
     <child link="car_frame_intermediate_1"/>
