Commit message: fix problem with new reference of link 1

File: relax_urdf/urdf/properties/inertial_properties.urdf.xacro (robot description, xacro)
@@ -6,5 +6,6 @@
 <xacro:property name="Link_1_x" value=" ${-1.8991406e+00*mmTom} "/>
 <xacro:property name="Link_1_y" value=" ${ 2.2645162e+01*mmTom} "/>
-<xacro:property name="Link_1_z" value=" ${ 1.6741297e+02*mmTom} "/>
+<!-- With the new ref frame of the link on the base of the link -->
+<xacro:property name="Link_1_z" value=" ${ (1.6741297e+02 - 54.16)*mmTom} "/>
 <!-- Mass -->
 <xacro:property name="Link_1_mass" value="6.2381702e+00"/>

File: relax_urdf/urdf/properties/kinematics_properties.urdf.xacro (robot description, xacro)
@@ -18,5 +18,6 @@
 <xacro:property name="Joint_1_Ox" value="  0.0 "/>
 <xacro:property name="Joint_1_Oy" value=" ${ 131.660*mmTom} "/>
-<xacro:property name="Joint_1_Oz" value=" ${ 249.660*mmTom} "/>
+<!-- With the new ref frame of the link on the base of the link -->
+<xacro:property name="Joint_1_Oz" value=" ${ (249.660-54.16)*mmTom} "/>
 <xacro:property name="Joint_1_Oroll" value=" -1.5707963 "/>
 <xacro:property name="Joint_1_Opitch" value=" 0.0 "/>
